File: circuit/1_Power.sch (KiCad schematic (older format))
At the start: 43 parts

Commit message: Adjust the schematic layout and add annotations to make the schematic more beautiful.
Parts:
- removed C?: 10uF, symbol Device:C
Connections:
- wire segments 124 -> 123
Other:
- note added: "3.3V Power Supply & Reference Voltage"
- note added: "5V Power Supply"
- note added: "Electronic Switch"
- note added: "Servo Power Supply"
- moved on the sheet: C?, L?, Q?, R?, SW?, U?

Commit message: Add the battery voltage detection circuit and complete the circuit connection of XPT2046.
Parts:
- added R? (x2): 100kR, symbol Device:R
Connections:
- net labels added: VBAT
- wire segments 123 -> 128
Other:
- moved on the sheet: C?, Q?, R?, SW?

Commit message: Assign general-purpose GPIO pins to the LCD. Add annotations to the Connector subdiagram. Label the component markers.
Parts:
- R6: renamed from R?; value 100kR -> 10kR
- R7: renamed from R?; value 100kR -> 1kR
- gave numbers to parts that had none: 42

Commit message: Add packages for standard components and set the basic rules and layers of the PCB.
Parts:
- C1, C11, C12, C13, C2, C4, C6, C9: footprint (none) -> Capacitor_SMD:C_0603_1608Metric
- C10, C14, C3: footprint (none) -> Capacitor_SMD:C_0805_2012Metric
- C15, C16, C5, C7, C8: footprint (none) -> Capacitor_SMD:CP_Elec_6.3x7.7
- J1: footprint (none) -> Connector_AMASS:AMASS_XT30PW-M_1x02_P2.50mm_Horizontal
- L1: footprint (none) -> Inductor_SMD:L_10.4x10.4_H4.8
- L2: footprint (none) -> Inductor_SMD:L_Abracon_ASPI-0630LR
- R1, R10, R11, R12, R13, R14, R15, R2, R3, R4, R5, R6, R7, R8, R9: footprint (none) -> Resistor_SMD:R_0603_1608Metric
- SW1: footprint (none) -> Button_Switch_SMD:SW_SPST_CK_RS282G05A3
Changed lines of the file:
@@
 F 0 "R4" H 4320 2196 50  0000 L CNN
 F 1 "1MR" H 4320 2105 50  0000 L CNN
-F 2 "" V 4180 2150 50  0001 C CNN
+F 2 "Resistor_SMD:R_0603_1608Metric" V 4180 2150 50  0001 C CNN
 F 3 "~" H 4250 2150 50  0001 C CNN
 	1    4250 2150
@@
 F 0 "C3" H 4365 3196 50  0000 L CNN
 F 1 "10uF" H 4365 3105 50  0000 L CNN
-F 2 "" H 4288 3000 50  0001 C CNN
+F 2 "Capacitor_SMD:C_0805_2012Metric" H 4288 3000 50  0001 C CNN
 F 3 "~" H 4250 3150 50  0001 C CNN
 	1    4250 3150
@@
 F 0 "R5" H 4820 2196 50  0000 L CNN
 F 1 "100kR" H 4820 2105 50  0000 L CNN
-F 2 "" V 4680 2150 50  0001 C CNN
+F 2 "Resistor_SMD:R_0603_1608Metric" V 4680 2150 50  0001 C CNN
 F 3 "~" H 4750 2150 50  0001 C CNN
 	1    4750 2150
@@
 F 0 "R1" H 2120 2046 50  0000 L CNN
 F 1 "100kR" H 2120 1955 50  0000 L CNN
-F 2 "" V 1980 2000 50  0001 C CNN
+F 2 "Resistor_SMD:R_0603_1608Metric" V 1980 2000 50  0001 C CNN
 F 3 "~" H 2050 2000 50  0001 C CNN
 	1    2050 2000
@@
 F 0 "R3" H 3270 2196 50  0000 L CNN
 F 1 "100kR" H 3270 2105 50  0000 L CNN
-F 2 "" V 3130 2150 50  0001 C CNN
+F 2 "Resistor_SMD:R_0603_1608Metric" V 3130 2150 50  0001 C CNN
 F 3 "~" H 3200 2150 50  0001 C CNN
 	1    3200 2150
@@
 F 0 "SW1" H 3700 2450 50  0000 C CNN
 F 1 "SW_DIP_x01" H 3700 2726 50  0001 C CNN
-F 2 "" H 3700 2550 50  0001 C CNN
+F 2 "Button_Switch_SMD:SW_SPST_CK_RS282G05A3" H 3700 2550 50  0001 C CNN
 F 3 "~" H 3700 2550 50  0001 C CNN
 	1    3700 2550
@@
 F 0 "R2" H 3120 3296 50  0000 L CNN
 F 1 "10kR" H 3120 3205 50  0000 L CNN
-F 2 "" V 2980 3250 50  0001 C CNN
+F 2 "Resistor_SMD:R_0603_1608Metric" V 2980 3250 50  0001 C CNN
 F 3 "~" H 3050 3250 50  0001 C CNN
 	1    3050 3250
@@
 F 0 "R11" H 7920 2896 50  0000 L CNN
 F 1 "47kR" H 7920 2805 50  0000 L CNN
-F 2 "" V 7780 2850 50  0001 C CNN
+F 2 "Resistor_SMD:R_0603_1608Metric" V 7780 2850 50  0001 C CNN
 F 3 "~" H 7850 2850 50  0001 C CNN
 	1    7850 2850
@@
 F 0 "R9" H 7520 2796 50  0000 L CNN
 F 1 "13.6kR" H 7520 2705 50  0000 L CNN
-F 2 "" V 7380 2750 50  0001 C CNN
+F 2 "Resistor_SMD:R_0603_1608Metric" V 7380 2750 50  0001 C CNN
 F 3 "~" H 7450 2750 50  0001 C CNN
 	1    7450 2750
@@
 F 0 "R8" H 7520 1996 50  0000 L CNN
 F 1 "100kR" H 7520 1905 50  0000 L CNN
-F 2 "" V 7380 1950 50  0001 C CNN
+F 2 "Resistor_SMD:R_0603_1608Metric" V 7380 1950 50  0001 C CNN
 F 3 "~" H 7450 1950 50  0001 C CNN
 	1    7450 1950
@@
 F 0 "L2" V 9800 2600 50  0000 C CNN
 F 1 "4.7uH" V 9600 2550 50  0000 C CNN
-F 2 "" H 9700 2550 50  0001 C CNN
+F 2 "Inductor_SMD:L_Abracon_ASPI-0630LR" H 9700 2550 50  0001 C CNN
 F 3 "~" H 9700 2550 50  0001 C CNN
 	1    9700 2550
@@
 F 0 "R12" H 9170 1996 50  0000 L CNN
 F 1 "100kR" H 9170 1905 50  0000 L CNN
-F 2 "" V 9030 1950 50  0001 C CNN
+F 2 "Resistor_SMD:R_0603_1608Metric" V 9030 1950 50  0001 C CNN
 F 3 "~" H 9100 1950 50  0001 C CNN
 	1    9100 1950
@@
 F 0 "C12" V 9050 2500 50  0000 L CNN
 F 1 "10nF" V 9150 2500 50  0000 L CNN
-F 2 "" H 9238 2300 50  0001 C CNN
+F 2 "Capacitor_SMD:C_0603_1608Metric" H 9238 2300 50  0001 C CNN
 F 3 "~" H 9200 2450 50  0001 C CNN
 	1    9200 2450
@@
 F 0 "C14" H 10115 3146 50  0000 L CNN
 F 1 "22uF" H 10115 3055 50  0000 L CNN
-F 2 "" H 10038 2950 50  0001 C CNN
+F 2 "Capacitor_SMD:C_0805_2012Metric" H 10038 2950 50  0001 C CNN
 F 3 "~" H 10000 3100 50  0001 C CNN
 	1    10000 3100
@@
 F 0 "C10" H 8965 3146 50  0000 L CNN
 F 1 "10uF" H 8965 3055 50  0000 L CNN
-F 2 "" H 8888 2950 50  0001 C CNN
+F 2 "Capacitor_SMD:C_0805_2012Metric" H 8888 2950 50  0001 C CNN
 F 3 "~" H 8850 3100 50  0001 C CNN
 	1    8850 3100
@@
 F 0 "C1" H 3065 6096 50  0000 L CNN
 F 1 "22uF" H 3065 6005 50  0000 L CNN
-F 2 "" H 2988 5900 50  0001 C CNN
+F 2 "Capacitor_SMD:C_0603_1608Metric" H 2988 5900 50  0001 C CNN
 F 3 "~" H 2950 6050 50  0001 C CNN
 	1    2950 6050
@@
 F 0 "C7" H 7118 2596 50  0000 L CNN
 F 1 "100uF" H 7118 2505 50  0000 L CNN
-F 2 "" H 7038 2400 50  0001 C CNN
+F 2 "Capacitor_SMD:CP_Elec_6.3x7.7" H 7038 2400 50  0001 C CNN
 F 3 "~" H 7000 2550 50  0001 C CNN
 	1    7000 2550
@@
 F 0 "C5" H 5768 2596 50  0000 L CNN
 F 1 "100uF" H 5768 2505 50  0000 L CNN
-F 2 "" H 5688 2400 50  0001 C CNN
+F 2 "Capacitor_SMD:CP_Elec_6.3x7.7" H 5688 2400 50  0001 C CNN
 F 3 "~" H 5650 2550 50  0001 C CNN
 	1    5650 2550
@@
 F 0 "C6" H 5815 6096 50  0000 L CNN
 F 1 "100nF" H 5815 6005 50  0000 L CNN
-F 2 "" H 5738 5900 50  0001 C CNN
+F 2 "Capacitor_SMD:C_0603_1608Metric" H 5738 5900 50  0001 C CNN
 F 3 "~" H 5700 6050 50  0001 C CNN
 	1    5700 6050
@@
 F 0 "C4" H 4365 6096 50  0000 L CNN
 F 1 "100nF" H 4365 6005 50  0000 L CNN
-F 2 "" H 4288 5900 50  0001 C CNN
+F 2 "Capacitor_SMD:C_0603_1608Metric" H 4288 5900 50  0001 C CNN
 F 3 "~" H 4250 6050 50  0001 C CNN
 	1    4250 6050
@@
 F 0 "C2" H 3465 5746 50  0000 L CNN
 F 1 "100nF" H 3465 5655 50  0000 L CNN
-F 2 "" H 3388 5550 50  0001 C CNN
+F 2 "Capacitor_SMD:C_0603_1608Metric" H 3388 5550 50  0001 C CNN
 F 3 "~" H 3350 5700 50  0001 C CNN
 	1    3350 5700
@@
 F 0 "J1" H 1400 2400 50  0000 C CNN
 F 1 "VIN" H 1350 2700 50  0000 C CNN
-F 2 "" H 1350 2600 50  0001 C CNN
+F 2 "Connector_AMASS:AMASS_XT30PW-M_1x02_P2.50mm_Horizontal" H 1350 2600 50  0001 C CNN
 F 3 "~" H 1350 2600 50  0001 C CNN
 	1    1350 2600
@@
 F 0 "R10" H 7670 6246 50  0000 L CNN
 F 1 "86.6kR" H 7670 6155 50  0000 L CNN
-F 2 "" V 7530 6200 50  0001 C CNN
+F 2 "Resistor_SMD:R_0603_1608Metric" V 7530 6200 50  0001 C CNN
 F 3 "~" H 7600 6200 50  0001 C CNN
 	1    7600 6200
@@
 F 0 "R15" H 9870 6196 50  0000 L CNN
 F 1 "10kR" H 9870 6105 50  0000 L CNN
-F 2 "" V 9730 6150 50  0001 C CNN
+F 2 "Resistor_SMD:R_0603_1608Metric" V 9730 6150 50  0001 C CNN
 F 3 "~" H 9800 6150 50  0001 C CNN
 	1    9800 6150
@@
 F 0 "R14" H 9870 5346 50  0000 L CNN
 F 1 "82kR" H 9870 5255 50  0000 L CNN
-F 2 "" V 9730 5300 50  0001 C CNN
+F 2 "Resistor_SMD:R_0603_1608Metric" V 9730 5300 50  0001 C CNN
 F 3 "~" H 9800 5300 50  0001 C CNN
 	1    9800 5300
@@
 F 0 "R13" H 9470 5946 50  0000 L CNN
 F 1 "23.7kR" H 9470 5855 50  0000 L CNN
-F 2 "" V 9330 5900 50  0001 C CNN
+F 2 "Resistor_SMD:R_0603_1608Metric" V 9330 5900 50  0001 C CNN
 F 3 "~" H 9400 5900 50  0001 C CNN
 	1    9400 5900
@@
 F 0 "C11" H 9215 6196 50  0000 L CNN
 F 1 "32pF" H 9215 6105 50  0000 L CNN
-F 2 "" H 9138 6000 50  0001 C CNN
+F 2 "Capacitor_SMD:C_0603_1608Metric" H 9138 6000 50  0001 C CNN
 F 3 "~" H 9100 6150 50  0001 C CNN
 	1    9100 6150
@@
 F 0 "C13" H 9515 6446 50  0000 L CNN
 F 1 "620pF" H 9515 6355 50  0000 L CNN
-F 2 "" H 9438 6250 50  0001 C CNN
+F 2 "Capacitor_SMD:C_0603_1608Metric" H 9438 6250 50  0001 C CNN
 F 3 "~" H 9400 6400 50  0001 C CNN
 	1    9400 6400
@@
 F 0 "C9" V 8050 5150 50  0000 L CNN
 F 1 "100nF" V 8150 5150 50  0000 L CNN
-F 2 "" H 8238 4900 50  0001 C CNN
+F 2 "Capacitor_SMD:C_0603_1608Metric" H 8238 4900 50  0001 C CNN
 F 3 "~" H 8200 5050 50  0001 C CNN
 	1    8200 5050
@@
 F 0 "L1" V 9200 5500 50  0000 C CNN
 F 1 "3.3uH" V 9050 5300 50  0000 C CNN
-F 2 "" H 9100 5400 50  0001 C CNN
+F 2 "Inductor_SMD:L_10.4x10.4_H4.8" H 9100 5400 50  0001 C CNN
 F 3 "~" H 9100 5400 50  0001 C CNN
 	1    9100 5400
@@
 F 0 "C8" H 7268 6246 50  0000 L CNN
 F 1 "100uF" H 7268 6155 50  0000 L CNN
-F 2 "" H 7188 6050 50  0001 C CNN
+F 2 "Capacitor_SMD:CP_Elec_6.3x7.7" H 7188 6050 50  0001 C CNN
 F 3 "~" H 7150 6200 50  0001 C CNN
 	1    7150 6200
@@
 F 0 "C15" H 10218 5896 50  0000 L CNN
 F 1 "100uF" H 10218 5805 50  0000 L CNN
-F 2 "" H 10138 5700 50  0001 C CNN
+F 2 "Capacitor_SMD:CP_Elec_6.3x7.7" H 10138 5700 50  0001 C CNN
 F 3 "~" H 10100 5850 50  0001 C CNN
 	1    10100 5850
@@
 F 0 "C16" H 10468 2596 50  0000 L CNN
 F 1 "100uF" H 10468 2505 50  0000 L CNN
-F 2 "" H 10388 2400 50  0001 C CNN
+F 2 "Capacitor_SMD:CP_Elec_6.3x7.7" H 10388 2400 50  0001 C CNN
 F 3 "~" H 10350 2550 50  0001 C CNN
 	1    10350 2550
@@
 F 0 "R7" H 5220 3046 50  0000 L CNN
 F 1 "1kR" H 5220 2955 50  0000 L CNN
-F 2 "" V 5080 3000 50  0001 C CNN
+F 2 "Resistor_SMD:R_0603_1608Metric" V 5080 3000 50  0001 C CNN
 F 3 "~" H 5150 3000 50  0001 C CNN
 	1    5150 3000
@@
 F 0 "R6" H 5220 2196 50  0000 L CNN
 F 1 "10kR" H 5220 2105 50  0000 L CNN
-F 2 "" V 5080 2150 50  0001 C CNN
+F 2 "Resistor_SMD:R_0603_1608Metric" V 5080 2150 50  0001 C CNN
 F 3 "~" H 5150 2150 50  0001 C CNN
 	1    5150 2150

Commit message: Eliminate design rule errors in schematics.
Connections:
- wire segments 128 -> 133
Changed lines of the file:
@@
 Wire Wire Line
 	5150 2550 5150 2850
+$Comp
+L power:PWR_FLAG #FLG0101
+U 1 1 61A86577
+P 1650 1600
+F 0 "#FLG0101" H 1650 1675 50  0001 C CNN
+F 1 "PWR_FLAG" H 1650 1773 50  0001 C CNN
+F 2 "" H 1650 1600 50  0001 C CNN
+F 3 "~" H 1650 1600 50  0001 C CNN
+	1    1650 1600
+	1    0    0    -1
+$EndComp
+Connection ~ 1550 1600
+Wire Wire Line
+	1550 1600 1650 1600
+$Comp
+L power:PWR_FLAG #FLG0102
+U 1 1 61A97945
+P 4350 1600
+F 0 "#FLG0102" H 4350 1675 50  0001 C CNN
+F 1 "PWR_FLAG" H 4350 1773 50  0001 C CNN
+F 2 "" H 4350 1600 50  0001 C CNN
+F 3 "~" H 4350 1600 50  0001 C CNN
+	1    4350 1600
+	1    0    0    -1
+$EndComp
+Wire Wire Line
+	4350 1600 4250 1600
+Connection ~ 4250 1600
+$Comp
+L power:PWR_FLAG #FLG0103
+U 1 1 61AA8539
+P 10200 4900
+F 0 "#FLG0103" H 10200 4975 50  0001 C CNN
+F 1 "PWR_FLAG" H 10200 5073 50  0001 C CNN
+F 2 "" H 10200 4900 50  0001 C CNN
+F 3 "~" H 10200 4900 50  0001 C CNN
+	1    10200 4900
+	1    0    0    -1
+$EndComp
+Wire Wire Line
+	10200 4900 10100 4900
+Connection ~ 10100 4900
+$Comp
+L power:PWR_FLAG #FLG0104
+U 1 1 61AB1F2C
+P 10100 1600
+F 0 "#FLG0104" H 10100 1675 50  0001 C CNN
+F 1 "PWR_FLAG" H 10100 1773 50  0001 C CNN
+F 2 "" H 10100 1600 50  0001 C CNN
+F 3 "~" H 10100 1600 50  0001 C CNN
+	1    10100 1600
+	1    0    0    -1
+$EndComp
+Wire Wire Line
+	10100 1600 10000 1600
+Connection ~ 10000 1600
+$Comp
+L power:PWR_FLAG #FLG0105
+U 1 1 61C90DF1
+P 1650 3450
+F 0 "#FLG0105" H 1650 3525 50  0001 C CNN
+F 1 "PWR_FLAG" H 1650 3623 50  0001 C CNN
+F 2 "" H 1650 3450 50  0001 C CNN
+F 3 "~" H 1650 3450 50  0001 C CNN
+	1    1650 3450
+	-1   0    0    1
+$EndComp
+Wire Wire Line
+	1650 3450 1550 3450
+Connection ~ 1550 3450
 $EndSCHEMATC

Commit message: Complete PCB design and export Gerber files.
Parts:
- added C51: 22uF, Capacitor_SMD:C_0805_2012Metric, symbol Device:C
Connections:
- wire segments 133 -> 135
Other:
- moved on the sheet: C11, C13, C15, C8, C9, L1, R10, R13, R14, R15

Commit message: Modify the circuit to modify the electronic switch section to disconnect via microcontroller control.
Parts:
- removed C3: 10uF, Capacitor_SMD:C_0805_2012Metric, symbol Device:C
- removed Q3: WST3400A, Package_TO_SOT_SMD:SOT-23, symbol Transistor_FET:AO3400A
- removed Q4: S8050, Package_TO_SOT_SMD:SOT-23, symbol MM32_Periph:S8050
- removed R4: 1MR, Resistor_SMD:R_0603_1608Metric, symbol Device:R
- added D4, D5: 1N4007, Diode_SMD:D_SOD-123, symbol Diode:1N4007
- R3: value 100kR -> 100R
- R5: value 100kR -> 10kR
Connections:
- net labels added: PWR_DET
- wire segments 135 -> 127
Other:
- moved on the sheet: Q1, R1, R2, R5, SW1
