File: circuit/2_MCU.sch (KiCad schematic (older format))
At the start: 6 parts

Commit message: Add reference voltage source to the circuit
Connections:
- net +3V3: no longer U?.32 (VREF+)
- net PWR_EN: now reaches U?.88 (PG3)
- new net +3V0: U?.32 (VREF+)
Changed lines of the file:
@@
 L power:+3.3V #PWR0138
 U 1 1 619E466A
-P 1850 5250
-F 0 "#PWR0138" H 1850 5100 50  0001 C CNN
-F 1 "+3.3V" V 1850 5500 50  0000 C CNN
-F 2 "" H 1850 5250 50  0001 C CNN
-F 3 "" H 1850 5250 50  0001 C CNN
-	1    1850 5250
+P 1850 5350
+F 0 "#PWR0138" H 1850 5200 50  0001 C CNN
+F 1 "+3.3V" V 1850 5600 50  0000 C CNN
+F 2 "" H 1850 5350 50  0001 C CNN
+F 3 "" H 1850 5350 50  0001 C CNN
+	1    1850 5350
 	0    -1   -1   0
 $EndComp
-Wire Wire Line
-	1850 5250 2250 5250
-Wire Wire Line
-	2600 5350 2250 5350
-Wire Wire Line
-	2250 5350 2250 5250
-Connection ~ 2250 5250
-Wire Wire Line
-	2250 5250 2600 5250
 $Comp
 L power:+3.3V #PWR0139
@@
 Wire Wire Line
 	1850 4550 2600 4550
+Text HLabel 7600 4150 2    50   Input ~ 0
+PWR_EN
+Wire Wire Line
+	6900 4150 7600 4150
+$Comp
+L power:+3V0 #PWR?
+U 1 1 619B9817
+P 1850 5250
+F 0 "#PWR?" H 1850 5100 50  0001 C CNN
+F 1 "+3V0" V 1850 5400 50  0000 L CNN
+F 2 "" H 1850 5250 50  0001 C CNN
+F 3 "" H 1850 5250 50  0001 C CNN
+	1    1850 5250
+	0    -1   -1   0
+$EndComp
+Wire Wire Line
+	1850 5350 2600 5350
+Wire Wire Line
+	1850 5250 2600 5250
 $EndSCHEMATC

Commit message: Add filter cap to MCU circuit and add sensor sch
Parts:
- added C? (x12): 100nF, symbol Device:C
Connections:
- net +3V3: now also C?.1, C?.1, C?.1, C?.1, C?.1, C?.1, C?.1, C?.1, C?.1, C?.1, C?.1, C?.1
- net GND: now also U?.30 (VSSA), C?.2, C?.2, C?.2, C?.2, C?.2, C?.2, C?.2, C?.2, C?.2, C?.2, C?.2, C?.2
- net PWR_EN: no longer U?.88 (PG3)
Other:
- moved on the sheet: C?, R?, U?, Y?

Commit message: Connect SPI2 of the microcontroller to the IMU.
Connections:
- net SPI2_CLK: now reaches U?.1 (PE2)
- net SPI2_CS: now reaches U?.2 (PE3)
- net SPI2_MISO: now reaches U?.4 (PE5)
- net SPI2_MOSI: now reaches U?.5 (PE6)
Changed lines of the file:
@@
 Wire Wire Line
 	8750 6850 9200 6850
+Text HLabel 1450 2150 0    50   Output ~ 0
+SPI2_CLK
+Text HLabel 1450 2250 0    50   Output ~ 0
+SPI2_CS
+Text HLabel 1450 2450 0    50   Input ~ 0
+SPI2_MISO
+Text HLabel 1450 2550 0    50   Output ~ 0
+SPI2_MOSI
+Wire Wire Line
+	1450 2150 2050 2150
+Wire Wire Line
+	2050 2250 1450 2250
+Wire Wire Line
+	1450 2450 2050 2450
+Wire Wire Line
+	2050 2550 1450 2550
 $EndSCHEMATC

Commit message: Improve the minimum system circuit of the microcontroller by adding two LEDs and a keypad. Pin out the debug pins of the microcontroller.
Parts:
- added C?: 100nF, symbol Device:C
- added D? (x2): LED, symbol Device:LED
- added K?: SW_DIP_x01, symbol Switch:SW_DIP_x01
- added R? (x2): 1kR, symbol Device:R
- added R? (x2): 10kR, symbol Device:R
Connections:
- net +3V3: now also R?.1, R?.1, R?.1
- net GND: now also C?.2, K?.1, R?.1
- net PWR_EN: now also U?.53 (PF13)
- net UART1_TX: now reaches U?.101 (PA9)
- net UART1_RX: now reaches U?.102 (PA10)
- net SWDIO: now reaches U?.105 (PA13)
- net SWDCLK: now reaches U?.109 (PA14)
- net at U?.138 (PH3): now also R?.2
- net IMU_RST: now reaches U?.142 (PE1)
- net IMU_DR: now reaches U?.3 (PE4)
- net LED1: now reaches U?.49 (PF11)
- net LED1: now also D?.1 (K)
- net LED2: now reaches U?.50 (PF12)
- net LED2: now also D?.1 (K)
- new net: D?.2 (A), R?.2 (x2)
- new net: C?.1, K?.2, R?.2
Other:
- moved on the sheet: C?, R?, Y?

Commit message: Added the debugger's schematic library and improved the circuit of the power section.
Connections:
- net KEY: now reaches U?.93 (PG8)
- net KEY: now also C?.1, K?.2, R?.2
Changed lines of the file:
@@
 	8800 4250 8100 4250
 $Comp
-L power:+3.3V #PWR?
+L power:+3.3V #PWR0225
 U 1 1 61D01329
 P 10150 3850
-F 0 "#PWR?" H 10150 3700 50  0001 C CNN
+F 0 "#PWR0225" H 10150 3700 50  0001 C CNN
 F 1 "+3.3V" V 10150 4100 50  0000 C CNN
 F 2 "" H 10150 3850 50  0001 C CNN
@@
 $EndComp
 $Comp
-L power:+3.3V #PWR?
+L power:+3.3V #PWR0226
 U 1 1 61D01D01
 P 10150 4250
-F 0 "#PWR?" H 10150 4100 50  0001 C CNN
+F 0 "#PWR0226" H 10150 4100 50  0001 C CNN
 F 1 "+3.3V" V 10150 4500 50  0000 C CNN
 F 2 "" H 10150 4250 50  0001 C CNN
@@
 $EndComp
 $Comp
-L power:+3.3V #PWR?
+L power:+3.3V #PWR0227
 U 1 1 61D96B9D
 P 10150 3200
-F 0 "#PWR?" H 10150 3050 50  0001 C CNN
+F 0 "#PWR0227" H 10150 3050 50  0001 C CNN
 F 1 "+3.3V" V 10150 3450 50  0000 C CNN
 F 2 "" H 10150 3200 50  0001 C CNN
@@
 	9450 3200 9650 3200
 $Comp
-L power:GND #PWR?
+L power:GND #PWR0228
 U 1 1 61DE545E
 P 8250 3200
-F 0 "#PWR?" H 8250 2950 50  0001 C CNN
+F 0 "#PWR0228" H 8250 2950 50  0001 C CNN
 F 1 "GND" H 8255 3027 50  0000 C CNN
 F 2 "" H 8250 3200 50  0001 C CNN
@@
 $EndComp
 $Comp
-L power:GND #PWR?
+L power:GND #PWR0229
 U 1 1 61DFA0CD
 P 3050 1100
-F 0 "#PWR?" H 3050 850 50  0001 C CNN
+F 0 "#PWR0229" H 3050 850 50  0001 C CNN
 F 1 "GND" V 3055 972 50  0000 R CNN
 F 2 "" H 3050 1100 50  0001 C CNN
@@
 Wire Wire Line
 	6900 2750 6350 2750
+Text Label 9450 3200 0    50   ~ 0
+KEY
+Text Label 7150 3650 2    50   ~ 0
+KEY
+Wire Wire Line
+	6350 3650 7150 3650
 $EndSCHEMATC

Commit message: Added brushless motor communication interface and LCD control interface.
Connections:
- net SPI1_CLK: now reaches U?.133 (PB3)
- net SPI1_MISO: now reaches U?.134 (PB4)
- net SPI1_MOSI: now reaches U?.135 (PB5)
- net UART3_TX: now reaches U?.77 (PD8)
- net UART3_RX: now reaches U?.78 (PD9)
Changed lines of the file:
@@
 Wire Wire Line
 	6350 3650 7150 3650
+Text HLabel 6850 5250 2    50   Output ~ 0
+UART3_TX
+Text HLabel 6850 5150 2    50   Input ~ 0
+UART3_RX
+Wire Wire Line
+	6850 5150 6350 5150
+Wire Wire Line
+	6350 5250 6850 5250
+Text HLabel 3550 1400 1    50   Output ~ 0
+SPI1_CLK
+Text HLabel 3450 1400 1    50   Input ~ 0
+SPI1_MISO
+Text HLabel 3350 1400 1    50   Output ~ 0
+SPI1_MOSI
+Wire Wire Line
+	3550 1400 3550 1850
+Wire Wire Line
+	3450 1850 3450 1400
+Wire Wire Line
+	3350 1400 3350 1850
 $EndSCHEMATC
