File: circuit/2_MCU.sch (KiCad schematic (older format))
At the start: 26 parts

Commit message: Add annotations to the microcontroller subdiagram.
Other:
- note added: "Filter"
- note added: "LED & KEY"
- note added: "XTAL & RST"
- moved on the sheet: C?, D?, R?, SW?, Y?

Commit message: Assign general-purpose GPIO pins to the LCD. Add annotations to the Connector subdiagram. Label the component markers.
Parts:
- gave numbers to parts that had none: 26
Connections:
- net ADC23_IN14: now reaches U5.44 (PC4)
- net UART6_TX: now reaches U5.46 (PB0)
- net UART6_RX: now reaches U5.47 (PB1)
- net PG2: now reaches U5.87 (PG2)
- net PG3: now reaches U5.88 (PG3)
- net PG4: now reaches U5.89 (PG4)
- net PG5: now reaches U5.90 (PG5)
- net PG6: now reaches U5.91 (PG6)
- net IMU_DR renamed PE4
- net IMU_RST renamed PE1
- net PWR_EN renamed PF13
- net SPI2_CS renamed PE3

Commit message: Add packages for standard components and set the basic rules and layers of the PCB.
Parts:
- C17, C18, C19, C20, C21, C22, C23, C24, C25, C26, C27, C28, C29, C30, C31, C32: footprint (none) -> Capacitor_SMD:C_0603_1608Metric
- D2, D3: footprint (none) -> LED_SMD:LED_0603_1608Metric
- R16, R17, R18, R19, R20: footprint (none) -> Resistor_SMD:R_0603_1608Metric
- SW2: footprint (none) -> Button_Switch_SMD:SW_SPST_CK_RS282G05A3
Changed lines of the file:
@@
 F 0 "C19" H 8315 2096 50  0000 L CNN
 F 1 "18pF" H 8315 2005 50  0000 L CNN
-F 2 "" H 8238 1900 50  0001 C CNN
+F 2 "Capacitor_SMD:C_0603_1608Metric" H 8238 1900 50  0001 C CNN
 F 3 "~" H 8200 2050 50  0001 C CNN
 	1    8200 2050
@@
 F 0 "C25" H 9465 2096 50  0000 L CNN
 F 1 "18pF" H 9465 2005 50  0000 L CNN
-F 2 "" H 9388 1900 50  0001 C CNN
+F 2 "Capacitor_SMD:C_0603_1608Metric" H 9388 1900 50  0001 C CNN
 F 3 "~" H 9350 2050 50  0001 C CNN
 	1    9350 2050
@@
 F 0 "R20" H 10320 1646 50  0000 L CNN
 F 1 "10kR" H 10320 1555 50  0000 L CNN
-F 2 "" V 10180 1600 50  0001 C CNN
+F 2 "Resistor_SMD:R_0603_1608Metric" V 10180 1600 50  0001 C CNN
 F 3 "~" H 10250 1600 50  0001 C CNN
 	1    10250 1600
@@
 F 0 "C30" H 10365 2146 50  0000 L CNN
 F 1 "100nF" H 10365 2055 50  0000 L CNN
-F 2 "" H 10288 1950 50  0001 C CNN
+F 2 "Capacitor_SMD:C_0603_1608Metric" H 10288 1950 50  0001 C CNN
 F 3 "~" H 10250 2100 50  0001 C CNN
 	1    10250 2100
@@
 F 0 "C17" H 8215 5346 50  0000 L CNN
 F 1 "100nF" H 8215 5255 50  0000 L CNN
-F 2 "" H 8138 5150 50  0001 C CNN
+F 2 "Capacitor_SMD:C_0603_1608Metric" H 8138 5150 50  0001 C CNN
 F 3 "~" H 8100 5300 50  0001 C CNN
 	1    8100 5300
@@
 F 0 "C20" H 8665 5346 50  0000 L CNN
 F 1 "100nF" H 8665 5255 50  0000 L CNN
-F 2 "" H 8588 5150 50  0001 C CNN
+F 2 "Capacitor_SMD:C_0603_1608Metric" H 8588 5150 50  0001 C CNN
 F 3 "~" H 8550 5300 50  0001 C CNN
 	1    8550 5300
@@
 F 0 "C22" H 9115 5346 50  0000 L CNN
 F 1 "100nF" H 9115 5255 50  0000 L CNN
-F 2 "" H 9038 5150 50  0001 C CNN
+F 2 "Capacitor_SMD:C_0603_1608Metric" H 9038 5150 50  0001 C CNN
 F 3 "~" H 9000 5300 50  0001 C CNN
 	1    9000 5300
@@
 F 0 "C26" H 9615 5346 50  0000 L CNN
 F 1 "100nF" H 9615 5255 50  0000 L CNN
-F 2 "" H 9538 5150 50  0001 C CNN
+F 2 "Capacitor_SMD:C_0603_1608Metric" H 9538 5150 50  0001 C CNN
 F 3 "~" H 9500 5300 50  0001 C CNN
 	1    9500 5300
@@
 F 0 "C28" H 10065 5346 50  0000 L CNN
 F 1 "100nF" H 10065 5255 50  0000 L CNN
-F 2 "" H 9988 5150 50  0001 C CNN
+F 2 "Capacitor_SMD:C_0603_1608Metric" H 9988 5150 50  0001 C CNN
 F 3 "~" H 9950 5300 50  0001 C CNN
 	1    9950 5300
@@
 F 0 "C31" H 10515 5346 50  0000 L CNN
 F 1 "100nF" H 10515 5255 50  0000 L CNN
-F 2 "" H 10438 5150 50  0001 C CNN
+F 2 "Capacitor_SMD:C_0603_1608Metric" H 10438 5150 50  0001 C CNN
 F 3 "~" H 10400 5300 50  0001 C CNN
 	1    10400 5300
@@
 F 0 "C18" H 8215 6496 50  0000 L CNN
 F 1 "100nF" H 8215 6405 50  0000 L CNN
-F 2 "" H 8138 6300 50  0001 C CNN
+F 2 "Capacitor_SMD:C_0603_1608Metric" H 8138 6300 50  0001 C CNN
 F 3 "~" H 8100 6450 50  0001 C CNN
 	1    8100 6450
@@
 F 0 "C21" H 8665 6496 50  0000 L CNN
 F 1 "100nF" H 8665 6405 50  0000 L CNN
-F 2 "" H 8588 6300 50  0001 C CNN
+F 2 "Capacitor_SMD:C_0603_1608Metric" H 8588 6300 50  0001 C CNN
 F 3 "~" H 8550 6450 50  0001 C CNN
 	1    8550 6450
@@
 F 0 "C23" H 9115 6496 50  0000 L CNN
 F 1 "100nF" H 9115 6405 50  0000 L CNN
-F 2 "" H 9038 6300 50  0001 C CNN
+F 2 "Capacitor_SMD:C_0603_1608Metric" H 9038 6300 50  0001 C CNN
 F 3 "~" H 9000 6450 50  0001 C CNN
 	1    9000 6450
@@
 F 0 "C27" H 9615 6496 50  0000 L CNN
 F 1 "100nF" H 9615 6405 50  0000 L CNN
-F 2 "" H 9538 6300 50  0001 C CNN
+F 2 "Capacitor_SMD:C_0603_1608Metric" H 9538 6300 50  0001 C CNN
 F 3 "~" H 9500 6450 50  0001 C CNN
 	1    9500 6450
@@
 F 0 "C29" H 10065 6496 50  0000 L CNN
 F 1 "100nF" H 10065 6405 50  0000 L CNN
-F 2 "" H 9988 6300 50  0001 C CNN
+F 2 "Capacitor_SMD:C_0603_1608Metric" H 9988 6300 50  0001 C CNN
 F 3 "~" H 9950 6450 50  0001 C CNN
 	1    9950 6450
@@
 F 0 "C32" H 10515 6496 50  0000 L CNN
 F 1 "100nF" H 10515 6405 50  0000 L CNN
-F 2 "" H 10438 6300 50  0001 C CNN
+F 2 "Capacitor_SMD:C_0603_1608Metric" H 10438 6300 50  0001 C CNN
 F 3 "~" H 10400 6450 50  0001 C CNN
 	1    10400 6450
@@
 F 0 "D2" H 8950 3950 50  0000 C CNN
 F 1 "LED" H 8943 3976 50  0001 C CNN
-F 2 "" H 8950 3850 50  0001 C CNN
+F 2 "LED_SMD:LED_0603_1608Metric" H 8950 3850 50  0001 C CNN
 F 3 "~" H 8950 3850 50  0001 C CNN
 	1    8950 3850
@@
 F 0 "D3" H 8950 4200 50  0000 C CNN
 F 1 "LED" H 8943 4226 50  0001 C CNN
-F 2 "" H 8950 4100 50  0001 C CNN
+F 2 "LED_SMD:LED_0603_1608Metric" H 8950 4100 50  0001 C CNN
 F 3 "~" H 8950 4100 50  0001 C CNN
 	1    8950 4100
@@
 F 0 "R17" V 9550 3850 50  0000 C CNN
 F 1 "1kR" V 9700 4050 50  0000 C CNN
-F 2 "" V 9580 3850 50  0001 C CNN
+F 2 "Resistor_SMD:R_0603_1608Metric" V 9580 3850 50  0001 C CNN
 F 3 "~" H 9650 3850 50  0001 C CNN
 	1    9650 3850
@@
 F 0 "R18" V 9550 4100 50  0000 C CNN
 F 1 "1kR" V 9700 4300 50  0000 C CNN
-F 2 "" V 9580 4100 50  0001 C CNN
+F 2 "Resistor_SMD:R_0603_1608Metric" V 9580 4100 50  0001 C CNN
 F 3 "~" H 9650 4100 50  0001 C CNN
 	1    9650 4100
@@
 F 0 "SW2" H 9050 3400 50  0000 C CNN
 F 1 "SW_DIP_x01" H 9050 3476 50  0001 C CNN
-F 2 "" H 9050 3300 50  0001 C CNN
+F 2 "Button_Switch_SMD:SW_SPST_CK_RS282G05A3" H 9050 3300 50  0001 C CNN
 F 3 "~" H 9050 3300 50  0001 C CNN
 	1    9050 3300
@@
 F 0 "R19" V 9593 3500 50  0000 C CNN
 F 1 "10kR" V 9684 3500 50  0000 C CNN
-F 2 "" V 9730 3500 50  0001 C CNN
+F 2 "Resistor_SMD:R_0603_1608Metric" V 9730 3500 50  0001 C CNN
 F 3 "~" H 9800 3500 50  0001 C CNN
 	1    9800 3500
@@
 F 0 "C24" V 9165 3546 50  0000 L CNN
 F 1 "100nF" V 9250 3550 50  0000 L CNN
-F 2 "" H 9088 3350 50  0001 C CNN
+F 2 "Capacitor_SMD:C_0603_1608Metric" H 9088 3350 50  0001 C CNN
 F 3 "~" H 9050 3500 50  0001 C CNN
 	1    9050 3500
@@
 F 0 "R16" H 3120 1546 50  0000 L CNN
 F 1 "10kR" H 3120 1455 50  0000 L CNN
-F 2 "" V 2980 1500 50  0001 C CNN
+F 2 "Resistor_SMD:R_0603_1608Metric" V 2980 1500 50  0001 C CNN
 F 3 "~" H 3050 1500 50  0001 C CNN
 	1    3050 1500

Commit message: Eliminate design rule errors in schematics.
Connections:
- no-connect marks 0 -> 86
Changed lines of the file:
@@
 Wire Wire Line
 	7000 4250 6350 4250
+NoConn ~ 4750 5950
+NoConn ~ 4650 5950
+NoConn ~ 4550 5950
+NoConn ~ 4450 5950
+NoConn ~ 4350 5950
+NoConn ~ 4250 5950
+NoConn ~ 4150 5950
+NoConn ~ 3550 5950
+NoConn ~ 3250 5950
+NoConn ~ 3050 5950
+NoConn ~ 2950 5950
+NoConn ~ 2850 5950
+NoConn ~ 2750 5950
+NoConn ~ 2450 5950
+NoConn ~ 2050 5450
+NoConn ~ 2050 5550
+NoConn ~ 2050 5650
+NoConn ~ 5750 5950
+NoConn ~ 5650 5950
+NoConn ~ 5550 5950
+NoConn ~ 5450 5950
+NoConn ~ 5350 5950
+NoConn ~ 5250 5950
+NoConn ~ 5150 5950
+NoConn ~ 5050 5950
+NoConn ~ 6350 5650
+NoConn ~ 6350 5550
+NoConn ~ 6350 5450
+NoConn ~ 6350 5350
+NoConn ~ 6350 5050
+NoConn ~ 6350 4950
+NoConn ~ 6350 4850
+NoConn ~ 6350 4750
+NoConn ~ 6350 4450
+NoConn ~ 6350 4350
+NoConn ~ 6350 3750
+NoConn ~ 6350 3350
+NoConn ~ 6350 3250
+NoConn ~ 6350 3150
+NoConn ~ 6350 3050
+NoConn ~ 6350 2950
+NoConn ~ 6350 2650
+NoConn ~ 6350 2550
+NoConn ~ 6350 2350
+NoConn ~ 5850 1850
+NoConn ~ 4950 1850
+NoConn ~ 5050 1850
+NoConn ~ 5150 1850
+NoConn ~ 5250 1850
+NoConn ~ 5350 1850
+NoConn ~ 5450 1850
+NoConn ~ 5550 1850
+NoConn ~ 5650 1850
+NoConn ~ 5750 1850
+NoConn ~ 2750 1850
+NoConn ~ 2850 1850
+NoConn ~ 2950 1850
+NoConn ~ 3150 1850
+NoConn ~ 3250 1850
+NoConn ~ 3650 1850
+NoConn ~ 3950 1850
+NoConn ~ 4050 1850
+NoConn ~ 4150 1850
+NoConn ~ 4250 1850
+NoConn ~ 4350 1850
+NoConn ~ 4450 1850
+NoConn ~ 4550 1850
+NoConn ~ 4650 1850
+NoConn ~ 2050 3550
+NoConn ~ 2050 3450
+NoConn ~ 2050 3350
+NoConn ~ 2050 3250
+NoConn ~ 2050 3150
+NoConn ~ 2050 3050
+NoConn ~ 2050 2950
+NoConn ~ 2050 2850
+NoConn ~ 2050 2750
+NoConn ~ 2050 3850
+NoConn ~ 2050 3950
+NoConn ~ 2050 4050
+NoConn ~ 2050 4150
+NoConn ~ 2050 4250
+NoConn ~ 2050 4650
+NoConn ~ 2050 4750
+NoConn ~ 2050 4850
+NoConn ~ 2050 4950
 $EndSCHEMATC

Commit message: Add Servo Interface
Connections:
- net TIM1_CH1: now reaches U5.60 (PE9)
- no-connect marks 86 -> 85
Changed lines of the file:
@@
 Wire Wire Line
 	7000 4250 6350 4250
-NoConn ~ 4750 5950
 NoConn ~ 4650 5950
 NoConn ~ 4550 5950
@@
 NoConn ~ 2050 4850
 NoConn ~ 2050 4950
+Text HLabel 4750 6400 3    50   Output ~ 0
+TIM1_CH1
+Wire Wire Line
+	4750 6400 4750 5950
 $EndSCHEMATC

Commit message: Adjust the pin order to make the wiring smoother.
Connections:
- net KEY: now also U5.54 (PF14); no longer U5.93 (PG8)
- net PG15: now reaches U5.132 (PG15)
- net PB6: now reaches U5.136 (PB6)
- net PB7: now reaches U5.137 (PB7)
- net PB9: now reaches U5.140 (PB9)
- net PE0: now reaches U5.141 (PE0)
- net PG2: no longer names the net of U5.87 (PG2)
- net PG3: no longer names the net of U5.88 (PG3)
- net PG4: no longer names the net of U5.89 (PG4)
- net PG5: no longer names the net of U5.90 (PG5)
- net PG6: no longer names the net of U5.91 (PG6)
- no-connect marks 85 -> 84
Changed lines of the file:
@@
 Text HLabel 1450 2150 0    50   Output ~ 0
 SPI2_CLK
-Text HLabel 1450 2250 0    50   Output ~ 0
-PE3
 Text HLabel 1450 2450 0    50   Input ~ 0
 SPI2_MISO
@@
 Wire Wire Line
 	1450 2150 2050 2150
-Wire Wire Line
-	2050 2250 1450 2250
 Wire Wire Line
 	1450 2450 2050 2450
@@
 Wire Wire Line
 	3650 5950 3650 6750
-Text HLabel 1450 2350 0    50   Input ~ 0
-PE4
-Wire Wire Line
-	1450 2350 2050 2350
-Text HLabel 2650 1350 1    50   Output ~ 0
-PE1
-Wire Wire Line
-	2650 1350 2650 1850
+Text HLabel 3250 1200 1    50   Output ~ 0
+PB6
+Wire Wire Line
+	3250 1200 3250 1850
 Wire Wire Line
 	4050 6450 4050 5950
@@
 Text Label 9450 3500 0    50   ~ 0
 KEY
-Text Label 7150 3650 2    50   ~ 0
+Text Label 4150 6750 1    50   ~ 0
 KEY
 Wire Wire Line
-	6350 3650 7150 3650
+	4150 6750 4150 5950
 Text HLabel 6850 5250 2    50   Output ~ 0
 UART3_TX
@@
 Wire Wire Line
 	3150 6300 3150 5950
-Text HLabel 7000 4250 2    50   Input ~ 0
-PG2
-Text HLabel 7000 4150 2    50   Output ~ 0
-PG3
-Text HLabel 7000 4050 2    50   Output ~ 0
-PG4
-Text HLabel 7000 3950 2    50   Output ~ 0
-PG5
-Text HLabel 7000 3850 2    50   Output ~ 0
-PG6
-Wire Wire Line
-	7000 3850 6350 3850
-Wire Wire Line
-	6350 3950 7000 3950
-Wire Wire Line
-	7000 4050 6350 4050
-Wire Wire Line
-	6350 4150 7000 4150
-Wire Wire Line
-	7000 4250 6350 4250
+Text HLabel 2750 1200 1    50   Input ~ 0
+PE0
+Text HLabel 2650 1200 1    50   Output ~ 0
+PE1
+Text HLabel 2850 1200 1    50   Output ~ 0
+PB9
+Wire Wire Line
+	2850 1200 2850 1850
+Wire Wire Line
+	2650 1850 2650 1200
+Wire Wire Line
+	2750 1200 2750 1850
 NoConn ~ 4650 5950
 NoConn ~ 4550 5950
@@
 NoConn ~ 4350 5950
 NoConn ~ 4250 5950
-NoConn ~ 4150 5950
 NoConn ~ 3550 5950
 NoConn ~ 3250 5950
@@
 NoConn ~ 5650 1850
 NoConn ~ 5750 1850
-NoConn ~ 2750 1850
-NoConn ~ 2850 1850
 NoConn ~ 2950 1850
-NoConn ~ 3150 1850
-NoConn ~ 3250 1850
-NoConn ~ 3650 1850
-NoConn ~ 3950 1850
-NoConn ~ 4050 1850
-NoConn ~ 4150 1850
-NoConn ~ 4250 1850
-NoConn ~ 4350 1850
 NoConn ~ 4450 1850
 NoConn ~ 4550 1850
@@
 Wire Wire Line
 	4750 6400 4750 5950
+NoConn ~ 6350 3850
+NoConn ~ 6350 3950
+NoConn ~ 6350 4050
+NoConn ~ 6350 4150
+NoConn ~ 6350 4250
+Text HLabel 3150 1200 1    50   Output ~ 0
+PB7
+Wire Wire Line
+	3150 1200 3150 1850
+Text HLabel 3650 1200 1    50   Input ~ 0
+PG15
+Wire Wire Line
+	3650 1200 3650 1850
+Text HLabel 1450 2250 0    50   Output ~ 0
+PE3
+Wire Wire Line
+	1450 2250 2050 2250
+Text HLabel 1450 2350 0    50   Output ~ 0
+PE4
+Wire Wire Line
+	1450 2350 2050 2350
+NoConn ~ 4050 1850
+NoConn ~ 4150 1850
+NoConn ~ 3950 1850
+NoConn ~ 4350 1850
+NoConn ~ 4250 1850
 $EndSCHEMATC

Commit message: Modify the circuit to modify the electronic switch section to disconnect via microcontroller control.
Connections:
- net KEY: now also U5.55 (PF15); no longer U5.54 (PF14)
- new net PF14: U5.54 (PF14)
- no-connect marks 84 -> 83
Changed lines of the file:
@@
 Sheet 3 5
 Title "MM32_Board"
-Date "2021-12-01"
-Rev "1.0.1"
+Date "2021-12-21"
+Rev "1.0.2"
 Comp ""
 Comment1 ""
@@
 Wire Wire Line
 	1300 4550 2050 4550
-Text HLabel 4050 6450 3    50   Input ~ 0
+Text HLabel 4050 6450 3    50   Output ~ 0
 PF13
 $Comp
@@
 Text Label 9450 3500 0    50   ~ 0
 KEY
-Text Label 4150 6750 1    50   ~ 0
+Text Label 4250 6750 1    50   ~ 0
 KEY
 Wire Wire Line
-	4150 6750 4150 5950
+	4250 6750 4250 5950
 Text HLabel 6850 5250 2    50   Output ~ 0
 UART3_TX
@@
 NoConn ~ 4450 5950
 NoConn ~ 4350 5950
-NoConn ~ 4250 5950
 NoConn ~ 3550 5950
 NoConn ~ 3250 5950
@@
 NoConn ~ 4350 1850
 NoConn ~ 4250 1850
+Text HLabel 4150 6450 3    50   Input ~ 0
+PF14
+Wire Wire Line
+	4150 6450 4150 5950
 $EndSCHEMATC
