File: circuit/project.sch (KiCad schematic (older format))
At the start: 0 parts

Commit message: Connect SPI2 of the microcontroller to the IMU.
Changed lines of the file:
@@
 $EndSheet
 $Sheet
-S 2650 700  1850 1600
+S 2550 700  1850 1600
 U 6194FB75
 F0 "MCU" 50
 F1 "2_MCU.sch" 50
-F2 "PWR_EN" I L 2650 1000 50
+F2 "PWR_EN" I L 2550 1000 50
+F3 "SPI2_CS" O R 4400 1450 50
+F4 "SPI2_MISO" I R 4400 1350 50
+F5 "SPI2_MOSI" O R 4400 1250 50
+F6 "SPI2_CLK" O R 4400 1150 50
 $EndSheet
 $Sheet
-S 4750 700  1400 1600
+S 5150 700  1400 1600
 U 61A493C9
 F0 "IMU" 50
 F1 "3_IMU.sch" 50
+F2 "IMU_CS" I L 5150 1450 50
+F3 "IMU_RST" I L 5150 1600 50
+F4 "IMU_DR" O L 5150 1700 50
+F5 "IMU_CLK" I L 5150 1150 50
+F6 "IMU_MOSI" I L 5150 1250 50
+F7 "IMU_MISO" O L 5150 1350 50
 $EndSheet
+Wire Wire Line
+	4400 1150 5150 1150
+Wire Wire Line
+	4400 1250 5150 1250
+Wire Wire Line
+	5150 1350 4400 1350
+Wire Wire Line
+	4400 1450 5150 1450
 $EndSCHEMATC

Commit message: Improve the minimum system circuit of the microcontroller by adding two LEDs and a keypad. Pin out the debug pins of the microcontroller.
Changed lines of the file:
@@
 F5 "SPI2_MOSI" O R 4400 1250 50
 F6 "SPI2_CLK" O R 4400 1150 50
+F7 "IMU_DR" I R 4400 1700 50
+F8 "IMU_RST" O R 4400 1600 50
+F9 "SWDIO" B L 2550 2100 50
+F10 "SWDCLK" I L 2550 2000 50
+F11 "UART1_TX" O L 2550 1900 50
+F12 "UART1_RX" I L 2550 1800 50
 $EndSheet
 $Sheet
@@
 Wire Wire Line
 	4400 1450 5150 1450
+Wire Wire Line
+	4400 1600 5150 1600
+Wire Wire Line
+	5150 1700 4400 1700
+Wire Wire Line
+	2200 1000 2550 1000
 $EndSCHEMATC

Commit message: Added servo power supply circuit and organized top-level schematic.
Changed lines of the file:
@@
 $Descr A4 11693 8268
 encoding utf-8
-Sheet 1 4
+Sheet 1 5
 Title "MM32_Board"
 Date "2021-11-14"
@@
 $EndDescr
 $Sheet
-S 900  700  1300 1000
+S 3150 3300 1300 500
 U 6191448D
 F0 "Power" 50
 F1 "1_Power.sch" 50
-F2 "PWR_EN" I R 2200 1000 50
+F2 "PWR_EN" I R 4450 3600 50
 $EndSheet
 $Sheet
-S 2550 700  1850 1600
+S 4800 3300 1800 1900
 U 6194FB75
 F0 "MCU" 50
 F1 "2_MCU.sch" 50
-F2 "PWR_EN" I L 2550 1000 50
-F3 "SPI2_CS" O R 4400 1450 50
-F4 "SPI2_MISO" I R 4400 1350 50
-F5 "SPI2_MOSI" O R 4400 1250 50
-F6 "SPI2_CLK" O R 4400 1150 50
-F7 "IMU_DR" I R 4400 1700 50
-F8 "IMU_RST" O R 4400 1600 50
-F9 "SWDIO" B L 2550 2100 50
-F10 "SWDCLK" I L 2550 2000 50
-F11 "UART1_TX" O L 2550 1900 50
-F12 "UART1_RX" I L 2550 1800 50
+F2 "PWR_EN" I L 4800 3600 50
+F3 "SPI2_CLK" O L 4800 4300 50
+F4 "SPI2_CS" O L 4800 4200 50
+F5 "SPI2_MISO" I L 4800 4500 50
+F6 "SPI2_MOSI" O L 4800 4400 50
+F7 "IMU_DR" I L 4800 4900 50
+F8 "IMU_RST" O L 4800 4800 50
+F9 "SWDIO" B R 6600 3400 50
+F10 "SWDCLK" I R 6600 3500 50
+F11 "UART1_TX" O R 6600 3600 50
+F12 "UART1_RX" I R 6600 3700 50
 $EndSheet
 $Sheet
-S 5150 700  1400 1600
+S 3150 4050 1300 1150
 U 61A493C9
 F0 "IMU" 50
 F1 "3_IMU.sch" 50
-F2 "IMU_CS" I L 5150 1450 50
-F3 "IMU_RST" I L 5150 1600 50
-F4 "IMU_DR" O L 5150 1700 50
-F5 "IMU_CLK" I L 5150 1150 50
-F6 "IMU_MOSI" I L 5150 1250 50
-F7 "IMU_MISO" O L 5150 1350 50
+F2 "IMU_CS" I R 4450 4200 50
+F3 "IMU_RST" I R 4450 4800 50
+F4 "IMU_DR" O R 4450 4900 50
+F5 "IMU_CLK" I R 4450 4300 50
+F6 "IMU_MOSI" I R 4450 4400 50
+F7 "IMU_MISO" O R 4450 4500 50
 $EndSheet
 Wire Wire Line
-	4400 1150 5150 1150
+	4450 3600 4800 3600
+$Sheet
+S 7000 3300 1050 1900
+U 61E2DD2B
+F0 "Connector" 50
+F1 "4_Connector.sch" 50
+$EndSheet
 Wire Wire Line
-	4400 1250 5150 1250
+	4450 4200 4800 4200
 Wire Wire Line
-	5150 1350 4400 1350
+	4450 4300 4800 4300
 Wire Wire Line
-	4400 1450 5150 1450
+	4450 4400 4800 4400
 Wire Wire Line
-	4400 1600 5150 1600
+	4450 4500 4800 4500
 Wire Wire Line
-	5150 1700 4400 1700
+	4800 4800 4450 4800
 Wire Wire Line
-	2200 1000 2550 1000
+	4450 4900 4800 4900
 $EndSCHEMATC

Commit message: Added the debugger's schematic library and improved the circuit of the power section.
Changed lines of the file:
@@
 F0 "Power" 50
 F1 "1_Power.sch" 50
-F2 "PWR_EN" I R 4450 3600 50
+F2 "PWR_EN" I R 4450 3550 50
 $EndSheet
 $Sheet
@@
 F0 "MCU" 50
 F1 "2_MCU.sch" 50
-F2 "PWR_EN" I L 4800 3600 50
+F2 "PWR_EN" I L 4800 3550 50
 F3 "SPI2_CLK" O L 4800 4300 50
 F4 "SPI2_CS" O L 4800 4200 50
@@
 $EndSheet
 Wire Wire Line
-	4450 3600 4800 3600
+	4450 3550 4800 3550
 $Sheet
 S 7000 3300 1050 1900
@@
 F0 "Connector" 50
 F1 "4_Connector.sch" 50
+F2 "SWDIO" B L 7000 3400 50
+F3 "SWDCLK" O L 7000 3500 50
+F4 "UART_TX" O L 7000 3700 50
+F5 "UART_RX" I L 7000 3600 50
 $EndSheet
 Wire Wire Line
@@
 Wire Wire Line
 	4450 4900 4800 4900
+Wire Wire Line
+	6600 3400 7000 3400
+Wire Wire Line
+	7000 3500 6600 3500
+Wire Wire Line
+	6600 3600 7000 3600
+Wire Wire Line
+	7000 3700 6600 3700
 $EndSCHEMATC

Commit message: Added brushless motor communication interface and LCD control interface.
Changed lines of the file:
@@
 $EndDescr
 $Sheet
-S 3150 3300 1300 500
+S 3850 3200 700  500
 U 6191448D
 F0 "Power" 50
 F1 "1_Power.sch" 50
-F2 "PWR_EN" I R 4450 3550 50
+F2 "PWR_EN" I R 4550 3450 50
 $EndSheet
 $Sheet
-S 4800 3300 1800 1900
+S 4950 3200 1800 1900
 U 6194FB75
 F0 "MCU" 50
 F1 "2_MCU.sch" 50
-F2 "PWR_EN" I L 4800 3550 50
-F3 "SPI2_CLK" O L 4800 4300 50
-F4 "SPI2_CS" O L 4800 4200 50
-F5 "SPI2_MISO" I L 4800 4500 50
-F6 "SPI2_MOSI" O L 4800 4400 50
-F7 "IMU_DR" I L 4800 4900 50
-F8 "IMU_RST" O L 4800 4800 50
-F9 "SWDIO" B R 6600 3400 50
-F10 "SWDCLK" I R 6600 3500 50
-F11 "UART1_TX" O R 6600 3600 50
-F12 "UART1_RX" I R 6600 3700 50
+F2 "PWR_EN" I L 4950 3450 50
+F3 "SPI2_CLK" O L 4950 4300 50
+F4 "SPI2_CS" O L 4950 4200 50
+F5 "SPI2_MISO" I L 4950 4500 50
+F6 "SPI2_MOSI" O L 4950 4400 50
+F7 "IMU_DR" I L 4950 4900 50
+F8 "IMU_RST" O L 4950 4800 50
+F9 "SWDIO" B R 6750 3300 50
+F10 "SWDCLK" I R 6750 3400 50
+F11 "UART1_TX" O R 6750 3500 50
+F12 "UART1_RX" I R 6750 3600 50
+F13 "UART3_TX" O R 6750 3900 50
+F14 "UART3_RX" I R 6750 3800 50
+F15 "SPI1_CLK" O R 6750 4600 50
+F16 "SPI1_MISO" I R 6750 4400 50
+F17 "SPI1_MOSI" O R 6750 4500 50
 $EndSheet
 $Sheet
-S 3150 4050 1300 1150
+S 3850 3950 700  1150
 U 61A493C9
 F0 "IMU" 50
 F1 "3_IMU.sch" 50
-F2 "IMU_CS" I R 4450 4200 50
-F3 "IMU_RST" I R 4450 4800 50
-F4 "IMU_DR" O R 4450 4900 50
-F5 "IMU_CLK" I R 4450 4300 50
-F6 "IMU_MOSI" I R 4450 4400 50
-F7 "IMU_MISO" O R 4450 4500 50
+F2 "IMU_CS" I R 4550 4200 50
+F3 "IMU_RST" I R 4550 4800 50
+F4 "IMU_DR" O R 4550 4900 50
+F5 "IMU_CLK" I R 4550 4300 50
+F6 "IMU_MOSI" I R 4550 4400 50
+F7 "IMU_MISO" O R 4550 4500 50
 $EndSheet
 Wire Wire Line
-	4450 3550 4800 3550
+	4550 3450 4950 3450
 $Sheet
-S 7000 3300 1050 1900
+S 7150 3200 800  1900
 U 61E2DD2B
 F0 "Connector" 50
 F1 "4_Connector.sch" 50
-F2 "SWDIO" B L 7000 3400 50
-F3 "SWDCLK" O L 7000 3500 50
-F4 "UART_TX" O L 7000 3700 50
-F5 "UART_RX" I L 7000 3600 50
+F2 "SWDIO" B L 7150 3300 50
+F3 "SWDCLK" O L 7150 3400 50
+F4 "LCD_CS" I L 7150 4950 50
+F5 "LCD_CLK" I L 7150 4600 50
+F6 "LCD_MOSI" I L 7150 4500 50
+F7 "LCD_A0" I L 7150 4850 50
+F8 "LCD_RST" I L 7150 4750 50
+F9 "LCD_MISO" O L 7150 4400 50
+F10 "TOUCH_CS" I L 7150 5050 50
+F11 "DEBUG_TX" O L 7150 3600 50
+F12 "DEBUG_RX" I L 7150 3500 50
+F13 "MOTOR_TX" I L 7150 3800 50
+F14 "MOTOR_RX" O L 7150 3900 50
 $EndSheet
 Wire Wire Line
-	4450 4200 4800 4200
+	4550 4200 4950 4200
 Wire Wire Line
-	4450 4300 4800 4300
+	4550 4300 4950 4300
 Wire Wire Line
-	4450 4400 4800 4400
+	4550 4400 4950 4400
 Wire Wire Line
-	4450 4500 4800 4500
+	4550 4500 4950 4500
 Wire Wire Line
-	4800 4800 4450 4800
+	4950 4800 4550 4800
 Wire Wire Line
-	4450 4900 4800 4900
+	4550 4900 4950 4900
 Wire Wire Line
-	6600 3400 7000 3400
+	6750 3300 7150 3300
 Wire Wire Line
-	7000 3500 6600 3500
+	7150 3400 6750 3400
 Wire Wire Line
-	6600 3600 7000 3600
+	6750 3500 7150 3500
 Wire Wire Line
-	7000 3700 6600 3700
+	7150 3600 6750 3600
+Wire Wire Line
+	6750 3800 7150 3800
+Wire Wire Line
+	6750 3900 7150 3900
+Wire Wire Line
+	6750 4400 7150 4400
+Wire Wire Line
+	6750 4500 7150 4500
+Wire Wire Line
+	6750 4600 7150 4600
 $EndSCHEMATC

Commit message: Add the battery voltage detection circuit and complete the circuit connection of XPT2046.
Changed lines of the file:
@@
 F0 "Power" 50
 F1 "1_Power.sch" 50
-F2 "PWR_EN" I R 4550 3450 50
+F2 "PWR_EN" I R 4550 3400 50
+F3 "VBAT" O R 4550 3500 50
 $EndSheet
 $Sheet
@@
 F0 "MCU" 50
 F1 "2_MCU.sch" 50
-F2 "PWR_EN" I L 4950 3450 50
+F2 "PWR_EN" I L 4950 3400 50
 F3 "SPI2_CLK" O L 4950 4300 50
 F4 "SPI2_CS" O L 4950 4200 50
@@
 F13 "UART3_TX" O R 6750 3900 50
 F14 "UART3_RX" I R 6750 3800 50
-F15 "SPI1_CLK" O R 6750 4600 50
-F16 "SPI1_MISO" I R 6750 4400 50
-F17 "SPI1_MOSI" O R 6750 4500 50
+F15 "SPI1_CLK" O R 6750 4250 50
+F16 "SPI1_MISO" I R 6750 4050 50
+F17 "SPI1_MOSI" O R 6750 4150 50
 $EndSheet
 $Sheet
@@
 $EndSheet
 Wire Wire Line
-	4550 3450 4950 3450
+	4550 3400 4950 3400
 $Sheet
 S 7150 3200 800  1900
@@
 F2 "SWDIO" B L 7150 3300 50
 F3 "SWDCLK" O L 7150 3400 50
-F4 "LCD_CS" I L 7150 4950 50
-F5 "LCD_CLK" I L 7150 4600 50
-F6 "LCD_MOSI" I L 7150 4500 50
-F7 "LCD_A0" I L 7150 4850 50
-F8 "LCD_RST" I L 7150 4750 50
-F9 "LCD_MISO" O L 7150 4400 50
-F10 "TOUCH_CS" I L 7150 5050 50
+F4 "LCD_CS" I L 7150 4600 50
+F5 "LCD_CLK" I L 7150 4250 50
+F6 "LCD_MOSI" I L 7150 4150 50
+F7 "LCD_A0" I L 7150 4500 50
+F8 "LCD_RST" I L 7150 4400 50
+F9 "LCD_MISO" O L 7150 4050 50
+F10 "TOUCH_CS" I L 7150 4700 50
 F11 "DEBUG_TX" O L 7150 3600 50
 F12 "DEBUG_RX" I L 7150 3500 50
 F13 "MOTOR_TX" I L 7150 3800 50
 F14 "MOTOR_RX" O L 7150 3900 50
+F15 "TOUCH_IT" O L 7150 4800 50
 $EndSheet
 Wire Wire Line
@@
 	6750 3900 7150 3900
 Wire Wire Line
-	6750 4400 7150 4400
+	6750 4050 7150 4050
 Wire Wire Line
-	6750 4500 7150 4500
+	6750 4150 7150 4150
 Wire Wire Line
-	6750 4600 7150 4600
+	6750 4250 7150 4250
 $EndSCHEMATC

Commit message: Add GPS module circuit.
Changed lines of the file:
@@
 $EndSheet
 $Sheet
-S 4950 3200 1800 1900
+S 4950 3200 1800 2000
 U 6194FB75
 F0 "MCU" 50
@@
 F13 "UART3_TX" O R 6750 3900 50
 F14 "UART3_RX" I R 6750 3800 50
-F15 "SPI1_CLK" O R 6750 4250 50
-F16 "SPI1_MISO" I R 6750 4050 50
-F17 "SPI1_MOSI" O R 6750 4150 50
+F15 "SPI1_CLK" O R 6750 4550 50
+F16 "SPI1_MISO" I R 6750 4350 50
+F17 "SPI1_MOSI" O R 6750 4450 50
 $EndSheet
 $Sheet
@@
 	4550 3400 4950 3400
 $Sheet
-S 7150 3200 800  1900
+S 7150 3200 800  2000
 U 61E2DD2B
 F0 "Connector" 50
@@
 F2 "SWDIO" B L 7150 3300 50
 F3 "SWDCLK" O L 7150 3400 50
-F4 "LCD_CS" I L 7150 4600 50
-F5 "LCD_CLK" I L 7150 4250 50
-F6 "LCD_MOSI" I L 7150 4150 50
-F7 "LCD_A0" I L 7150 4500 50
-F8 "LCD_RST" I L 7150 4400 50
-F9 "LCD_MISO" O L 7150 4050 50
-F10 "TOUCH_CS" I L 7150 4700 50
+F4 "LCD_CS" I L 7150 4900 50
+F5 "LCD_CLK" I L 7150 4550 50
+F6 "LCD_MOSI" I L 7150 4450 50
+F7 "LCD_A0" I L 7150 4800 50
+F8 "LCD_RST" I L 7150 4700 50
+F9 "LCD_MISO" O L 7150 4350 50
+F10 "TOUCH_CS" I L 7150 5000 50
 F11 "DEBUG_TX" O L 7150 3600 50
 F12 "DEBUG_RX" I L 7150 3500 50
 F13 "MOTOR_TX" I L 7150 3800 50
 F14 "MOTOR_RX" O L 7150 3900 50
-F15 "TOUCH_IT" O L 7150 4800 50
+F15 "TOUCH_IT" O L 7150 5100 50
+F16 "GPS_RXD" I L 7150 4050 50
+F17 "GPS_TXD" O L 7150 4150 50
 $EndSheet
 Wire Wire Line
@@
 	6750 3900 7150 3900
 Wire Wire Line
-	6750 4050 7150 4050
+	6750 4350 7150 4350
 Wire Wire Line
-	6750 4150 7150 4150
+	6750 4450 7150 4450
 Wire Wire Line
-	6750 4250 7150 4250
+	6750 4550 7150 4550
 $EndSCHEMATC

Commit message: Assign general-purpose GPIO pins to the LCD. Add annotations to the Connector subdiagram. Label the component markers.
Changed lines of the file:
@@
 F0 "MCU" 50
 F1 "2_MCU.sch" 50
-F2 "PWR_EN" I L 4950 3400 50
-F3 "SPI2_CLK" O L 4950 4300 50
-F4 "SPI2_CS" O L 4950 4200 50
-F5 "SPI2_MISO" I L 4950 4500 50
-F6 "SPI2_MOSI" O L 4950 4400 50
-F7 "IMU_DR" I L 4950 4900 50
-F8 "IMU_RST" O L 4950 4800 50
-F9 "SWDIO" B R 6750 3300 50
-F10 "SWDCLK" I R 6750 3400 50
-F11 "UART1_TX" O R 6750 3500 50
-F12 "UART1_RX" I R 6750 3600 50
-F13 "UART3_TX" O R 6750 3900 50
-F14 "UART3_RX" I R 6750 3800 50
-F15 "SPI1_CLK" O R 6750 4550 50
-F16 "SPI1_MISO" I R 6750 4350 50
-F17 "SPI1_MOSI" O R 6750 4450 50
+F2 "SPI2_CLK" O L 4950 4300 50
+F3 "SPI2_MISO" I L 4950 4500 50
+F4 "SPI2_MOSI" O L 4950 4400 50
+F5 "SWDIO" B R 6750 3300 50
+F6 "SWDCLK" I R 6750 3400 50
+F7 "UART1_TX" O R 6750 3500 50
+F8 "UART1_RX" I R 6750 3600 50
+F9 "UART3_TX" O R 6750 3900 50
+F10 "UART3_RX" I R 6750 3800 50
+F11 "SPI1_CLK" O R 6750 4550 50
+F12 "SPI1_MISO" I R 6750 4350 50
+F13 "SPI1_MOSI" O R 6750 4450 50
+F14 "UART6_TX" O R 6750 4050 50
+F15 "UART6_RX" I R 6750 4150 50
+F16 "PF13" I L 4950 3400 50
+F17 "PE3" O L 4950 4200 50
+F18 "PE4" I L 4950 4900 50
+F19 "PE1" O L 4950 4800 50
+F20 "PG2" I R 6750 5100 50
+F21 "PG3" O R 6750 5000 50
+F22 "PG4" O R 6750 4900 50
+F23 "PG5" O R 6750 4800 50
+F24 "PG6" O R 6750 4700 50
+F25 "ADC23_IN14" I L 4950 3500 50
 $EndSheet
 $Sheet
-S 3850 3950 700  1150
+S 3850 3950 700  1250
 U 61A493C9
 F0 "IMU" 50
@@
 F14 "MOTOR_RX" O L 7150 3900 50
 F15 "TOUCH_IT" O L 7150 5100 50
-F16 "GPS_RXD" I L 7150 4050 50
-F17 "GPS_TXD" O L 7150 4150 50
+F16 "GPS_RX" I L 7150 4050 50
+F17 "GPS_TX" O L 7150 4150 50
 $EndSheet
 Wire Wire Line
@@
 Wire Wire Line
 	6750 4550 7150 4550
+Wire Wire Line
+	6750 4050 7150 4050
+Wire Wire Line
+	7150 4150 6750 4150
+Wire Wire Line
+	4550 3500 4950 3500
+Wire Wire Line
+	6750 4700 7150 4700
+Wire Wire Line
+	7150 4800 6750 4800
+Wire Wire Line
+	6750 4900 7150 4900
+Wire Wire Line
+	7150 5000 6750 5000
+Wire Wire Line
+	6750 5100 7150 5100
 $EndSCHEMATC
