File: circuit/project.sch (KiCad schematic (older format))
At the start: 0 parts

Commit message: Add Servo Interface
Changed lines of the file:
@@
 $EndSheet
 $Sheet
-S 4950 3200 1800 2000
+S 4950 3200 1800 2200
 U 6194FB75
 F0 "MCU" 50
 F1 "2_MCU.sch" 50
-F2 "SPI2_CLK" O L 4950 4300 50
-F3 "SPI2_MISO" I L 4950 4500 50
-F4 "SPI2_MOSI" O L 4950 4400 50
+F2 "SPI2_CLK" O L 4950 4400 50
+F3 "SPI2_MISO" I L 4950 4600 50
+F4 "SPI2_MOSI" O L 4950 4500 50
 F5 "SWDIO" B R 6750 3300 50
 F6 "SWDCLK" I R 6750 3400 50
@@
 F15 "UART6_RX" I R 6750 4150 50
 F16 "PF13" I L 4950 3400 50
-F17 "PE3" O L 4950 4200 50
-F18 "PE4" I L 4950 4900 50
-F19 "PE1" O L 4950 4800 50
+F17 "PE3" O L 4950 4300 50
+F18 "PE4" I L 4950 5000 50
+F19 "PE1" O L 4950 4900 50
 F20 "PG2" I R 6750 5100 50
 F21 "PG3" O R 6750 5000 50
@@
 F24 "PG6" O R 6750 4700 50
 F25 "ADC23_IN14" I L 4950 3500 50
+F26 "TIM1_CH1" O R 6750 5250 50
 $EndSheet
 $Sheet
-S 3850 3950 700  1250
+S 3850 4050 700  1350
 U 61A493C9
 F0 "IMU" 50
 F1 "3_IMU.sch" 50
-F2 "IMU_CS" I R 4550 4200 50
-F3 "IMU_RST" I R 4550 4800 50
-F4 "IMU_DR" O R 4550 4900 50
-F5 "IMU_CLK" I R 4550 4300 50
-F6 "IMU_MOSI" I R 4550 4400 50
-F7 "IMU_MISO" O R 4550 4500 50
+F2 "IMU_CS" I R 4550 4300 50
+F3 "IMU_RST" I R 4550 4900 50
+F4 "IMU_DR" O R 4550 5000 50
+F5 "IMU_CLK" I R 4550 4400 50
+F6 "IMU_MOSI" I R 4550 4500 50
+F7 "IMU_MISO" O R 4550 4600 50
 $EndSheet
 Wire Wire Line
 	4550 3400 4950 3400
 $Sheet
-S 7150 3200 800  2000
+S 7150 3200 800  2200
 U 61E2DD2B
 F0 "Connector" 50
@@
 F16 "GPS_RX" I L 7150 4050 50
 F17 "GPS_TX" O L 7150 4150 50
+F18 "Servo_PWM" I L 7150 5250 50
 $EndSheet
-Wire Wire Line
-	4550 4200 4950 4200
 Wire Wire Line
 	4550 4300 4950 4300
@@
 	4550 4500 4950 4500
 Wire Wire Line
-	4950 4800 4550 4800
+	4550 4600 4950 4600
 Wire Wire Line
-	4550 4900 4950 4900
+	4950 4900 4550 4900
+Wire Wire Line
+	4550 5000 4950 5000
 Wire Wire Line
 	6750 3300 7150 3300
@@
 Wire Wire Line
 	6750 5100 7150 5100
+Wire Wire Line
+	6750 5250 7150 5250
 $EndSCHEMATC

Commit message: Adjust the pin order to make the wiring smoother.
Changed lines of the file:
@@
 F0 "MCU" 50
 F1 "2_MCU.sch" 50
-F2 "SPI2_CLK" O L 4950 4400 50
-F3 "SPI2_MISO" I L 4950 4600 50
-F4 "SPI2_MOSI" O L 4950 4500 50
-F5 "SWDIO" B R 6750 3300 50
-F6 "SWDCLK" I R 6750 3400 50
-F7 "UART1_TX" O R 6750 3500 50
-F8 "UART1_RX" I R 6750 3600 50
-F9 "UART3_TX" O R 6750 3900 50
-F10 "UART3_RX" I R 6750 3800 50
-F11 "SPI1_CLK" O R 6750 4550 50
-F12 "SPI1_MISO" I R 6750 4350 50
-F13 "SPI1_MOSI" O R 6750 4450 50
-F14 "UART6_TX" O R 6750 4050 50
-F15 "UART6_RX" I R 6750 4150 50
-F16 "PF13" I L 4950 3400 50
-F17 "PE3" O L 4950 4300 50
-F18 "PE4" I L 4950 5000 50
-F19 "PE1" O L 4950 4900 50
-F20 "PG2" I R 6750 5100 50
-F21 "PG3" O R 6750 5000 50
-F22 "PG4" O R 6750 4900 50
-F23 "PG5" O R 6750 4800 50
-F24 "PG6" O R 6750 4700 50
-F25 "ADC23_IN14" I L 4950 3500 50
-F26 "TIM1_CH1" O R 6750 5250 50
+F2 "SWDIO" B R 6750 3300 50
+F3 "SWDCLK" I R 6750 3400 50
+F4 "UART1_TX" O R 6750 3500 50
+F5 "UART1_RX" I R 6750 3600 50
+F6 "UART3_TX" O R 6750 3900 50
+F7 "UART3_RX" I R 6750 3800 50
+F8 "UART6_TX" O R 6750 4050 50
+F9 "UART6_RX" I R 6750 4150 50
+F10 "PF13" I L 4950 3400 50
+F11 "ADC23_IN14" I L 4950 3500 50
+F12 "TIM1_CH1" O R 6750 5250 50
+F13 "SPI2_CLK" O R 6750 4550 50
+F14 "SPI2_MISO" I R 6750 4350 50
+F15 "SPI2_MOSI" O R 6750 4450 50
+F16 "SPI1_CLK" O L 4950 4400 50
+F17 "SPI1_MISO" I L 4950 4600 50
+F18 "SPI1_MOSI" O L 4950 4500 50
+F19 "PB6" O L 4950 4300 50
+F20 "PB7" O L 4950 4900 50
+F21 "PG15" I L 4950 5000 50
+F22 "PG12" O L 4950 5300 50
+F23 "PG13" O L 4950 5200 50
+F24 "PE3" O R 6750 4700 50
+F25 "PE4" O R 6750 4800 50
+F26 "PE0" I R 6750 5100 50
+F27 "PE1" O R 6750 5000 50
+F28 "PB9" O R 6750 4900 50
 $EndSheet
 $Sheet

Commit message: Modify the circuit to modify the electronic switch section to disconnect via microcontroller control.
Changed lines of the file:
@@
 Sheet 1 5
 Title "MM32_Board"
-Date "2021-12-01"
-Rev "1.0.1"
+Date "2021-12-21"
+Rev "1.0.2"
 Comp ""
 Comment1 ""
@@
 $EndDescr
 $Sheet
-S 3850 3200 700  500
+S 3850 3200 700  550
 U 6191448D
 F0 "Power" 50
@@
 F2 "PWR_EN" I R 4550 3400 50
 F3 "VBAT" O R 4550 3500 50
+F4 "PWR_DET" O R 4550 3600 50
 $EndSheet
 $Sheet
@@
 F8 "UART6_TX" O R 6750 4050 50
 F9 "UART6_RX" I R 6750 4150 50
-F10 "PF13" I L 4950 3400 50
-F11 "ADC23_IN14" I L 4950 3500 50
-F12 "TIM1_CH1" O R 6750 5250 50
-F13 "SPI2_CLK" O R 6750 4550 50
-F14 "SPI2_MISO" I R 6750 4350 50
-F15 "SPI2_MOSI" O R 6750 4450 50
-F16 "SPI1_CLK" O L 4950 4400 50
-F17 "SPI1_MISO" I L 4950 4600 50
-F18 "SPI1_MOSI" O L 4950 4500 50
-F19 "PB6" O L 4950 4300 50
-F20 "PB7" O L 4950 4900 50
-F21 "PG15" I L 4950 5000 50
-F22 "PG12" O L 4950 5300 50
-F23 "PG13" O L 4950 5200 50
-F24 "PE3" O R 6750 4700 50
-F25 "PE4" O R 6750 4800 50
-F26 "PE0" I R 6750 5100 50
-F27 "PE1" O R 6750 5000 50
-F28 "PB9" O R 6750 4900 50
+F10 "ADC23_IN14" I L 4950 3500 50
+F11 "TIM1_CH1" O R 6750 5250 50
+F12 "SPI2_CLK" O R 6750 4550 50
+F13 "SPI2_MISO" I R 6750 4350 50
+F14 "SPI2_MOSI" O R 6750 4450 50
+F15 "SPI1_CLK" O L 4950 4400 50
+F16 "SPI1_MISO" I L 4950 4600 50
+F17 "SPI1_MOSI" O L 4950 4500 50
+F18 "PB6" O L 4950 4300 50
+F19 "PB7" O L 4950 4900 50
+F20 "PG15" I L 4950 5000 50
+F21 "PE3" O R 6750 4700 50
+F22 "PE4" O R 6750 4800 50
+F23 "PE0" I R 6750 5100 50
+F24 "PE1" O R 6750 5000 50
+F25 "PB9" O R 6750 4900 50
+F26 "PF13" O L 4950 3400 50
+F27 "PF14" I L 4950 3600 50
 $EndSheet
 $Sheet
@@
 Wire Wire Line
 	6750 5250 7150 5250
+Wire Wire Line
+	4550 3600 4950 3600
 $EndSCHEMATC
