File: circuit/3_IMU.sch (KiCad schematic (older format))
At the start: 10 parts

Commit message: Connect SPI2 of the microcontroller to the IMU.
Parts:
- added C? (x8): 100nF, symbol Device:C
Connections:
- net +3.3VA: now also C?.1, C?.1, C?.1, C?.1, C?.1, C?.1, C?.1, C?.1
- net GNDA: now also C?.2, C?.2, C?.2, C?.2, C?.2, C?.2, C?.2, C?.2
- net IMU_CS: now also U?.3 (IN_A)
- net IMU_DR: now also U?.5 (OUT_C)
- net IMU_RST: now also U?.4 (IN_B)
- net IMU_CLK: now reaches U?.3 (IN_A)
- net IMU_MOSI: now reaches U?.4 (IN_B)
- net IMU_MISO: now reaches U?.5 (OUT_C)
Other:
- moved on the sheet: C?, L?, U?

Commit message: Added the debugger's schematic library and improved the circuit of the power section.
Parts:
- added C? (x5): 100nF, symbol Device:C
Connections:
- net +3.3VA: now also C?.1, C?.1
- net +3V3: now also C?.1, C?.1
- net +5VA: now also C?.1
- net GNDA: now also C?.2, C?.2, C?.2, C?.2, C?.2
Other:
- moved on the sheet: U?

Commit message: Adjust the schematic layout and add annotations to make the schematic more beautiful.
Parts:
- removed C? (x11): 100nF, symbol Device:C
- removed U? (x2): π131M31, Package_SO:SOIC-16_3.9x9.9mm_P1.27mm, symbol MM32_Periph:π131M31
- added C? (x11): 100nF, symbol Device:C
- added U? (x2): π131M31, Package_SO:SOIC-16_3.9x9.9mm_P1.27mm, symbol MM32_Periph:π131M31
Connections:
- net +3.3VA: now also C?.1, C?.1, C?.1, C?.1, C?.1, C?.1, C?.1, C?.1, C?.1, U?.16 (VDD2), U?.16 (VDD2)
- net +3V3: now also C?.1, C?.1, U?.1 (VDD1), U?.1 (VDD1)
- net GND: now also U?.2 (GND1), U?.2 (GND1), U?.8 (GND1), U?.8 (GND1)
- net GNDA: now also C?.2, C?.2, C?.2, C?.2, C?.2, C?.2, C?.2, C?.2, C?.2, C?.2, C?.2, U?.15 (GND2), U?.15 (GND2), U?.9 (GND2), U?.9 (GND2)
- net IMU_CLK: now also U?.3 (IN_A)
- net IMU_CS: now also U?.14 (OUT_A), U?.3 (IN_A)
- net IMU_DIN: now also U?.13 (OUT_B)
- net IMU_DOUT: now also U?.12 (IN_C)
- net IMU_DR: now also U?.12 (IN_C), U?.5 (OUT_C)
- net IMU_MISO: now also U?.5 (OUT_C)
- net IMU_MOSI: now also U?.4 (IN_B)
- net IMU_RST: now also U?.13 (OUT_B), U?.4 (IN_B)
- net IMU_SCLK: now also U?.14 (OUT_A)
Other:
- note added: "Filter"
- note added: "IMU"
- note added: "Isolated Power Supply"
- note added: "Signal Isolation"
- moved on the sheet: C?, L?, U?

Commit message: Add annotations to the microcontroller subdiagram.
Other:
- note added: "Power Supply Isolation"
- note removed: "Isolated Power Supply"
Changed lines of the file:
@@
 Filter
 Text Notes 1050 5350 0    150  ~ 0
-Isolated Power Supply
+Power Supply Isolation
 Text Notes 7250 1350 0    150  ~ 0
 Signal Isolation

Commit message: Assign general-purpose GPIO pins to the LCD. Add annotations to the Connector subdiagram. Label the component markers.
Parts:
- gave numbers to parts that had none: 23

Commit message: Add packages for standard components and set the basic rules and layers of the PCB.
Parts:
- C33, C34, C35, C36, C37, C38, C39, C40, C41, C42, C43, C44, C45, C46, C47, C48, C49: footprint (none) -> Capacitor_SMD:C_0603_1608Metric
Changed lines of the file:
@@
 F 0 "C33" H 1465 6646 50  0000 L CNN
 F 1 "10uF" H 1465 6555 50  0000 L CNN
-F 2 "" H 1388 6450 50  0001 C CNN
+F 2 "Capacitor_SMD:C_0603_1608Metric" H 1388 6450 50  0001 C CNN
 F 3 "~" H 1350 6600 50  0001 C CNN
 	1    1350 6600
@@
 F 0 "C34" H 2165 6646 50  0000 L CNN
 F 1 "10uF" H 2165 6555 50  0000 L CNN
-F 2 "" H 2088 6450 50  0001 C CNN
+F 2 "Capacitor_SMD:C_0603_1608Metric" H 2088 6450 50  0001 C CNN
 F 3 "~" H 2050 6600 50  0001 C CNN
 	1    2050 6600
@@
 F 0 "C35" H 3615 6496 50  0000 L CNN
 F 1 "10uF" H 3615 6405 50  0000 L CNN
-F 2 "" H 3538 6300 50  0001 C CNN
+F 2 "Capacitor_SMD:C_0603_1608Metric" H 3538 6300 50  0001 C CNN
 F 3 "~" H 3500 6450 50  0001 C CNN
 	1    3500 6450
@@
 F 0 "C43" H 6165 6846 50  0000 L CNN
 F 1 "22uF" H 6165 6755 50  0000 L CNN
-F 2 "" H 6088 6650 50  0001 C CNN
+F 2 "Capacitor_SMD:C_0603_1608Metric" H 6088 6650 50  0001 C CNN
 F 3 "~" H 6050 6800 50  0001 C CNN
 	1    6050 6800
@@
 F 0 "C38" H 4965 4046 50  0000 L CNN
 F 1 "100nF" H 4965 3955 50  0000 L CNN
-F 2 "" H 4888 3850 50  0001 C CNN
+F 2 "Capacitor_SMD:C_0603_1608Metric" H 4888 3850 50  0001 C CNN
 F 3 "~" H 4850 4000 50  0001 C CNN
 	1    4850 4000
@@
 F 0 "C36" H 4015 6496 50  0000 L CNN
 F 1 "100nF" H 4015 6405 50  0000 L CNN
-F 2 "" H 3938 6300 50  0001 C CNN
+F 2 "Capacitor_SMD:C_0603_1608Metric" H 3938 6300 50  0001 C CNN
 F 3 "~" H 3900 6450 50  0001 C CNN
 	1    3900 6450
@@
 F 0 "C49" H 10415 5396 50  0000 L CNN
 F 1 "100nF" H 10415 5305 50  0000 L CNN
-F 2 "" H 10338 5200 50  0001 C CNN
+F 2 "Capacitor_SMD:C_0603_1608Metric" H 10338 5200 50  0001 C CNN
 F 3 "~" H 10300 5350 50  0001 C CNN
 	1    10300 5350
@@
 F 0 "C48" H 10415 2946 50  0000 L CNN
 F 1 "100nF" H 10415 2855 50  0000 L CNN
-F 2 "" H 10338 2750 50  0001 C CNN
+F 2 "Capacitor_SMD:C_0603_1608Metric" H 10338 2750 50  0001 C CNN
 F 3 "~" H 10300 2900 50  0001 C CNN
 	1    10300 2900
@@
 F 0 "C47" H 7465 5396 50  0000 L CNN
 F 1 "100nF" H 7465 5305 50  0000 L CNN
-F 2 "" H 7388 5200 50  0001 C CNN
+F 2 "Capacitor_SMD:C_0603_1608Metric" H 7388 5200 50  0001 C CNN
 F 3 "~" H 7350 5350 50  0001 C CNN
 	1    7350 5350
@@
 F 0 "C46" H 7465 2946 50  0000 L CNN
 F 1 "100nF" H 7465 2855 50  0000 L CNN
-F 2 "" H 7388 2750 50  0001 C CNN
+F 2 "Capacitor_SMD:C_0603_1608Metric" H 7388 2750 50  0001 C CNN
 F 3 "~" H 7350 2900 50  0001 C CNN
 	1    7350 2900
@@
 F 0 "C40" H 5415 4046 50  0000 L CNN
 F 1 "100nF" H 5415 3955 50  0000 L CNN
-F 2 "" H 5338 3850 50  0001 C CNN
+F 2 "Capacitor_SMD:C_0603_1608Metric" H 5338 3850 50  0001 C CNN
 F 3 "~" H 5300 4000 50  0001 C CNN
 	1    5300 4000
@@
 F 0 "C42" H 5865 4046 50  0000 L CNN
 F 1 "100nF" H 5865 3955 50  0000 L CNN
-F 2 "" H 5788 3850 50  0001 C CNN
+F 2 "Capacitor_SMD:C_0603_1608Metric" H 5788 3850 50  0001 C CNN
 F 3 "~" H 5750 4000 50  0001 C CNN
 	1    5750 4000
@@
 F 0 "C45" H 6315 4046 50  0000 L CNN
 F 1 "100nF" H 6315 3955 50  0000 L CNN
-F 2 "" H 6238 3850 50  0001 C CNN
+F 2 "Capacitor_SMD:C_0603_1608Metric" H 6238 3850 50  0001 C CNN
 F 3 "~" H 6200 4000 50  0001 C CNN
 	1    6200 4000
@@
 F 0 "C37" H 4965 2396 50  0000 L CNN
 F 1 "100nF" H 4965 2305 50  0000 L CNN
-F 2 "" H 4888 2200 50  0001 C CNN
+F 2 "Capacitor_SMD:C_0603_1608Metric" H 4888 2200 50  0001 C CNN
 F 3 "~" H 4850 2350 50  0001 C CNN
 	1    4850 2350
@@
 F 0 "C39" H 5415 2396 50  0000 L CNN
 F 1 "100nF" H 5415 2305 50  0000 L CNN
-F 2 "" H 5338 2200 50  0001 C CNN
+F 2 "Capacitor_SMD:C_0603_1608Metric" H 5338 2200 50  0001 C CNN
 F 3 "~" H 5300 2350 50  0001 C CNN
 	1    5300 2350
@@
 F 0 "C41" H 5865 2396 50  0000 L CNN
 F 1 "100nF" H 5865 2305 50  0000 L CNN
-F 2 "" H 5788 2200 50  0001 C CNN
+F 2 "Capacitor_SMD:C_0603_1608Metric" H 5788 2200 50  0001 C CNN
 F 3 "~" H 5750 2350 50  0001 C CNN
 	1    5750 2350
@@
 F 0 "C44" H 6315 2396 50  0000 L CNN
 F 1 "100nF" H 6315 2305 50  0000 L CNN
-F 2 "" H 6238 2200 50  0001 C CNN
+F 2 "Capacitor_SMD:C_0603_1608Metric" H 6238 2200 50  0001 C CNN
 F 3 "~" H 6200 2350 50  0001 C CNN
 	1    6200 2350
