File: circuit/3_IMU.sch (KiCad schematic (older format))
At the start: 23 parts, among them U10 π131M31, U6 ADIS16470AMLZ, U7 B0505S-1WR3, U8 HX9193, U9 π131M31

Commit message: Eliminate design rule errors in schematics.
Connections:
- net labels added: CS, DIN, DOUT, DR, RST, SCLK
- net labels removed: IMU_DIN, IMU_DOUT, IMU_SCLK
- wire segments 163 -> 164
Changed lines of the file:
@@
 NoConn ~ 2050 2550
 Text Label 1150 2650 0    50   ~ 0
-IMU_DOUT
+DOUT
 Text Label 1150 2450 0    50   ~ 0
-IMU_SCLK
+SCLK
 Text Label 1150 2350 0    50   ~ 0
-IMU_RST
+RST
 Text Label 1150 2250 0    50   ~ 0
-IMU_DR
+DR
 Text Label 1150 2150 0    50   ~ 0
-IMU_DIN
+DIN
 Text Label 1150 2050 0    50   ~ 0
-IMU_CS
+CS
 Wire Wire Line
 	1150 2050 2050 2050
@@
 	8550 5050 8650 5050
 Text Label 9750 5450 0    50   ~ 0
-IMU_DOUT
+DOUT
 Text Label 9750 3000 0    50   ~ 0
-IMU_DR
+DR
 Wire Wire Line
 	9500 3000 9750 3000
@@
 	9500 5450 9750 5450
 Text Label 9750 5250 0    50   ~ 0
-IMU_SCLK
+SCLK
 Text Label 9750 5350 0    50   ~ 0
-IMU_DIN
+DIN
 Wire Wire Line
 	9500 5350 9750 5350
@@
 	9750 5250 9500 5250
 Text Label 9750 2900 0    50   ~ 0
-IMU_RST
+RST
 Text Label 9750 2800 0    50   ~ 0
-IMU_CS
+CS
 Wire Wire Line
 	9500 2800 9750 2800
@@
 Text Notes 7250 1350 0    150  ~ 0
 Signal Isolation
+$Comp
+L power:PWR_FLAG #FLG0106
+U 1 1 61CA638A
+P 2350 5750
+F 0 "#FLG0106" H 2350 5825 50  0001 C CNN
+F 1 "PWR_FLAG" H 2350 5923 50  0000 C CNN
+F 2 "" H 2350 5750 50  0001 C CNN
+F 3 "~" H 2350 5750 50  0001 C CNN
+	1    2350 5750
+	1    0    0    -1
+$EndComp
+Wire Wire Line
+	2350 5750 2350 6400
+Connection ~ 2350 6400
 $EndSCHEMATC

Commit message: Adjust the pin order to make the wiring smoother.
Changed lines of the file:
@@
-	1    0    0    -1
-$EndComp
-$Comp
-L power:GNDA #PWR0130
-U 1 1 61E07F79
-P 7350 6050
-F 0 "#PWR0130" H 7350 5800 50  0001 C CNN
-F 1 "GNDA" H 7355 5877 50  0000 C CNN
-F 2 "" H 7350 6050 50  0001 C CNN
-F 3 "" H 7350 6050 50  0001 C CNN
-	1    7350 6050
 	1    0    0    -1
 $EndComp
@@
 	1    0    0    -1
 $EndComp
-$Comp
-L power:GNDA #PWR0128
-U 1 1 61E07F8D
-P 7350 3600
-F 0 "#PWR0128" H 7350 3350 50  0001 C CNN
-F 1 "GNDA" H 7355 3427 50  0000 C CNN
-F 2 "" H 7350 3600 50  0001 C CNN
-F 3 "" H 7350 3600 50  0001 C CNN
-	1    7350 3600
-	1    0    0    -1
-$EndComp
 Wire Wire Line
 	7350 2200 7350 2750
@@
 	2350 5750 2350 6400
 Connection ~ 2350 6400
+$Comp
+L power:GND #PWR0128
+U 1 1 61BFE812
+P 7350 3600
+F 0 "#PWR0128" H 7350 3350 50  0001 C CNN
+F 1 "GND" H 7355 3427 50  0000 C CNN
+F 2 "" H 7350 3600 50  0001 C CNN
+F 3 "" H 7350 3600 50  0001 C CNN
+	1    7350 3600
+	1    0    0    -1
+$EndComp
+$Comp
+L power:GND #PWR0130
+U 1 1 61BFEED7
+P 7350 6050
+F 0 "#PWR0130" H 7350 5800 50  0001 C CNN
+F 1 "GND" H 7355 5877 50  0000 C CNN
+F 2 "" H 7350 6050 50  0001 C CNN
+F 3 "" H 7350 6050 50  0001 C CNN
+	1    7350 6050
+	1    0    0    -1
+$EndComp
 $EndSCHEMATC
