File: circuit/4_Connector.sch (KiCad schematic (older format))
At the start: 0 parts

Commit message: Added the debugger's schematic library and improved the circuit of the power section.
Parts:
- added J?: VOUT, symbol Connector_Generic:Conn_01x02
- added M?: Debugger, symbol MM32_Periph:Debugger
Connections:
- net labels added: +15V, +3.3V, GND, SWDCLK, SWDIO, UART_RX, UART_TX
- wire segments 0 -> 14
Changed lines of the file:
@@
 Comment4 ""
 $EndDescr
+Text HLabel 1850 2450 0    50   BiDi ~ 0
+SWDIO
+Text HLabel 1850 2550 0    50   Output ~ 0
+SWDCLK
+Text HLabel 3650 2550 2    50   Output ~ 0
+UART_TX
+Text HLabel 3650 2450 2    50   Input ~ 0
+UART_RX
+$Comp
+L MM32_Periph:Debugger M?
+U 1 1 619F71DE
+P 2400 2750
+F 0 "M?" H 2450 3300 50  0000 C CNN
+F 1 "Debugger" H 2600 2700 50  0000 C CNN
+F 2 "" H 2450 3300 50  0001 C CNN
+F 3 "" H 2450 3300 50  0001 C CNN
+	1    2400 2750
+	1    0    0    -1
+$EndComp
+Wire Wire Line
+	3250 2450 3650 2450
+Wire Wire Line
+	3650 2550 3250 2550
+Wire Wire Line
+	1850 2450 2300 2450
+Wire Wire Line
+	2300 2550 1850 2550
+$Comp
+L power:+3.3V #PWR0240
+U 1 1 619F94A5
+P 3450 1700
+F 0 "#PWR0240" H 3450 1550 50  0001 C CNN
+F 1 "+3.3V" H 3465 1873 50  0000 C CNN
+F 2 "" H 3450 1700 50  0001 C CNN
+F 3 "" H 3450 1700 50  0001 C CNN
+	1    3450 1700
+	1    0    0    -1
+$EndComp
+$Comp
+L power:GND #PWR0241
+U 1 1 619F9BA6
+P 3450 3400
+F 0 "#PWR0241" H 3450 3150 50  0001 C CNN
+F 1 "GND" H 3455 3227 50  0000 C CNN
+F 2 "" H 3450 3400 50  0001 C CNN
+F 3 "" H 3450 3400 50  0001 C CNN
+	1    3450 3400
+	1    0    0    -1
+$EndComp
+$Comp
+L power:GND #PWR0242
+U 1 1 619F9F09
+P 2100 3400
+F 0 "#PWR0242" H 2100 3150 50  0001 C CNN
+F 1 "GND" H 2105 3227 50  0000 C CNN
+F 2 "" H 2100 3400 50  0001 C CNN
+F 3 "" H 2100 3400 50  0001 C CNN
+	1    2100 3400
+	1    0    0    -1
+$EndComp
+$Comp
+L power:+3.3V #PWR0243
+U 1 1 619FA449
+P 2100 1700
+F 0 "#PWR0243" H 2100 1550 50  0001 C CNN
+F 1 "+3.3V" H 2115 1873 50  0000 C CNN
+F 2 "" H 2100 1700 50  0001 C CNN
+F 3 "" H 2100 1700 50  0001 C CNN
+	1    2100 1700
+	1    0    0    -1
+$EndComp
+Wire Wire Line
+	2100 1700 2100 2350
+Wire Wire Line
+	2100 2350 2300 2350
+Wire Wire Line
+	3450 1700 3450 2350
+Wire Wire Line
+	3450 2350 3250 2350
+Wire Wire Line
+	3250 2650 3450 2650
+Wire Wire Line
+	3450 2650 3450 3400
+Wire Wire Line
+	2300 2650 2100 2650
+Wire Wire Line
+	2100 2650 2100 3400
+$Comp
+L Connector_Generic:Conn_01x02 J?
+U 1 1 61B1D9F4
+P 4750 2500
+F 0 "J?" H 4700 2600 50  0000 L CNN
+F 1 "VOUT" H 4700 2300 50  0000 L CNN
+F 2 "" H 4750 2500 50  0001 C CNN
+F 3 "~" H 4750 2500 50  0001 C CNN
+	1    4750 2500
+	1    0    0    -1
+$EndComp
+$Comp
+L power:+15V #PWR?
+U 1 1 61B26E64
+P 4550 1700
+F 0 "#PWR?" H 4550 1550 50  0001 C CNN
+F 1 "+15V" H 4565 1873 50  0000 C CNN
+F 2 "" H 4550 1700 50  0001 C CNN
+F 3 "" H 4550 1700 50  0001 C CNN
+	1    4550 1700
+	1    0    0    -1
+$EndComp
+Wire Wire Line
+	4550 1700 4550 2500
+$Comp
+L power:GND #PWR?
+U 1 1 61B26FE3
+P 4550 3400
+F 0 "#PWR?" H 4550 3150 50  0001 C CNN
+F 1 "GND" H 4555 3227 50  0000 C CNN
+F 2 "" H 4550 3400 50  0001 C CNN
+F 3 "" H 4550 3400 50  0001 C CNN
+	1    4550 3400
+	1    0    0    -1
+$EndComp
+Wire Wire Line
+	4550 2600 4550 3400
 $EndSCHEMATC

Commit message: Added brushless motor communication interface and LCD control interface.
Parts:
- added J?: Camera, symbol MM32_Periph:Camera
- added J?: Conn_01x03, symbol Connector_Generic:Conn_01x03
- added LCD?: 1.8inch-TFT-LCD, symbol MM32_Periph:1.8inch-TFT-LCD
- added U?: XPT2046TS, Package_SO:TSSOP-16_4.4x5mm_P0.65mm, symbol Driver_Display:XPT2046TS
Connections:
- net labels added: CLK, DEBUG_RX, DEBUG_TX, DIN, LCD_A0, LCD_CLK, LCD_CS, LCD_MISO, LCD_MOSI, LCD_RST, MOTOR_RX, MOTOR_TX, TOUCH_CS, T_XM, T_XP, T_YM, T_YP
- net labels removed: UART_RX, UART_TX
- wire segments 14 -> 51

Commit message: Add the battery voltage detection circuit and complete the circuit connection of XPT2046.
Connections:
- net labels added: TOUCH_IT
- wire segments 51 -> 56
- no-connect marks 0 -> 4

Commit message: Add GPS module circuit.
Parts:
- removed J?: Camera, symbol MM32_Periph:Camera
- added BT?: Battery_Cell, Battery:BatteryHolder_Keystone_1060_1x2032, symbol Device:Battery_Cell
- added C?: C, symbol Device:C
- added J?: Conn_01x02, symbol Connector_Generic:Conn_01x02
- added L?: 47nH, symbol Device:L
- added U?: ATGM336H, RF_GPS:ublox_MAX, symbol MM32_Periph:ATGM336H
Connections:
- net labels added: GPS_RXD, GPS_TXD
- wire segments 56 -> 75
- no-connect marks 4 -> 7

Commit message: Assign general-purpose GPIO pins to the LCD. Add annotations to the Connector subdiagram. Label the component markers.
Parts:
- C50: renamed from C?; value C -> 10uF
- J2: renamed from J?; value Conn_01x02 -> ANT
- gave numbers to parts that had none: 8
Connections:
- net labels added: GPS_RX, GPS_TX
- net labels removed: GPS_RXD, GPS_TXD
Other:
- note added: "Debugger"
- note added: "GPS"
- note added: "LCD"
- note added: "Motor"
- moved on the sheet: C50, L4

Commit message: Add packages for standard components and set the basic rules and layers of the PCB.
Parts:
- C50: footprint (none) -> Capacitor_SMD:C_0603_1608Metric
- J2: footprint (none) -> Connector_Coaxial:SMA_Molex_73251-2200_Horizontal
- J3: footprint (none) -> Connector_JST:JST_GH_SM03B-GHS-TB_1x03-1MP_P1.25mm_Horizontal
- J4: footprint (none) -> Connector_AMASS:AMASS_XT30PW-F_1x02_P2.50mm_Horizontal
- L4: footprint (none) -> Inductor_SMD:L_0805_2012Metric_Pad1.15x1.40mm_HandSolder
Changed lines of the file:
@@
 F 0 "J4" H 10000 2550 50  0000 L CNN
 F 1 "VOUT" H 10000 2850 50  0000 L CNN
-F 2 "" H 10050 2750 50  0001 C CNN
+F 2 "Connector_AMASS:AMASS_XT30PW-F_1x02_P2.50mm_Horizontal" H 10050 2750 50  0001 C CNN
 F 3 "~" H 10050 2750 50  0001 C CNN
 	1    10050 2750
@@
 F 0 "J3" H 9150 2900 50  0000 L CNN
 F 1 "Conn_01x03" H 9050 2500 50  0000 L CNN
-F 2 "" H 9200 2700 50  0001 C CNN
+F 2 "Connector_JST:JST_GH_SM03B-GHS-TB_1x03-1MP_P1.25mm_Horizontal" H 9200 2700 50  0001 C CNN
 F 3 "~" H 9200 2700 50  0001 C CNN
 	1    9200 2700
@@
 F 0 "J2" H 3950 6000 50  0000 L CNN
 F 1 "ANT" H 3950 5700 50  0000 L CNN
-F 2 "" H 4000 5900 50  0001 C CNN
+F 2 "Connector_Coaxial:SMA_Molex_73251-2200_Horizontal" H 4000 5900 50  0001 C CNN
 F 3 "~" H 4000 5900 50  0001 C CNN
 	1    4000 5900
@@
 F 0 "L4" H 3503 5796 50  0000 L CNN
 F 1 "47nH" H 3503 5705 50  0000 L CNN
-F 2 "" H 3450 5750 50  0001 C CNN
+F 2 "Inductor_SMD:L_0805_2012Metric_Pad1.15x1.40mm_HandSolder" H 3450 5750 50  0001 C CNN
 F 3 "~" H 3450 5750 50  0001 C CNN
 	1    3450 5750
@@
 F 0 "C50" H 2015 6246 50  0000 L CNN
 F 1 "10uF" H 2015 6155 50  0000 L CNN
-F 2 "" H 1938 6050 50  0001 C CNN
+F 2 "Capacitor_SMD:C_0603_1608Metric" H 1938 6050 50  0001 C CNN
 F 3 "~" H 1900 6200 50  0001 C CNN
 	1    1900 6200

Commit message: Add packages for the remaining components.
Parts:
- LCD1: footprint (none) -> Display:TFT-LCD1.8inch
- M1: footprint (none) -> Connector:Gernic_Debugger
Changed lines of the file:
@@
 F 0 "M1" H 2350 3500 50  0000 C CNN
 F 1 "Debugger" H 2500 2900 50  0000 C CNN
-F 2 "" H 2350 3500 50  0001 C CNN
+F 2 "Connector:Gernic_Debugger" H 2350 3500 50  0001 C CNN
 F 3 "" H 2350 3500 50  0001 C CNN
 	1    2300 2950
@@
 F 0 "LCD1" H 6100 4300 50  0000 C CNN
 F 1 "1.8inch-TFT-LCD" H 6350 3200 50  0000 C CNN
-F 2 "" H 6100 4300 50  0001 C CNN
+F 2 "Display:TFT-LCD1.8inch" H 6100 4300 50  0001 C CNN
 F 3 "" H 6100 4300 50  0001 C CNN
 	1    6000 3250

Commit message: Eliminate design rule errors in schematics.
Connections:
- wire segments 75 -> 76
- no-connect marks 7 -> 9
Changed lines of the file:
@@
 Text Notes 1400 4550 0    150  ~ 0
 GPS
+NoConn ~ 2250 5600
+NoConn ~ 2250 5500
+$Comp
+L power:PWR_FLAG #FLG0107
+U 1 1 61CB58F4
+P 1500 4900
+F 0 "#FLG0107" H 1500 4975 50  0001 C CNN
+F 1 "PWR_FLAG" H 1500 5073 50  0000 C CNN
+F 2 "" H 1500 4900 50  0001 C CNN
+F 3 "~" H 1500 4900 50  0001 C CNN
+	1    1500 4900
+	1    0    0    -1
+$EndComp
+Wire Wire Line
+	1500 4900 1500 5700
+Connection ~ 1500 5700
 $EndSCHEMATC
