File: circuit/4_Connector.sch (KiCad schematic (older format))
At the start: 10 parts, among them J2 ANT, J3 Conn_01x03, J4 VOUT, M1 Debugger, U11 ATGM336H, U12 XPT2046TS

Commit message: Add Servo Interface
Parts:
- added J5: Conn_01x03, Connector_PinHeader_2.54mm:PinHeader_1x03_P2.54mm_Horizontal, symbol Connector_Generic:Conn_01x03
Connections:
- net labels added: +7.5V, Servo_PWM
- wire segments 76 -> 81
Other:
- note added: "Servo"
Changed lines of the file:
@@
 	1500 4900 1500 5700
 Connection ~ 1500 5700
+$Comp
+L Connector_Generic:Conn_01x03 J5
+U 1 1 61A932D6
+P 9850 5700
+F 0 "J5" H 9800 5900 50  0000 L CNN
+F 1 "Conn_01x03" H 9700 5500 50  0000 L CNN
+F 2 "Connector_PinHeader_2.54mm:PinHeader_1x03_P2.54mm_Horizontal" H 9850 5700 50  0001 C CNN
+F 3 "~" H 9850 5700 50  0001 C CNN
+	1    9850 5700
+	1    0    0    -1
+$EndComp
+$Comp
+L power:GND #PWR0162
+U 1 1 61A93E0F
+P 9450 6450
+F 0 "#PWR0162" H 9450 6200 50  0001 C CNN
+F 1 "GND" H 9455 6277 50  0000 C CNN
+F 2 "" H 9450 6450 50  0001 C CNN
+F 3 "" H 9450 6450 50  0001 C CNN
+	1    9450 6450
+	1    0    0    -1
+$EndComp
+$Comp
+L power:+7.5V #PWR?
+U 1 1 61A9B489
+P 9450 4900
+AR Path="/6191448D/61A9B489" Ref="#PWR?"  Part="1"
+AR Path="/61E2DD2B/61A9B489" Ref="#PWR0163"  Part="1"
+F 0 "#PWR0163" H 9450 4750 50  0001 C CNN
+F 1 "+7.5V" H 9465 5073 50  0000 C CNN
+F 2 "" H 9450 4900 50  0001 C CNN
+F 3 "" H 9450 4900 50  0001 C CNN
+	1    9450 4900
+	1    0    0    -1
+$EndComp
+Wire Wire Line
+	9450 4900 9450 5700
+Wire Wire Line
+	9450 5700 9650 5700
+Wire Wire Line
+	9650 5800 9450 5800
+Wire Wire Line
+	9450 5800 9450 6450
+Text HLabel 9250 5600 0    50   Input ~ 0
+Servo_PWM
+Wire Wire Line
+	9250 5600 9650 5600
+Wire Notes Line
+	8100 4200 10500 4200
+Wire Notes Line
+	10500 4200 10500 6900
+Wire Notes Line
+	10500 6900 8100 6900
+Wire Notes Line
+	8100 6900 8100 4200
+Text Notes 8250 4550 0    150  ~ 0
+Servo
 $EndSCHEMATC

Commit message: Add servo interface.
Parts:
- removed BT1: Battery_Cell, Battery:BatteryHolder_Keystone_1060_1x2032, symbol Device:Battery_Cell
Connections:
- wire segments 81 -> 79
Changed lines of the file:
@@
 Wire Wire Line
 	1900 6350 1900 6450
-$Comp
-L Device:Battery_Cell BT1
-U 1 1 61A84728
-P 1500 6150
-F 0 "BT1" H 1618 6200 50  0000 L CNN
-F 1 "Battery_Cell" H 1618 6155 50  0001 L CNN
-F 2 "Battery:BatteryHolder_Keystone_1060_1x2032" V 1500 6210 50  0001 C CNN
-F 3 "~" V 1500 6210 50  0001 C CNN
-	1    1500 6150
-	1    0    0    -1
-$EndComp
 Wire Wire Line
-	1900 4900 1900 5900
-Wire Wire Line
-	1500 5950 1500 5700
-Wire Wire Line
-	1500 5700 2250 5700
-$Comp
-L power:GND #PWR0143
-U 1 1 61A8DC9F
-P 1500 6450
-F 0 "#PWR0143" H 1500 6200 50  0001 C CNN
-F 1 "GND" H 1505 6277 50  0000 C CNN
-F 2 "" H 1500 6450 50  0001 C CNN
-F 3 "" H 1500 6450 50  0001 C CNN
-	1    1500 6450
-	1    0    0    -1
-$EndComp
-Wire Wire Line
-	1500 6450 1500 6250
+	1900 4900 1900 5700
 NoConn ~ 2250 6000
 Text HLabel 1850 5400 0    50   Input ~ 0
@@
 NoConn ~ 2250 5600
 NoConn ~ 2250 5500
-$Comp
-L power:PWR_FLAG #FLG0107
-U 1 1 61CB58F4
-P 1500 4900
-F 0 "#FLG0107" H 1500 4975 50  0001 C CNN
-F 1 "PWR_FLAG" H 1500 5073 50  0000 C CNN
-F 2 "" H 1500 4900 50  0001 C CNN
-F 3 "~" H 1500 4900 50  0001 C CNN
-	1    1500 4900
-	1    0    0    -1
-$EndComp
-Wire Wire Line
-	1500 4900 1500 5700
-Connection ~ 1500 5700
 $Comp
 L Connector_Generic:Conn_01x03 J5
@@
 Text Notes 8250 4550 0    150  ~ 0
 Servo
+Wire Wire Line
+	2250 5700 1900 5700
+Connection ~ 1900 5700
+Wire Wire Line
+	1900 5700 1900 5900
 $EndSCHEMATC

Commit message: Complete PCB design and export Gerber files.
Parts:
- added C52: 22uF, Capacitor_SMD:C_0805_2012Metric, symbol Device:C
- added C53, C54, C55, C56, C57, C58: 100nF, Capacitor_SMD:C_0603_1608Metric, symbol Device:C
Connections:
- wire segments 79 -> 107
Changed lines of the file:
@@
 Wire Wire Line
 	9450 5800 9450 6450
-Text HLabel 9250 5600 0    50   Input ~ 0
+Text HLabel 9050 5600 0    50   Input ~ 0
 Servo_PWM
 Wire Wire Line
-	9250 5600 9650 5600
+	9050 5600 9650 5600
 Wire Notes Line
 	8100 4200 10500 4200
@@
 Wire Wire Line
 	1900 5700 1900 5900
+$Comp
+L Device:C C?
+U 1 1 61AFDD59
+P 9150 5950
+AR Path="/6191448D/61AFDD59" Ref="C?"  Part="1"
+AR Path="/61E2DD2B/61AFDD59" Ref="C52"  Part="1"
+F 0 "C52" H 9265 5996 50  0000 L CNN
+F 1 "22uF" H 9265 5905 50  0000 L CNN
+F 2 "Capacitor_SMD:C_0805_2012Metric" H 9188 5800 50  0001 C CNN
+F 3 "~" H 9150 5950 50  0001 C CNN
+	1    9150 5950
+	1    0    0    -1
+$EndComp
+$Comp
+L power:+7.5V #PWR?
+U 1 1 61B022AD
+P 9150 4900
+AR Path="/6191448D/61B022AD" Ref="#PWR?"  Part="1"
+AR Path="/61E2DD2B/61B022AD" Ref="#PWR0165"  Part="1"
+F 0 "#PWR0165" H 9150 4750 50  0001 C CNN
+F 1 "+7.5V" H 9165 5073 50  0000 C CNN
+F 2 "" H 9150 4900 50  0001 C CNN
+F 3 "" H 9150 4900 50  0001 C CNN
+	1    9150 4900
+	1    0    0    -1
+$EndComp
+$Comp
+L power:GND #PWR0166
+U 1 1 61B026B8
+P 9150 6450
+F 0 "#PWR0166" H 9150 6200 50  0001 C CNN
+F 1 "GND" H 9155 6277 50  0000 C CNN
+F 2 "" H 9150 6450 50  0001 C CNN
+F 3 "" H 9150 6450 50  0001 C CNN
+	1    9150 6450
+	1    0    0    -1
+$EndComp
+Wire Wire Line
+	9150 4900 9150 5800
+Wire Wire Line
+	9150 6450 9150 6100
+$Comp
+L Device:C C?
+U 1 1 61B30203
+P 5150 4250
+AR Path="/6194FB75/61B30203" Ref="C?"  Part="1"
+AR Path="/61E2DD2B/61B30203" Ref="C53"  Part="1"
+F 0 "C53" H 5265 4296 50  0000 L CNN
+F 1 "100nF" H 5265 4205 50  0000 L CNN
+F 2 "Capacitor_SMD:C_0603_1608Metric" H 5188 4100 50  0001 C CNN
+F 3 "~" H 5150 4250 50  0001 C CNN
+	1    5150 4250
+	1    0    0    -1
+$EndComp
+$Comp
+L Device:C C?
+U 1 1 61B30209
+P 5600 4250
+AR Path="/6194FB75/61B30209" Ref="C?"  Part="1"
+AR Path="/61E2DD2B/61B30209" Ref="C54"  Part="1"
+F 0 "C54" H 5715 4296 50  0000 L CNN
+F 1 "100nF" H 5715 4205 50  0000 L CNN
+F 2 "Capacitor_SMD:C_0603_1608Metric" H 5638 4100 50  0001 C CNN
+F 3 "~" H 5600 4250 50  0001 C CNN
+	1    5600 4250
+	1    0    0    -1
+$EndComp
+$Comp
+L Device:C C?
+U 1 1 61B3020F
+P 6050 4250
+AR Path="/6194FB75/61B3020F" Ref="C?"  Part="1"
+AR Path="/61E2DD2B/61B3020F" Ref="C55"  Part="1"
+F 0 "C55" H 6165 4296 50  0000 L CNN
+F 1 "100nF" H 6165 4205 50  0000 L CNN
+F 2 "Capacitor_SMD:C_0603_1608Metric" H 6088 4100 50  0001 C CNN
+F 3 "~" H 6050 4250 50  0001 C CNN
+	1    6050 4250
+	1    0    0    -1
+$EndComp
+$Comp
+L Device:C C?
+U 1 1 61B30215
+P 6550 4250
+AR Path="/6194FB75/61B30215" Ref="C?"  Part="1"
+AR Path="/61E2DD2B/61B30215" Ref="C56"  Part="1"
+F 0 "C56" H 6665 4296 50  0000 L CNN
+F 1 "100nF" H 6665 4205 50  0000 L CNN
+F 2 "Capacitor_SMD:C_0603_1608Metric" H 6588 4100 50  0001 C CNN
+F 3 "~" H 6550 4250 50  0001 C CNN
+	1    6550 4250
+	1    0    0    -1
+$EndComp
+$Comp
+L Device:C C?
+U 1 1 61B3021B
+P 7000 4250
+AR Path="/6194FB75/61B3021B" Ref="C?"  Part="1"
+AR Path="/61E2DD2B/61B3021B" Ref="C57"  Part="1"
+F 0 "C57" H 7115 4296 50  0000 L CNN
+F 1 "100nF" H 7115 4205 50  0000 L CNN
+F 2 "Capacitor_SMD:C_0603_1608Metric" H 7038 4100 50  0001 C CNN
+F 3 "~" H 7000 4250 50  0001 C CNN
+	1    7000 4250
+	1    0    0    -1
+$EndComp
+$Comp
+L Device:C C?
+U 1 1 61B30221
+P 7450 4250
+AR Path="/6194FB75/61B30221" Ref="C?"  Part="1"
+AR Path="/61E2DD2B/61B30221" Ref="C58"  Part="1"
+F 0 "C58" H 7565 4296 50  0000 L CNN
+F 1 "100nF" H 7565 4205 50  0000 L CNN
+F 2 "Capacitor_SMD:C_0603_1608Metric" H 7488 4100 50  0001 C CNN
+F 3 "~" H 7450 4250 50  0001 C CNN
+	1    7450 4250
+	1    0    0    -1
+$EndComp
+$Comp
+L power:+3.3V #PWR?
+U 1 1 61B30227
+P 6300 3900
+AR Path="/6194FB75/61B30227" Ref="#PWR?"  Part="1"
+AR Path="/61E2DD2B/61B30227" Ref="#PWR0167"  Part="1"
+F 0 "#PWR0167" H 6300 3750 50  0001 C CNN
+F 1 "+3.3V" H 6300 4050 50  0000 C CNN
+F 2 "" H 6300 3900 50  0001 C CNN
+F 3 "" H 6300 3900 50  0001 C CNN
+	1    6300 3900
+	1    0    0    -1
+$EndComp
+Wire Wire Line
+	5150 4100 5150 3950
+Wire Wire Line
+	5150 3950 5600 3950
+Wire Wire Line
+	6300 3950 6300 3900
+Wire Wire Line
+	6300 3950 6550 3950
+Wire Wire Line
+	7450 3950 7450 4100
+Connection ~ 6300 3950
+Wire Wire Line
+	7000 4100 7000 3950
+Connection ~ 7000 3950
+Wire Wire Line
+	7000 3950 7450 3950
+Wire Wire Line
+	6550 4100 6550 3950
+Connection ~ 6550 3950
+Wire Wire Line
+	6550 3950 7000 3950
+Wire Wire Line
+	6050 4100 6050 3950
+Connection ~ 6050 3950
+Wire Wire Line
+	6050 3950 6300 3950
+Wire Wire Line
+	5600 4100 5600 3950
+Connection ~ 5600 3950
+Wire Wire Line
+	5600 3950 6050 3950
+$Comp
+L power:GND #PWR?
+U 1 1 61B3023F
+P 6300 4600
+AR Path="/6194FB75/61B3023F" Ref="#PWR?"  Part="1"
+AR Path="/61E2DD2B/61B3023F" Ref="#PWR0168"  Part="1"
+F 0 "#PWR0168" H 6300 4350 50  0001 C CNN
+F 1 "GND" H 6350 4450 50  0000 R CNN
+F 2 "" H 6300 4600 50  0001 C CNN
+F 3 "" H 6300 4600 50  0001 C CNN
+	1    6300 4600
+	1    0    0    -1
+$EndComp
+Wire Wire Line
+	5150 4400 5150 4550
+Wire Wire Line
+	5150 4550 5600 4550
+Wire Wire Line
+	6300 4600 6300 4550
+Wire Wire Line
+	6300 4550 6550 4550
+Wire Wire Line
+	7450 4550 7450 4400
+Connection ~ 6300 4550
+Wire Wire Line
+	7000 4400 7000 4550
+Connection ~ 7000 4550
+Wire Wire Line
+	7000 4550 7450 4550
+Wire Wire Line
+	6550 4400 6550 4550
+Connection ~ 6550 4550
+Wire Wire Line
+	6550 4550 7000 4550
+Wire Wire Line
+	6050 4400 6050 4550
+Connection ~ 6050 4550
+Wire Wire Line
+	6050 4550 6300 4550
+Wire Wire Line
+	5600 4400 5600 4550
+Connection ~ 5600 4550
+Wire Wire Line
+	5600 4550 6050 4550
 $EndSCHEMATC
