File: circuit/project.kicad_pcb (KiCad board)
At the start: 2 copper layers, 61 x 28.4 mm, 34 parts, among them J1 IN, J2 OUT, Q1 NTMFS5C670, Q2 NTMFS5C670, U1 LM5117

Commit message: Add reference voltage source to the circuit
Parts:
- removed C1, C13, C18: 100uF, Capacitor_SMD:CP_Elec_6.3x5.2
- removed C10, C12: 100nF, Capacitor_SMD:C_0603_1608Metric
- removed C11: 820pF, Capacitor_SMD:C_0603_1608Metric
- removed C14: 470nF, Capacitor_SMD:C_0603_1608Metric
- removed C15, C16, C17, C2, C3, C4, C5: 10uF, Capacitor_SMD:C_1206_3216Metric
- removed C6: 390nF, Capacitor_SMD:C_0603_1608Metric
- removed C7: 150nF, Capacitor_SMD:C_0603_1608Metric
- removed C8: 100pF, Capacitor_SMD:C_0603_1608Metric
- removed C9: 3.9nF, Capacitor_SMD:C_0603_1608Metric
- removed D1: 1N4007, Diode_SMD:D_SMA
- removed J1: IN, Connector_AMASS:AMASS_XT30PW-M_1x02_P2.50mm_Horizontal
- removed J2: OUT, Connector_AMASS:AMASS_XT30PW-F_1x02_P2.50mm_Horizontal
- removed L1: 4.7uH, Inductor_SMD:L_12x12mm_H8mm
- removed Q1, Q2: NTMFS5C670, Package_SO:NTMFS5C673NLT1G
- removed R1: 56k, Resistor_SMD:R_0603_1608Metric
- removed R2: 4.7k, Resistor_SMD:R_0603_1608Metric
- removed R3: 9.1k, Resistor_SMD:R_0603_1608Metric
- removed R4: 13k, Resistor_SMD:R_0603_1608Metric
- removed R5, R6: 1k, Resistor_SMD:R_0603_1608Metric
- removed R7: 43k, Resistor_SMD:R_0603_1608Metric
- removed R8: 5mR, Resistor_SMD:R_1206_3216Metric
- removed R9: 110k, Resistor_SMD:R_0603_1608Metric
- removed U1: LM5117, Package_SO:HTSSOP-20-1EP_4.4x6.5mm_P0.65mm_EP2.85x4mm
Routing:
- net +24V: track 24.3 -> 0.00 mm, vias 20 -> 0
- net +12V: track 18.0 -> 0.00 mm
- net Net-(Q1-Pad2): track 17.1 -> 0.00 mm, vias 2 -> 0
- net Net-(Q2-Pad3): track 16.7 -> 0.00 mm, vias 2 -> 0
- net Net-(Q2-Pad2): track 13.6 -> 0.00 mm, vias 2 -> 0
- net VCC: track 12.5 -> 0.00 mm, vias 2 -> 0
- net Net-(C10-Pad2): track 12.1 -> 0.00 mm
- net Net-(C10-Pad1): track 9.90 -> 0.00 mm
- net Net-(C8-Pad2): track 8.71 -> 0.00 mm
- net Net-(C6-Pad1): track 7.91 -> 0.00 mm, vias 1 -> 0
- net Net-(C7-Pad1): track 7.33 -> 0.00 mm, vias 1 -> 0
- net Net-(R3-Pad1): track 6.19 -> 0.00 mm, vias 1 -> 0
- net Net-(R4-Pad2): track 5.79 -> 0.00 mm
- net Net-(C8-Pad1): track 5.28 -> 0.00 mm
- net Net-(R1-Pad2): track 4.69 -> 0.00 mm
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- removed copper zone on F.Cu, net +12V
- removed copper zone on B.Cu, net +24V
- removed copper zone on F.Cu, net +24V
- removed copper zone on B.Cu, net 0
- removed copper zone on F.Cu, net 0
- removed copper zone on F.Cu, net Net-(C10-Pad2)
- removed copper zone on F.Cu, net Net-(Q2-Pad3)
Other:
- board outline removed
- net class Default: trace_width 0.254 -> 0.25; via_dia 0.6 -> 0.8; via_drill 0.3 -> 0.4
- rule via_min_size: 0.6 -> 0.4

Commit message: Add packages for standard components and set the basic rules and layers of the PCB.
Other:
- copper layers 2 -> 4
- net class Default: trace_width 0.25 -> 0.254; via_dia 0.8 -> 0.6; via_drill 0.4 -> 0.3
Changed lines of the file:
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@@
   )
   (page A4)
+  (title_block
+    (title MM32_Board)
+    (date 2021-11-30)
+    (rev 1.0.1)
+  )
   (layers
     (0 F.Cu signal)
+    (1 In1.Cu signal)
+    (2 In2.Cu signal)
     (31 B.Cu signal)
     (32 B.Adhes user)
@@
   )
   (setup
-    (last_trace_width 0.25)
+    (last_trace_width 0.254)
+    (user_trace_width 0.2)
+    (user_trace_width 0.254)
+    (user_trace_width 0.3)
+    (user_trace_width 0.5)
     (trace_clearance 0.2)
     (zone_clearance 0.508)
     (zone_45_only no)
     (trace_min 0.2)
-    (via_size 0.8)
-    (via_drill 0.4)
+    (via_size 0.6)
+    (via_drill 0.3)
     (via_min_size 0.4)
     (via_min_drill 0.3)
+    (user_via 0.6 0.3)
     (uvia_size 0.3)
     (uvia_drill 0.1)
@@
     (pad_to_mask_clearance 0)
     (aux_axis_origin 0 0)
-    (visible_elements FFFFFF7F)
+    (visible_elements 7FFFFFFF)
     (pcbplotparams
       (layerselection 0x010fc_ffffffff)
@@
   (net_class Default 这是默认网络类。
     (clearance 0.2)
-    (trace_width 0.25)
-    (via_dia 0.8)
-    (via_drill 0.4)
+    (trace_width 0.254)
+    (via_dia 0.6)
+    (via_drill 0.3)
     (uvia_dia 0.3)
     (uvia_drill 0.1)
+    (diff_pair_width 0.2)
+    (diff_pair_gap 0.2)
   )
 )

Commit message: Modify schematic title and date and generate PCB file.
Parts:
- added BT1: Battery_Cell, Battery:BatteryHolder_Keystone_1060_1x2032, F.Cu at (132.5, 108.8)
- added C1: 22uF, Capacitor_SMD:C_0603_1608Metric, F.Cu at (226.5, 96.4)
- added C10: 10uF, Capacitor_SMD:C_0805_2012Metric, F.Cu at (179.9, 106.6)
- added C11: 32pF, Capacitor_SMD:C_0603_1608Metric, F.Cu at (205.5, 90.8)
- added C12: 10nF, Capacitor_SMD:C_0603_1608Metric, F.Cu at (209.5, 90.8)
- added C13: 620pF, Capacitor_SMD:C_0603_1608Metric, F.Cu at (213.5, 90.8)
- added C14: 22uF, Capacitor_SMD:C_0805_2012Metric, F.Cu at (184.4, 106.6)
- added C15: 100uF, Capacitor_SMD:CP_Elec_6.3x7.7, F.Cu at (221.3, 80.4)
- added C16: 100uF, Capacitor_SMD:CP_Elec_6.3x7.7, F.Cu at (205.9, 96.6)
- added C17: 100nF, Capacitor_SMD:C_0603_1608Metric, F.Cu at (120.9, 136.6)
- added C18: 100nF, Capacitor_SMD:C_0603_1608Metric, F.Cu at (110.0, 151.8)
- added C19: 18pF, Capacitor_SMD:C_0603_1608Metric, F.Cu at (118.0, 144.2)
- added C2: 100nF, Capacitor_SMD:C_0603_1608Metric, F.Cu at (222.5, 93.9)
- added C20: 100nF, Capacitor_SMD:C_0603_1608Metric, F.Cu at (114.0, 146.8)
- added C21: 100nF, Capacitor_SMD:C_0603_1608Metric, F.Cu at (119.3, 141.6)
- added C22: 100nF, Capacitor_SMD:C_0603_1608Metric, F.Cu at (119.3, 139.1)
- added C23: 100nF, Capacitor_SMD:C_0603_1608Metric, F.Cu at (106.0, 153.6)
- added C24: 100nF, Capacitor_SMD:C_0603_1608Metric, F.Cu at (106.0, 156.1)
- added C25: 18pF, Capacitor_SMD:C_0603_1608Metric, F.Cu at (116.8, 136.6)
- added C26: 100nF, Capacitor_SMD:C_0603_1608Metric, F.Cu at (106.0, 146.1)
- added C27: 100nF, Capacitor_SMD:C_0603_1608Metric, F.Cu at (111.2, 141.7)
- added C28: 100nF, Capacitor_SMD:C_0603_1608Metric, F.Cu at (120.9, 134.0)
- added C29: 100nF, Capacitor_SMD:C_0603_1608Metric, F.Cu at (110.0, 149.3)
- added C3: 10uF, Capacitor_SMD:C_0805_2012Metric, F.Cu at (201.5, 107.5)
- added C30: 100nF, Capacitor_SMD:C_0603_1608Metric, F.Cu at (110.0, 144.2)
- added C31: 100nF, Capacitor_SMD:C_0603_1608Metric, F.Cu at (106.0, 148.6)
- added C32: 100nF, Capacitor_SMD:C_0603_1608Metric, F.Cu at (115.3, 139.1)
- added C33: 10uF, Capacitor_SMD:C_0603_1608Metric, F.Cu at (214.7, 125.8)
- added C34: 10uF, Capacitor_SMD:C_0603_1608Metric, F.Cu at (208.8, 132.9)
- added C35: 10uF, Capacitor_SMD:C_0603_1608Metric, F.Cu at (214.7, 123.3)
- added C36: 100nF, Capacitor_SMD:C_0603_1608Metric, F.Cu at (210.7, 127.2)
- added C37: 100nF, Capacitor_SMD:C_0603_1608Metric, F.Cu at (204.8, 132.9)
- added C38: 100nF, Capacitor_SMD:C_0603_1608Metric, F.Cu at (214.7, 120.8)
- added C39: 100nF, Capacitor_SMD:C_0603_1608Metric, F.Cu at (214.7, 118.3)
- added C4: 100nF, Capacitor_SMD:C_0603_1608Metric, F.Cu at (213.2, 98.5)
- added C40: 100nF, Capacitor_SMD:C_0603_1608Metric, F.Cu at (210.7, 124.7)
- added C41: 100nF, Capacitor_SMD:C_0603_1608Metric, F.Cu at (184.6, 129.9)
- added C42: 100nF, Capacitor_SMD:C_0603_1608Metric, F.Cu at (214.7, 115.8)
- added C43: 22uF, Capacitor_SMD:C_0603_1608Metric, F.Cu at (184.6, 133.0)
- added C44: 100nF, Capacitor_SMD:C_0603_1608Metric, F.Cu at (196.6, 133.0)
- added C45: 100nF, Capacitor_SMD:C_0603_1608Metric, F.Cu at (200.8, 132.9)
- added C46: 100nF, Capacitor_SMD:C_0603_1608Metric, F.Cu at (192.6, 133.0)
- added C47: 100nF, Capacitor_SMD:C_0603_1608Metric, F.Cu at (214.7, 113.3)
- added C48: 100nF, Capacitor_SMD:C_0603_1608Metric, F.Cu at (188.6, 133.0)
- added C49: 100nF, Capacitor_SMD:C_0603_1608Metric, F.Cu at (200.8, 121.5)
- added C5: 100uF, Capacitor_SMD:CP_Elec_6.3x7.7, F.Cu at (210.4, 85.5)
- added C50: 10uF, Capacitor_SMD:C_0603_1608Metric, F.Cu at (86.4, 126.7)
- added C6: 100nF, Capacitor_SMD:C_0603_1608Metric, F.Cu at (217.2, 98.5)
- added C7: 100uF, Capacitor_SMD:CP_Elec_6.3x7.7, F.Cu at (195.5, 97.3)
- added C8: 100uF, Capacitor_SMD:CP_Elec_6.3x7.7, F.Cu at (198.3, 88.4)
- added C9: 100nF, Capacitor_SMD:C_0603_1608Metric, F.Cu at (209.8, 106.4)
- added D1: SVM1550UB, Package_TO_SOT_SMD:TO-277B, F.Cu at (229.3, 80.7)
- added D2: LED, LED_SMD:LED_0603_1608Metric, F.Cu at (111.3, 139.2)
- added D3: LED, LED_SMD:LED_0603_1608Metric, F.Cu at (116.9, 134.0)
- added J1: VIN, Connector_AMASS:AMASS_XT30PW-M_1x02_P2.50mm_Horizontal, F.Cu at (187.9, 90.4)
- added J2: ANT, Connector_Coaxial:SMA_Molex_73251-2200_Horizontal, F.Cu at (161.8, 93.8)
- added J3: Conn_01x03, Connector_JST:JST_GH_SM03B-GHS-TB_1x03-1MP_P1.25mm_Horizontal, F.Cu at (120.2, 123.8)
- added J4: VOUT, Connector_AMASS:AMASS_XT30PW-F_1x02_P2.50mm_Horizontal, F.Cu at (154.7, 113.6)
- added L1: 3.3uH, Inductor_SMD:L_10.4x10.4_H4.8, F.Cu at (184.0, 99.2)
- added L2: 4.7uH, Inductor_SMD:L_Abracon_ASPI-0630LR, F.Cu at (220.6, 88.5)
- added L3: 6.8uH, Inductor_SMD:L_Abracon_ASPI-0630LR, F.Cu at (203.7, 127.6)
- added L4: 47nH, Inductor_SMD:L_0805_2012Metric_Pad1.15x1.40mm_HandSolder, F.Cu at (82.0, 126.9)
- added LCD1: 1.8inch-TFT-LCD, Display:TFT-LCD1.8inch, F.Cu at (80.6, 124.4)
- added M1: Debugger, Connector:Gernic_Debugger, F.Cu at (116.3, 96.8)
- added Q1: S8050, Package_TO_SOT_SMD:SOT-23, F.Cu at (227.8, 87.4)
- added Q2: ME85P03, Package_TO_SOT_SMD:TO-252-2, F.Cu at (199.1, 80.3)
- added Q3: WST3400A, Package_TO_SOT_SMD:SOT-23, F.Cu at (206.4, 102.9)
- added Q4: S8050, Package_TO_SOT_SMD:SOT-23, F.Cu at (210.8, 102.9)
- added R1: 100kR, Resistor_SMD:R_0603_1608Metric, F.Cu at (227.6, 90.9)
- added R10: 86.6kR, Resistor_SMD:R_0603_1608Metric, F.Cu at (219.1, 103.6)
- added R11: 47kR, Resistor_SMD:R_0603_1608Metric, F.Cu at (232.1, 88.9)
- added R12: 100kR, Resistor_SMD:R_0603_1608Metric, F.Cu at (226.5, 93.9)
- added R13: 23.7kR, Resistor_SMD:R_0603_1608Metric, F.Cu at (222.5, 96.4)
- added R14: 82kR, Resistor_SMD:R_0603_1608Metric, F.Cu at (219.1, 101.1)
- added R15: 10kR, Resistor_SMD:R_0603_1608Metric, F.Cu at (213.8, 106.4)
- added R16: 10kR, Resistor_SMD:R_0603_1608Metric, F.Cu at (114.0, 144.2)
- added R17: 1kR, Resistor_SMD:R_0603_1608Metric, F.Cu at (106.0, 151.1)
- added R18: 1kR, Resistor_SMD:R_0603_1608Metric, F.Cu at (115.3, 141.7)
- added R19: 10kR, Resistor_SMD:R_0603_1608Metric, F.Cu at (110.0, 146.8)
- added R2: 10kR, Resistor_SMD:R_0603_1608Metric, F.Cu at (232.1, 86.4)
- added R20: 10kR, Resistor_SMD:R_0603_1608Metric, F.Cu at (106.0, 143.6)
- added R3: 100kR, Resistor_SMD:R_0603_1608Metric, F.Cu at (215.1, 103.6)
- added R4: 1MR, Resistor_SMD:R_0603_1608Metric, F.Cu at (215.1, 101.1)
- added R5: 100kR, Resistor_SMD:R_0603_1608Metric, F.Cu at (223.1, 101.4)
- added R6: 10kR, Resistor_SMD:R_0603_1608Metric, F.Cu at (223.1, 98.9)
- added R7: 1kR, Resistor_SMD:R_0603_1608Metric, F.Cu at (205.8, 107.2)
- added R8: 100kR, Resistor_SMD:R_0603_1608Metric, F.Cu at (231.6, 91.4)
- added R9: 13.6kR, Resistor_SMD:R_0603_1608Metric, F.Cu at (217.8, 106.1)
- added SW1: SW_DIP_x01, Button_Switch_SMD:SW_SPST_CK_RS282G05A3, F.Cu at (210.6, 78.9)
- added SW2: SW_DIP_x01, Button_Switch_SMD:SW_SPST_CK_RS282G05A3, F.Cu at (109.4, 135.3)
- added U1: HX9193, Package_TO_SOT_SMD:SOT-23-5, F.Cu at (213.6, 95.0)
- added U10: π131M31, Package_SO:SOIC-16_3.9x9.9mm_P1.27mm, F.Cu at (208.5, 117.8)
- added U11: ATGM336H, RF_GPS:ublox_MAX, F.Cu at (155.9, 122.2)
- added U12: XPT2046TS, Package_SO:TSSOP-16_4.4x5mm_P0.65mm, F.Cu at (129.2, 123.3)
- added U2: REF3030, Package_TO_SOT_SMD:SOT-23, F.Cu at (218.2, 94.9)
- added U3: TPS54540, Package_SO:TI_SO-PowerPAD-8, F.Cu at (194.8, 104.6)
- added U4: SY8303, Package_TO_SOT_SMD:SOT-23-8, F.Cu at (201.7, 103.7)
- added U5: MM32F3277G9P, Package_QFP:LQFP-144_20x20mm_P0.5mm, F.Cu at (91.8, 144.9)
- added U6: ADIS16470AMLZ, Sensor_Motion:ADIS16470AMLZ, F.Cu at (184.0, 120.3)
- added U7: B0505S-1WR3, Package_SIP:SIP-4_B0505S_1WR3, F.Cu at (193.4, 118.2)
- added U8: HX9193, Package_TO_SOT_SMD:SOT-23-5, F.Cu at (180.1, 131.0)
- added U9: π131M31, Package_SO:SOIC-16_3.9x9.9mm_P1.27mm, F.Cu at (194.5, 126.0)
- added Y1: 8MHz, Crystal:Crystal_SMD_3225-4Pin_3.2x2.5mm, F.Cu at (106.6, 140.1)

Commit message: Update the PCB board frame and layout.
Parts:
- moved C18 141.1 mm to (251.1, 150.6)
- moved C19 141.1 mm to (259.1, 143.0)
- moved C25 141.1 mm to (257.9, 135.4)
- moved C28 141.1 mm to (262.0, 132.8)
- moved C29 141.1 mm to (251.1, 148.1)
- moved C30 141.1 mm to (251.1, 143.1)
- moved D2 141.1 mm to (252.4, 138.0)
- moved R19 141.1 mm to (251.1, 145.6)
- moved SW2 141.1 mm to (250.5, 134.1)
- moved C17 141.1 mm to (262.0, 135.4)
- moved C20 141.1 mm to (255.1, 145.6)
- moved C21 141.1 mm to (260.4, 140.4)
- moved C22 141.1 mm to (260.4, 137.9)
- moved C32 141.1 mm to (256.4, 138.0)
- moved R16 141.1 mm to (255.1, 143.1)
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Other:
- board outline added: 95 x 50 mm
- net class Default: clearance 0.2 -> 0.1; via_dia 0.6 -> 0.4; via_drill 0.3 -> 0.2
- rule trace_clearance: 0.2 -> 0.1
- rule trace_min: 0.2 -> 0.1
- rule via_min_drill: 0.3 -> 0.2

Commit message: Add Servo Interface
Parts:
- added J5: Conn_01x03, Connector_PinHeader_2.54mm:PinHeader_1x03_P2.54mm_Horizontal, F.Cu at (148.5, 143.3)
Connections:
- U5 pad 60: Net-(U5-Pad60) -> /Connector/Servo_PWM

Commit message: Basic completion of PCB layout.
Parts:
- removed BT1: Battery_Cell, Battery:BatteryHolder_Keystone_1060_1x2032
- C1, C10, C12, C14, C15, C16, C19, C2, C25, C30, C34, C36, C37, C4, C40, C42, C44, C45, C47, C48, C49, C5, C6, C7, C8, C9, D1, J3, L1, L2, Q1, Q2, Q3, Q4, R1, R10, R11, R12, R14, R15, R2, R20, R3, R4, R6, R7, R8, R9, U1, U12, U2, U3, U4, U5, Y1: moved to B.Cu
- moved J2 135.1 mm to (195.3, 87.8), turned to 270 degrees
- moved R2 133.6 mm to (127.7, 91.3), turned to 90 degrees
- moved R5 131.8 mm to (123.0, 76.0)
- moved R13 130.4 mm to (121.3, 94.7), turned to 270 degrees
- moved R1 129.9 mm to (127.0, 86.3)
- moved L4 129.7 mm to (189.7, 86.8), turned to 270 degrees
- moved R11 128.1 mm to (134.3, 72.2), turned to 180 degrees
- moved R8 127.9 mm to (133.6, 78.6), turned to 90 degrees
- moved Q1 126.4 mm to (130.6, 87.3), turned to 90 degrees
- moved R10 124.5 mm to (124.0, 96.3), turned to 90 degrees
- moved R3 123.4 mm to (124.3, 75.3), turned to 90 degrees
- moved R4 122.5 mm to (123.4, 81.5), turned to 180 degrees
- moved D1 122.5 mm to (136.4, 91.8), turned to 270 degrees
- moved SW1 122.5 mm to (117.5, 72.8)
- moved C5 120.1 mm to (120.6, 102.1), turned to 270 degrees
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Connections:
- C46 pad 2: GNDA -> EP
- C47 pad 2: GNDA -> EP
- U11 pad 6: Net-(BT1-Pad1) -> +3V3
- U12 pad 11: /MCU/PG2 -> /MCU/PE0
- U12 pad 15: /MCU/PG3 -> /MCU/PE1
- U5 pad 1: /IMU/IMU_CLK -> /Connector/LCD_CLK
- U5 pad 132: Net-(U5-Pad132) -> /IMU/IMU_DR
- U5 pad 133: /Connector/LCD_CLK -> /IMU/IMU_CLK
- U5 pad 134: /Connector/LCD_MISO -> /IMU/IMU_MISO
- U5 pad 135: /Connector/LCD_MOSI -> /IMU/IMU_MOSI
- U5 pad 136: Net-(U5-Pad136) -> /IMU/IMU_CS
- U5 pad 137: Net-(U5-Pad137) -> /IMU/IMU_RST
- U5 pad 140: Net-(U5-Pad140) -> /Connector/LCD_CS
- U5 pad 141: Net-(U5-Pad141) -> /MCU/PE0
- U5 pad 142: /IMU/IMU_RST -> /MCU/PE1
- U5 pad 2: /IMU/IMU_CS -> /Connector/LCD_RST
- U5 pad 3: /IMU/IMU_DR -> /Connector/LCD_A0
- U5 pad 4: /IMU/IMU_MISO -> /Connector/LCD_MISO
- U5 pad 5: /IMU/IMU_MOSI -> /Connector/LCD_MOSI
- U5 pad 54: Net-(U5-Pad54) -> /MCU/KEY
- U5 pad 87: /MCU/PG2 -> Net-(U5-Pad87)
- U5 pad 88: /MCU/PG3 -> Net-(U5-Pad88)
- U5 pad 89: /Connector/LCD_CS -> Net-(U5-Pad89)
- U5 pad 90: /Connector/LCD_A0 -> Net-(U5-Pad90)
- U5 pad 91: /Connector/LCD_RST -> Net-(U5-Pad91)
- U5 pad 93: /MCU/KEY -> Net-(U5-Pad93)
Routing:
- net +3.3VA: track 0.00 -> 95.3 mm, vias 0 -> 11
- net /Connector/LCD_CS: track 0.00 -> 40.7 mm, vias 0 -> 1
- net /MCU/PE0: track 0.00 -> 32.9 mm, vias 0 -> 2
- net /Connector/LCD_MOSI: track 0.00 -> 29.1 mm, vias 0 -> 2
- net /Connector/LCD_CLK: track 0.00 -> 29.0 mm, vias 0 -> 2
- net /Connector/LCD_MISO: track 0.00 -> 28.0 mm, vias 0 -> 2
- net /MCU/PE1: track 0.00 -> 27.8 mm, vias 0 -> 2
- net +3V3: track 0.00 -> 27.0 mm, vias 0 -> 1
- net +5VA: track 0.00 -> 25.3 mm
- net /Connector/LCD_A0: track 0.00 -> 22.6 mm, vias 0 -> 1
- net /IMU/SCLK: track 0.00 -> 22.0 mm, vias 0 -> 2
- net /Connector/LCD_RST: track 0.00 -> 21.7 mm, vias 0 -> 1
- net +15V: track 0.00 -> 21.3 mm
- net /IMU/DIN: track 0.00 -> 20.0 mm, vias 0 -> 2
- net /IMU/IMU_DR: track 0.00 -> 17.8 mm, vias 0 -> 1
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Other:
- outline, holes or cut-outs redrawn

Commit message: Add copper laying for high power areas and complete small parts of wiring.
Parts:
- R4: moved to F.Cu
- moved C28 19.0 mm to (183.6, 95.1), turned to 90 degrees
- moved C11 3.27 mm to (123.6, 93.7)
- moved C13 2.32 mm to (121.6, 91.8)
- moved R16 1.99 mm to (164.8, 95.4)
- moved C33 1.88 mm to (161.0, 95.4)
- moved R10 0.90 mm to (124.9, 96.3)
- moved R13 0.69 mm to (121.6, 95.3), turned to 90 degrees
- moved R4 0.49 mm to (123.1, 81.9)
- moved C34 0.43 mm to (164.3, 110.5)
- moved C10 0.11 mm to (126.2, 103.1), turned to 0 degrees
Routing:
- net +15V: track 21.3 -> 62.2 mm, vias 0 -> 17
- net /Connector/Servo_PWM: track 0.00 -> 21.9 mm
- net /IMU/DR: track 0.00 -> 19.0 mm, vias 0 -> 2
- net /IMU/RST: track 0.00 -> 18.5 mm, vias 0 -> 2
- net Net-(Q1-Pad1): track 14.4 -> 32.3 mm, vias 1 -> 3
- net +3V3: track 27.0 -> 43.7 mm, vias 1 -> 2
- net Net-(C11-Pad1): track 0.00 -> 15.9 mm, vias 0 -> 1
- net /IMU/CS: track 0.00 -> 15.5 mm, vias 0 -> 2
- net /Connector/GPS_RX: track 0.00 -> 15.2 mm, vias 0 -> 1
- net /Connector/GPS_TX: track 0.00 -> 13.9 mm, vias 0 -> 1
- net VDD: track 0.00 -> 9.49 mm
- net /MCU/ADC23_IN14: track 0.00 -> 5.54 mm
- net Net-(C12-Pad1): track 6.72 -> 1.92 mm
- net Net-(R14-Pad2): track 0.00 -> 4.79 mm
- net Net-(C9-Pad1): track 0.00 -> 4.39 mm
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- added copper zone on B.Cu, net +15V
- added copper zone on F.Cu, net +15V
- added copper zone on B.Cu, net +5V
- added copper zone on B.Cu, net +7.5V
- added copper zone on B.Cu, net GNDA
- added copper zone on F.Cu, net GNDA
- added copper zone on B.Cu, net Net-(C12-Pad1)
- added copper zone on B.Cu, net Net-(C9-Pad1)
- added copper zone on B.Cu, net VDD

Commit message: Basic completion of PCB layout wiring design and silkscreen placement.
Parts:
- added C51: 22uF, Capacitor_SMD:C_0805_2012Metric, B.Cu at (148.7, 103.8)
- added C52: 22uF, Capacitor_SMD:C_0805_2012Metric, F.Cu at (190.0, 79.9)
- added C53: 100nF, Capacitor_SMD:C_0603_1608Metric, B.Cu at (183.3, 88.8)
- added C54: 100nF, Capacitor_SMD:C_0603_1608Metric, B.Cu at (183.2, 83.3)
- added C55: 100nF, Capacitor_SMD:C_0603_1608Metric, F.Cu at (109.8, 111.5)
- added C56: 100nF, Capacitor_SMD:C_0603_1608Metric, B.Cu at (170.5, 101.5)
- added C57: 100nF, Capacitor_SMD:C_0603_1608Metric, F.Cu at (109.8, 114.8)
- added C58: 100nF, Capacitor_SMD:C_0603_1608Metric, B.Cu at (153.6, 74.4)
- C21, C22, C32: moved to B.Cu
- moved C22 63.5 mm to (139.2, 107.1), turned to 180 degrees
- moved C32 63.3 mm to (139.4, 111.9), turned to 90 degrees
- moved C21 55.4 mm to (147.1, 107.2)
- moved C29 53.0 mm to (161.9, 78.3), turned to 180 degrees
- moved C31 48.7 mm to (161.6, 80.9), turned to 270 degrees
- moved C18 47.8 mm to (161.8, 92.4), turned to 90 degrees
- moved C23 46.5 mm to (161.8, 88.9), turned to 270 degrees
- moved C20 42.7 mm to (173.4, 78.3), turned to 180 degrees
- moved C17 40.4 mm to (168.3, 78.3), turned to 180 degrees
- moved C26 36.2 mm to (179.3, 73.5), turned to 90 degrees
- moved C27 33.5 mm to (173.9, 96.5)
- moved C28 0.30 mm to (183.3, 95.1)
Routing:
- net +3V3: track 43.7 -> 318.7 mm, vias 2 -> 21
- net /Connector/MOTOR_TX: track 0.00 -> 93.2 mm, vias 0 -> 2
- net /Connector/MOTOR_RX: track 0.00 -> 89.9 mm, vias 0 -> 2
- net /Connector/SWDIO: track 0.00 -> 78.5 mm, vias 0 -> 2
- net /Connector/SWDCLK: track 0.00 -> 78.4 mm, vias 0 -> 2
- net /Connector/DEBUG_RX: track 0.00 -> 75.6 mm, vias 0 -> 2
- net /Connector/DEBUG_TX: track 0.00 -> 74.6 mm, vias 0 -> 2
- net +7.5V: track 0.00 -> 70.2 mm, vias 0 -> 5
- net /MCU/PF13: track 1.94 -> 53.8 mm, vias 0 -> 2
- net +5V: track 12.5 -> 54.1 mm, vias 0 -> 5
- net +15V: track 62.2 -> 47.1 mm
- net EP: track 0.00 -> 13.2 mm, vias 0 -> 139
- net /MCU/RST: track 1.71 -> 13.2 mm, vias 0 -> 2
- net GNDA: vias 0 -> 33
- net /IMU/SCLK: vias 2 -> 3
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- added copper zone on B.Cu, net +3V3
- added copper zone on B.Cu, net EP
- added copper zone on F.Cu, net EP
- added copper zone on In1.Cu, net EP
- added copper zone on In2.Cu, net EP
- added copper zone on In1.Cu, net GNDA
- added copper zone on In2.Cu, net GNDA
Other:
- rule trace_min: 0.1 -> 0.2
- board text added: "2021/12/05"
- board text added: "GDUT"
