File: circuit/Compass&Storage.kicad_sch (KiCad schematic)
At the start: 9 parts, among them U13 HMC5883L, U14 AT24C02

Commit message: Modify the circuit diagram of the GPS to swap the pin order of the serial port. Add borders to the Compass schematic.
Other:
- note added: "Cmpass"
- note added: "EEPROM"
- moved on the sheet: C69, C70, C71, C72, C73, R10, R9, U13, U14
