File: circuit/ControlMCU.kicad_sch (KiCad schematic)
At the start: 21 parts

Commit message: Update circuit and ADIS16470 footprint reference datasheet.
Connections:
- net +3V3 renamed +3.3VP

Commit message: Basically finished schematic drawing and annotation, not yet package selection.
Parts:
- gave numbers to parts that had none: 21
Connections:
- net TIM2_CH1: now reaches U11.34 (PA0)
- no-connect marks 106 -> 105

Commit message: Basically finished all the design of the schematic and selected the package for the components.
Connections:
- net UART3_TX: now reaches U11.77 (PD8)
- net UART3_RX: now reaches U11.78 (PD9)
- no-connect marks 105 -> 103
Changed lines of the file:
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@@
   (title_block
     (title "MM32_Board")
-    (date "2022-01-11")
-    (rev "1.0.2")
+    (date "2022-01-16")
+    (rev "1.2.1")
   )
   (junction (at 217.17 134.62) (diameter 0) (color 0 0 0 0)
@@
   (no_connect (at 161.29 113.03))
   (no_connect (at 161.29 123.19))
-  (no_connect (at 161.29 130.81))
-  (no_connect (at 161.29 133.35))
   (no_connect (at 140.97 151.13))
   (no_connect (at 128.27 151.13))
@@
     (stroke (width 0) (type default) (color 0 0 0 0))
   )
+  (wire (pts (xy 173.99 130.81) (xy 161.29 130.81))
+    (stroke (width 0) (type default) (color 0 0 0 0))
+  )
   (wire (pts (xy 234.95 163.83) (xy 241.3 163.83))
     (stroke (width 0) (type default) (color 0 0 0 0))
@@
   )
   (wire (pts (xy 95.25 27.94) (xy 95.25 46.99))
+    (stroke (width 0) (type default) (color 0 0 0 0))
+  )
+  (wire (pts (xy 161.29 133.35) (xy 173.99 133.35))
     (stroke (width 0) (type default) (color 0 0 0 0))
   )
@@
     (effects (font (size 1.27 1.27)) (justify right))
   )
+  (hierarchical_label "UART3_TX" (shape output) (at 173.99 133.35 0)
+    (effects (font (size 1.27 1.27)) (justify left))
+  )
   (hierarchical_label "SWDCLK" (shape input) (at 151.13 34.29 90)
     (effects (font (size 1.27 1.27)) (justify left))
@@
     (effects (font (size 1.27 1.27)) (justify left))
   )
+  (hierarchical_label "UART3_RX" (shape input) (at 173.99 130.81 0)
+    (effects (font (size 1.27 1.27)) (justify left))
+  )

Commit message: Revised and finalized the final circuit schematic.
Connections:
- net LED1: now also U11.1 (PE2); no longer U11.49 (PF11)
- net TIM3_CH1: now reaches U11.134 (PB4)
- net UART7_TX: now reaches U11.136 (PB6)
- net UART7_RX: now reaches U11.137 (PB7)
- net TIM2_CH1: no longer names the net of U11.34 (PA0)
- net UART3_RX: no longer names the net of U11.78 (PD9)
- net UART3_TX: no longer names the net of U11.77 (PD8)
Changed lines of the file:
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@@
   (title_block
     (title "MM32_Board")
-    (date "2022-01-16")
-    (rev "1.2.1")
+    (date "2022-01-18")
+    (rev "1.2.2")
   )
   (junction (at 217.17 134.62) (diameter 0) (color 0 0 0 0)
@@
   (no_connect (at 92.71 46.99))
   (no_connect (at 90.17 46.99))
-  (no_connect (at 87.63 46.99))
   (no_connect (at 72.39 46.99))
   (no_connect (at 69.85 46.99))
   (no_connect (at 67.31 46.99))
   (no_connect (at 85.09 46.99))
-  (no_connect (at 82.55 46.99))
-  (no_connect (at 80.01 46.99))
   (no_connect (at 143.51 151.13))
   (no_connect (at 161.29 97.79))
@@
   (no_connect (at 118.11 151.13))
   (no_connect (at 52.07 120.65))
-  (no_connect (at 146.05 46.99))
   (no_connect (at 105.41 46.99))
   (no_connect (at 52.07 102.87))
@@
   (no_connect (at 135.89 151.13))
   (no_connect (at 113.03 46.99))
+  (no_connect (at 161.29 133.35))
+  (no_connect (at 161.29 130.81))
+  (no_connect (at 92.71 151.13))
   (no_connect (at 52.07 85.09))
   (no_connect (at 161.29 138.43))
   (no_connect (at 161.29 92.71))
+  (no_connect (at 52.07 138.43))
   (no_connect (at 52.07 72.39))
   (no_connect (at 138.43 151.13))
@@
   (no_connect (at 52.07 59.69))
   (no_connect (at 52.07 57.15))
-  (no_connect (at 52.07 54.61))
   (no_connect (at 74.93 151.13))
   (no_connect (at 161.29 85.09))
-  (no_connect (at 143.51 46.99))
   (no_connect (at 110.49 46.99))
   (no_connect (at 52.07 62.23))
@@
   (no_connect (at 82.55 151.13))
   (no_connect (at 161.29 82.55))
+  (no_connect (at 146.05 46.99))
+  (no_connect (at 143.51 46.99))
   (no_connect (at 130.81 151.13))
   (no_connect (at 161.29 64.77))
@@
     (stroke (width 0) (type default) (color 0 0 0 0))
   )
-  (wire (pts (xy 40.64 138.43) (xy 52.07 138.43))
+  (wire (pts (xy 87.63 35.56) (xy 87.63 46.99))
     (stroke (width 0) (type default) (color 0 0 0 0))
   )
@@
     (stroke (width 0) (type default) (color 0 0 0 0))
   )
-  (wire (pts (xy 173.99 130.81) (xy 161.29 130.81))
+  (wire (pts (xy 80.01 34.29) (xy 80.01 46.99))
     (stroke (width 0) (type default) (color 0 0 0 0))
   )
@@
     (stroke (width 0) (type default) (color 0 0 0 0))
   )
-  (wire (pts (xy 92.71 151.13) (xy 92.71 171.45))
+  (wire (pts (xy 52.07 54.61) (xy 31.75 54.61))
     (stroke (width 0) (type default) (color 0 0 0 0))
   )
@@
     (stroke (width 0) (type default) (color 0 0 0 0))
   )
-  (wire (pts (xy 161.29 133.35) (xy 173.99 133.35))
+  (wire (pts (xy 82.55 46.99) (xy 82.55 34.29))
     (stroke (width 0) (type default) (color 0 0 0 0))
   )
@@
     (effects (font (size 1.27 1.27)) (justify left bottom))
   )
-  (label "LED1" (at 92.71 171.45 90)
+  (label "LED1" (at 31.75 54.61 0)
     (effects (font (size 1.27 1.27)) (justify left bottom))
   )
@@
     (effects (font (size 1.27 1.27)) (justify right))
   )
-  (hierarchical_label "TIM2_CH1" (shape output) (at 40.64 138.43 180)
-    (effects (font (size 1.27 1.27)) (justify right))
+  (hierarchical_label "TIM3_CH1" (shape output) (at 87.63 35.56 90)
+    (effects (font (size 1.27 1.27)) (justify left))
   )
   (hierarchical_label "UART6_TX" (shape output) (at 85.09 162.56 270)
     (effects (font (size 1.27 1.27)) (justify right))
   )
-  (hierarchical_label "UART3_TX" (shape output) (at 173.99 133.35 0)
+  (hierarchical_label "UART7_TX" (shape output) (at 82.55 34.29 90)
     (effects (font (size 1.27 1.27)) (justify left))
   )
@@
     (effects (font (size 1.27 1.27)) (justify left))
   )
-  (hierarchical_label "UART3_RX" (shape input) (at 173.99 130.81 0)
+  (hierarchical_label "UART7_RX" (shape input) (at 80.01 34.29 90)
     (effects (font (size 1.27 1.27)) (justify left))
   )
@@
   (symbol (lib_id "Device:R") (at 77.47 38.1 0) (unit 1)
     (in_bom yes) (on_board yes)
-    (property "Reference" "R4" (id 0) (at 79.248 36.9316 0)
-      (effects (font (size 1.27 1.27)) (justify left))
-    )
-    (property "Value" "10kR" (id 1) (at 79.248 39.243 0)
-      (effects (font (size 1.27 1.27)) (justify left))
-    )
+    (property "Reference" "R4" (id 0) (at 71.755 37.465 0)
+      (effects (font (size 1.27 1.27)) (justify left))
+    )
+    (property "Value" "10kR" (id 1) (at 70.485 40.005 0)
+      (effects (font (size 1.27 1.27)) (justify left))
+    )
