File: circuit/Debugger.kicad_sch (KiCad schematic)
At the start: 2 parts

Commit message: Basically finished schematic drawing and annotation, not yet package selection.
Parts:
- added C67: 10uF, Capacitor_SMD:C_0603_1608Metric, symbol Device:C
- added C68: 0.1uF, Capacitor_SMD:C_0603_1608Metric, symbol Device:C
- added R7: 1kR, Resistor_SMD:R_0603_1608Metric, symbol Device:R
- added SW1: SW_DIP_x01, symbol Switch:SW_DIP_x01
- gave numbers to parts that had none: 2
Connections:
- net +5V: now also C67.1, C68.1, R7.1
- net GND: now also U12.15 (#EN), C67.2, C68.2, SW1.1
- net SEL: now reaches U12.1 (SEL)
- net SEL: now also R7.2, SW1.2
Other:
- moved on the sheet: M1, U12

Commit message: Basically finished all the design of the schematic and selected the package for the components.
Parts:
- removed SW1: SW_DIP_x01, symbol Switch:SW_DIP_x01
- added SW1: SW_DIP_x02, Button_Switch_SMD:SW_DIP_SPSTx02_Slide_Copal_CHS-02B_W7.62mm_P1.27mm, symbol Switch:SW_DIP_x02
- C68: value 0.1uF -> 100nF
- M1: footprint Connector:Gernic_Debugger -> MM32_Library:Gernic_Debugger
- R7: value 1kR -> 10kR
Connections:
- net GND: now also SW1.1
- net SEL: now also SW1.4
- no-connect marks 0 -> 2
Changed lines of the file:
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@@
   (title_block
     (title "MM32_Board")
-    (date "2022-01-11")
-    (rev "1.0.2")
+    (date "2022-01-16")
+    (rev "1.2.1")
   )
   (junction (at 229.235 107.95) (diameter 0) (color 0 0 0 0)
   )
+  (no_connect (at 231.775 112.395))
+  (no_connect (at 231.775 127.635))
   (polyline (pts (xy 166.37 71.12) (xy 166.37 142.24))
     (stroke (width 0) (type default) (color 0 0 0 0))
@@
     (property "Reference" "M1" (id 0) (at 97.79 100.965 0))
     (property "Value" "Debugger" (id 1) (at 101.6 116.205 0))
-    (property "Footprint" "Connector:Gernic_Debugger" (id 2) (at 97.79 100.965 0)
+    (property "Footprint" "MM32_Library:Gernic_Debugger" (id 2) (at 97.79 100.965 0)
       (effects (font (size 1.27 1.27)) hide)
     )
@@
     (pin "2")
   )
+  (symbol (lib_id "Switch:SW_DIP_x02") (at 231.775 120.015 90) (unit 1)
+    (in_bom yes) (on_board yes) (fields_autoplaced)
+    (property "Reference" "SW1" (id 0) (at 233.045 118.7449 90)
+      (effects (font (size 1.27 1.27)) (justify right))
+    )
+    (property "Value" "SW_DIP_x02" (id 1) (at 233.045 121.2849 90)
+      (effects (font (size 1.27 1.27)) (justify right) hide)
+    )
+    (property "Footprint" "Button_Switch_SMD:SW_DIP_SPSTx02_Slide_Copal_CHS-02B_W7.62mm_P1.27mm" (id 2) (at 231.775 120.015 0)
+      (effects (font (size 1.27 1.27)) hide)
+    )
+    (property "Datasheet" "~" (id 3) (at 231.775 120.015 0)
+      (effects (font (size 1.27 1.27)) hide)
+    )
+    (pin "1")
+    (pin "2")
+    (pin "3")
+    (pin "4")
+  )
   (symbol (lib_id "power:+5V") (at 143.51 88.265 0) (unit 1)
     (in_bom yes) (on_board yes)
@@
     (in_bom yes) (on_board yes)
     (property "Reference" "R7" (id 0) (at 233.045 97.79 0))
-    (property "Value" "1kR" (id 1) (at 233.68 100.33 0))
+    (property "Value" "10kR" (id 1) (at 233.68 100.33 0))
     (property "Footprint" "Resistor_SMD:R_0603_1608Metric" (id 2) (at 227.457 97.79 90)
       (effects (font (size 1.27 1.27)) hide)
@@
     (pin "1")
   )
-  (symbol (lib_id "Switch:SW_DIP_x01") (at 229.235 120.015 90) (unit 1)
-    (in_bom yes) (on_board yes)
-    (property "Reference" "SW1" (id 0) (at 231.14 120.015 90)
-      (effects (font (size 1.27 1.27)) (justify right))
-    )
-    (property "Value" "SW_DIP_x01" (id 1) (at 231.14 121.2849 90)
-      (effects (font (size 1.27 1.27)) (justify right) hide)
-    )
-    (property "Footprint" "" (id 2) (at 229.235 120.015 0)
-      (effects (font (size 1.27 1.27)) hide)
-    )
-    (property "Datasheet" "~" (id 3) (at 229.235 120.015 0)
-      (effects (font (size 1.27 1.27)) hide)
-    )
-    (pin "1")
-    (pin "2")
-  )
   (symbol (lib_id "Device:C") (at 143.51 107.95 0) (unit 1)
     (in_bom yes) (on_board yes)
@@
       (effects (font (size 1.27 1.27)) (justify left))
     )
-    (property "Value" "0.1uF" (id 1) (at 146.431 109.093 0)
+    (property "Value" "100nF" (id 1) (at 146.431 109.093 0)
       (effects (font (size 1.27 1.27)) (justify left))
     )

Commit message: Revised and finalized the final circuit schematic.
Connections:
- net DBG_RX: now also M1.6 (U_TX), U12.9 (DC); no longer M1.7 (U_RX), U12.12 (DD)
- net DBG_RX1: now also U12.11 (S1C); no longer U12.14 (S1D)
- net DBG_RX2: now also U12.10 (S2C); no longer U12.13 (S2D)
- net DBG_TX: now also M1.7 (U_RX), U12.12 (DD); no longer M1.6 (U_TX), U12.9 (DC)
- net DBG_TX1: now also U12.14 (S1D); no longer U12.11 (S1C)
- net DBG_TX2: now also U12.13 (S2D); no longer U12.10 (S2C)
- net SWDCLK: now also U12.4 (DA); no longer U12.7 (DB)
- net SWDCLK1: now also U12.2 (S1A); no longer U12.5 (S1B)
- net SWDCLK2: now also U12.3 (S2A); no longer U12.6 (S2B)
- net SWDIO: now also U12.7 (DB); no longer U12.4 (DA)
- net SWDIO1: now also U12.5 (S1B); no longer U12.2 (S1A)
- net SWDIO2: now also U12.6 (S2B); no longer U12.3 (S2A)
