File: circuit/IMU.kicad_sch (KiCad schematic)
At the start: 23 parts, among them U10 π131M31, U6 ADIS16470AMLZ, U7 B0505S-1WR3, U8 HX9193, U9 π131M31

Commit message: Update circuit with control mcu.
Parts:
- renumbered C33 to C?, C34 to C?, C35 to C?, C36 to C?, C43 to C?, C38 to C?, C49 to C?, C48 to C?, C47 to C?, C46 to C?, C40 to C?, C42 to C?, C45 to C?, C37 to C?, C39 to C?, C41 to C?, C44 to C?, L3 to L?, U7 to U?, U8 to U?, U6 to U?, U9 to U?, U10 to U?

Commit message: Update circuit and ADIS16470 footprint reference datasheet.
Connections:
- net +3V3 is gone; now on net +3.3VA: C?.1, C?.1, U?.1 (VDD1), U?.1 (VDD1)
- net +3.3VA: no longer C?.1, C?.1, C?.1, C?.1, C?.1, C?.1, C?.1, C?.1, C?.1, C?.1, C?.1, U?.16 (VDD2), U?.16 (VDD2), U?.5 (VOUT), U?.C7 (VDD), U?.D6 (VDD), U?.E3 (VDD), U?.H1 (VDD), U?.J4 (VDD), U?.J5 (VDD), U?.K6 (VDD)
- new net +3.3VADC: C?.1, C?.1, C?.1, C?.1, C?.1, C?.1, C?.1, C?.1, C?.1, C?.1, C?.1, U?.16 (VDD2), U?.16 (VDD2), U?.5 (VOUT), U?.C7 (VDD), U?.D6 (VDD), U?.E3 (VDD), U?.H1 (VDD), U?.J4 (VDD), U?.J5 (VDD), U?.K6 (VDD)

Commit message: Basically finished schematic drawing and annotation, not yet package selection.
Parts:
- gave numbers to parts that had none: 23

Commit message: Basically finished all the design of the schematic and selected the package for the components.
Parts:
- U3: footprint Sensor_Motion:ADIS16470AMLZ -> MM32_Library:ADIS16470AMLZ
- U4: footprint Package_SIP:SIP-4_B0505S_1WR3 -> MM32_Library:SIP-4_B0505S_1WR3
Changed lines of the file:
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@@
   (title_block
     (title "MM32_Board")
-    (date "2022-01-11")
-    (rev "1.0.2")
+    (date "2022-01-16")
+    (rev "1.2.1")
   )
   (junction (at 101.6 100.33) (diameter 0) (color 0 0 0 0)
@@
     (property "Reference" "U4" (id 0) (at 63.5 158.75 0))
     (property "Value" "B0505S-1WR3" (id 1) (at 69.85 168.91 0))
-    (property "Footprint" "Package_SIP:SIP-4_B0505S_1WR3" (id 2) (at 69.85 171.45 0)
+    (property "Footprint" "MM32_Library:SIP-4_B0505S_1WR3" (id 2) (at 69.85 171.45 0)
       (effects (font (size 1.27 1.27)) hide)
     )
@@
     (property "Reference" "U3" (id 0) (at 60.96 33.02 0))
     (property "Value" "ADIS16470AMLZ" (id 1) (at 67.31 111.76 0))
-    (property "Footprint" "Sensor_Motion:ADIS16470AMLZ" (id 2) (at 60.96 33.02 0)
-      (effects (font (size 1.27 1.27)) hide)
-    )
+    (property "Footprint" "MM32_Library:ADIS16470AMLZ" (id 2) (at 60.96 33.02 0)
+      (effects (font (size 1.27 1.27)) hide)
+    )

Commit message: Revised and finalized the final circuit schematic.
Parts:
- added R8: 10kR, Resistor_SMD:R_0603_1608Metric, symbol Device:R
Connections:
- net GND: now also R8.1
- net GNDA: now also R8.2
Changed lines of the file:
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@@
   (title_block
     (title "MM32_Board")
-    (date "2022-01-16")
-    (rev "1.2.1")
+    (date "2022-01-18")
+    (rev "1.2.2")
   )
   (junction (at 101.6 100.33) (diameter 0) (color 0 0 0 0)
   )
   (junction (at 101.6 92.71) (diameter 0) (color 0 0 0 0)
+  )
+  (junction (at 80.01 177.165) (diameter 0) (color 0 0 0 0)
+  )
+  (junction (at 59.69 177.165) (diameter 0) (color 0 0 0 0)
   )
   (junction (at 101.6 72.39) (diameter 0) (color 0 0 0 0)
@@
     (stroke (width 0) (type default) (color 0 0 0 0))
   )
-  (wire (pts (xy 59.69 181.61) (xy 59.69 165.1))
+  (wire (pts (xy 59.69 181.61) (xy 59.69 177.165))
     (stroke (width 0) (type default) (color 0 0 0 0))
   )
@@
     (stroke (width 0) (type default) (color 0 0 0 0))
   )
+  (wire (pts (xy 59.69 177.165) (xy 59.69 165.1))
+    (stroke (width 0) (type default) (color 0 0 0 0))
+  )
   (wire (pts (xy 134.62 63.5) (xy 134.62 72.39))
     (stroke (width 0) (type default) (color 0 0 0 0))
@@
     (stroke (width 0) (type default) (color 0 0 0 0))
   )
+  (wire (pts (xy 73.66 177.165) (xy 80.01 177.165))
+    (stroke (width 0) (type default) (color 0 0 0 0))
+  )
   (wire (pts (xy 241.3 135.89) (xy 247.65 135.89))
     (stroke (width 0) (type default) (color 0 0 0 0))
@@
     (stroke (width 0) (type default) (color 0 0 0 0))
   )
-  (wire (pts (xy 80.01 165.1) (xy 80.01 181.61))
+  (wire (pts (xy 80.01 165.1) (xy 80.01 177.165))
     (stroke (width 0) (type default) (color 0 0 0 0))
   )
@@
     (stroke (width 0) (type default) (color 0 0 0 0))
   )
+  (wire (pts (xy 59.69 177.165) (xy 66.04 177.165))
+    (stroke (width 0) (type default) (color 0 0 0 0))
+  )
   (wire (pts (xy 101.6 114.3) (xy 101.6 107.95))
     (stroke (width 0) (type default) (color 0 0 0 0))
@@
   )
   (wire (pts (xy 59.69 146.05) (xy 59.69 162.56))
+    (stroke (width 0) (type default) (color 0 0 0 0))
+  )
+  (wire (pts (xy 80.01 177.165) (xy 80.01 181.61))
     (stroke (width 0) (type default) (color 0 0 0 0))
   )
@@
     (pin "1")
   )
+  (symbol (lib_id "Device:R") (at 69.85 177.165 90) (unit 1)
+    (in_bom yes) (on_board yes)
+    (property "Reference" "R8" (id 0) (at 69.85 174.625 90)
+      (effects (font (size 1.27 1.27)) (justify left))
+    )
+    (property "Value" "10kR" (id 1) (at 72.39 179.705 90)
+      (effects (font (size 1.27 1.27)) (justify left))
+    )
+    (property "Footprint" "Resistor_SMD:R_0603_1608Metric" (id 2) (at 69.85 178.943 90)
+      (effects (font (size 1.27 1.27)) hide)
+    )
+    (property "Datasheet" "~" (id 3) (at 69.85 177.165 0)
+      (effects (font (size 1.27 1.27)) hide)
+    )
+    (pin "1")
+    (pin "2")
+  )
   (symbol (lib_id "power:+3.3VADC") (at 123.19 88.9 0) (unit 1)
