File: circuit/LCD&GPS.kicad_sch (KiCad schematic)
At the start: 17 parts

Commit message: Basically finished schematic drawing and annotation, not yet package selection.
Parts:
- gave numbers to parts that had none: 17
Other:
- moved on the sheet: C1, C10, C11, C12, C2, C3, C4, C5, C6, C7, C8, C9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

Commit message: Basically finished all the design of the schematic and selected the package for the components.
Parts:
- J1: footprint (none) -> Connector_Coaxial:SMA_Molex_73251-2200_Horizontal
- L1: footprint (none) -> Inductor_SMD:L_0603_1608Metric
- LCD1: footprint Display:TFT-LCD1.8inch -> MM32_Library:TFT-LCD1.8inch
Changed lines of the file:
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@@
   (title_block
     (title "MM32_Board")
-    (date "2022-01-11")
-    (rev "1.0.2")
+    (date "2022-01-16")
+    (rev "1.2.1")
   )
   (junction (at 198.755 97.79) (diameter 0) (color 0 0 0 0)
@@
       (effects (font (size 1.27 1.27)) (justify right))
     )
-    (property "Footprint" "" (id 2) (at 128.905 57.15 0)
+    (property "Footprint" "Connector_Coaxial:SMA_Molex_73251-2200_Horizontal" (id 2) (at 128.905 57.15 0)
       (effects (font (size 1.27 1.27)) hide)
     )
@@
     (property "Reference" "L1" (id 0) (at 123.19 71.12 90))
     (property "Value" "39nH" (id 1) (at 125.095 75.565 90))
-    (property "Footprint" "" (id 2) (at 124.46 73.66 0)
+    (property "Footprint" "Inductor_SMD:L_0603_1608Metric" (id 2) (at 124.46 73.66 0)
       (effects (font (size 1.27 1.27)) hide)
     )
@@
     (property "Reference" "LCD1" (id 0) (at 187.325 53.34 0))
     (property "Value" "1.8inch-TFT-LCD" (id 1) (at 193.675 81.28 0))
-    (property "Footprint" "Display:TFT-LCD1.8inch" (id 2) (at 187.325 53.34 0)
-      (effects (font (size 1.27 1.27)) hide)
-    )
+    (property "Footprint" "MM32_Library:TFT-LCD1.8inch" (id 2) (at 187.325 53.34 0)
+      (effects (font (size 1.27 1.27)) hide)
+    )

Commit message: Modify the circuit diagram of the GPS to swap the pin order of the serial port. Add borders to the Compass schematic.
Connections:
- net GPS_RX: now also U1.21 (UIN0); no longer U1.20 (UOUT0)
- net GPS_TX: now also U1.20 (UOUT0); no longer U1.21 (UIN0)
Changed lines of the file:
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@@
     (effects (font (size 1.27 1.27)) (justify left))
   )
-  (hierarchical_label "GPS_RX" (shape input) (at 74.93 86.36 180)
+  (hierarchical_label "GPS_RX" (shape input) (at 74.93 88.9 180)
     (effects (font (size 1.27 1.27)) (justify right))
   )
@@
     (effects (font (size 1.27 1.27)) (justify left))
   )
-  (hierarchical_label "GPS_TX" (shape output) (at 74.93 88.9 180)
+  (hierarchical_label "GPS_TX" (shape output) (at 74.93 86.36 180)
     (effects (font (size 1.27 1.27)) (justify right))
   )
