File: circuit/Power.kicad_sch (KiCad schematic)
At the start: 7 parts

Commit message: Basically finished schematic drawing and annotation, not yet package selection.
Parts:
- added C45, C46: 10uF, Capacitor_SMD:C_0603_1608Metric, symbol Device:C
- added C47: 0.1uF, Capacitor_SMD:C_0603_1608Metric, symbol Device:C
- gave numbers to parts that had none: 7
Connections:
- net +5V: now also C45.1, C46.1, C47.1
- net GND: now also C45.2, C46.2, C47.2
Other:
- moved on the sheet: C48, C49, C50, C51, J2, U10, U9

Commit message: Basically finished all the design of the schematic and selected the package for the components.
Parts:
- C47: value 0.1uF -> 100nF
- J2: footprint (none) -> Connector_JST:JST_PH_S8B-PH-K_1x08_P2.00mm_Horizontal
Changed lines of the file:
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@@
   (title_block
     (title "MM32_Board")
-    (date "2022-01-11")
-    (rev "1.0.2")
+    (date "2022-01-16")
+    (rev "1.2.1")
   )
   (junction (at 240.03 102.235) (diameter 0) (color 0 0 0 0)
@@
       (effects (font (size 1.27 1.27)) hide)
     )
-    (property "Footprint" "" (id 2) (at 40.005 105.41 0)
+    (property "Footprint" "Connector_JST:JST_PH_S8B-PH-K_1x08_P2.00mm_Horizontal" (id 2) (at 40.005 105.41 0)
       (effects (font (size 1.27 1.27)) hide)
     )
@@
       (effects (font (size 1.27 1.27)) (justify left))
     )
-    (property "Value" "0.1uF" (id 1) (at 99.441 105.918 0)
-      (effects (font (size 1.27 1.27)) (justify left))
-    )
+    (property "Value" "100nF" (id 1) (at 99.441 105.918 0)
+      (effects (font (size 1.27 1.27)) (justify left))
+    )

Commit message: Revised and finalized the final circuit schematic.
Connections:
- net MOTOR_RX: now also J2.5 (Pin_5); no longer J2.4 (Pin_4)
- net MOTOR_TX: now also J2.4 (Pin_4); no longer J2.5 (Pin_5)
Changed lines of the file:
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@@
   (title_block
     (title "MM32_Board")
-    (date "2022-01-16")
-    (rev "1.2.1")
+    (date "2022-01-18")
+    (rev "1.2.2")
   )
   (junction (at 240.03 102.235) (diameter 0) (color 0 0 0 0)
@@
     (stroke (width 0) (type default) (color 0 0 0 0))
   )
-  (wire (pts (xy 75.565 108.585) (xy 75.565 128.27))
+  (wire (pts (xy 74.295 108.585) (xy 74.295 128.27))
     (stroke (width 0) (type default) (color 0 0 0 0))
   )
@@
     (stroke (width 0) (type default) (color 0 0 0 0))
   )
-  (wire (pts (xy 75.565 83.185) (xy 75.565 100.965))
+  (wire (pts (xy 74.295 83.185) (xy 74.295 100.965))
     (stroke (width 0) (type default) (color 0 0 0 0))
   )
@@
     (effects (font (size 1.27 1.27)) (justify left))
   )
-  (hierarchical_label "MOTOR_RX" (shape input) (at 57.785 105.41 0)
+  (hierarchical_label "MOTOR_RX" (shape input) (at 57.785 102.87 0)
     (effects (font (size 1.27 1.27)) (justify left))
   )
-  (hierarchical_label "MOTOR_TX" (shape output) (at 57.785 102.87 0)
+  (hierarchical_label "MOTOR_TX" (shape output) (at 57.785 105.41 0)
     (effects (font (size 1.27 1.27)) (justify left))
   )
@@
     (pin "2")
   )
-  (symbol (lib_id "power:+5V") (at 75.565 83.185 0) (unit 1)
-    (in_bom yes) (on_board yes)
-    (property "Reference" "#PWR0104" (id 0) (at 75.565 86.995 0)
-      (effects (font (size 1.27 1.27)) hide)
-    )
-    (property "Value" "+5V" (id 1) (at 75.946 78.7908 0))
-    (property "Footprint" "" (id 2) (at 75.565 83.185 0)
-      (effects (font (size 1.27 1.27)) hide)
-    )
-    (property "Datasheet" "" (id 3) (at 75.565 83.185 0)
-      (effects (font (size 1.27 1.27)) hide)
-    )
-    (pin "1")
+  (symbol (lib_id "power:+5V") (at 74.295 83.185 0) (unit 1)
+    (in_bom yes) (on_board yes)
+    (property "Reference" "#PWR0104" (id 0) (at 74.295 86.995 0)
+      (effects (font (size 1.27 1.27)) hide)
+    )
+    (property "Value" "+5V" (id 1) (at 74.676 78.7908 0))
+    (property "Footprint" "" (id 2) (at 74.295 83.185 0)
+      (effects (font (size 1.27 1.27)) hide)
+    )
+    (property "Datasheet" "" (id 3) (at 74.295 83.185 0)
+      (effects (font (size 1.27 1.27)) hide)
+    )
+    (pin "1")
+  )
+  (symbol (lib_id "Device:C") (at 74.295 104.775 0) (unit 1)
+    (in_bom yes) (on_board yes)
+    (property "Reference" "C45" (id 0) (at 77.216 103.6066 0)
+      (effects (font (size 1.27 1.27)) (justify left))
+    )
+    (property "Value" "10uF" (id 1) (at 77.216 105.918 0)
+      (effects (font (size 1.27 1.27)) (justify left))
+    )
+    (property "Footprint" "Capacitor_SMD:C_0603_1608Metric" (id 2) (at 75.2602 108.585 0)
+      (effects (font (size 1.27 1.27)) hide)
+    )
+    (property "Datasheet" "~" (id 3) (at 74.295 104.775 0)
+      (effects (font (size 1.27 1.27)) hide)
+    )
+    (pin "1")
+    (pin "2")
   )
   (symbol (lib_id "power:PWR_FLAG") (at 55.88 128.27 180) (unit 1)
@@
     (pin "1")
   )
-  (symbol (lib_id "Device:C") (at 75.565 104.775 0) (unit 1)
-    (in_bom yes) (on_board yes)
-    (property "Reference" "C45" (id 0) (at 78.486 103.6066 0)
-      (effects (font (size 1.27 1.27)) (justify left))
-    )
-    (property "Value" "10uF" (id 1) (at 78.486 105.918 0)
-      (effects (font (size 1.27 1.27)) (justify left))
-    )
-    (property "Footprint" "Capacitor_SMD:C_0603_1608Metric" (id 2) (at 76.5302 108.585 0)
-      (effects (font (size 1.27 1.27)) hide)
-    )
-    (property "Datasheet" "~" (id 3) (at 75.565 104.775 0)
-      (effects (font (size 1.27 1.27)) hide)
-    )
-    (pin "1")
-    (pin "2")
-  )
   (symbol (lib_id "power:+5V") (at 52.705 83.82 0) (unit 1)
     (in_bom yes) (on_board yes)
@@
     (pin "1")
   )
-  (symbol (lib_id "power:GND") (at 75.565 128.27 0) (unit 1)
-    (in_bom yes) (on_board yes)
-    (property "Reference" "#PWR0105" (id 0) (at 75.565 134.62 0)
-      (effects (font (size 1.27 1.27)) hide)
-    )
-    (property "Value" "GND" (id 1) (at 75.692 132.6642 0))
-    (property "Footprint" "" (id 2) (at 75.565 128.27 0)
-      (effects (font (size 1.27 1.27)) hide)
-    )
-    (property "Datasheet" "" (id 3) (at 75.565 128.27 0)
-      (effects (font (size 1.27 1.27)) hide)
-    )
+  (symbol (lib_id "power:GND") (at 74.295 128.27 0) (unit 1)
+    (in_bom yes) (on_board yes)
+    (property "Reference" "#PWR0105" (id 0) (at 74.295 134.62 0)
+      (effects (font (size 1.27 1.27)) hide)
+    )
+    (property "Value" "GND" (id 1) (at 74.422 132.6642 0))
+    (property "Footprint" "" (id 2) (at 74.295 128.27 0)
+      (effects (font (size 1.27 1.27)) hide)
+    )
+    (property "Datasheet" "" (id 3) (at 74.295 128.27 0)
+      (effects (font (size 1.27 1.27)) hide)
+    )
