File: circuit/ProcessMCU.kicad_sch (KiCad schematic)
At the start: 26 parts, among them SW2 SW_DIP_x01, U5 MM32F3277G9P, Y1 8MHz

Commit message: Update circuit with control mcu.
Parts:
- removed C17, C18, C20, C21, C22, C23, C24, C26, C27, C28, C29, C30, C31, C32: 100nF, Capacitor_SMD:C_0603_1608Metric, symbol Device:C
- removed C19, C25: 18pF, Capacitor_SMD:C_0603_1608Metric, symbol Device:C
- removed D2, D3: LED, LED_SMD:LED_0603_1608Metric, symbol Device:LED
- removed R16, R19, R20: 10kR, Resistor_SMD:R_0603_1608Metric, symbol Device:R
- removed R17, R18: 1kR, Resistor_SMD:R_0603_1608Metric, symbol Device:R
- removed SW2: SW_DIP_x01, Button_Switch_SMD:SW_SPST_CK_RS282G05A3, symbol Switch:SW_DIP_x01
- removed U5: MM32F3277G9P, Package_QFP:LQFP-144_20x20mm_P0.5mm, symbol MM32_Periph:MM32F3277G9P
- removed Y1: 8MHz, Crystal:Crystal_SMD_3225-4Pin_3.2x2.5mm, symbol Device:Crystal_GND24
- added C? (x13): 100nF, Capacitor_SMD:C_0603_1608Metric, symbol Device:C
- added C? (x2): 18pF, Capacitor_SMD:C_0603_1608Metric, symbol Device:C
- added D?: LED, LED_SMD:LED_0603_1608Metric, symbol Device:LED
- added R? (x2): 10kR, Resistor_SMD:R_0603_1608Metric, symbol Device:R
- added R?: 1kR, Resistor_SMD:R_0603_1608Metric, symbol Device:R
- added U?: MM32F3277G9P, Package_QFP:LQFP-144_20x20mm_P0.5mm, symbol MM32_Periph:MM32F3277G9P
- added Y?: 8MHz, Crystal:Crystal_SMD_3225-4Pin_3.2x2.5mm, symbol Device:Crystal_GND24
Connections:
- net GND: now also C?.2, C?.2, C?.2, C?.2, C?.2, C?.2, C?.2, C?.2, C?.2, C?.2, C?.2, C?.2, C?.2, C?.2, C?.2, R?.1, U?.107 (VSS), U?.120 (VSS), U?.130 (VSS), U?.143 (VSS), U?.16 (VSS), U?.30 (VSSA), U?.31 (VREF-), U?.38 (VSS), U?.51 (VSS), U?.61 (VSS), U?.71 (VSS), U?.83 (VSS), U?.94 (VSS), Y?.2, Y?.4
- net LED1: now also D?.1 (K), U?.49 (PF11)
- net PB6: now also U?.136 (PB6)
- net PB7: now also U?.137 (PB7)
- net PB9: now also U?.140 (PB9)
- net PE0: now also U?.141 (PE0)
- net PE1: now also U?.142 (PE1)
- net PE3: now also U?.2 (PE3)
- net PE4: now also U?.3 (PE4)
- net PG15: now also U?.132 (PG15)
- net RST: now also C?.1, R?.2, U?.25 (nRST)
- net SPI1_CLK: now also U?.133 (PB3)
- net SPI1_MISO: now also U?.134 (PB4)
- net SPI1_MOSI: now also U?.135 (PB5)
- net SPI2_CLK: now also U?.1 (PE2)
- net SPI2_MOSI: now also U?.5 (PE6)
- net SWDCLK: now also U?.109 (PA14)
- net SWDIO: now also U?.105 (PA13)
- net UART1_RX: now also U?.102 (PA10)
- net UART1_TX: now also U?.101 (PA9)
- net UART3_RX: now also U?.78 (PD9)
- net UART3_TX: now also U?.77 (PD8)
- net UART6_RX: now also U?.47 (PB1)
- net UART6_TX: now also U?.46 (PB0)
- net XTAL_IN: now also C?.1, U?.23 (PH0), Y?.3
- net XTAL_OUT: now also C?.1, U?.24 (PH1), Y?.1
- new net: R?.2, U?.138 (PH3)
- new net: D?.2 (A), R?.2
- new net +3.3VA: C?.1, C?.1, C?.1, C?.1, C?.1, C?.1, C?.1, C?.1, C?.1, C?.1, C?.1, C?.1, R?.1, R?.1, U?.108 (VDD), U?.121 (VDD), U?.131 (VDD), U?.144 (VDD), U?.17 (VDD), U?.32 (VREF+), U?.33 (VDDA), U?.39 (VDD), U?.52 (VDD), U?.6 (VBAT), U?.62 (VDD), U?.72 (VDD), U?.84 (VDD), U?.95 (VDD)
- new net SPI3_CLK: U?.81 (PD12)
- new net SPI3_MISO: U?.82 (PD13)
- new net SPI3_MOSI: U?.85 (PD14)
- no-connect marks 84 -> 88
Other:
- note added: "LED"
- note removed: "LED & KEY"

Commit message: Basically finished schematic drawing and annotation, not yet package selection.
Parts:
- gave numbers to parts that had none: 21

Commit message: Basically finished all the design of the schematic and selected the package for the components.
Connections:
- net UART4_TX: now reaches U8.34 (PA0)
- net UART4_RX: now reaches U8.35 (PA1)
- no-connect marks 88 -> 86
Changed lines of the file:
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@@
   (title_block
     (title "MM32_Board")
-    (date "2022-01-11")
-    (rev "1.0.2")
+    (date "2022-01-16")
+    (rev "1.2.1")
   )
   (junction (at 217.17 133.985) (diameter 0) (color 0 0 0 0)
@@
   (no_connect (at 52.07 82.55))
   (no_connect (at 52.07 90.17))
-  (no_connect (at 52.07 140.97))
   (no_connect (at 161.29 140.97))
   (no_connect (at 161.29 105.41))
@@
   (no_connect (at 128.27 46.99))
   (no_connect (at 125.73 46.99))
-  (no_connect (at 52.07 138.43))
   (no_connect (at 52.07 74.93))
   (no_connect (at 52.07 123.19))
@@
     (stroke (width 0) (type default) (color 0 0 0 0))
   )
+  (wire (pts (xy 38.1 140.97) (xy 52.07 140.97))
+    (stroke (width 0) (type default) (color 0 0 0 0))
+  )
   (polyline (pts (xy 275.59 21.59) (xy 198.12 21.59))
     (stroke (width 0) (type default) (color 0 0 0 0))
@@
   )
   (wire (pts (xy 252.73 163.195) (xy 264.16 163.195))
+    (stroke (width 0) (type default) (color 0 0 0 0))
+  )
+  (wire (pts (xy 38.1 138.43) (xy 52.07 138.43))
     (stroke (width 0) (type default) (color 0 0 0 0))
   )
@@
     (effects (font (size 1.27 1.27)) (justify right))
   )
+  (hierarchical_label "UART4_RX" (shape input) (at 38.1 140.97 180)
+    (effects (font (size 1.27 1.27)) (justify right))
+  )
   (hierarchical_label "PB6" (shape output) (at 82.55 30.48 90)
     (effects (font (size 1.27 1.27)) (justify left))
@@
     (effects (font (size 1.27 1.27)) (justify left))
   )
+  (hierarchical_label "UART4_TX" (shape output) (at 38.1 138.43 180)
+    (effects (font (size 1.27 1.27)) (justify right))
+  )
   (hierarchical_label "SPI2_MOSI" (shape output) (at 36.83 64.77 180)

Commit message: Revised and finalized the final circuit schematic.
Connections:
- net +3.3VA: no longer R2.1
- net LED1: now also U8.37 (PA3); no longer U8.49 (PF11)
- net SPI3_CLK: now also U8.118 (PD4); no longer U8.81 (PD12)
- net SPI3_MISO: now also U8.119 (PD5); no longer U8.82 (PD13)
- net SPI3_MOSI: now also U8.122 (PD6); no longer U8.85 (PD14)
- net PF0: now reaches U8.10 (PF0)
- net SPI3_NSS: now reaches U8.123 (PD7)
- net PG9: now reaches U8.124 (PG9)
- net PG10: now reaches U8.125 (PG10)
- net IIC1_SCL: now reaches U8.79 (PD10)
- net IIC1_SDA: now reaches U8.80 (PD11)
- net PB6: no longer names the net of U8.136 (PB6)
- net PB7: no longer names the net of U8.137 (PB7)
- net PB9: no longer names the net of U8.140 (PB9)
- net PE3 renamed SPI2_NSS
- net PG15: no longer names the net of U8.132 (PG15)
- new net +3.3VP: R2.1
- new net PD12: U8.81 (PD12)
- no-connect marks 86 -> 83
