File: circuit/project.kicad_sch (KiCad schematic)
At the start: 0 parts

Commit message: Update circuit with control mcu.
Other:
- sheet Connector renamed Miscellaneous
- sheet MCU renamed Process_MCU
- added sheet Control_MCU (ControlMCU.kicad_sch)
- sheet IMU: file 3_IMU.kicad_sch -> IMU.kicad_sch
- sheet Miscellaneous: file 4_Connector.kicad_sch -> Miscellaneous.kicad_sch
- sheet Miscellaneous ports: added TOUCH_CLK, TOUCH_MISO, TOUCH_MOSI; removed LCD_MISO, MOTOR_RX, MOTOR_TX, Servo_PWM
- sheet Power: file 1_Power.kicad_sch -> Power.kicad_sch
- sheet Power ports: added MOTOR_RX, MOTOR_TX, PWR_RX, PWR_TX, Servo_PWM; removed PWR_DET, PWR_EN, VBAT
- sheet Process_MCU: file 2_MCU.kicad_sch -> ProcessMCU.kicad_sch
- sheet Process_MCU ports: added SPI3_CLK, SPI3_MISO, SPI3_MOSI; removed ADC23_IN14, PF13, PF14, SPI2_MISO, TIM1_CH1

Commit message: Update circuit and ADIS16470 footprint reference datasheet.
Other:
- sheet Miscellaneous renamed LCD&GPS
- added sheet Debugger (Debugger.kicad_sch)
- sheet LCD&GPS: file Miscellaneous.kicad_sch -> LCD&GPS.kicad_sch
- sheet LCD&GPS ports: added none; removed DEBUG_RX, DEBUG_TX, SWDCLK, SWDIO

Commit message: Basically finished schematic drawing and annotation, not yet package selection.
Other:
- sheet Control_MCU ports: added TIM2_CH1; removed none

Commit message: Basically finished all the design of the schematic and selected the package for the components.
Other:
- sheet Control_MCU ports: added UART3_RX, UART3_TX; removed none
- sheet Process_MCU ports: added UART4_RX, UART4_TX; removed none
Changed lines of the file:
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@@
   (title_block
     (title "MM32_Board")
-    (date "2022-01-11")
-    (rev "1.0.2")
+    (date "2022-01-16")
+    (rev "1.2.1")
+  )
+  (wire (pts (xy 101.6 97.155) (xy 141.605 97.155))
+    (stroke (width 0) (type default) (color 0 0 0 0))
   )
   (wire (pts (xy 187.325 99.06) (xy 197.485 99.06))
@@
   )
   (wire (pts (xy 101.6 79.375) (xy 113.665 79.375))
+    (stroke (width 0) (type default) (color 0 0 0 0))
+  )
+  (wire (pts (xy 101.6 94.615) (xy 141.605 94.615))
     (stroke (width 0) (type default) (color 0 0 0 0))
   )
@@
       (effects (font (size 1.27 1.27)) (justify right))
     )
+    (pin "UART4_TX" output (at 141.605 94.615 180)
+      (effects (font (size 1.27 1.27)) (justify left))
+    )
+    (pin "UART4_RX" input (at 141.605 97.155 180)
+      (effects (font (size 1.27 1.27)) (justify left))
+    )
   )
   (sheet (at 113.665 101.6) (size 16.51 25.4) (fields_autoplaced)
@@
     )
     (pin "TIM2_CH1" output (at 101.6 79.375 0)
+      (effects (font (size 1.27 1.27)) (justify right))
+    )
+    (pin "UART3_TX" output (at 101.6 97.155 0)
+      (effects (font (size 1.27 1.27)) (justify right))
+    )
+    (pin "UART3_RX" input (at 101.6 94.615 0)
       (effects (font (size 1.27 1.27)) (justify right))
     )
@@
     )
     (path "/00000000-0000-0000-0000-00006191448d/d31a625f-432d-4db7-81fa-5bdb5957e6bf"
-      (reference "C47") (unit 1) (value "0.1uF") (footprint "Capacitor_SMD:C_0603_1608Metric")
+      (reference "C47") (unit 1) (value "100nF") (footprint "Capacitor_SMD:C_0603_1608Metric")
     )
     (path "/00000000-0000-0000-0000-00006191448d/00000000-0000-0000-0000-0000619e4d63"
@@
     )
     (path "/b932d339-7888-4506-92dc-7b9f4a021ec5/f0f75b81-72fe-4a7f-8a1a-a9c6f0a003a6"
-      (reference "C68") (unit 1) (value "0.1uF") (footprint "Capacitor_SMD:C_0603_1608Metric")
+      (reference "C68") (unit 1) (value "100nF") (footprint "Capacitor_SMD:C_0603_1608Metric")
     )
     (path "/00000000-0000-0000-0000-00006194fb75/a012f378-e2e1-4b18-8c88-ccb430b11cee"
@@
     )
     (path "/00000000-0000-0000-0000-000061e2dd2b/25b39db8-8576-4473-b331-b912323e85f4"
-      (reference "J1") (unit 1) (value "ANT") (footprint "")
+      (reference "J1") (unit 1) (value "ANT") (footprint "Connector_Coaxial:SMA_Molex_73251-2200_Horizontal")
     )
     (path "/00000000-0000-0000-0000-00006191448d/1d417c7a-b772-4095-9f25-27b4cd8ff3f9"
-      (reference "J2") (unit 1) (value "Conn_01x08") (footprint "")
+      (reference "J2") (unit 1) (value "Conn_01x08") (footprint "Connector_JST:JST_PH_S8B-PH-K_1x08_P2.00mm_Horizontal")
     )
     (path "/00000000-0000-0000-0000-000061e2dd2b/2f8ebbbf-0f11-4a15-9648-1d28e5593127"
-      (reference "L1") (unit 1) (value "39nH") (footprint "")
+      (reference "L1") (unit 1) (value "39nH") (footprint "Inductor_SMD:L_0603_1608Metric")
     )
     (path "/00000000-0000-0000-0000-000061a493c9/00000000-0000-0000-0000-0000619da865"
@@
     )
     (path "/00000000-0000-0000-0000-000061e2dd2b/cad44c02-7fd2-4e9a-b93a-e1b73d6a3ee6"
-      (reference "LCD1") (unit 1) (value "1.8inch-TFT-LCD") (footprint "Display:TFT-LCD1.8inch")
+      (reference "LCD1") (unit 1) (value "1.8inch-TFT-LCD") (footprint "MM32_Library:TFT-LCD1.8inch")
     )
     (path "/b932d339-7888-4506-92dc-7b9f4a021ec5/00000000-0000-0000-0000-0000619f71de"
-      (reference "M1") (unit 1) (value "Debugger") (footprint "Connector:Gernic_Debugger")
+      (reference "M1") (unit 1) (value "Debugger") (footprint "MM32_Library:Gernic_Debugger")
     )
     (path "/00000000-0000-0000-0000-00006194fb75/0e701b31-0d3a-4461-babd-26744d455b3e"
@@
     )
     (path "/b932d339-7888-4506-92dc-7b9f4a021ec5/c1a18f74-a42c-4afc-acea-8274e502b185"
-      (reference "R7") (unit 1) (value "1kR") (footprint "Resistor_SMD:R_0603_1608Metric")
-    )
-    (path "/b932d339-7888-4506-92dc-7b9f4a021ec5/ecded0f9-a77b-4680-92eb-b2427606c506"
-      (reference "SW1") (unit 1) (value "SW_DIP_x01") (footprint "")
+      (reference "R7") (unit 1) (value "10kR") (footprint "Resistor_SMD:R_0603_1608Metric")
+    )
+    (path "/b932d339-7888-4506-92dc-7b9f4a021ec5/5be3d2d4-2465-422c-8da7-9722bb04468f"
+      (reference "SW1") (unit 1) (value "SW_DIP_x02") (footprint "Button_Switch_SMD:SW_DIP_SPSTx02_Slide_Copal_CHS-02B_W7.62mm_P1.27mm")
     )
     (path "/00000000-0000-0000-0000-000061e2dd2b/da151d0a-a1fa-4865-aa78-eb4b6082fbfd"
@@
     )
     (path "/00000000-0000-0000-0000-000061a493c9/00000000-0000-0000-0000-000061a49918"
-      (reference "U3") (unit 1) (value "ADIS16470AMLZ") (footprint "Sensor_Motion:ADIS16470AMLZ")
+      (reference "U3") (unit 1) (value "ADIS16470AMLZ") (footprint "MM32_Library:ADIS16470AMLZ")
     )
     (path "/00000000-0000-0000-0000-000061a493c9/00000000-0000-0000-0000-0000619c904b"
-      (reference "U4") (unit 1) (value "B0505S-1WR3") (footprint "Package_SIP:SIP-4_B0505S_1WR3")
+      (reference "U4") (unit 1) (value "B0505S-1WR3") (footprint "MM32_Library:SIP-4_B0505S_1WR3")
     )
     (path "/00000000-0000-0000-0000-000061a493c9/00000000-0000-0000-0000-000061a111e1"

Commit message: Revised and finalized the final circuit schematic.
Other:
- added sheet Compass&Storage (Compass&Storage.kicad_sch)
- sheet Control_MCU ports: added TIM3_CH1, UART7_RX, UART7_TX; removed TIM2_CH1, UART3_RX, UART3_TX
- sheet Process_MCU ports: added IIC1_SCL, IIC1_SDA, PD12, PF0, PG10, PG9, SPI2_NSS, SPI3_NSS; removed PB6, PB7, PB9, PE3, PG15
