File: circuit/wireless_debugger/ESP8266.kicad_pcb (KiCad board)
At the start: 2 copper layers, 40 x 20 mm, 39 parts, among them J1 Conn_02x04_Odd_Even, K1 SW_DIP_x01, K2 SW_DIP_x01, P1 USB_C_Plug_USB2.0, U1 W25Q64, U2 ESP8266EX, U3 HX9193, U4 CH330N, Y1 26MHz

Commit message: Modify the ESP8266 circuit and swap the SPI line sequence.
Connections:
- U1 pad 3: /SD_DATA2 -> /SD_DATA3
- U1 pad 7: /SD_DATA3 -> /SD_DATA2
Routing:
- net /SD_DATA3: track 12.6 -> 9.60 mm
- net /SD_DATA2: track 8.70 -> 11.5 mm
- net GND: vias 41 -> 51
Other:
- board text added: "2022/02/19"
- board text added: "Version 1.2.2"
- board text removed: "2022/02/09"
- board text removed: "Version 1.2.1"

Commit message: Change the ceramic antenna of wireless debugger to IPEX terminal and external antenna.
Parts:
- removed ANT1: Conn_01x02, RF_Antenna:Johanson_2450AT18x100
- added J2: Conn_01x03, ESP8266:IPEX 1G, F.Cu at (131.5, 97.6)
Routing:
- net GND: vias 51 -> 52
- net (no net): vias 1 -> 0
Other:
- board text added: "2022/03/10"
- board text added: "Version 1.2.3"
- board text added: "White"
- board text added: "电介质层 1"
- board text removed: "2022/02/19"
- board text removed: "Version 1.2.2"
