File: circuit/wireless_debugger/ESP8266.kicad_sch (KiCad schematic)
At the start: 39 parts, among them J1 Conn_02x04_Odd_Even, K1 SW_DIP_x01, K2 SW_DIP_x01, P1 USB_C_Plug_USB2.0, U1 W25Q64, U2 ESP8266EX, U3 HX9193, U4 CH330N, Y1 26MHz

Commit message: Change the ceramic antenna of wireless debugger to IPEX terminal and external antenna.
Parts:
- removed ANT1: Conn_01x02, RF_Antenna:Johanson_2450AT18x100, symbol Connector_Generic:Conn_01x02
- added J2: Conn_01x03, ESP8266:IPEX 1G, symbol Connector_Generic:Conn_01x03
Connections:
- net GND: now also J2.1 (Pin_1), J2.2 (Pin_2)
- net at C2.1, L1.1: now also J2.3 (Pin_3)
- no-connect marks 8 -> 7
Changed lines of the file:
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@@
   (title_block
     (title "ESP8266 Wireless DAP")
-    (date "2022-02-19")
-    (rev "Version 1.2.2")
+    (date "2022-03-10")
+    (rev "Version 1.2.3")
   )
   (junction (at 121.92 127.635) (diameter 0) (color 0 0 0 0)
@@
   (junction (at 125.73 55.88) (diameter 0) (color 0 0 0 0)
   )
+  (junction (at 33.02 98.425) (diameter 0) (color 0 0 0 0)
+  )
   (junction (at 77.47 100.33) (diameter 0) (color 0 0 0 0)
   )
@@
   (junction (at 109.22 142.24) (diameter 0) (color 0 0 0 0)
   )
-  (no_connect (at 33.02 95.885))
   (no_connect (at 238.76 149.225))
   (no_connect (at 99.06 125.73))
@@
     (stroke (width 0) (type default) (color 0 0 0 0))
   )
+  (wire (pts (xy 33.02 95.885) (xy 33.02 98.425))
+    (stroke (width 0) (type default) (color 0 0 0 0))
+  )
   (wire (pts (xy 205.74 162.56) (xy 208.28 162.56))
     (stroke (width 0) (type default) (color 0 0 0 0))
@@
   )
   (wire (pts (xy 104.14 53.975) (xy 101.6 53.975))
+    (stroke (width 0) (type default) (color 0 0 0 0))
+  )
+  (wire (pts (xy 33.02 98.425) (xy 33.02 107.95))
     (stroke (width 0) (type default) (color 0 0 0 0))
   )
@@
     (pin "1")
     (pin "2")
+  )
+  (symbol (lib_id "power:GND") (at 33.02 107.95 0) (unit 1)
+    (in_bom yes) (on_board yes)
+    (property "Reference" "#PWR04" (id 0) (at 33.02 114.3 0)
+      (effects (font (size 1.27 1.27)) hide)
+    )
+    (property "Value" "GND" (id 1) (at 33.02 111.76 0))
+    (property "Footprint" "" (id 2) (at 33.02 107.95 0)
+      (effects (font (size 1.27 1.27)) hide)
+    )
+    (property "Datasheet" "" (id 3) (at 33.02 107.95 0)
+      (effects (font (size 1.27 1.27)) hide)
+    )
+    (pin "1")
   )
   (symbol (lib_id "Device:C") (at 125.73 60.96 0) (unit 1)
@@
     )
     (pin "1")
+  )
+  (symbol (lib_id "Connector_Generic:Conn_01x03") (at 27.94 95.885 180) (unit 1)
+    (in_bom yes) (on_board yes)
+    (property "Reference" "J2" (id 0) (at 27.94 90.805 0))
+    (property "Value" "Conn_01x03" (id 1) (at 24.765 94.6151 0)
+      (effects (font (size 1.27 1.27)) (justify left) hide)
+    )
+    (property "Footprint" "ESP8266:IPEX 1G" (id 2) (at 27.94 95.885 0)
+      (effects (font (size 1.27 1.27)) hide)
+    )
+    (property "Datasheet" "~" (id 3) (at 27.94 95.885 0)
+      (effects (font (size 1.27 1.27)) hide)
+    )
+    (pin "1")
+    (pin "2")
+    (pin "3")
   )
   (symbol (lib_id "Device:R") (at 260.35 53.975 180) (unit 1)
@@
     (pin "2")
   )
-  (symbol (lib_id "Connector_Generic:Conn_01x02") (at 27.94 95.885 180) (unit 1)
-    (in_bom yes) (on_board yes)
-    (property "Reference" "ANT1" (id 0) (at 27.94 90.805 0))
-    (property "Value" "Conn_01x02" (id 1) (at 27.94 89.535 0)
-      (effects (font (size 1.27 1.27)) hide)
-    )
-    (property "Footprint" "RF_Antenna:Johanson_2450AT18x100" (id 2) (at 27.94 95.885 0)
-      (effects (font (size 1.27 1.27)) hide)
-    )
-    (property "Datasheet" "~" (id 3) (at 27.94 95.885 0)
-      (effects (font (size 1.27 1.27)) hide)
-    )
-    (pin "1")
-    (pin "2")
-  )
   (symbol (lib_id "power:+3.3V") (at 49.53 122.555 90) (unit 1)
     (in_bom yes) (on_board yes)
@@
       (reference "#PWR03") (unit 1) (value "GND") (footprint "")
     )
+    (path "/331d14c6-fab9-40b7-92ff-996d4fe14e95"
+      (reference "#PWR04") (unit 1) (value "GND") (footprint "")
+    )
     (path "/77fe20ea-7bba-42b5-a357-0ffdc2e402f0"
       (reference "#PWR05") (unit 1) (value "GND") (footprint "")
@@
       (reference "#PWR045") (unit 1) (value "+5V") (footprint "")
     )
-    (path "/807cdbf3-f7bf-4198-9154-360bb7c5dad3"
-      (reference "ANT1") (unit 1) (value "Conn_01x02") (footprint "RF_Antenna:Johanson_2450AT18x100")
-    )
     (path "/1b3ca2b7-8fee-45a4-95e6-06fd80318255"
       (reference "C1") (unit 1) (value "10uF") (footprint "Capacitor_SMD:C_0603_1608Metric")
@@
       (reference "J1") (unit 1) (value "Conn_02x04_Odd_Even") (footprint "Connector_PinHeader_1.27mm:PinHeader_2x04_P1.27mm_Vertical_SMD")
     )
+    (path "/66ab6bde-fb3a-4560-ab6b-bd9f8fb34cc8"
+      (reference "J2") (unit 1) (value "Conn_01x03") (footprint "ESP8266:IPEX 1G")
+    )
     (path "/ff38afa2-64ac-4bdb-b08d-1f66bbb39b07"

Commit message: Add the circuit design of serial port pass-through PC side.
Parts:
- C1, C10, C11, C12, C13, C14, C15, C16, C17, C2, C3, C4, C5, C6, C7, C8, C9: footprint Capacitor_SMD:C_0603_1608Metric -> ESP8266:C_0603_1608Metric
- D1: footprint LED_SMD:LED_0603_1608Metric -> ESP8266:LED_0603_1608Metric
- J1: footprint Connector_PinHeader_1.27mm:PinHeader_2x04_P1.27mm_Vertical_SMD -> ESP8266:PinHeader_2x04_P1.27mm_Vertical_SMD
- K1, K2: footprint Button_Switch_SMD:SW_Push_SPST_NO_Alps_SKRK -> ESP8266:SW_Push_SPST_NO_Alps_SKRK
- L1: footprint Inductor_SMD:L_0603_1608Metric -> ESP8266:L_0603_1608Metric
- P1: footprint Connector_USB:USB_C_Receptacle_HRO_TYPE-C-31-M-12 -> ESP8266:USB_C_Receptacle_HRO_TYPE-C-31-M-12
- R1, R10, R2, R3, R4, R5, R6, R7, R8, R9: footprint Resistor_SMD:R_0603_1608Metric -> ESP8266:R_0603_1608Metric
- U1: footprint Package_SO:SOIC-8_5.23x5.23mm_P1.27mm -> ESP8266:SOIC-8_5.23x5.23mm_P1.27mm
- U3: footprint Package_TO_SOT_SMD:SOT-23-5 -> ESP8266:SOT-23-5
- U4: footprint Package_SO:SOIC-8_3.9x4.9mm_P1.27mm -> ESP8266:SOIC-8_3.9x4.9mm_P1.27mm
- Y1: footprint Crystal:Crystal_SMD_3225-4Pin_3.2x2.5mm -> ESP8266:Crystal_SMD_3225-4Pin_3.2x2.5mm
