File: circuit/uart_tt_pc/project.kicad_pcb (KiCad board)
At the start: 2 copper layers, 36.5 x 25.9 mm, 13 parts, among them J1 Conn_02x03_Odd_Even, P1 USB_C_Plug_USB2.0, U1 E220-900T22S, U2 HX9193, U3 CH330N

Commit message: Adding level conversion circuitry to the serial port pass-through PC module
Parts:
- added U1: RS0101YH6, Package_TO_SOT_SMD:SOT-23-6, B.Cu at (151.9, 90.0)
- added U3: RS0101YH6, Package_TO_SOT_SMD:SOT-23-6, B.Cu at (149.1, 87.2)
- C1, C2, C3, C4: footprint Capacitor_SMD:C_0603_1608Metric -> TTLibrary:C_0603_1608Metric
- J1: footprint Connector_PinHeader_2.54mm:PinHeader_2x03_P2.54mm_Vertical -> TTLibrary:PinHeader_2x03_P2.54mm_Vertical
- R1, R2, R3, R4: footprint Resistor_SMD:R_0603_1608Metric -> TTLibrary:R_0603_1608Metric
- U4: renamed from U2; footprint Package_TO_SOT_SMD:SOT-23-5 -> TTLibrary:SOT-23-5
- U5: renamed from U3; footprint Package_SO:SOIC-8_3.9x4.9mm_P1.27mm -> TTLibrary:SOIC-8_3.9x4.9mm_P1.27mm
- renumbered U1 to U2
Connections:
- U2 pad 22: /U0_RXD -> /U_RXD
- U2 pad 23: /U0_TXD -> /U_TXD
Routing:
- net +5V: track 39.7 -> 55.3 mm
- net +3V3: track 28.1 -> 36.6 mm, vias 2 -> 3
- net /U_RXD: track 0.00 -> 5.34 mm, vias 0 -> 1
- net /U0_TXD: track 15.1 -> 10.6 mm, vias 0 -> 1
- net /U0_RXD: track 15.5 -> 12.2 mm, vias 0 -> 1
- net /U_TXD: track 0.00 -> 1.84 mm, vias 0 -> 1
- net GND: vias 21 -> 24
