File: circuit/uart_tt_pc/project.kicad_sch (KiCad schematic)
At the start: 13 parts, among them J1 Conn_02x03_Odd_Even, P1 USB_C_Plug_USB2.0, U1 E220-900T22S, U2 HX9193, U3 CH330N

Commit message: Adding level conversion circuitry to the serial port pass-through PC module
Parts:
- added U1, U3: RS0101YH6, TTLibrary:SOT-23-6, symbol TTLibrary:RS0101YH6
- renumbered U1 to U2, U2 to U4, U3 to U5
Connections:
- net +3V3: now also U1.1 (VCCA), U3.1 (VCCA)
- net +5V: now also U1.5 (OE), U1.6 (VCCB), U3.5 (OE), U3.6 (VCCB)
- net GND: now also U1.2 (GND), U3.2 (GND)
- net U0_RXD: now also U1.4 (B); no longer U2.22 (RXD)
- net U0_TXD: now also U3.4 (B); no longer U2.23 (TXD)
- new net U_RXD: U1.3 (A), U2.22 (RXD)
- new net U_TXD: U2.23 (TXD), U3.3 (A)
Other:
- moved on the sheet: J1, R1, R2, R3, R4, U2
