File: circuit/uart_tt_mcu/project.kicad_pcb (KiCad board)
At the start: 2 copper layers, 40 x 20 mm, 11 parts, among them J1 Conn_02x03_Odd_Even, J2 Conn_02x04_Odd_Even, U1 E220-900T22S, U2 HX9193

Commit message: Finished uart transparent transmit mcu side circuit design.
Parts:
- removed the J1 at (183.2, 118.1)
- added C4: 100nF, TTLibrary:C_0603_1608Metric, F.Cu at (165.6, 91.0)
- added P1: USB_C_Plug_USB2.0, TTLibrary:USB_C_Receptacle_HRO_TYPE-C-31-M-12, F.Cu at (171.7, 96.1)
- added U3: RS0101YH6, TTLibrary:SOT-23-6, B.Cu at (159.3, 90.0)
- added U4: HX9193, TTLibrary:SOT-23-5, F.Cu at (164.0, 101.4)
- added U5: CH330N, TTLibrary:SOIC-8_3.9x4.9mm_P1.27mm, F.Cu at (167.9, 87.3)
- C2, C3: moved to B.Cu
- U2: value HX9193 -> RS0101YH6; footprint TTLibrary:SOT-23-5 -> TTLibrary:SOT-23-6; moved to B.Cu
- moved R1 46.1 mm to (141.3, 84.8)
- moved R2 45.2 mm to (138.2, 84.8), turned to 0 degrees
- moved R3 42.7 mm to (144.5, 84.8), turned to 0 degrees
- moved R4 35.5 mm to (147.7, 84.8)
- moved U2 32.8 mm to (159.3, 86.3), turned to 0 degrees
- moved C2 29.2 mm to (138.4, 88.3)
- moved C3 28.6 mm to (138.4, 86.7)
- moved C1 20.1 mm to (164.0, 98.4), turned to 0 degrees
- moved U1 4.83 mm to (135.8, 102.7)
- renumbered J2 to J1
Connections:
- R1 pad 2: Net-(J1-Pad1) -> Net-(U1-Pad21)
- R2 pad 2: Net-(J1-Pad5) -> Net-(U1-Pad21)
- R3 pad 2: Net-(J1-Pad2) -> Net-(U1-Pad20)
- R4 pad 2: Net-(J1-Pad6) -> Net-(U1-Pad20)
- U1 pad 20: /M0 -> Net-(U1-Pad20)
- U1 pad 21: /M1 -> Net-(U1-Pad21)
- U2 pad 1: +5V -> +3V3
- U2 pad 3: +5V -> /U_RXD
- U2 pad 4: unconnected-(U2-Pad4) -> /U0_RXD
- U2 pad 5: +3V3 -> +5V
Routing:
- net +5V: track 0.00 -> 58.1 mm, vias 0 -> 2
- net +3V3: track 0.00 -> 51.2 mm, vias 0 -> 6
- net /U_RXD: track 0.00 -> 26.2 mm, vias 0 -> 2
- net /U_TXD: track 0.00 -> 25.5 mm, vias 0 -> 1
- net /USB_DM: track 0.00 -> 14.9 mm
- net /USB_DP: track 0.00 -> 11.5 mm
- net Net-(U1-Pad21): track 0.00 -> 6.39 mm, vias 0 -> 2
- net /U0_RXD: track 0.00 -> 5.53 mm, vias 0 -> 1
- net /U0_TXD: track 0.00 -> 5.49 mm, vias 0 -> 1
- net Net-(U1-Pad20): track 0.00 -> 3.48 mm
- net Net-(C4-Pad1): track 0.00 -> 2.04 mm
- net GND: vias 1 -> 16
- added copper zone on B.Cu, net GND
- added copper zone on F.Cu, net GND
Other:
- board text added: "0"
- board text added: "0 mm"
- board text added: "0.01 mm"
- board text added: "0.02"
- board text added: "0.035 mm"
- board text added: "0.2000 mm / 0.2000 mm"
- board text added: "0.3000 mm"
- board text added: "1"
- board text added: "1.51 mm"
- board text added: "1.6000 mm"
- board text added: "2"
- board text added: "3.3"
- board text added: "4.5"
- board text added: "40.0804 mm x 20.0652 mm"
- board text added: "B.Cu"
- board text added: "B.Mask"
- board text added: "B.Paste"
- board text added: "B.Silkscreen"
- board text added: "BOARD CHARACTERISTICS"
- board text added: "Bottom Silk Screen"
- board text added: "Bottom Solder Mask"
- board text added: "Bottom Solder Paste"
- board text added: "Epsilon R（相对介电常数）"
- board text added: "F.Cu"
- board text added: "F.Mask"
- board text added: "F.Paste"
- board text added: "F.Silkscreen"
- board text added: "FR4"
- board text added: "GDUT 2022/03/18"
- board text added: "JLCJLCJLCJLC"
- board text added: "Jesus Team"
- board text added: "Loss Tangent（损耗切线）"
- board text added: "None"
- board text added: "Not specified"
- board text added: "R1 R3 PULLUP"
- board text added: "R2 R4 PULLDOWN"
- board text added: "Top Silk Screen"
- board text added: "Top Solder Mask"
- board text added: "Top Solder Paste"
- board text added: "UART TT MCU"
- board text added: "Version 1.0.1"
- board text added: "copper"
- board text added: "core"
- board text added: "否"
- board text added: "孔最小直径："
- board text added: "层名称"
- board text added: "最小布线/间距："
- board text added: "材料"
- board text added: "板子整体尺寸："
- board text added: "电介质层 1"
- board text added: "电路板厚度："
- board text added: "电镀板边："
- board text added: "类型"
- board text added: "粗细 (mm)"
- board text added: "边缘卡连接器："
- board text added: "邮票孔："
- board text added: "铜层数量："
- board text added: "铜表面处理（镀铜）："
- board text added: "阻抗控制"
- board text added: "颜色"
