File: circuit/uart_tt_mcu/project.kicad_sch (KiCad schematic)
At the start: 11 parts, among them J1 Conn_02x03_Odd_Even, J2 Conn_02x04_Odd_Even, U1 E220-900T22S, U2 HX9193

Commit message: Finished uart transparent transmit mcu side circuit design.
Parts:
- removed J1: Conn_02x03_Odd_Even, TTLibrary:PinHeader_2x03_P2.54mm_Vertical, symbol Connector_Generic:Conn_02x03_Odd_Even
- removed U2: HX9193, TTLibrary:SOT-23-5, symbol ESP8266:HX9193
- added C4: 100nF, TTLibrary:C_0603_1608Metric, symbol Device:C
- added P1: USB_C_Plug_USB2.0, TTLibrary:USB_C_Receptacle_HRO_TYPE-C-31-M-12, symbol Connector:USB_C_Plug_USB2.0
- added U2, U3: RS0101YH6, TTLibrary:SOT-23-6, symbol TTLibrary:RS0101YH6
- added U4: HX9193, TTLibrary:SOT-23-5, symbol ESP8266:HX9193
- added U5: CH330N, TTLibrary:SOIC-8_3.9x4.9mm_P1.27mm, symbol Interface_USB:CH330N
- renumbered J2 to J1
Connections:
- net M0 is gone; now on an unnamed net: U1.20 (M0)
- net M1 is gone; now on an unnamed net: U1.21 (M1)
- net +3V3: now also U2.1 (VCCA), U3.1 (VCCA), U4.5 (VOUT)
- net +5V: now also P1.A4 (VBUS), P1.A9 (VBUS), P1.B4 (VBUS), P1.B9 (VBUS), U2.5 (OE), U2.6 (VCCB), U3.5 (OE), U3.6 (VCCB), U4.1 (VIN), U4.3 (EN), U5.5 (VCC)
- net GND: now also C4.2, P1.A1 (GND), P1.A12 (GND), P1.B1 (GND), P1.B12 (GND), U2.2 (GND), U3.2 (GND), U4.2 (GND), U5.3 (GND)
- net U_RXD: now also U2.3 (A)
- net U_TXD: now also U3.3 (A)
- net at R3.2: now also R4.2
- net at R1.2: now also R2.2
- new net: C4.1, U5.8 (V3)
- new net U0_RXD: U2.4 (B), U5.6 (TXD)
- new net U0_TXD: U3.4 (B), U5.7 (RXD)
- new net USB_DM: P1.A7 (D-), P1.B7 (D-), U5.2 (UD-)
- new net USB_DP: P1.A6 (D+), P1.B6 (D+), U5.1 (UD+)
- no-connect marks 4 -> 5
Other:
- note added: "USB TO TTL"
- note removed: "Connector"
- moved on the sheet: J1
