File: circuit/bldc_driver/Driver.kicad_sch (KiCad schematic)
At the start: 21 parts

Commit message: Update BLDC 6-Step Driver schematic, Version 1.0.1
Parts:
- added J3: MR30, Connector_AMASS:AMASS_MR30PW-FB_1x03_P3.50mm_Horizontal, symbol Library:MR30
- R30, R31, R32, R33, R35, R36, R37, R41, R42, R43, R44: renamed from R?; footprint (none) -> Resistor_SMD:R_0805_2012Metric
- R34, R39, R40: renamed from R?; footprint (none) -> Resistor_SMD:R_2512_6332Metric
- R38: renamed from R?; footprint (none) -> Resistor_SMD:R_0603_1608Metric
- gave numbers to parts that had none: 6
Connections:
- net VS1: now also J3.1 (Pin_1)
- net VS2: now also J3.2 (Pin_2)
- net VS3: now also J3.3 (Pin_3)

Commit message: Modify the scheme of brushless motor driver board to reduce the use of resistors and capacitors to reduce the size of the circuit.
Parts:
- J4: renamed from J3; footprint Connector_AMASS:AMASS_MR30PW-FB_1x03_P3.50mm_Horizontal -> BLDC_Driver:MR30_Vertical
- R21: renamed from R30; footprint Resistor_SMD:R_0805_2012Metric -> Resistor_SMD:R_0603_1608Metric
- R22: renamed from R31; footprint Resistor_SMD:R_0805_2012Metric -> Resistor_SMD:R_0603_1608Metric
- R23: renamed from R32; footprint Resistor_SMD:R_0805_2012Metric -> Resistor_SMD:R_0603_1608Metric
- R24: renamed from R33; footprint Resistor_SMD:R_0805_2012Metric -> Resistor_SMD:R_0603_1608Metric
- R25: renamed from R34; footprint Resistor_SMD:R_2512_6332Metric -> Resistor_SMD:R_1206_3216Metric
- R26: renamed from R35; footprint Resistor_SMD:R_0805_2012Metric -> Resistor_SMD:R_0603_1608Metric
- R27: renamed from R36; footprint Resistor_SMD:R_0805_2012Metric -> Resistor_SMD:R_0603_1608Metric
- R28: renamed from R37; footprint Resistor_SMD:R_0805_2012Metric -> Resistor_SMD:R_0603_1608Metric
- R30: renamed from R39; footprint Resistor_SMD:R_2512_6332Metric -> Resistor_SMD:R_1206_3216Metric
- R31: renamed from R40; footprint Resistor_SMD:R_2512_6332Metric -> Resistor_SMD:R_1206_3216Metric
- R32: renamed from R41; footprint Resistor_SMD:R_0805_2012Metric -> Resistor_SMD:R_0603_1608Metric
- R33: renamed from R42; footprint Resistor_SMD:R_0805_2012Metric -> Resistor_SMD:R_0603_1608Metric
- R34: renamed from R43; footprint Resistor_SMD:R_0805_2012Metric -> Resistor_SMD:R_0603_1608Metric
- R35: renamed from R44; footprint Resistor_SMD:R_0805_2012Metric -> Resistor_SMD:R_0603_1608Metric
- renumbered R38 to R29
Other:
- note added: "MOSFET"
- moved on the sheet: J4, Q1, Q2, Q3, Q4, Q5, Q6, R21, R22, R23, R24, R25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

Commit message: Some components in the six-step commutation brushless drive were modified to achieve a smaller size.
Connections:
- net HO1: now also R32.1; no longer R21.1
- net HO3: now also R21.1; no longer R32.1
- net IA: now also Q6.1 (S), Q6.2 (S), Q6.3 (S); no longer Q2.1 (S), Q2.2 (S), Q2.3 (S)
- net ISUM: now also Q2.1 (S), Q2.2 (S), Q2.3 (S); no longer Q6.1 (S), Q6.2 (S), Q6.3 (S)
- net LO1: now also R33.1; no longer R22.1
- net LO3: now also R22.1; no longer R33.1
- net VS1: now also J4.3 (Pin_3), Q5.1 (S), Q5.2 (S), Q5.3 (S), Q6.5 (D), R34.1; no longer J4.1 (Pin_1), Q1.1 (S), Q1.2 (S), Q1.3 (S), Q2.5 (D), R23.1
- net VS3: now also J4.1 (Pin_1), Q1.1 (S), Q1.2 (S), Q1.3 (S), Q2.5 (D), R23.1; no longer J4.3 (Pin_3), Q5.1 (S), Q5.2 (S), Q5.3 (S), Q6.5 (D), R34.1
Other:
- moved on the sheet: R25

Commit message: Update the schematic and package library of BLDC Driver.
Parts:
- Q1, Q2, Q3, Q4, Q5, Q6: footprint Package_TO_SOT_SMD:TDSON-8-1 -> BLDC_Driver:TDSON-8-1
- R21, R22, R23, R24, R26, R27, R28, R29, R32, R33, R34, R35: footprint Resistor_SMD:R_0603_1608Metric -> BLDC_Driver:R_0603_1608Metric
- R25, R30, R31: footprint Resistor_SMD:R_1206_3216Metric -> BLDC_Driver:R_1206_3216Metric
Connections:
- net GND: now also R35.1
- net ISUM: no longer R35.1

Commit message: Modified the BLDC driver circuit by deleting the crystal and adding decoupling capacitors. Replaced the buck chip with JW5017s chip for power supply.
Parts:
- R21, R22, R26, R27, R32, R33: value 100R -> 33R
Changed lines of the file:
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@@
   (title_block
     (title "BLDC Driver 6-Step")
-    (date "2022-03-26")
-    (rev "1.1.2")
+    (date "2022-04-07")
+    (rev "1.2.4")
   )
   (junction (at 93.98 132.08) (diameter 0) (color 0 0 0 0)
@@
     (in_bom yes) (on_board yes)
     (property "Reference" "R22" (id 0) (at 70.485 111.76 90))
-    (property "Value" "100R" (id 1) (at 71.755 116.84 90))
+    (property "Value" "33R" (id 1) (at 71.755 116.84 90))
     (property "Footprint" "BLDC_Driver:R_0603_1608Metric" (id 2) (at 71.755 116.078 90)
       (effects (font (size 1.27 1.27)) hide)
@@
     (in_bom yes) (on_board yes)
     (property "Reference" "R32" (id 0) (at 203.835 79.375 90))
-    (property "Value" "100R" (id 1) (at 205.105 84.455 90))
+    (property "Value" "33R" (id 1) (at 205.105 84.455 90))
     (property "Footprint" "BLDC_Driver:R_0603_1608Metric" (id 2) (at 205.105 83.693 90)
       (effects (font (size 1.27 1.27)) hide)
@@
     (in_bom yes) (on_board yes)
     (property "Reference" "R33" (id 0) (at 203.835 111.76 90))
-    (property "Value" "100R" (id 1) (at 205.105 116.84 90))
+    (property "Value" "33R" (id 1) (at 205.105 116.84 90))
     (property "Footprint" "BLDC_Driver:R_0603_1608Metric" (id 2) (at 205.105 116.078 90)
       (effects (font (size 1.27 1.27)) hide)
@@
     (in_bom yes) (on_board yes)
     (property "Reference" "R26" (id 0) (at 137.795 79.375 90))
-    (property "Value" "100R" (id 1) (at 139.065 84.455 90))
+    (property "Value" "33R" (id 1) (at 139.065 84.455 90))
     (property "Footprint" "BLDC_Driver:R_0603_1608Metric" (id 2) (at 139.065 83.693 90)
       (effects (font (size 1.27 1.27)) hide)
@@
     (in_bom yes) (on_board yes)
     (property "Reference" "R21" (id 0) (at 70.485 79.375 90))
-    (property "Value" "100R" (id 1) (at 71.755 84.455 90))
+    (property "Value" "33R" (id 1) (at 71.755 84.455 90))
     (property "Footprint" "BLDC_Driver:R_0603_1608Metric" (id 2) (at 71.755 83.693 90)
       (effects (font (size 1.27 1.27)) hide)
@@
     (in_bom yes) (on_board yes)
     (property "Reference" "R27" (id 0) (at 137.795 111.76 90))
-    (property "Value" "100R" (id 1) (at 139.065 116.84 90))
+    (property "Value" "33R" (id 1) (at 139.065 116.84 90))
     (property "Footprint" "BLDC_Driver:R_0603_1608Metric" (id 2) (at 139.065 116.078 90)
       (effects (font (size 1.27 1.27)) hide)
