File: circuit/bldc_driver/controller.kicad_sch (KiCad schematic)
At the start: 6 parts

Commit message: Add BLDC driver circuit.
Parts:
- added C? (x3): 10uF, ControlBoard:C_0603_1608Metric, symbol Device:C
- added R? (x3): 10kR, symbol Device:R
- added R?: 1kR, symbol Device:R
Connections:
- net GND: now also U?.1 (GND), U?.24 (GND), U?.49 (GND), R?.2
- net RST: now also U?.8 (~{RST})
- net XTAL_IN: now also U?.6 (OSC_IN)
- net XTAL_OUT: now also U?.7 (OSC_OUT)
- net at U?.14 (PA4/OP1_INP): now also R?.1
- net at U?.15 (PA5/OP1_INM): now also R?.1
- net +9V: now reaches U?.2 (VCC)
- net +5V: now reaches U?.23 (VDDIO)
- net +5V: now also U?.3 (VDDIO), U?.9 (VDDA), R?.1
- net SWDIO: now reaches U?.33 (PA13/SWDIO)
- net SWDCLK: now reaches U?.36 (PA14/SWDCLK)
- net LO3: now reaches U?.37 (LO3)
- net VS3: now reaches U?.38 (VS3)
- net VS3: now also C?.2
- net HO3: now reaches U?.39 (HO3)
- net at U?.40 (VB3): now also C?.1
- net LO2: now reaches U?.41 (LO2)
- net VS2: now reaches U?.42 (VS2)
- net VS2: now also C?.2
- net HO2: now reaches U?.43 (HO2)
- net at U?.44 (VB2): now also C?.1
- net LO1: now reaches U?.45 (LO1)
- net VS1: now reaches U?.46 (VS1)
- net VS1: now also C?.2
- net HO1: now reaches U?.47 (HO1)
- net at U?.48 (VB1): now also C?.1
- net +3.3VA renamed +3V3
- new net: R?.1, R?.2
- new net ISUN: R?.2
Other:
- title: (none) -> BLDC Driver 6-Step

Commit message: Update BLDC 6-Step Driver schematic, Version 1.0.1
Parts:
- removed R? (x3): 10kR, symbol Device:R
- removed R?: 1kR, symbol Device:R
- added C1: 1uF, Capacitor_SMD:C_0201_0603Metric, symbol Device:C
- added C8: 100nF, Capacitor_SMD:C_0603_1608Metric, symbol Device:C
- added D1, D2, D3, D4: LED, LED_SMD:LED_0603_1608Metric, symbol Device:LED
- added M1: Debugger, BLDC_Driver:Gernic_Debugger, symbol MM32_Periph:Debugger
- added R1, R19, R20, R21, R23: 10KR, Resistor_SMD:R_0603_1608Metric, symbol Device:R
- added R10, R9: 1kR, Resistor_SMD:R_0603_1608Metric, symbol Device:R
- added R11, R12, R15, R16: 100KR, Resistor_SMD:R_0603_1608Metric, symbol Device:R
- added R13, R14, R5, R6: 10kR, Resistor_SMD:R_0603_1608Metric, symbol Device:R
- added R17: 47kR, Resistor_SMD:R_0603_1608Metric, symbol Device:R
- added R18: 20KR, Resistor_SMD:R_0603_1608Metric, symbol Device:R
- added R2: 100R, Resistor_SMD:R_0603_1608Metric, symbol Device:R
- added R22: 40KR, Resistor_SMD:R_0603_1608Metric, symbol Device:R
- added R3, R4, R7, R8: 1KR, Resistor_SMD:R_0603_1608Metric, symbol Device:R
- C2, C3, C4: renamed from C?; footprint ControlBoard:C_0603_1608Metric -> Capacitor_SMD:C_1206_3216Metric
- C5, C6, C7: renamed from C?; footprint ControlBoard:C_0603_1608Metric -> Capacitor_SMD:C_0603_1608Metric
- R24: renamed from R?; footprint ControlBoard:R_0603_1608Metric -> Resistor_SMD:R_0603_1608Metric
- Y1: renamed from Y?; footprint ControlBoard:Crystal_SMD_3225-4Pin_3.2x2.5mm -> Crystal:Crystal_SMD_3225-4Pin_3.2x2.5mm
- gave numbers to parts that had none: 1
Connections:
- net +5V: now also M1.1 (5V), M1.8 (5V), R18.1, R19.1, R20.1, R21.1, R5.1, R6.1
- net GND: now also C1.2, C8.2, D4.1 (K), M1.4 (GND), M1.5 (GND), R13.2, R14.2, R23.2, R9.1
- net IA: now also R7.2
- net IB: now also R8.2
- net SWDCLK: now also M1.3 (SWDCLK)
- net SWDIO: now also M1.2 (SWDIO)
- net PA0: now reaches U1.10 (PA0)
- net PA1: now reaches U1.11 (PA1)
- net PA2: now reaches U1.12 (PA2)
- net at U1.13 (PA3): now also C1.1, R1.2
- net PA4: now reaches U1.14 (PA4/OP1_INP)
- net PA4: now also R10.1
- net PA5: now reaches U1.15 (PA5/OP1_INM)
- net PA5: now also R17.2, R9.2
- net PA6: now reaches U1.16 (PA6/OP1_OUT)
- net PA6: now also R1.1, R17.1
- net PA7: now reaches U1.17 (PA7)
- net PB0: now reaches U1.18 (PB0/OP2_INP)
- net PB0: now also R11.1, R7.1
- net PB1: now reaches U1.19 (PB1/OP2_INM)
- net PB1: now also R15.2, R3.1
- net PB2: now reaches U1.20 (PB2/OP2_OUT)
- net PB2: now also R15.1
- net PB10: now reaches U1.21 (PB10/OP3_OUT)
- net PB10: now also R16.1
- net PB11: now reaches U1.22 (PB11/OP3_INM)
- net PB11: now also R16.2, R4.1
- net PB12: now reaches U1.25 (PB12/OP3_INP)
- net PB13: now reaches U1.26 (PB13)
- net PB13: now also D1.1 (K)
- net PB15: now reaches U1.28 (PB15)
- net PB15: now also C8.1, R22.2, R23.1
- net M_RX: now reaches U1.29 (PA9)
- net M_RX: now also M1.6 (U_TX)
- net M_TX: now reaches U1.30 (PA10)
- net M_TX: now also M1.7 (U_RX)
- net at U1.35 (PD3/CMP4_INP): now also R2.1
- net PC14: now reaches U1.4 (PC14)
- net PC14: now also D3.1 (K)
- net PC15: now reaches U1.5 (PC15)
- net PC15: now also D2.1 (K)
- new net: D3.2 (A), R20.2
- new net: R11.2, R13.1, R5.2
- new net: R12.2, R14.1, R6.2
- new net: D1.2 (A), R18.2
- new net: D2.2 (A), R19.2
- new net: D4.2 (A), R21.2
- new net +15V: R22.1
- new net ISUM: R10.2, R3.2, R4.2
- new net P12: R12.1, R8.1
- new net PA3: R2.2
Other:
- moved on the sheet: C2, C3, C4, U1

Commit message: Modify the scheme of brushless motor driver board to reduce the use of resistors and capacitors to reduce the size of the circuit.
Parts:
- removed D2, D3: LED, LED_SMD:LED_0603_1608Metric, symbol Device:LED
- removed M1: Debugger, BLDC_Driver:Gernic_Debugger, symbol MM32_Periph:Debugger
- removed R13, R14, R5, R6: 10kR, Resistor_SMD:R_0603_1608Metric, symbol Device:R
- removed R19, R20: 10KR, Resistor_SMD:R_0603_1608Metric, symbol Device:R
- removed R2: 100R, Resistor_SMD:R_0603_1608Metric, symbol Device:R
- added J1: Conn_01x04, Connector_PinSocket_2.54mm:PinSocket_1x04_P2.54mm_Vertical, symbol Connector_Generic:Conn_01x04
- added U2: REF3025, Package_TO_SOT_SMD:SOT-23, symbol Reference_Voltage:REF3025
- C2, C3, C4: footprint Capacitor_SMD:C_1206_3216Metric -> Capacitor_SMD:C_0603_1608Metric
- R13: renamed from R18; value 20KR -> 2kR
- R14: renamed from R21; value 10KR -> 2kR
- renumbered D4 to D2, R15 to R10, R16 to R11, R17 to R12, R22 to R15, R23 to R16, R24 to R17, R3 to R2, R4 to R3, R7 to R4, R8 to R5, R9 to R6, R10 to R7, R11 to R8, R12 to R9
Connections:
- net +3V3 is gone; now on net +5V: R17.1
- net +5V: now also J1.1 (Pin_1), U2.1 (VCC)
- net GND: now also J1.4 (Pin_4), U2.3 (GND)
- net PA3: now also C1.1, R1.2, U1.13 (PA3), U1.35 (PD3/CMP4_INP)
- net SWDCLK: now also J1.2 (Pin_2)
- net SWDIO: now also J1.3 (Pin_3)
- net +2V5: now reaches R8.2
- net +2V5: now also R9.2, U2.2 (OUT)
- net M_RX renamed UART1_TX
- net M_TX renamed UART1_RX
- no-connect marks 0 -> 4
Other:
- note added: "Current Sample"
- note added: "Debug Port"
- note added: "LED"
- note added: "Microcontroller"
- moved on the sheet: C1, C2, C3, C4, C8, D1, D2, R1, R10, R11, R12, R13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

Commit message: Some components in the six-step commutation brushless drive were modified to achieve a smaller size.
Parts:
- C1: footprint Capacitor_SMD:C_0201_0603Metric -> Capacitor_SMD:C_0603_1608Metric
Connections:
- net P12 is gone; now on net PB12: R5.1, R9.1
- net PC14: no longer names the net of U1.4 (PC14)
- net PC15: no longer names the net of U1.5 (PC15)
- no-connect marks 4 -> 6
Changed lines of the file:
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@@
   (no_connect (at 53.34 136.525))
   (no_connect (at 53.34 133.985))
+  (no_connect (at 53.34 103.505))
+  (no_connect (at 53.34 100.965))
   (wire (pts (xy 258.445 112.395) (xy 258.445 109.855))
     (stroke (width 0) (type default) (color 0 0 0 0))
@@
     (stroke (width 0) (type default) (color 0 0 0 0))
   )
-  (wire (pts (xy 25.4 103.505) (xy 53.34 103.505))
-    (stroke (width 0) (type default) (color 0 0 0 0))
-  )
   (wire (pts (xy 207.645 85.725) (xy 207.645 102.235))
     (stroke (width 0) (type default) (color 0 0 0 0))
@@
     (stroke (width 0) (type default) (color 0 0 0 0))
   )
-  (wire (pts (xy 25.4 100.965) (xy 53.34 100.965))
-    (stroke (width 0) (type default) (color 0 0 0 0))
-  )
   (wire (pts (xy 207.645 102.235) (xy 210.185 102.235))
     (stroke (width 0) (type default) (color 0 0 0 0))
@@
     (effects (font (size 1.27 1.27)) (justify left bottom))
   )
-  (label "PC15" (at 25.4 103.505 0)
-    (effects (font (size 1.27 1.27)) (justify left bottom))
-  )
   (label "PA6" (at 194.31 68.58 180)
     (effects (font (size 1.27 1.27)) (justify right bottom))
@@
     (effects (font (size 1.27 1.27)) (justify left bottom))
   )
-  (label "P12" (at 175.26 140.97 180)
+  (label "PB12" (at 175.26 140.97 180)
     (effects (font (size 1.27 1.27)) (justify right bottom))
   )
@@
     (effects (font (size 1.27 1.27)) (justify left bottom))
   )
-  (label "PC14" (at 25.4 100.965 0)
-    (effects (font (size 1.27 1.27)) (justify left bottom))
-  )
   (label "PA3" (at 124.46 116.205 180)
     (effects (font (size 1.27 1.27)) (justify right bottom))
@@
       (effects (font (size 1.27 1.27)) (justify left))
     )
-    (property "Footprint" "Capacitor_SMD:C_0201_0603Metric" (id 2) (at 42.8752 145.415 0)
+    (property "Footprint" "Capacitor_SMD:C_0603_1608Metric" (id 2) (at 42.8752 145.415 0)
       (effects (font (size 1.27 1.27)) hide)
     )

Commit message: Update the schematic and package library of BLDC Driver.
Parts:
- C1, C2, C3, C4, C5, C6, C7, C8: footprint Capacitor_SMD:C_0603_1608Metric -> BLDC_Driver:C_0603_1608Metric
- D1, D2: footprint LED_SMD:LED_0603_1608Metric -> BLDC_Driver:LED_0603_1608Metric
- J1: footprint Connector_PinSocket_2.54mm:PinSocket_1x04_P2.54mm_Vertical -> BLDC_Driver:PinSocket_1x04_P2.54mm_Vertical
- R1, R10, R11, R12, R13, R14, R15, R16, R17, R2, R3, R4, R5, R6, R7, R8, R9: footprint Resistor_SMD:R_0603_1608Metric -> BLDC_Driver:R_0603_1608Metric
- U1: footprint Package_QFP:TQFP-48-1EP_7x7mm_P0.5mm_EP5x5mm -> BLDC_Driver:QFN-48-1EP_6x6mm_P0.4mm_EP4.2x4.2mm
- U2: footprint Package_TO_SOT_SMD:SOT-23 -> BLDC_Driver:SOT-23
- Y1: footprint Crystal:Crystal_SMD_3225-4Pin_3.2x2.5mm -> BLDC_Driver:Crystal_SMD_3225-4Pin_3.2x2.5mm

Commit message: Modified the BLDC driver circuit by deleting the crystal and adding decoupling capacitors. Replaced the buck chip with JW5017s chip for power supply.
Parts:
- removed C5, C6: 18pF, BLDC_Driver:C_0603_1608Metric, symbol Device:C
- removed Y1: 8MHz, BLDC_Driver:Crystal_SMD_3225-4Pin_3.2x2.5mm, symbol Device:Crystal_GND24
- R1, R16: value 10KR -> 10kR
- R10, R11, R8, R9: value 100KR -> 100kR
- R15: value 40KR -> 40kR
- R2, R3, R4, R5: value 1KR -> 1kR
Connections:
- net +9V renamed +12V
- net XTAL_IN: no longer names the net of U1.6 (OSC_IN)
- net XTAL_OUT: no longer names the net of U1.7 (OSC_OUT)
- no-connect marks 6 -> 8
Other:
- note added: "RST"
- note removed: "XTAL & RST"
- moved on the sheet: C7, R17
