File: circuit/bldc_driver/power.kicad_sch (KiCad schematic)
At the start: 10 parts

Commit message: Update BLDC 6-Step Driver schematic, Version 1.0.1
Parts:
- removed C?: 100nF, symbol Device:C
- added C10, C15, C9: 100uF, Capacitor_SMD:CP_Elec_6.3x9.9, symbol Device:C_Polarized
- added C14: 22uF, Capacitor_SMD:C_1206_3216Metric, symbol Device:C
- added J1: XT30, Connector_AMASS:AMASS_XT30PW-M_1x02_P2.50mm_Horizontal, symbol Library:XT30
- added J2: GH1.25-3P, Connector_JST:JST_GH_SM03B-GHS-TB_1x03-1MP_P1.25mm_Horizontal, symbol Library:GH1.25-3P
- added R28: 124KR, Resistor_SMD:R_0603_1608Metric, symbol Device:R
- added R29: 12.1KR, Resistor_SMD:R_0603_1608Metric, symbol Device:R
- C11: renamed from C?; footprint (none) -> Capacitor_SMD:C_0603_1608Metric
- C12: renamed from C?; value 100nF -> 750pF; footprint (none) -> Capacitor_SMD:C_0603_1608Metric
- C13: renamed from C?; value 100nF -> 8.2pF; footprint (none) -> Capacitor_SMD:C_0603_1608Metric
- L1: renamed from L?; footprint (none) -> Inductor_SMD:L_6.3x6.3_H3
- R25: renamed from R?; value R -> 100KR; footprint (none) -> Resistor_SMD:R_0603_1608Metric
- R26: renamed from R?; value R -> 68.1KR; footprint (none) -> Resistor_SMD:R_0603_1608Metric
- R27: renamed from R?; value R -> 36.5KR; footprint (none) -> Resistor_SMD:R_0603_1608Metric
- gave numbers to parts that had none: 2
Connections:
- net +15V: now also C10.1, C9.1, J1.1 (Pin_1)
- net +9V: now also C14.2, C15.1, R28.1
- net EP: now also C12.1, C13.1, D5.1 (A), D5.2 (A), R26.2, C10.2, C14.1, C15.2, C9.2, J1.2 (Pin_2), J2.3 (Pin_3), R29.2
- net at R27.1: now also C13.2, U2.6 (COMP); no longer C12.1
- net at U2.5 (FB): now also R28.2, R29.1
- removed net GND: C13.1, D5.1 (A), D5.2 (A), R26.2, R27.2
- new net: C12.2, R27.2
- new net M_RX: J2.1 (Pin_1)
- new net M_TX: J2.2 (Pin_2)
Other:
- moved on the sheet: C11, C12, C13, D5, L1, R25, R26, R27, U2

Commit message: Modify the scheme of brushless motor driver board to reduce the use of resistors and capacitors to reduce the size of the circuit.
Parts:
- removed C10, C15, C9: 100uF, Capacitor_SMD:CP_Elec_6.3x9.9, symbol Device:C_Polarized
- removed C12: 750pF, Capacitor_SMD:C_0603_1608Metric, symbol Device:C
- removed D5: SVM1550UB, Package_TO_SOT_SMD:TO-277B, symbol Library:SVM1550UB
- removed R25: 100KR, Resistor_SMD:R_0603_1608Metric, symbol Device:R
- removed R27: 36.5KR, Resistor_SMD:R_0603_1608Metric, symbol Device:R
- removed U2: TPS54540, Package_SO:HSOP-8-1EP_3.9x4.9mm_P1.27mm_EP2.41x3.1mm, symbol Library:TPS54540
- added C10, C9: 22uF, Capacitor_SMD:C_1206_3216Metric, symbol Device:C
- added U3: TPS56339DDC, Package_TO_SOT_SMD:SOT-23-6, symbol Regulator_Switching:TPS56339DDC
- C13: value 8.2pF -> 22uF; footprint Capacitor_SMD:C_0603_1608Metric -> Capacitor_SMD:C_1206_3216Metric
- J2: renamed from J1; footprint Connector_AMASS:AMASS_XT30PW-M_1x02_P2.50mm_Horizontal -> Connector_AMASS:AMASS_XT30U-M_1x02_P5.0mm_Vertical
- L1: value 4.7uH -> 10uH
- R18: renamed from R26; value 68.1KR -> 30R
- R19: renamed from R28; value 124KR -> 140kR
- R20: renamed from R29; value 12.1KR -> 10kR
- renumbered C14 to C12, J2 to J3
Connections:
- net +15V: now also C10.2, C9.2, U3.3 (VIN)
- net +9V: now also C13.2
- net at R19.2, R20.1: now also U3.4 (FB)
- net at C11.1: now also R18.2
- net at C11.2, L1.1: now also U3.2 (SW)
- net at R18.1: now also U3.6 (BOOT)
- net EP renamed GND
- net GND: now also C10.1, C9.1, U3.1 (GND); no longer R18.2
- no-connect marks 0 -> 1
Other:
- note added: "Power Supply"
- moved on the sheet: C11, C12, J2, J3, L1, R18, R19, R20

Commit message: Update the schematic and package library of BLDC Driver.
Parts:
- C10, C12, C13, C9: footprint Capacitor_SMD:C_1206_3216Metric -> BLDC_Driver:C_1206_3216Metric
- C11: footprint Capacitor_SMD:C_0603_1608Metric -> BLDC_Driver:C_0603_1608Metric
- J2: footprint Connector_AMASS:AMASS_XT30U-M_1x02_P5.0mm_Vertical -> BLDC_Driver:AMASS_XT30U-M_1x02_P5.0mm_Vertical
- J3: footprint Connector_JST:JST_GH_SM03B-GHS-TB_1x03-1MP_P1.25mm_Horizontal -> BLDC_Driver:JST_GH_SM03B-GHS-TB_1x03-1MP_P1.25mm_Horizontal
- L1: footprint Inductor_SMD:L_6.3x6.3_H3 -> BLDC_Driver:L_6.3x6.3_H3
- R18, R19, R20: footprint Resistor_SMD:R_0603_1608Metric -> BLDC_Driver:R_0603_1608Metric
- U3: footprint Package_TO_SOT_SMD:SOT-23-6 -> BLDC_Driver:SOT-23-6
Changed lines of the file:
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@@
   (title_block
     (title "BLDC Driver 6-Step")
-    (date "2022-03-25")
-    (rev "1.1.1")
+    (date "2022-03-26")
+    (rev "1.1.2")
   )
   (junction (at 188.595 99.06) (diameter 0) (color 0 0 0 0)
@@
       (effects (font (size 1.27 1.27)) (justify left))
     )
-    (property "Footprint" "Resistor_SMD:R_0603_1608Metric" (id 2) (at 177.927 106.68 90)
+    (property "Footprint" "BLDC_Driver:R_0603_1608Metric" (id 2) (at 177.927 106.68 90)
       (effects (font (size 1.27 1.27)) hide)
     )
@@
     (property "Reference" "C10" (id 0) (at 93.345 101.6 0))
     (property "Value" "22uF" (id 1) (at 93.98 104.14 0))
-    (property "Footprint" "Capacitor_SMD:C_1206_3216Metric" (id 2) (at 86.6648 99.06 0)
+    (property "Footprint" "BLDC_Driver:C_1206_3216Metric" (id 2) (at 86.6648 99.06 0)
       (effects (font (size 1.27 1.27)) hide)
     )
@@
     (property "Reference" "C11" (id 0) (at 155.575 93.345 90))
     (property "Value" "100nF" (id 1) (at 156.21 95.25 90))
-    (property "Footprint" "Capacitor_SMD:C_0603_1608Metric" (id 2) (at 159.385 98.0948 0)
+    (property "Footprint" "BLDC_Driver:C_0603_1608Metric" (id 2) (at 159.385 98.0948 0)
       (effects (font (size 1.27 1.27)) hide)
     )
@@
     (property "Reference" "C13" (id 0) (at 209.55 100.33 0))
     (property "Value" "22uF" (id 1) (at 210.185 102.87 0))
-    (property "Footprint" "Capacitor_SMD:C_1206_3216Metric" (id 2) (at 202.8698 97.79 0)
+    (property "Footprint" "BLDC_Driver:C_1206_3216Metric" (id 2) (at 202.8698 97.79 0)
       (effects (font (size 1.27 1.27)) hide)
     )
@@
     (property "Reference" "U3" (id 0) (at 127 95.25 0))
     (property "Value" "TPS56339DDC" (id 1) (at 132.08 107.95 0))
-    (property "Footprint" "Package_TO_SOT_SMD:SOT-23-6" (id 2) (at 134.62 107.95 0)
+    (property "Footprint" "BLDC_Driver:SOT-23-6" (id 2) (at 134.62 107.95 0)
       (effects (font (size 1.27 1.27)) (justify left) hide)
     )
@@
     (property "Reference" "R18" (id 0) (at 146.05 93.345 90))
     (property "Value" "30R" (id 1) (at 146.05 95.885 90))
-    (property "Footprint" "Resistor_SMD:R_0603_1608Metric" (id 2) (at 146.05 100.838 90)
+    (property "Footprint" "BLDC_Driver:R_0603_1608Metric" (id 2) (at 146.05 100.838 90)
       (effects (font (size 1.27 1.27)) hide)
     )
@@
     (property "Reference" "L1" (id 0) (at 170.815 93.345 90))
     (property "Value" "10uH" (id 1) (at 170.815 95.885 90))
-    (property "Footprint" "Inductor_SMD:L_6.3x6.3_H3" (id 2) (at 170.815 99.06 0)
+    (property "Footprint" "BLDC_Driver:L_6.3x6.3_H3" (id 2) (at 170.815 99.06 0)
       (effects (font (size 1.27 1.27)) hide)
     )
@@
     (property "Reference" "C9" (id 0) (at 80.645 101.6 0))
     (property "Value" "22uF" (id 1) (at 81.28 104.14 0))
-    (property "Footprint" "Capacitor_SMD:C_1206_3216Metric" (id 2) (at 73.9648 99.06 0)
+    (property "Footprint" "BLDC_Driver:C_1206_3216Metric" (id 2) (at 73.9648 99.06 0)
       (effects (font (size 1.27 1.27)) hide)
     )
@@
     (property "Reference" "C12" (id 0) (at 194.31 111.76 0))
     (property "Value" "22uF" (id 1) (at 194.945 114.3 0))
-    (property "Footprint" "Capacitor_SMD:C_1206_3216Metric" (id 2) (at 187.6298 109.22 0)
+    (property "Footprint" "BLDC_Driver:C_1206_3216Metric" (id 2) (at 187.6298 109.22 0)
       (effects (font (size 1.27 1.27)) hide)
     )
@@
       (effects (font (size 1.27 1.27)) (justify left))
     )
-    (property "Footprint" "Connector_JST:JST_GH_SM03B-GHS-TB_1x03-1MP_P1.25mm_Horizontal" (id 2) (at 242.57 109.22 0)
+    (property "Footprint" "BLDC_Driver:JST_GH_SM03B-GHS-TB_1x03-1MP_P1.25mm_Horizontal" (id 2) (at 242.57 109.22 0)
       (effects (font (size 1.27 1.27)) hide)
     )
@@
     (property "Reference" "J2" (id 0) (at 52.705 95.25 0))
     (property "Value" "XT30" (id 1) (at 52.705 97.79 0))
-    (property "Footprint" "Connector_AMASS:AMASS_XT30U-M_1x02_P5.0mm_Vertical" (id 2) (at 56.515 109.22 0)
+    (property "Footprint" "BLDC_Driver:AMASS_XT30U-M_1x02_P5.0mm_Vertical" (id 2) (at 56.515 109.22 0)
       (effects (font (size 1.27 1.27)) hide)
     )
@@
       (effects (font (size 1.27 1.27)) (justify left))
     )
-    (property "Footprint" "Resistor_SMD:R_0603_1608Metric" (id 2) (at 177.927 118.11 90)
-      (effects (font (size 1.27 1.27)) hide)
-    )
+    (property "Footprint" "BLDC_Driver:R_0603_1608Metric" (id 2) (at 177.927 118.11 90)
+      (effects (font (size 1.27 1.27)) hide)
+    )

Commit message: Modified the BLDC driver circuit by deleting the crystal and adding decoupling capacitors. Replaced the buck chip with JW5017s chip for power supply.
Parts:
- removed U3: TPS56339DDC, BLDC_Driver:SOT-23-6, symbol Regulator_Switching:TPS56339DDC
- added C15, C6: 1uF, BLDC_Driver:C_0603_1608Metric, symbol Device:C
- added C5: 4.7uF, BLDC_Driver:C_0603_1608Metric, symbol Device:C
- added U3: JW5015s, Package_TO_SOT_SMD:SOT-23-6, symbol Library:JW5015s
- C10, C13: value 22uF -> 47uF
- C12, C9: value 22uF -> 10uF
- L1: value 10uH -> 4.7uH; footprint BLDC_Driver:L_6.3x6.3_H3 -> Inductor_SMD:L_Bourns-SRN4018
- R18: value 30R -> 100kR
Connections:
- net +15V: now also J2.2 (Pin_2), R18.1, U3.5 (VIN); no longer J2.1 (Pin_1)
- net GND: now also J2.1 (Pin_1), C15.1, C5.1, C6.1, U3.2 (GND); no longer J2.2 (Pin_2)
- net at R19.2, R20.1: now also U3.3 (FB)
- net at C11.1: now also U3.1 (BST); no longer R18.2
- net at C11.2, L1.1: now also U3.6 (SW)
- net +9V renamed +12V
- net +12V: now also C5.2
- new net: R18.2, U3.4 (EN)
- new net +5V: C15.2, C6.2
- no-connect marks 1 -> 0
Other:
- moved on the sheet: C10, C11, C12, C13, L1, R19, R20
