File: circuit/bldc_driver/project.kicad_sch (KiCad schematic)
At the start: 0 parts

Commit message: Add BLDC driver circuit.
Other:
- added sheet Driver (Driver.kicad_sch)
- added sheet Power (power.kicad_sch)
- sheet Controller ports: added HO1, HO2, HO3, IA, IB, ISUN, LO1, LO2, LO3, VS1, VS2, VS3; removed none
- title: BLDC Driver -> BLDC Driver 6-Step

Commit message: Update BLDC 6-Step Driver schematic, Version 1.0.1
Other:
- added sheet Connector (connector.kicad_sch)
- sheet Controller ports: added ISUM, M_RX, M_TX, PA0, PA1, PA2, PA7; removed ISUN
- sheet Power ports: added M_RX, M_TX; removed none

Commit message: Modify the scheme of brushless motor driver board to reduce the use of resistors and capacitors to reduce the size of the circuit.
Other:
- sheet Connector ports: added HA, HB, HC, NTC; removed PA0, PA1, PA2, PA7
- sheet Controller ports: added UART1_RX, UART1_TX; removed M_RX, M_TX
