File: circuit/bldc_driver/project.kicad_pcb (KiCad board)
At the start: 2 copper layers, 91 parts, among them J1 XT30, J2 GH1.25-3P, J3 MR30, J4 PH2.0_6P, M1 Debugger, Q1 CSD18540Q5B, Q2 CSD18540Q5B, Q3 CSD18540Q5B, Q4 CSD18540Q5B, Q5 CSD18540Q5B, Q6 CSD18540Q5B, U1 MM32SPIN360C, U2 TPS54540, Y1 8MHz

Commit message: Complete the design of BLDC Driver PCB and export the interactive BOM.
Parts:
- removed the C12 at (193.6, 73.0)
- removed C15: 100uF, Capacitor_SMD:CP_Elec_6.3x9.9
- removed C16, C17, C18: 100nF, Capacitor_SMD:C_0603_1608Metric
- removed the D2 at (101.7, 97.8)
- removed D3: LED, LED_SMD:LED_0603_1608Metric
- removed D5: SVM1550UB, Package_TO_SOT_SMD:TO-277B
- removed M1: Debugger, BLDC_Driver:Gernic_Debugger
- removed the R13 at (141.3, 70.5)
- removed the R14 at (139.6, 78.1)
- removed the R19 at (131.6, 82.2)
- removed the R2 at (117.7, 99.3)
- removed the R20 at (120.6, 91.8)
- removed the R25 at (188.0, 78.3)
- removed the R27 at (173.4, 92.6)
- removed R45, R50, R51, R52: 100R, Resistor_SMD:R_0603_1608Metric
- removed R46, R47, R48: 4.7KR, Resistor_SMD:R_0603_1608Metric
- removed the R5 at (139.6, 75.6)
- removed the R6 at (131.6, 77.2)
- added J1: Conn_01x04, Connector_PinSocket_2.54mm:PinSocket_1x04_P2.54mm_Vertical, F.Cu at (146.2, 81.0)
- added U3: TPS56339DDC, Package_TO_SOT_SMD:SOT-23-6, F.Cu at (148.3, 86.7)
- added U4: 74HC1G126GW, Package_TO_SOT_SMD:SOT-353_SC-70-5, B.Cu at (140.1, 88.5)
- added U5: 74HC1G126GW, Package_TO_SOT_SMD:SOT-353_SC-70-5, B.Cu at (140.1, 85.8)
- added U6: 74HC1G126GW, Package_TO_SOT_SMD:SOT-353_SC-70-5, B.Cu at (140.1, 83.2)
- C1: footprint Capacitor_SMD:C_0201_0603Metric -> Capacitor_SMD:C_0603_1608Metric; moved to B.Cu
- C10, C9: value 100uF -> 22uF; footprint Capacitor_SMD:CP_Elec_6.3x9.9 -> Capacitor_SMD:C_1206_3216Metric; moved to B.Cu
- C13: value 8.2pF -> 22uF; footprint Capacitor_SMD:C_0603_1608Metric -> Capacitor_SMD:C_1206_3216Metric
- C14: renamed from C19; moved to B.Cu
- C2, C3, C4: footprint Capacitor_SMD:C_1206_3216Metric -> Capacitor_SMD:C_0603_1608Metric; moved to B.Cu
- C5, C6, C8, R1, Y1: moved to B.Cu
- J2: renamed from J1; footprint Connector_AMASS:AMASS_XT30PW-M_1x02_P2.50mm_Horizontal -> Connector_AMASS:AMASS_XT30U-M_1x02_P5.0mm_Vertical
- J4: renamed from J3; footprint Connector_AMASS:AMASS_MR30PW-FB_1x03_P3.50mm_Horizontal -> BLDC_Driver:MR30_Vertical
- J5: renamed from J4; value PH2.0_6P -> GH1.25_6P; footprint Connector_JST:JST_PH_B6B-PH-SM4-TB_1x06-1MP_P2.00mm_Vertical -> Connector_JST:JST_GH_BM06B-GHS-TBT_1x06-1MP_P1.25mm_Vertical
- L1: value 4.7uH -> 10uH
- R10: renamed from R15; moved to B.Cu
- R11: renamed from R16; moved to B.Cu
- R12: renamed from R17; moved to B.Cu
- R13: renamed from R18; value 20KR -> 2kR
- R14: renamed from R21; value 10KR -> 2kR
- R15: renamed from R22; moved to B.Cu
- R16: renamed from R23; moved to B.Cu
- R18: renamed from R26; value 68.1KR -> 30R
- R19: renamed from R28; value 124KR -> 140kR
- R2: renamed from R3; moved to B.Cu
- R20: renamed from R29; value 12.1KR -> 10kR
- R21: renamed from R30; footprint Resistor_SMD:R_0805_2012Metric -> Resistor_SMD:R_0603_1608Metric; moved to B.Cu
- R22: renamed from R31; footprint Resistor_SMD:R_0805_2012Metric -> Resistor_SMD:R_0603_1608Metric; moved to B.Cu
- R23: renamed from R32; footprint Resistor_SMD:R_0805_2012Metric -> Resistor_SMD:R_0603_1608Metric; moved to B.Cu
- R24: renamed from R33; footprint Resistor_SMD:R_0805_2012Metric -> Resistor_SMD:R_0603_1608Metric
- R25: renamed from R34; footprint Resistor_SMD:R_2512_6332Metric -> Resistor_SMD:R_1206_3216Metric
- R26: renamed from R35; footprint Resistor_SMD:R_0805_2012Metric -> Resistor_SMD:R_0603_1608Metric; moved to B.Cu
- R27: renamed from R36; footprint Resistor_SMD:R_0805_2012Metric -> Resistor_SMD:R_0603_1608Metric; moved to B.Cu
- R28: renamed from R37; footprint Resistor_SMD:R_0805_2012Metric -> Resistor_SMD:R_0603_1608Metric; moved to B.Cu
- R3: renamed from R4; moved to B.Cu
- R30: renamed from R39; footprint Resistor_SMD:R_2512_6332Metric -> Resistor_SMD:R_1206_3216Metric; moved to B.Cu
- R31: renamed from R40; footprint Resistor_SMD:R_2512_6332Metric -> Resistor_SMD:R_1206_3216Metric
- R32: renamed from R41; footprint Resistor_SMD:R_0805_2012Metric -> Resistor_SMD:R_0603_1608Metric; moved to B.Cu
- R33: renamed from R42; footprint Resistor_SMD:R_0805_2012Metric -> Resistor_SMD:R_0603_1608Metric; moved to B.Cu
- R34: renamed from R43; footprint Resistor_SMD:R_0805_2012Metric -> Resistor_SMD:R_0603_1608Metric; moved to B.Cu
- R35: renamed from R44; footprint Resistor_SMD:R_0805_2012Metric -> Resistor_SMD:R_0603_1608Metric
- R36: renamed from R49; moved to B.Cu
- R4: renamed from R7; moved to B.Cu
- R6: renamed from R9; moved to B.Cu
- R7: renamed from R10; moved to B.Cu
- R8: renamed from R11; moved to B.Cu
- R9: renamed from R12; moved to B.Cu
- U1: footprint Package_QFP:TQFP-48-1EP_7x7mm_P0.5mm_EP5x5mm -> Package_DFN_QFN:QFN-48-1EP_6x6mm_P0.4mm_EP4.2x4.2mm; moved to B.Cu
- U2: value TPS54540 -> REF3025; footprint Package_SO:HSOP-8-1EP_3.9x4.9mm_P1.27mm_EP2.41x3.1mm -> Package_TO_SOT_SMD:SOT-23; moved to B.Cu
- moved R24 76.1 mm to (163.2, 107.7), turned to -90 degrees
- moved R31 75.2 mm to (162.8, 99.1), turned to 180 degrees
- moved R29 69.9 mm to (157.5, 99.3), turned to -90 degrees
- moved U1 66.6 mm to (160.6, 95.5)
- moved Q4 62.6 mm to (159.4, 104.2), turned to -90 degrees
- moved R9 60.3 mm to (164.5, 87.0), turned to 90 degrees
- moved R4 58.9 mm to (159.0, 87.0), turned to 90 degrees
- moved C3 57.9 mm to (159.3, 103.2), turned to -90 degrees
- moved Q2 57.1 mm to (164.7, 113.3), turned to -90 degrees
- moved R15 56.7 mm to (166.3, 97.0), turned to 90 degrees
- moved R13 53.9 mm to (161.6, 86.7), turned to -90 degrees
- moved R25 53.6 mm to (159.3, 92.2), turned to 180 degrees
- moved D2 53.5 mm to (165.9, 87.5), turned to 180 degrees
- moved R22 52.3 mm to (164.9, 106.7), turned to -90 degrees
- moved R12 51.6 mm to (156.3, 86.1), turned to 180 degrees
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- renumbered C14 to C12, D4 to D2, J2 to J3, R24 to R17, R38 to R29, R8 to R5
Connections:
- net /Controller/DBG_RX renamed /Controller/UART1_TX
- net /Controller/DBG_TX renamed /Controller/UART1_RX
- C1 pad 1: Net-(C1-Pad1) -> /Controller/PA3
- C1 pad 2: EP -> GND
- C10 pad 1: +15V -> GND
- C10 pad 2: EP -> +15V
- C12 pad 1: EP -> GND
- C13 pad 1: EP -> GND
- C13 pad 2: Net-(C13-Pad2) -> +9V
- C14 pad 1: EP -> GND
- C14 pad 2: /Connector/MNTC -> /Connector/NTC
- C5 pad 2: EP -> GND
- C6 pad 2: EP -> GND
- C7 pad 2: EP -> GND
- C8 pad 2: EP -> GND
- C9 pad 1: +15V -> GND
- C9 pad 2: EP -> +15V
- D2 pad 1: EP -> GND
- J2 pad 2: EP -> GND
- J3 pad 3: EP -> GND
- J4 pad 1: /Controller/VS1 -> /Controller/VS3
- J4 pad 3: /Controller/VS3 -> /Controller/VS1
- J5 pad 2: /Connector/MNTC -> /Connector/NTC
- J5 pad 6: EP -> GND
- Q1 pad 1: /Controller/VS1 -> /Controller/VS3
- Q1 pad 2: /Controller/VS1 -> /Controller/VS3
- Q1 pad 3: /Controller/VS1 -> /Controller/VS3
- Q2 pad 1: /Controller/IA -> /Controller/ISUM
- Q2 pad 2: /Controller/IA -> /Controller/ISUM
- Q2 pad 3: /Controller/IA -> /Controller/ISUM
- Q2 pad 5: /Controller/VS1 -> /Controller/VS3
- Q5 pad 1: /Controller/VS3 -> /Controller/VS1
- Q5 pad 2: /Controller/VS3 -> /Controller/VS1
- Q5 pad 3: /Controller/VS3 -> /Controller/VS1
- Q6 pad 1: /Controller/ISUM -> /Controller/IA
- Q6 pad 2: /Controller/ISUM -> /Controller/IA
- Q6 pad 3: /Controller/ISUM -> /Controller/IA
- Q6 pad 5: /Controller/VS3 -> /Controller/VS1
- R1 pad 2: Net-(C1-Pad1) -> /Controller/PA3
- R16 pad 2: EP -> GND
- R17 pad 1: +3V3 -> +5V
- R18 pad 1: Net-(R26-Pad1) -> Net-(R18-Pad1)
- R18 pad 2: EP -> Net-(C11-Pad1)
- R19 pad 2: Net-(R28-Pad2) -> Net-(R19-Pad2)
- R20 pad 1: Net-(R28-Pad2) -> Net-(R19-Pad2)
- R20 pad 2: EP -> GND
- R21 pad 1: /Controller/HO1 -> /Controller/HO3
- R22 pad 1: /Controller/LO1 -> /Controller/LO3
- R23 pad 1: /Controller/VS1 -> /Controller/VS3
- R30 pad 1: EP -> GND
- R32 pad 1: /Controller/HO3 -> /Controller/HO1
- R33 pad 1: /Controller/LO3 -> /Controller/LO1
- R34 pad 1: /Controller/VS3 -> /Controller/VS1
- R35 pad 1: /Controller/ISUM -> GND
- R36 pad 2: /Connector/MNTC -> /Connector/NTC
- R5 pad 1: /Controller/P12 -> /Controller/PB12
- R6 pad 1: EP -> GND
- R8 pad 2: Net-(R11-Pad2) -> +2V5
- R9 pad 1: /Controller/P12 -> /Controller/PB12
- R9 pad 2: Net-(R12-Pad2) -> +2V5
- U1 pad 1: EP -> GND
- U1 pad 10: /Connector/PA0 -> /Connector/HA
- U1 pad 11: /Connector/PA1 -> /Connector/HB
- U1 pad 12: /Connector/PA2 -> /Connector/HC
- U1 pad 13: Net-(C1-Pad1) -> /Controller/PA3
- U1 pad 17: /Connector/PA7 -> /Connector/NTC
- U1 pad 24: EP -> GND
- U1 pad 35: Net-(R2-Pad1) -> /Controller/PA3
- U1 pad 4: /Controller/PC14 -> unconnected-(U1-Pad4)
- U1 pad 49: EP -> GND
- U1 pad 5: /Controller/PC15 -> unconnected-(U1-Pad5)
- U2 pad 1: Net-(C11-Pad1) -> +5V
- U2 pad 2: +15V -> +2V5
- U2 pad 3: Net-(R25-Pad2) -> GND
- Y1 pad 2: EP -> GND
- Y1 pad 4: EP -> GND
Routing:
- net +5V: track 0.00 -> 103.1 mm, vias 0 -> 5
- net /Controller/RST: track 0.00 -> 34.9 mm, vias 0 -> 2
- net +9V: track 0.00 -> 30.8 mm, vias 0 -> 2
- net Net-(Q4-Pad4): track 0.00 -> 30.1 mm, vias 0 -> 1
- net Net-(Q6-Pad4): track 0.00 -> 29.4 mm, vias 0 -> 1
- net /Controller/ISUM: track 0.00 -> 28.1 mm, vias 0 -> 20
- net /Controller/SWDIO: track 0.00 -> 27.5 mm, vias 0 -> 1
- net +15V: track 0.00 -> 27.3 mm, vias 0 -> 29
- net /Controller/SWDCLK: track 0.00 -> 27.2 mm, vias 0 -> 1
- net /Connector/NTC: track 0.00 -> 27.0 mm, vias 0 -> 2
- net /Controller/PA3: track 0.00 -> 26.2 mm, vias 0 -> 2
- net /Connector/HC: track 0.00 -> 22.3 mm
- net /Controller/VS3: track 0.00 -> 20.5 mm, vias 0 -> 3
- net /Controller/UART1_RX: track 0.00 -> 20.2 mm, vias 0 -> 2
- net /Connector/HB: track 0.00 -> 20.1 mm
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- added copper zone on B.Cu, net +15V
- added copper zone on F.Cu, net +15V
- added copper zone on F.Cu, net +9V
- added copper zone on F.Cu, net /Controller/IA
- added copper zone on F.Cu, net /Controller/IB
- added copper zone on B.Cu, net /Controller/ISUM
- added copper zone on F.Cu, net /Controller/ISUM
- added copper zone on F.Cu, net /Controller/VS1
- added copper zone on F.Cu, net /Controller/VS2
- added copper zone on F.Cu, net /Controller/VS3
- added copper zone on B.Cu, net GND
- added copper zone on F.Cu, net GND
- added copper zone on In1.Cu, net GND
- added copper zone on In2.Cu, net GND
Other:
- board outline added: 30 x 40 mm
- copper layers 2 -> 4
- board text added: "0"
- board text added: "0 mm"
- board text added: "0.01 mm"
- board text added: "0.0175 mm"
- board text added: "0.02"
- board text added: "0.035 mm"
- board text added: "0.2 mm"
- board text added: "0.2000 mm"
- board text added: "0.2000 mm / 0.2000 mm"
- board text added: "1"
- board text added: "1.075 mm"
- board text added: "1.6000 mm"
- board text added: "2022/03/16"
- board text added: "3.3"
- board text added: "30.1000 mm x 40.1000 mm"
- board text added: "4"
- board text added: "4.5"
- board text added: "B.Cu"
- board text added: "B.Mask"
- board text added: "B.Paste"
- board text added: "B.Silkscreen"
- board text added: "BLDC Driver"
- board text added: "BOARD CHARACTERISTICS"
- board text added: "Bottom Silk Screen"
- board text added: "Bottom Solder Mask"
- board text added: "Bottom Solder Paste"
- board text added: "Direct Printing"
- board text added: "Dry Film"
- board text added: "Epsilon R（相对介电常数）"
- board text added: "F.Cu"
- board text added: "F.Mask"
- board text added: "F.Paste"
- board text added: "F.Silkscreen"
- board text added: "FR4"
- board text added: "G I C V"
- board text added: "GDUT"
- board text added: "Green"
- board text added: "In1.Cu"
- board text added: "In2.Cu"
- board text added: "Jesus Team"
- board text added: "LaoZhu Design"
- board text added: "Loss Tangent（损耗切线）"
- board text added: "None"
- board text added: "Top Silk Screen"
- board text added: "Top Solder Mask"
- board text added: "Top Solder Paste"
- board text added: "Ver 1.1.2"
- board text added: "White"
- board text added: "copper"
- board text added: "core"
- board text added: "否"
- board text added: "孔最小直径："
- board text added: "层名称"
- board text added: "最小布线/间距："
- board text added: "材料"
- board text added: "板子整体尺寸："
- board text added: "电介质层 1"
- board text added: "电介质层 2"
- board text added: "电介质层 3"
- board text added: "电路板厚度："
- board text added: "电镀板边："
- board text added: "类型"
- board text added: "粗细 (mm)"
- board text added: "边缘卡连接器："
- board text added: "邮票孔："
- board text added: "铜层数量："
- board text added: "铜表面处理（镀铜）："
- board text added: "阻抗控制"
- board text added: "颜色"

Commit message: Completed PCB layout wiring of BLDC driver circuit and exported the interactive BOM.
Parts:
- removed Y1: 8MHz, Crystal:Crystal_SMD_3225-4Pin_3.2x2.5mm
- added C15: 1uF, BLDC_Driver:C_0603_1608Metric, B.Cu at (154.4, 93.7)
- C1, C11, C14, C2, C3, C4, C8: footprint Capacitor_SMD:C_0603_1608Metric -> BLDC_Driver:C_0603_1608Metric
- C10, C13: value 22uF -> 47uF; footprint Capacitor_SMD:C_1206_3216Metric -> BLDC_Driver:C_1206_3216Metric
- C12, C9: value 22uF -> 10uF; footprint Capacitor_SMD:C_1206_3216Metric -> BLDC_Driver:C_1206_3216Metric
- C5: value 18pF -> 4.7uF; footprint Capacitor_SMD:C_0603_1608Metric -> BLDC_Driver:C_0603_1608Metric
- C6: value 18pF -> 1uF; footprint Capacitor_SMD:C_0603_1608Metric -> BLDC_Driver:C_0603_1608Metric
- C7: footprint Capacitor_SMD:C_0603_1608Metric -> BLDC_Driver:C_0603_1608Metric; moved to B.Cu
- D1, D2: footprint LED_SMD:LED_0603_1608Metric -> BLDC_Driver:LED_0603_1608Metric
- J1: footprint Connector_PinSocket_2.54mm:PinSocket_1x04_P2.54mm_Vertical -> BLDC_Driver:PinSocket_1x04_P2.54mm_Vertical
- J2: footprint Connector_AMASS:AMASS_XT30U-M_1x02_P5.0mm_Vertical -> BLDC_Driver:AMASS_XT30U-M_1x02_P5.0mm_Vertical
- J3: footprint Connector_JST:JST_GH_SM03B-GHS-TB_1x03-1MP_P1.25mm_Horizontal -> BLDC_Driver:JST_GH_SM03B-GHS-TB_1x03-1MP_P1.25mm_Horizontal
- J5: footprint Connector_JST:JST_GH_BM06B-GHS-TBT_1x06-1MP_P1.25mm_Vertical -> BLDC_Driver:JST_GH_BM06B-GHS-TBT_1x06-1MP_P1.25mm_Vertical
- L1: value 10uH -> 4.7uH; footprint Inductor_SMD:L_6.3x6.3_H3 -> Inductor_SMD:L_Bourns-SRN4018
- Q1, Q2, Q3, Q4, Q5, Q6: footprint Package_TO_SOT_SMD:TDSON-8-1 -> BLDC_Driver:TDSON-8-1
- R1, R16, R36: value 10KR -> 10kR; footprint Resistor_SMD:R_0603_1608Metric -> BLDC_Driver:R_0603_1608Metric
- R10, R11, R8, R9: value 100KR -> 100kR; footprint Resistor_SMD:R_0603_1608Metric -> BLDC_Driver:R_0603_1608Metric
- R12, R13, R14, R19, R20, R21, R22, R23, R24, R26, R27, R28, R29, R32, R33, R34, R35, R6, R7: footprint Resistor_SMD:R_0603_1608Metric -> BLDC_Driver:R_0603_1608Metric
- R15: value 40KR -> 40kR; footprint Resistor_SMD:R_0603_1608Metric -> BLDC_Driver:R_0603_1608Metric
- R17: footprint Resistor_SMD:R_0603_1608Metric -> BLDC_Driver:R_0603_1608Metric; moved to B.Cu
- R18: value 30R -> 100kR; footprint Resistor_SMD:R_0603_1608Metric -> BLDC_Driver:R_0603_1608Metric
- R2, R3, R4, R5: value 1KR -> 1kR; footprint Resistor_SMD:R_0603_1608Metric -> BLDC_Driver:R_0603_1608Metric
- R25, R30, R31: footprint Resistor_SMD:R_1206_3216Metric -> BLDC_Driver:R_1206_3216Metric
- U1: footprint Package_DFN_QFN:QFN-48-1EP_6x6mm_P0.4mm_EP4.2x4.2mm -> BLDC_Driver:QFN-48-1EP_6x6mm_P0.4mm_EP4.2x4.2mm
- U2: footprint Package_TO_SOT_SMD:SOT-23 -> BLDC_Driver:SOT-23
- U3: value TPS56339DDC -> JW5015s
- U4, U5, U6: footprint Package_TO_SOT_SMD:SOT-353_SC-70-5 -> BLDC_Driver:SOT-353_SC-70-5
- moved R17 8.71 mm to (151.3, 95.3)
- moved C5 6.14 mm to (154.4, 98.5), turned to 0 degrees
- moved C7 5.71 mm to (154.4, 95.3)
- moved C11 4.77 mm to (149.4, 86.7)
- moved C13 3.72 mm to (153.7, 83.5), turned to 180 degrees
- moved R18 3.59 mm to (146.2, 89.6), turned to 180 degrees
- moved C12 2.61 mm to (156.7, 88.1)
- moved C6 2.40 mm to (154.4, 97.0)
- moved U3 1.60 mm to (146.7, 86.8), turned to -90 degrees
- moved L1 1.10 mm to (153.3, 87.2)
Connections:
- C12 pad 2: +9V -> +12V
- C13 pad 2: +9V -> +12V
- C5 pad 1: /Controller/XTAL_OUT -> GND
- C5 pad 2: GND -> +12V
- C6 pad 1: /Controller/XTAL_IN -> GND
- C6 pad 2: GND -> +5V
- J2 pad 1: +15V -> GND
- J2 pad 2: GND -> +15V
- L1 pad 2: +9V -> +12V
- R18 pad 1: Net-(R18-Pad1) -> +15V
- R18 pad 2: Net-(C11-Pad1) -> Net-(R18-Pad2)
- R19 pad 1: +9V -> +12V
- U1 pad 2: +9V -> +12V
- U1 pad 6: /Controller/XTAL_IN -> unconnected-(U1-Pad6)
- U1 pad 7: /Controller/XTAL_OUT -> unconnected-(U1-Pad7)
- U3 pad 1: GND -> Net-(C11-Pad1)
- U3 pad 2: Net-(C11-Pad2) -> GND
- U3 pad 3: +15V -> Net-(R19-Pad2)
- U3 pad 4: Net-(R19-Pad2) -> Net-(R18-Pad2)
- U3 pad 5: unconnected-(U3-Pad5) -> +15V
- U3 pad 6: Net-(R18-Pad1) -> Net-(C11-Pad2)
Routing:
- net +9V: track 30.8 -> 0.00 mm, vias 2 -> 0
- net /Controller/RST: track 34.9 -> 6.33 mm, vias 2 -> 0
- net +12V: track 0.00 -> 19.6 mm, vias 0 -> 2
- net GND: track 14.8 -> 0.00 mm, vias 89 -> 66
- net +5V: track 103.1 -> 91.4 mm
- net /Controller/XTAL_IN: track 8.18 -> 0.00 mm
- net /Controller/XTAL_OUT: track 6.24 -> 0.00 mm
- net +15V: track 27.3 -> 23.1 mm
- net Net-(C11-Pad2): track 10.9 -> 8.85 mm
- net Net-(R18-Pad1): track 2.07 -> 0.00 mm
- net Net-(R18-Pad2): track 0.00 -> 1.82 mm
- net /Connector/HC: track 22.3 -> 21.1 mm
- net /Controller/ISUM: vias 20 -> 21
- added copper zone on F.Cu, net +12V
- removed copper zone on F.Cu, net +9V
Other:
- board text added: "2022/04/07"
- board text added: "Ver 1.2.4"
- board text removed: "2022/03/16"
- board text removed: "Ver 1.1.2"
