File: circuit/control_board/project.kicad_pcb (KiCad board)
At the start: 4 copper layers, 95 x 50 mm, 108 parts, among them J1 ANT, J2 Conn_01x08, M1 Debugger, SW1 SW_DIP_x02, U1 TAU1201, U10 HX9193, U11 MM32F3277G9P, U12 CH440R, U13 HMC5883L, U14 AT24C02, U2 XPT2046TS, U3 ADIS16470AMLZ, U4 B0505S-1WR3, U5 HX9193, U6 π131M31, U7 π131M31, U8 MM32F3277G9P, U9 HX9193, Y1 8MHz, Y2 8MHz

Commit message: Complete PCB layout wiring, screen printing adjustment. But not yet checked the circuit.
Parts:
- removed the C26 at (170.4, 110.7)
- removed the C27 at (148.2, 83.5)
- removed the C28 at (191.6, 105.8)
- removed the C29 at (190.9, 113.4)
- removed C72: 100nF, Capacitor_SMD:C_0603_1608Metric
- removed the U6 at (170.4, 116.6)
- removed the U7 at (170.4, 104.8)
- added C67: 100nF, ControlBoard:C_0603_1608Metric, B.Cu at (176.5, 101.8)
- added C68: 18pF, ControlBoard:C_0603_1608Metric, B.Cu at (164.7, 110.8)
- added D3: LED, ControlBoard:LED_0603_1608Metric, F.Cu at (181.2, 120.8)
- added J3: Conn_01x04, ControlBoard:SWD_Connector, F.Cu at (170.0, 121.8)
- added R10: 121R, ControlBoard:R_0603_1608Metric, F.Cu at (191.3, 101.9)
- added R11: 121R, ControlBoard:R_0603_1608Metric, F.Cu at (194.6, 101.7)
- added R12: 121R, ControlBoard:R_0603_1608Metric, F.Cu at (194.8, 98.4)
- added R13: 121R, ControlBoard:R_0603_1608Metric, F.Cu at (194.8, 95.0)
- added R14: 121R, ControlBoard:R_0603_1608Metric, F.Cu at (192.4, 94.5)
- added R15: 121R, ControlBoard:R_0603_1608Metric, F.Cu at (189.3, 94.5)
- added R16: PN13101(Z), ControlBoard:PN13101, F.Cu at (195.9, 104.7)
- added R17: PN13104(XY), ControlBoard:PN13104, F.Cu at (197.1, 94.1)
- added R18: PN13104(XY), ControlBoard:PN13104, F.Cu at (189.1, 91.5)
- added R21: 10kR, ControlBoard:R_0603_1608Metric, B.Cu at (170.8, 120.2)
- added R22: 1kR, ControlBoard:R_0603_1608Metric, F.Cu at (184.3, 120.8)
- added R23: 10kR, ControlBoard:R_0603_1608Metric, B.Cu at (164.7, 109.2)
- added R9: 33kR, ControlBoard:R_0603_1608Metric, F.Cu at (186.0, 97.3)
- added U11: RM3100_13156, ControlBoard:QFN-28-1EP_4x4mm_P0.4mm_EP2.4x2.4mm, F.Cu at (190.7, 98.1)
- added U14: π131M31, ControlBoard:SOIC-16_3.9x9.9mm_P1.27mm, B.Cu at (181.3, 98.0)
- added Y3: 8MHz, ControlBoard:Crystal_SMD_3225-4Pin_3.2x2.5mm, B.Cu at (164.7, 114.0)
- C1, C10, C11, C12, C2, C3, C4, C5, C6, C8, C9: footprint Capacitor_SMD:C_0603_1608Metric -> ControlBoard:C_0603_1608Metric
- C13: renamed from C17; footprint Capacitor_SMD:C_0603_1608Metric -> ControlBoard:C_0603_1608Metric
- C14: renamed from C18; footprint Capacitor_SMD:C_0603_1608Metric -> ControlBoard:C_0603_1608Metric; moved to B.Cu
- C15: renamed from C19; footprint Capacitor_SMD:C_0603_1608Metric -> ControlBoard:C_0603_1608Metric; moved to F.Cu
- C16: renamed from C20; footprint Capacitor_SMD:C_0603_1608Metric -> ControlBoard:C_0603_1608Metric
- C17: renamed from C21; footprint Capacitor_SMD:C_0603_1608Metric -> ControlBoard:C_0603_1608Metric
- C18: renamed from C22; footprint Capacitor_SMD:C_0603_1608Metric -> ControlBoard:C_0603_1608Metric
- C19: renamed from C24; footprint Capacitor_SMD:C_0603_1608Metric -> ControlBoard:C_0603_1608Metric
- C20: renamed from C25; footprint Capacitor_SMD:C_0603_1608Metric -> ControlBoard:C_0603_1608Metric
- C21: renamed from C13; footprint Capacitor_SMD:C_0603_1608Metric -> ControlBoard:C_0603_1608Metric
- C22: renamed from C16; footprint Capacitor_SMD:C_0603_1608Metric -> ControlBoard:C_0603_1608Metric
- C23: renamed from C14; footprint Capacitor_SMD:C_0603_1608Metric -> ControlBoard:C_0603_1608Metric
- C24: renamed from C23; footprint Capacitor_SMD:C_0603_1608Metric -> ControlBoard:C_0603_1608Metric
- C25: renamed from C15; footprint Capacitor_SMD:C_0603_1608Metric -> ControlBoard:C_0603_1608Metric
- C26: renamed from C30; footprint Capacitor_SMD:C_0603_1608Metric -> ControlBoard:C_0603_1608Metric
- C27: renamed from C31; footprint Capacitor_SMD:C_0603_1608Metric -> ControlBoard:C_0603_1608Metric
- C28: renamed from C32; footprint Capacitor_SMD:C_0603_1608Metric -> ControlBoard:C_0603_1608Metric
- C29: renamed from C33; footprint Capacitor_SMD:C_0603_1608Metric -> ControlBoard:C_0603_1608Metric
- C30: renamed from C34; footprint Capacitor_SMD:C_0603_1608Metric -> ControlBoard:C_0603_1608Metric
- C31: renamed from C35; footprint Capacitor_SMD:C_0603_1608Metric -> ControlBoard:C_0603_1608Metric
- C32: renamed from C36; footprint Capacitor_SMD:C_0603_1608Metric -> ControlBoard:C_0603_1608Metric
- C33: renamed from C37; footprint Capacitor_SMD:C_0603_1608Metric -> ControlBoard:C_0603_1608Metric
- C34: renamed from C38; footprint Capacitor_SMD:C_0603_1608Metric -> ControlBoard:C_0603_1608Metric
- C35: renamed from C39; footprint Capacitor_SMD:C_0603_1608Metric -> ControlBoard:C_0603_1608Metric
- C36: renamed from C40; footprint Capacitor_SMD:C_0603_1608Metric -> ControlBoard:C_0603_1608Metric
- C37: renamed from C41; footprint Capacitor_SMD:C_0603_1608Metric -> ControlBoard:C_0603_1608Metric
- C38: renamed from C42; footprint Capacitor_SMD:C_0603_1608Metric -> ControlBoard:C_0603_1608Metric
- C39: renamed from C43; footprint Capacitor_SMD:C_0603_1608Metric -> ControlBoard:C_0603_1608Metric
- C40: renamed from C44; footprint Capacitor_SMD:C_0603_1608Metric -> ControlBoard:C_0603_1608Metric
- C41: renamed from C45; value 10uF -> 680uF; footprint Capacitor_SMD:C_0603_1608Metric -> ControlBoard:Cap_SinkBoard
- C42: renamed from C46; footprint Capacitor_SMD:C_0603_1608Metric -> ControlBoard:C_0603_1608Metric
- C43: renamed from C47; footprint Capacitor_SMD:C_0603_1608Metric -> ControlBoard:C_0603_1608Metric
- C44: renamed from C48; footprint Capacitor_SMD:C_0603_1608Metric -> ControlBoard:C_0603_1608Metric
- C45: renamed from C49; footprint Capacitor_SMD:C_0603_1608Metric -> ControlBoard:C_0603_1608Metric
- C46: renamed from C50; footprint Capacitor_SMD:C_0603_1608Metric -> ControlBoard:C_0603_1608Metric
- C47: renamed from C51; footprint Capacitor_SMD:C_0603_1608Metric -> ControlBoard:C_0603_1608Metric
- C48: renamed from C52; footprint Capacitor_SMD:C_0603_1608Metric -> ControlBoard:C_0603_1608Metric
- C49: renamed from C53; footprint Capacitor_SMD:C_0603_1608Metric -> ControlBoard:C_0603_1608Metric
- C50: renamed from C54; footprint Capacitor_SMD:C_0603_1608Metric -> ControlBoard:C_0603_1608Metric
- C51: renamed from C55; footprint Capacitor_SMD:C_0603_1608Metric -> ControlBoard:C_0603_1608Metric
- C52: renamed from C56; footprint Capacitor_SMD:C_0603_1608Metric -> ControlBoard:C_0603_1608Metric
- C53: renamed from C57; footprint Capacitor_SMD:C_0603_1608Metric -> ControlBoard:C_0603_1608Metric
- C54: renamed from C58; footprint Capacitor_SMD:C_0603_1608Metric -> ControlBoard:C_0603_1608Metric
- C55: renamed from C59; footprint Capacitor_SMD:C_0603_1608Metric -> ControlBoard:C_0603_1608Metric
- C56: renamed from C60; footprint Capacitor_SMD:C_0603_1608Metric -> ControlBoard:C_0603_1608Metric
- C57: renamed from C61; footprint Capacitor_SMD:C_0603_1608Metric -> ControlBoard:C_0603_1608Metric
- C58: renamed from C62; footprint Capacitor_SMD:C_0603_1608Metric -> ControlBoard:C_0603_1608Metric
- C59: renamed from C63; footprint Capacitor_SMD:C_0603_1608Metric -> ControlBoard:C_0603_1608Metric
- C60: renamed from C64; footprint Capacitor_SMD:C_0603_1608Metric -> ControlBoard:C_0603_1608Metric
- C61: renamed from C65; footprint Capacitor_SMD:C_0603_1608Metric -> ControlBoard:C_0603_1608Metric
- C62: renamed from C66; footprint Capacitor_SMD:C_0603_1608Metric -> ControlBoard:C_0603_1608Metric
- C63: renamed from C67; footprint Capacitor_SMD:C_0603_1608Metric -> ControlBoard:C_0603_1608Metric
- C64: renamed from C68; footprint Capacitor_SMD:C_0603_1608Metric -> ControlBoard:C_0603_1608Metric
- C65: renamed from C71; footprint Capacitor_SMD:C_0603_1608Metric -> ControlBoard:C_0603_1608Metric
- C66: renamed from C73; footprint Capacitor_SMD:C_0603_1608Metric -> ControlBoard:C_0603_1608Metric; moved to B.Cu
- C69: value 100nF -> 18pF; footprint Capacitor_SMD:C_0603_1608Metric -> ControlBoard:C_0603_1608Metric
- C7: footprint Capacitor_SMD:C_0603_1608Metric -> ControlBoard:C_0603_1608Metric; moved to F.Cu
- C70: value 220nF -> 100nF; footprint Capacitor_SMD:C_0603_1608Metric -> ControlBoard:C_0603_1608Metric; moved to B.Cu
- D1, D2: footprint LED_SMD:LED_0603_1608Metric -> ControlBoard:LED_0603_1608Metric
- J1: footprint Connector_Coaxial:SMA_Molex_73251-2200_Horizontal -> ControlBoard:SMA_Molex_73251-2200_Horizontal
- J2: footprint Connector_JST:JST_PH_S8B-PH-K_1x08_P2.00mm_Horizontal -> ControlBoard:JST_PH_S8B-PH-K_1x08_P2.00mm_Horizontal
- L1: footprint Inductor_SMD:L_0603_1608Metric -> ControlBoard:L_0603_1608Metric
- L2: footprint Inductor_SMD:L_Abracon_ASPI-0630LR -> ControlBoard:L_Abracon_ASPI-0630LR
- LCD1: footprint MM32_Library:TFT-LCD1.8inch -> ControlBoard:TFT-LCD1.8inch
- M1: footprint MM32_Library:Gernic_Debugger -> ControlBoard:Gernic_Debugger
- R1: renamed from R8; footprint Resistor_SMD:R_0603_1608Metric -> ControlBoard:R_0603_1608Metric
- R19: renamed from R9; value 2.2kR -> 10kR; footprint Resistor_SMD:R_0603_1608Metric -> ControlBoard:R_0603_1608Metric
- R2: renamed from R1; footprint Resistor_SMD:R_0603_1608Metric -> ControlBoard:R_0603_1608Metric
- R20: renamed from R10; value 2.2kR -> 10kR; footprint Resistor_SMD:R_0603_1608Metric -> ControlBoard:R_0603_1608Metric
- R3: renamed from R2; footprint Resistor_SMD:R_0603_1608Metric -> ControlBoard:R_0603_1608Metric
- R4: renamed from R3; footprint Resistor_SMD:R_0603_1608Metric -> ControlBoard:R_0603_1608Metric
- R5: renamed from R4; footprint Resistor_SMD:R_0603_1608Metric -> ControlBoard:R_0603_1608Metric
- R6: renamed from R5; footprint Resistor_SMD:R_0603_1608Metric -> ControlBoard:R_0603_1608Metric
- R7: renamed from R6; footprint Resistor_SMD:R_0603_1608Metric -> ControlBoard:R_0603_1608Metric
- R8: renamed from R7; footprint Resistor_SMD:R_0603_1608Metric -> ControlBoard:R_0603_1608Metric
- SW1: footprint Button_Switch_SMD:SW_DIP_SPSTx02_Slide_Copal_CHS-02B_W7.62mm_P1.27mm -> ControlBoard:SW_DIP_SPSTx02_Slide_Copal_CHS-02B_W7.62mm_P1.27mm
- U1: footprint RF_GPS:ublox_NEO -> ControlBoard:ublox_NEO
- U10: renamed from U12; footprint Package_SO:TSSOP-16_4.4x5mm_P0.65mm -> ControlBoard:TSSOP-16_4.4x5mm_P0.65mm
- U12: renamed from U14; footprint Package_SO:SOP-8_3.9x4.9mm_P1.27mm -> ControlBoard:SOP-8_3.9x4.9mm_P1.27mm
- U13: value HMC5883L -> MM32SPIN27PS; footprint MM32_Library:QFN-16_3x3_Pitch0.5mm -> Package_QFP:LQFP-64_10x10mm_P0.5mm; moved to B.Cu
- U2: footprint Package_SO:TSSOP-16_4.4x5mm_P0.65mm -> ControlBoard:TSSOP-16_4.4x5mm_P0.65mm
- U3: footprint MM32_Library:ADIS16470AMLZ -> ControlBoard:ADIS16470AMLZ
- U4: renamed from U5; footprint Package_TO_SOT_SMD:SOT-23-5 -> ControlBoard:SOT-23-5
- U5: renamed from U4; footprint MM32_Library:SIP-4_B0505S_1WR3 -> ControlBoard:SIP-4_B0505S_1WR3
- U6: renamed from U8; footprint Package_QFP:LQFP-144_20x20mm_P0.5mm -> ControlBoard:LQFP-144_20x20mm_P0.5mm
- U7: renamed from U9; footprint Package_TO_SOT_SMD:SOT-23-5 -> ControlBoard:SOT-23-5
- U8: renamed from U10; footprint Package_TO_SOT_SMD:SOT-23-5 -> ControlBoard:SOT-23-5
- U9: renamed from U11; footprint Package_QFP:LQFP-144_20x20mm_P0.5mm -> ControlBoard:LQFP-144_20x20mm_P0.5mm
- Y1, Y2: footprint Crystal:Crystal_SMD_3225-4Pin_3.2x2.5mm -> ControlBoard:Crystal_SMD_3225-4Pin_3.2x2.5mm
- moved C69 40.4 mm to (164.7, 117.1)
- moved C70 36.4 mm to (162.3, 110.0)
- moved C20 25.2 mm to (165.6, 106.6), turned to 90 degrees
- moved U13 24.2 mm to (173.5, 112.3)
- moved C14 22.5 mm to (191.3, 95.8), turned to 180 degrees
- moved C13 21.1 mm to (193.4, 111.8), turned to 90 degrees
- moved C16 19.9 mm to (186.4, 94.5), turned to 90 degrees
- moved C66 18.9 mm to (180.6, 79.8)
- moved C24 18.0 mm to (168.0, 110.8), turned to 0 degrees
- moved C65 17.4 mm to (180.5, 107.1), turned to 180 degrees
- moved C17 16.0 mm to (190.2, 120.8), turned to 0 degrees
- moved C19 14.5 mm to (191.3, 101.9)
- moved U4 14.0 mm to (168.1, 113.8), turned to 90 degrees
- moved C18 13.4 mm to (193.4, 115.4), turned to -90 degrees
- moved C15 12.5 mm to (171.5, 118.5), turned to 0 degrees
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Connections:
- C65 pad 1: Net-(C71-Pad1) -> +3.3VADC
- C65 pad 2: GND -> GNDA
- C69 pad 1: +3.3VP -> /Coprocessor/XTAL_IN
- C69 pad 2: GND -> GNDA
- C70 pad 1: Net-(C70-Pad1) -> /Coprocessor/RST
- C70 pad 2: Net-(C70-Pad2) -> GNDA
- R19 pad 2: /Compass&Storage/IIC_SDA -> /Compass&Storage/EEPROM_SDA
- R20 pad 2: /Compass&Storage/IIC_SCL -> /Compass&Storage/EEPROM_SCL
- U12 pad 5: /Compass&Storage/IIC_SDA -> /Compass&Storage/EEPROM_SDA
- U12 pad 6: /Compass&Storage/IIC_SCL -> /Compass&Storage/EEPROM_SCL
- U13 pad 1: /Compass&Storage/IIC_SCL -> unconnected-(U13-Pad1)
- U13 pad 10: Net-(C71-Pad1) -> unconnected-(U13-Pad10)
- U13 pad 11: GND -> unconnected-(U13-Pad11)
- U13 pad 12: Net-(C70-Pad1) -> GNDA
- U13 pad 13: +3.3VP -> +3.3VADC
- U13 pad 15: /Compass&Storage/COMPASS_RDY -> unconnected-(U13-Pad15)
- U13 pad 16: /Compass&Storage/IIC_SDA -> unconnected-(U13-Pad16)
- U13 pad 2: +3.3VP -> unconnected-(U13-Pad2)
- U13 pad 4: +3.3VP -> unconnected-(U13-Pad4)
- U13 pad 5: unconnected-(U13-Pad5) -> /Coprocessor/XTAL_IN
- U13 pad 6: unconnected-(U13-Pad6) -> /Coprocessor/XTAL_OUT
- U13 pad 7: unconnected-(U13-Pad7) -> /Coprocessor/RST
- U13 pad 8: Net-(C70-Pad2) -> unconnected-(U13-Pad8)
- U13 pad 9: GND -> unconnected-(U13-Pad9)
- U3 pad F3: /IMU/RST -> /Coprocessor/PC7
- U3 pad G3: /IMU/CS -> /Coprocessor/SPI2_NSS
- U3 pad G6: /IMU/DIN -> /Coprocessor/SPI2_MOSI
- U3 pad H3: /IMU/DOUT -> /Coprocessor/SPI2_MISO
- U3 pad H6: /IMU/SCLK -> /Coprocessor/SPI2_CLK
- U3 pad J6: /IMU/DR -> /Coprocessor/PC6
- U6 pad 1: /LCD&GPS/LCD_CLK -> /LCD&GPS/TOUCH_CLK
- U6 pad 10: /LCD&GPS/LCD_RST -> unconnected-(U6-Pad10)
- U6 pad 114: unconnected-(U8-Pad114) -> /Coprocessor/UART1_RX
- U6 pad 115: unconnected-(U8-Pad115) -> /Coprocessor/UART1_TX
- U6 pad 118: /IMU/IMU_CLK -> /LCD&GPS/LCD_CLK
- U6 pad 119: /IMU/IMU_MISO -> unconnected-(U6-Pad119)
- U6 pad 122: /IMU/IMU_MOSI -> /LCD&GPS/LCD_MOSI
- U6 pad 123: /IMU/IMU_CS -> /LCD&GPS/LCD_CS
- U6 pad 124: /IMU/IMU_RST -> unconnected-(U6-Pad124)
- U6 pad 125: /IMU/IMU_DR -> unconnected-(U6-Pad125)
- U6 pad 133: /LCD&GPS/TOUCH_CLK -> unconnected-(U6-Pad133)
- U6 pad 134: /LCD&GPS/TOUCH_MISO -> unconnected-(U6-Pad134)
- U6 pad 135: /LCD&GPS/TOUCH_MOSI -> unconnected-(U6-Pad135)
- U6 pad 141: /LCD&GPS/TOUCH_CS -> /LCD&GPS/LCD_RST
- U6 pad 142: /LCD&GPS/TOUCH_IT -> /LCD&GPS/LCD_A0
- U6 pad 2: /LCD&GPS/LCD_CS -> /LCD&GPS/TOUCH_CS
- U6 pad 3: /LCD&GPS/LCD_A0 -> /LCD&GPS/TOUCH_IT
- U6 pad 4: unconnected-(U8-Pad4) (its old number) -> /LCD&GPS/TOUCH_MISO
- U6 pad 5: /LCD&GPS/LCD_MOSI -> /LCD&GPS/TOUCH_MOSI
- U6 pad 79: /Compass&Storage/IIC_SCL -> /Compass&Storage/EEPROM_SCL
- U6 pad 80: /Compass&Storage/IIC_SDA -> /Compass&Storage/EEPROM_SDA
- U6 pad 81: /Compass&Storage/COMPASS_RDY -> unconnected-(U6-Pad81)
Routing:
- net +3.3VADC: track 76.9 -> 150.5 mm, vias 6 -> 10
- net /Coprocessor/UART_TX: track 0.00 -> 37.9 mm
- net /Coprocessor/UART_RX: track 0.00 -> 37.7 mm
- net /Compass&Storage/IIC_SCL: track 27.0 -> 0.00 mm, vias 1 -> 0
- net /Compass&Storage/COMPASS_RDY: track 26.1 -> 0.00 mm, vias 1 -> 0
- net /Compass&Storage/Compass_DR: track 0.00 -> 26.0 mm, vias 0 -> 3
- net /Compass&Storage/IIC_SDA: track 25.9 -> 0.00 mm, vias 1 -> 0
- net +3.3VP: track 199.5 -> 174.6 mm, vias 31 -> 29
- net /Compass&Storage/Compass_MISO: track 0.00 -> 23.8 mm, vias 0 -> 1
- net /Compass&Storage/Compass_CLK: track 0.00 -> 23.2 mm, vias 0 -> 1
- net /Compass&Storage/Compass_CS: track 0.00 -> 23.0 mm, vias 0 -> 1
- net /Compass&Storage/Compass_MOSI: track 0.00 -> 23.0 mm, vias 0 -> 1
- net /IMU/SCLK: track 21.1 -> 0.00 mm, vias 2 -> 0
- net /IMU/DIN: track 19.3 -> 0.00 mm, vias 2 -> 0
- net /IMU/IMU_DR: track 19.3 -> 0.00 mm, vias 1 -> 0
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- added copper zone on B.Cu, net GNDA
Other:
- outline, holes or cut-outs redrawn
- rule pad_to_mask_clearance: 0 -> 0.06
- board text added: "0.1500 mm / 0.1500 mm"
- board text added: "Designed By LaoZhu"
- board text added: "G R T R T G P 5V"
- board text added: "GDUT 2022/03/03"
- board text added: "GND"
- board text added: "VICG"
- board text added: "Version 1.3.3"
- board text added: "X"
- board text added: "Y"
- board text added: "是"
- board text added: "电介质"
- board text removed: "2022/02/09"
- board text removed: "Designed By"
- board text removed: "GDUT"
- board text removed: "LaoZhu"
- board text removed: "Version 1.2.3"

Commit message: Adjust PCB routing and copper laying, export schematic PDF file.
Routing:
- net +3.3VADC: track 150.5 -> 148.5 mm
- net +5V: track 151.2 -> 149.7 mm
- net +3.3VP: track 174.6 -> 175.3 mm
- net /LCD&GPS/LCD_CLK: track 32.7 -> 33.2 mm
- net GND: vias 73 -> 84
Other:
- rule pad_to_mask_clearance: 0.06 -> 0

Commit message: Update the ControlBoard's PCB and export the interactive BOM.
Parts:
- removed L2: 6.8uH, ControlBoard:L_Abracon_ASPI-0630LR
- removed Y3: 8MHz, ControlBoard:Crystal_SMD_3225-4Pin_3.2x2.5mm
- added G***: LOGO, LOGO, F.Cu at (175.5, 81.2)
- added J4: BAT_CR1220, ControlBoard:BAT_CR1220, F.Cu at (185.2, 101.0)
- added P1: USB_C_Plug_USB2.0, ControlBoard:USB_C_Receptacle_HRO_TYPE-C-31-M-12, F.Cu at (117.8, 76.5)
- added R24: 1kR, ControlBoard:R_0603_1608Metric, F.Cu at (188.3, 108.8)
- added R25: 10kR, ControlBoard:R_0603_1608Metric, F.Cu at (179.0, 102.9)
- added U15: W25Q64, Package_SO:SOIC-8_5.23x5.23mm_P1.27mm, B.Cu at (134.0, 108.6)
- C13, C42, C45: moved to B.Cu
- C19, C67, R1: moved to F.Cu
- C21, C23: value 10uF -> 100nF
- C22: value 100nF -> 22uF; moved to B.Cu
- C24: value 22uF -> 100nF
- C25: value 10uF -> 2.2nF
- C68: value 18pF -> 10uF; moved to F.Cu
- C69: value 18pF -> 100nF; moved to F.Cu
- U14: value π131M31 -> CH372C; footprint ControlBoard:SOIC-16_3.9x9.9mm_P1.27mm -> Package_SO:SSOP-20_4.4x6.5mm_P0.65mm; moved to F.Cu
- U3: value ADIS16470AMLZ -> ADXL350BCEZ; footprint ControlBoard:ADIS16470AMLZ -> ControlBoard:LGA-16-3.35mm_3.53mm; moved to B.Cu
- U5: value B0505S-1WR3 -> MPU-6050; footprint ControlBoard:SIP-4_B0505S_1WR3 -> Sensor_Motion:InvenSense_QFN-24_4x4mm_P0.5mm
- moved U14 63.8 mm to (118.6, 86.1), turned to -90 degrees
- moved C68 63.4 mm to (111.8, 75.9), turned to 90 degrees
- moved C67 56.5 mm to (123.6, 81.9), turned to 0 degrees
- moved C69 49.7 mm to (123.2, 89.8), turned to -90 degrees
- moved D2 41.3 mm to (159.9, 75.1)
- moved R6 41.3 mm to (159.9, 78.2)
- moved R3 40.4 mm to (161.9, 78.2)
- moved D1 40.4 mm to (161.9, 75.1)
- moved L1 39.9 mm to (183.6, 121.6), turned to 0 degrees
- moved C22 34.0 mm to (185.5, 87.5)
- moved SW1 32.8 mm to (106.4, 110.1)
- moved C19 32.6 mm to (161.8, 115.9), turned to 90 degrees
- moved J1 31.6 mm to (194.3, 112.8)
- moved C13 29.3 mm to (186.2, 83.4)
- moved C21 26.8 mm to (184.8, 86.5), turned to -90 degrees
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Connections:
- C13 pad 2: GNDA -> GND
- C14 pad 2: GNDA -> GND
- C15 pad 2: GNDA -> GND
- C16 pad 2: GNDA -> GND
- C17 pad 2: GNDA -> GND
- C18 pad 2: GNDA -> GND
- C19 pad 2: GNDA -> GND
- C20 pad 2: GNDA -> GND
- C21 pad 1: +5V -> +3.3VADC
- C22 pad 1: +5VA -> +3.3VADC
- C22 pad 2: GNDA -> GND
- C23 pad 1: Net-(C23-Pad1) -> +3.3VADC
- C24 pad 1: +3.3VADC -> Net-(C24-Pad1)
- C24 pad 2: GNDA -> GND
- C25 pad 1: +5VA -> Net-(C25-Pad1)
- C25 pad 2: GNDA -> GND
- C65 pad 2: GNDA -> GND
- C66 pad 1: +3.3VP -> +3.3VA
- C67 pad 1: +3.3VA -> Net-(C67-Pad1)
- C68 pad 1: /Coprocessor/XTAL_OUT -> +5V
- C68 pad 2: GNDA -> GND
- C69 pad 1: /Coprocessor/XTAL_IN -> +5V
- C69 pad 2: GNDA -> GND
- C70 pad 2: GNDA -> GND
- J3 pad 4: GNDA -> GND
- R1 pad 1: GND -> +3.3VADC
- R1 pad 2: GNDA -> /Coprocessor/IIC_SDA
- R19 pad 1: +3.3VP -> +3.3VA
- R20 pad 1: +3.3VP -> +3.3VA
- R21 pad 1: GNDA -> GND
- R3 pad 1: +3.3VP -> +3.3VA
- R6 pad 1: +3.3VP -> +3.3VA
- R9 pad 2: GNDA -> GND
- U1 pad 22: +3.3VP -> Net-(R24-Pad1)
- U11 pad 19: GNDA -> GND
- U11 pad 2: GNDA -> GND
- U11 pad 20: GNDA -> GND
- U11 pad 22: GNDA -> GND
- U11 pad 23: /Compass&Storage/Compass_DR -> unconnected-(U11-Pad23)
- U11 pad 29: GNDA -> GND
- U11 pad 5: GNDA -> GND
- U12 pad 8: +3.3VP -> +3.3VA
- U13 pad 12: GNDA -> GND
- U13 pad 22: /Compass&Storage/Compass_DR -> unconnected-(U13-Pad22)
- U13 pad 31: GNDA -> GND
- U13 pad 42: /Coprocessor/UART_TX -> /Coprocessor/UART1_TX
- U13 pad 43: /Coprocessor/UART_RX -> /Coprocessor/UART1_RX
- U13 pad 5: /Coprocessor/XTAL_IN -> unconnected-(U13-Pad5)
- U13 pad 51: unconnected-(U13-Pad51) -> /Coprocessor/LED1
- U13 pad 55: unconnected-(U13-Pad55) -> /Coprocessor/IIC_SDA
- U13 pad 56: unconnected-(U13-Pad56) -> /Coprocessor/IIC_CLK
- U13 pad 6: /Coprocessor/XTAL_OUT -> unconnected-(U13-Pad6)
- U13 pad 62: /Coprocessor/LED1 -> unconnected-(U13-Pad62)
- U13 pad 63: GNDA -> GND
- U14 pad 1: +3.3VA -> /Control_MCU/PE6
- U14 pad 10: unconnected-(U14-Pad10) -> /Control_MCU/PF3
- U14 pad 11: unconnected-(U14-Pad11) -> /Control_MCU/PF4
- U14 pad 12: /Coprocessor/UART_TX -> /Control_MCU/PF5
- U14 pad 13: /Coprocessor/UART_RX -> /Control_MCU/PF6
- U14 pad 14: unconnected-(U14-Pad14) -> /Control_MCU/PF7
- U14 pad 15: GNDA -> /Control_MCU/PF8
- U14 pad 16: +3.3VADC -> /Control_MCU/PF9
- U14 pad 2: GND -> /Control_MCU/PF0
- U14 pad 3: unconnected-(U14-Pad3) -> /Control_MCU/PF1
- U14 pad 4: /Coprocessor/UART1_RX -> /Control_MCU/PF2
- U14 pad 5: /Coprocessor/UART1_TX -> Net-(C67-Pad1)
- U14 pad 6: unconnected-(U14-Pad6) -> Net-(P1-PadA6)
- U14 pad 7: unconnected-(U14-Pad7) -> Net-(P1-PadA7)
- U14 pad 9: GNDA -> unconnected-(U14-Pad9)
- U4 pad 1: +5VA -> +5V
- U4 pad 2: GNDA -> GND
- U4 pad 3: +5VA -> +5V
- U5 pad 2: Net-(C23-Pad1) -> (no net)
- U5 pad 3: GNDA -> (no net)
- U5 pad 4: +5VA -> (no net)
- U6 pad 114: /Coprocessor/UART1_RX -> unconnected-(U6-Pad114)
- U6 pad 115: /Coprocessor/UART1_TX -> unconnected-(U6-Pad115)
- U6 pad 34: /Control_MCU/UART6_RX -> /LCD&GPS/GPS_RX
- U6 pad 36: unconnected-(U6-Pad36) -> /Coprocessor/UART1_RX
- U6 pad 37: /Process_MCU/LED1 -> /Coprocessor/UART1_TX
- U6 pad 40: unconnected-(U6-Pad40) -> /Process_MCU/LED1
- U6 pad 77: /LCD&GPS/GPS_RX -> /Control_MCU/UART6_RX
- U9 pad 1: /Control_MCU/LED1 -> unconnected-(U9-Pad1)
- U9 pad 10: unconnected-(U9-Pad10) -> /Control_MCU/PF0
- U9 pad 11: unconnected-(U9-Pad11) -> /Control_MCU/PF1
- U9 pad 12: unconnected-(U9-Pad12) -> /Control_MCU/PF2
- U9 pad 13: unconnected-(U9-Pad13) -> /Control_MCU/PF3
- U9 pad 14: unconnected-(U9-Pad14) -> /Control_MCU/PF4
- U9 pad 15: unconnected-(U9-Pad15) -> /Control_MCU/PF5
- U9 pad 18: unconnected-(U9-Pad18) -> /Control_MCU/PF6
- U9 pad 19: unconnected-(U9-Pad19) -> /Control_MCU/PF7
- U9 pad 20: unconnected-(U9-Pad20) -> /Control_MCU/PF8
- U9 pad 21: unconnected-(U9-Pad21) -> /Control_MCU/PF9
- U9 pad 22: unconnected-(U9-Pad22) -> /Control_MCU/PF10
- U9 pad 26: unconnected-(U9-Pad26) -> /Control_MCU/PC0
- U9 pad 36: unconnected-(U9-Pad36) -> /Control_MCU/LED1
- U9 pad 5: unconnected-(U9-Pad5) -> /Control_MCU/PE6
- U9 pad 81: unconnected-(U9-Pad81) -> /Control_MCU/SPI3_CLK
- U9 pad 82: unconnected-(U9-Pad82) -> /Control_MCU/SPI3_MISO
- U9 pad 85: unconnected-(U9-Pad85) -> /Control_MCU/SPI3_MOSI
- U9 pad 86: unconnected-(U9-Pad86) -> /Control_MCU/SPI3_NSS
Routing:
- net +5V: track 149.7 -> 195.4 mm, vias 11 -> 13
- net /Coprocessor/UART_TX: track 37.9 -> 0.00 mm
- net /Coprocessor/UART_RX: track 37.7 -> 0.00 mm
- net /LCD&GPS/GPS_RX: track 10.8 -> 45.0 mm
- net /Coprocessor/UART1_RX: track 12.5 -> 42.9 mm
- net /Coprocessor/UART1_TX: track 13.7 -> 42.6 mm
- net /Coprocessor/IIC_CLK: track 0.00 -> 28.2 mm, vias 0 -> 2
- net /Coprocessor/IIC_SDA: track 0.00 -> 27.9 mm, vias 0 -> 2
- net /Coprocessor/PC6: track 11.5 -> 37.4 mm
- net /Compass&Storage/Compass_DR: track 26.0 -> 0.00 mm, vias 3 -> 0
- net /Debugger/SEL: track 40.2 -> 14.9 mm
- net +3.3VP: track 175.3 -> 150.3 mm, vias 29 -> 26
- net /Process_MCU/LED1: track 36.1 -> 11.4 mm
- net /Control_MCU/UART6_RX: track 14.1 -> 36.3 mm, vias 0 -> 2
- net /Control_MCU/PC0: track 0.00 -> 20.9 mm, vias 0 -> 1
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- removed copper zone on B.Cu, net GNDA
- removed copper zone on F.Cu, net GNDA
- removed copper zone on In1.Cu, net GNDA
- removed copper zone on In2.Cu, net GNDA
- removed copper zone on F.Cu, net Net-(C23-Pad1)
Other:
- board text added: "Ctrl"
- board text added: "GDUT 2022/04/06"
- board text added: "Proc"
- board text added: "Version 1.5.2"
- board text removed: "GDUT 2022/03/03"
- board text removed: "GND"
- board text removed: "VICG"
- board text removed: "Version 1.3.3"
- board text removed: "X"
- board text removed: "Y"

Commit message: Update control board schematic pdf file.
Other:
- board text added: "V I C G"
Changed lines of the file:
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@@
     (property "Sheetname" "Process_MCU")
     (attr smd)
-    (fp_text reference "C28" (at 0 1.2916) (layer "B.SilkS")
+    (fp_text reference "C28" (at 1.9792 1.0342) (layer "B.SilkS")
       (effects (font (size 1 1) (thickness 0.15)) (justify mirror))
     )
@@
     (property "Sheetname" "Control_MCU")
     (attr smd)
-    (fp_text reference "C54" (at 2.9328 0.0176 180) (layer "B.SilkS")
+    (fp_text reference "C54" (at -0.0172 1.4664 180) (layer "B.SilkS")
       (effects (font (size 1 1) (thickness 0.15)) (justify mirror))
     )
@@
     (property "Sheetname" "LCD&GPS")
     (attr smd)
-    (fp_text reference "C5" (at 2.9328 0.0176 180) (layer "B.SilkS")
+    (fp_text reference "C5" (at -2.5141 0.0176 180) (layer "B.SilkS")
       (effects (font (size 1 1) (thickness 0.15)) (justify mirror))
     )
@@
     (property "Sheetname" "IMU")
     (attr smd)
-    (fp_text reference "C20" (at 0.099 1.299) (layer "B.SilkS")
+    (fp_text reference "C20" (at 2.8 0) (layer "B.SilkS")
       (effects (font (size 1 1) (thickness 0.15)) (justify mirror))
     )
@@
     (property "Sheetname" "LCD&GPS")
     (attr smd)
-    (fp_text reference "C4" (at 2.9328 0.0176 90) (layer "B.SilkS")
+    (fp_text reference "C4" (at 2.5 0 90) (layer "B.SilkS")
       (effects (font (size 1 1) (thickness 0.15)) (justify mirror))
     )
@@
     (fp_line (start 10.25 -9.15) (end 11.65 -9.15) (layer "B.CrtYd") (width 0.05))
     (fp_line (start 9.15 11.65) (end 9.15 10.25) (layer "B.CrtYd") (width 0.05))
-    (fp_line (start 0 -11.65) (end 9.15 -11.65) (layer "B.CrtYd") (width 0.05))
     (fp_line (start -9.15 11.65) (end -9.15 10.25) (layer "B.CrtYd") (width 0.05))
+    (fp_line (start -10.25 9.15) (end -11.65 9.15) (layer "B.CrtYd") (width 0.05))
     (fp_line (start 11.65 -9.15) (end 11.65 0) (layer "B.CrtYd") (width 0.05))
     (fp_line (start 0 -11.65) (end -9.15 -11.65) (layer "B.CrtYd") (width 0.05))
     (fp_line (start 10.25 -10.25) (end 10.25 -9.15) (layer "B.CrtYd") (width 0.05))
     (fp_line (start -10.25 10.25) (end -10.25 9.15) (layer "B.CrtYd") (width 0.05))
-    (fp_line (start -10.25 9.15) (end -11.65 9.15) (layer "B.CrtYd") (width 0.05))
+    (fp_line (start 0 -11.65) (end 9.15 -11.65) (layer "B.CrtYd") (width 0.05))
     (fp_line (start 9.15 10.25) (end 10.25 10.25) (layer "B.CrtYd") (width 0.05))
     (fp_line (start -11.65 -9.15) (end -11.65 0) (layer "B.CrtYd") (width 0.05))
@@
     (property "Sheetname" "Process_MCU")
     (attr smd)
-    (fp_text reference "C39" (at 2.9328 0.0176) (layer "B.SilkS")
+    (fp_text reference "C39" (at -2.8 0) (layer "B.SilkS")
       (effects (font (size 1 1) (thickness 0.15)) (justify mirror))
     )
@@
     (property "Sheetname" "Flash&USB")
     (attr smd)
-    (fp_text reference "U15" (at 0 3.56) (layer "B.SilkS")
+    (fp_text reference "U15" (at 0 -3.7) (layer "B.SilkS")
       (effects (font (size 1 1) (thickness 0.15)) (justify mirror))
     )
@@
     (property "Sheetname" "Control_MCU")
     (attr smd)
-    (fp_text reference "C62" (at 0.0724 1.2954 270) (layer "B.SilkS")
+    (fp_text reference "C62" (at 2.7484 0.0864 270) (layer "B.SilkS")
       (effects (font (size 1 1) (thickness 0.15)) (justify mirror))
     )
@@
     (property "Sheetname" "Coprocessor")
     (attr smd)
-    (fp_text reference "R23" (at -1.23 -2.953) (layer "B.SilkS")
+    (fp_text reference "R23" (at -2.8 0) (layer "B.SilkS")
       (effects (font (size 1 1) (thickness 0.15)) (justify mirror))
     )
@@
     (property "Sheetname" "Coprocessor")
     (attr smd)
-    (fp_text reference "C70" (at -1.086 1.243) (layer "B.SilkS")
+    (fp_text reference "C70" (at 2.8 0) (layer "B.SilkS")
       (effects (font (size 1 1) (thickness 0.15)) (justify mirror))
     )
@@
     (effects (font (size 1.5 1.5) (thickness 0.3)))
   )
+  (gr_text "V I C G" (at 164.9298 118.9266) (layer "F.SilkS")
+    (effects (font (size 1.2 1.2) (thickness 0.2)))
+  )
   (gr_text "GDUT 2022/04/06" (at 179.4798 74.9766) (layer "F.Mask")

Commit message: The main control board circuit modified the CH372C package, changed the serial port of the GPS and ControlMCU back, and moved the components a bit towards the middle so that they could be screwed on.
Parts:
- U14: footprint Package_SO:SSOP-20_4.4x6.5mm_P0.65mm -> Package_SO:SSOP-20_5.3x7.2mm_P0.65mm
- moved C43 20.7 mm to (109.3, 98.6)
- moved C6 3.68 mm to (119.3, 96.0)
- moved C69 3.45 mm to (122.2, 93.1), turned to 0 degrees
- moved C64 1.89 mm to (110.5, 113.7), turned to 90 degrees
- moved J2 1.21 mm to (110.2, 81.1)
- moved U14 1.00 mm to (118.6, 87.1)
- moved C2 0.94 mm to (119.3, 94.5)
Connections:
- U6 pad 34: /LCD&GPS/GPS_RX -> /Control_MCU/UART6_RX
- U6 pad 77: /Control_MCU/UART6_RX -> /LCD&GPS/GPS_RX
Routing:
- net /Control_MCU/UART6_RX: track 36.3 -> 13.9 mm
- net /LCD&GPS/GPS_RX: track 45.0 -> 28.2 mm
- net +3.3VP: track 150.3 -> 153.8 mm, vias 26 -> 23
- net +5V: track 195.4 -> 192.5 mm
- net /Control_MCU/PF4: track 18.8 -> 20.6 mm
- net /Control_MCU/PF5: track 18.9 -> 20.7 mm
- net /Control_MCU/PF6: track 19.9 -> 21.6 mm
- net /Control_MCU/PF7: track 20.1 -> 21.6 mm
- net /Control_MCU/PF8: track 20.1 -> 21.4 mm
- net /Control_MCU/PF9: track 20.2 -> 21.3 mm
- net /Control_MCU/PF0: track 8.77 -> 9.89 mm
- net /Control_MCU/PF2: track 12.3 -> 13.3 mm
- net /Control_MCU/PF3: track 17.2 -> 18.2 mm
- net /Control_MCU/PF10: track 20.2 -> 21.2 mm
- net /Control_MCU/PF1: track 10.5 -> 11.4 mm
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Other:
- board text added: "GDUT 2022/04/17"
- board text added: "Version 1.5.3"
- board text added: "X"
- board text added: "Y"
- board text removed: "GDUT 2022/04/06"
- board text removed: "Version 1.5.2"
