File: circuit/control_board/project.kicad_pcb (KiCad board)
At the start: 4 copper layers, 95 x 50 mm, 125 parts, among them J1 ANT, J2 Conn_01x08, J3 Conn_01x04, J4 BAT_CR1220, M1 Debugger, P1 USB_C_Plug_USB2.0, SW1 SW_DIP_x02, U1 TAU1201, U10 CH440R, U11 RM3100_13156, U12 AT24C02, U13 MM32SPIN27PS, U14 CH372C, U15 W25Q64, U2 XPT2046TS, U3 ADXL350BCEZ, U4 HX9193, U5 MPU-6050, U6 MM32F3277G9P, U7 HX9193, U8 HX9193, U9 MM32F3277G9P, Y1 8MHz, Y2 8MHz

Commit message: Updated the main control board circuit to change the GNSS feed line from microstrip line to ribbon line.
Routing:
- net GND: track 0.00 -> 11.2 mm, vias 128 -> 119
- net Net-(J1-Pad1): track 16.5 -> 16.1 mm, vias 0 -> 1
Other:
- board text added: "GDUT 2022/04/21"
- board text removed: "GDUT 2022/04/17"

Commit message: Slightly modify the ControlBoard package
Parts:
- U13: footprint Package_QFP:LQFP-64_10x10mm_P0.5mm -> ControlBoard:LQFP-64_10x10mm_P0.5mm
- U14: footprint Package_SO:SSOP-20_5.3x7.2mm_P0.65mm -> ControlBoard:SSOP-20_5.3x7.2mm_P0.65mm
- U15: footprint Package_SO:SOIC-8_5.23x5.23mm_P1.27mm -> ControlBoard:SOIC-8_5.23x5.23mm_P1.27mm
- U5: footprint Sensor_Motion:InvenSense_QFN-24_4x4mm_P0.5mm -> ControlBoard:InvenSense_QFN-24_4x4mm_P0.5mm
Routing:
- net GND: track 11.2 -> 20.3 mm
Other:
- board text added: "GDUT 2022/04/22"
- board text removed: "GDUT 2022/04/21"

Commit message: Modified a portion of the main control board circuit schematic.Added TF card and card reader chip.
Parts:
- removed R10, R11, R12, R13, R14, R15: 121R, ControlBoard:R_0603_1608Metric
- removed R16: PN13101(Z), ControlBoard:PN13101
- removed R17, R18: PN13104(XY), ControlBoard:PN13104
- removed R9: 33kR, ControlBoard:R_0603_1608Metric
- removed U11: RM3100_13156, ControlBoard:QFN-28-1EP_4x4mm_P0.4mm_EP2.4x2.4mm
- added J5: Conn_01x06, Connector_JST:JST_GH_SM06B-GHS-TB_1x06-1MP_P1.25mm_Horizontal, F.Cu at (195.4, 85.6)
- moved J1 1.28 mm to (193.7, 111.7)
- moved J4 1.22 mm to (185.4, 99.8)
Connections:
- U5 pad 25: GND -> (no net)
Routing:
- net +3.3VADC: track 132.8 -> 115.6 mm, vias 11 -> 9
- net Net-(J1-Pad1): track 16.1 -> 2.97 mm
- net GND: track 20.3 -> 9.14 mm, vias 119 -> 109
- net Net-(R14-Pad2): track 7.47 -> 0.00 mm
- net Net-(R11-Pad2): track 7.05 -> 0.00 mm
- net Net-(R13-Pad2): track 6.42 -> 0.00 mm
- net Net-(R12-Pad2): track 6.32 -> 0.00 mm
- net Net-(R15-Pad2): track 5.66 -> 0.00 mm
- net Net-(R10-Pad2): track 5.16 -> 0.00 mm
- net Net-(R11-Pad1): track 4.96 -> 0.00 mm
- net Net-(R13-Pad1): track 4.42 -> 0.00 mm
- net Net-(R9-Pad1): track 3.29 -> 0.00 mm
- net Net-(R15-Pad1): track 3.18 -> 0.00 mm
- net /Compass&Storage/Compass_MISO: track 43.4 -> 40.5 mm
- net /Compass&Storage/Compass_CS: track 40.6 -> 37.7 mm
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Other:
- board text added: "GDUT 2022/05/23"
- board text added: "Version 1.5.4"
- board text removed: "GDUT 2022/04/22"
- board text removed: "Version 1.5.3"

Commit message: Fixed part of the control board circuit and added SD card reading chip.
Parts:
- added U13: CH440R, ControlBoard:TSSOP-16_4.4x5mm_P0.65mm, F.Cu at (204.0, 94.8)
- added U14: MKDV1GCL-AB, ControlBoard:LGA-8060_8, F.Cu at (204.7, 103.7)
- renumbered C24 to C13, C21 to C14, C25 to C15, C13 to C16, C14 to C17, C15 to C18, C16 to C19, C17 to C20, C18 to C21, C19 to C22, C20 to C23, C26 to C24, C27 to C25, C28 to C26, C29 to C27, C30 to C28, C31 to C29, C32 to C30, C33 to C31, C34 to C32, C35 to C33, C36 to C34, C37 to C35, C38 to C36, C39 to C37, C40 to C38, C41 to C39, C42 to C40, C43 to C41, C22 to C42, C23 to C43, C46 to C45, C45 to C46, C70 to C67, J4 to J1, J1 to J2, J2 to J3, J5 to J4, J3 to J5, R24 to R1, R20 to R10, R21 to R11, R1 to R12, R25 to R13, R23 to R14, R22 to R15, R19 to R9, U12 to U11, U13 to U12, U5 to U3, U3 to U4, U6 to U5, U4 to U6
