File: circuit/control_board/IMU.kicad_sch (KiCad schematic)
At the start: 24 parts, among them U3 ADIS16470AMLZ, U4 B0505S-1WR3, U5 HX9193, U6 π131M31, U7 π131M31

Commit message: Modified the circuitry of the main control board to add a microcontroller for reading information from the magnetometer and IMU. Modified the SPI connection port of the Process MCU.
Parts:
- removed C26, C27, C28, C29: 100nF, Capacitor_SMD:C_0603_1608Metric, symbol Device:C
- removed U6, U7: π131M31, Package_SO:SOIC-16_3.9x9.9mm_P1.27mm, symbol MM32_Periph:π131M31
- C13, C14, C15, C16, C17, C18, C19, C20, C21, C22, C23, C24, C25: footprint Capacitor_SMD:C_0603_1608Metric -> ControlBoard:C_0603_1608Metric
- L2: footprint Inductor_SMD:L_Abracon_ASPI-0630LR -> ControlBoard:L_Abracon_ASPI-0630LR
- R8: footprint Resistor_SMD:R_0603_1608Metric -> ControlBoard:R_0603_1608Metric
- U3: footprint MM32_Library:ADIS16470AMLZ -> ControlBoard:ADIS16470AMLZ
- U4: footprint MM32_Library:SIP-4_B0505S_1WR3 -> ControlBoard:SIP-4_B0505S_1WR3
- U5: footprint Package_TO_SOT_SMD:SOT-23-5 -> ControlBoard:SOT-23-5
Connections:
- net CS is gone; now on net IMU_CS: U3.G3 (CS)
- net DIN is gone; now on net IMU_MOSI: U3.G6 (DIN)
- net DOUT is gone; now on net IMU_MISO: U3.H3 (DOUT)
- net DR is gone; now on net IMU_DR: U3.J6 (DR)
- net RST is gone; now on net IMU_RST: U3.F3 (RST)
- net SCLK is gone; now on net IMU_CLK: U3.H6 (SCLK)
Other:
- note removed: "Signal Isolation"
- moved on the sheet: C13, C14, C15, C16, C17, C18, C19, C20, C21, C22, C23, C24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

Commit message: Modify and complete the circuit schematic to make the interface easier to wire.
Parts:
- renumbered C17 to C13, C18 to C14, C19 to C15, C20 to C16, C21 to C17, C22 to C18, C24 to C19, C25 to C20, C13 to C21, C16 to C22, C14 to C23, C23 to C24, C15 to C25, R8 to R1, U5 to U4, U4 to U5
Other:
- title: MM32_Board -> MM32 Control Board

Commit message: Modify the main control board schematic, replace the IMU device and remove the isolation module.
Parts:
- removed C22: 100nF, ControlBoard:C_0603_1608Metric, symbol Device:C
- removed C23, C25: 10uF, ControlBoard:C_0603_1608Metric, symbol Device:C
- removed C24: 22uF, ControlBoard:C_0603_1608Metric, symbol Device:C
- removed L2: 6.8uH, ControlBoard:L_Abracon_ASPI-0630LR, symbol Device:L
- removed R1: 10kR, ControlBoard:R_0603_1608Metric, symbol Device:R
- removed U3: ADIS16470AMLZ, ControlBoard:ADIS16470AMLZ, symbol MM32_Periph:ADIS16470AMLZ
- removed U4: HX9193, ControlBoard:SOT-23-5, symbol MM32_Periph:HX9193
- removed U5: B0505S-1WR3, ControlBoard:SIP-4_B0505S_1WR3, symbol MM32_Periph:B0505S-1WR3
- added U3: ADXL350BCEZ, ControlBoard:LGA-16-3.35mm_3.53mm, symbol MM32_Periph:ADXL350BCEZ
- C21: value 10uF -> 100nF
Connections:
- net +5V is gone; now on net +3.3VADC: C21.1
- net GNDA is gone; now on net GND: C13.2, C14.2, C15.2, C16.2, C17.2, C18.2, C19.2, C20.2
- net +3.3VADC: now also U3.1 (VDDIO), U3.14 (VS)
- net GND: now also U3.13 (GND), U3.16 (GND)
- net IMU_CLK: now also U3.4 (CLK)
- net IMU_CS: now also U3.8 (~{CS})
- net IMU_MISO: now also U3.7 (MISO)
- net IMU_MOSI: now also U3.6 (MOSI)
- new net IMU_INT1: U3.11 (INT1)
- new net IMU_INT2: U3.9 (INT2)
- no-connect marks 1 -> 0
Other:
- note removed: "Power Supply Isolation"
- moved on the sheet: C13, C14, C15, C16, C17, C18, C19, C20

Commit message: Modify the ControlBoard schematic to add useful features.
Parts:
- added C24: 100nF, ControlBoard:C_0603_1608Metric, symbol Device:C
- added C25: 2.2nF, ControlBoard:C_0603_1608Metric, symbol Device:C
- added U5: MPU-6050, Sensor_Motion:InvenSense_QFN-24_4x4mm_P0.5mm, symbol Sensor_Motion:MPU-6050
Connections:
- net +3.3VADC: now also U5.13 (VDD), U5.8 (VDDIO)
- net GND: now also C24.2, C25.2, U5.1 (CLKIN), U5.18 (GND), U5.9 (AD0)
- net IMU_INT2: now also U5.12 (INT); no longer U3.9 (INT2)
- new net: C25.1, U5.20 (CPOUT)
- new net: C24.1, U5.10 (REGOUT)
- new net IIC_CLK: U5.23 (SCL)
- new net IIC_SDA: U5.24 (SDA)
- no-connect marks 0 -> 4
Other:
- moved on the sheet: C21, U3

Commit message: Slightly modify the ControlBoard package
Parts:
- U5: footprint Sensor_Motion:InvenSense_QFN-24_4x4mm_P0.5mm -> ControlBoard:InvenSense_QFN-24_4x4mm_P0.5mm
Changed lines of the file:
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@@
     (property "Reference" "U5" (id 0) (at 107.315 116.84 0))
     (property "Value" "MPU-6050" (id 1) (at 118.745 140.335 0))
-    (property "Footprint" "Sensor_Motion:InvenSense_QFN-24_4x4mm_P0.5mm" (id 2) (at 108.585 142.875 0)
+    (property "Footprint" "ControlBoard:InvenSense_QFN-24_4x4mm_P0.5mm" (id 2) (at 108.585 142.875 0)
       (effects (font (size 1.27 1.27)) hide)
     )
