File: circuit/control_board/IMU.kicad_sch (KiCad schematic)
At the start: 13 parts, among them U3 ADXL350BCEZ, U5 MPU-6050

Commit message: Fixed part of the control board circuit and added SD card reading chip.
Parts:
- renumbered C24 to C13, C21 to C14, C25 to C15, C13 to C16, C14 to C17, C15 to C18, C16 to C19, C17 to C20, C18 to C21, C19 to C22, C20 to C23, U5 to U3, U3 to U4
