File: circuit/control_board/LCD&GPS.kicad_sch (KiCad schematic)
At the start: 17 parts, among them J1 ANT, U1 TAU1201, U2 XPT2046TS

Commit message: Modified the circuitry of the main control board to add a microcontroller for reading information from the magnetometer and IMU. Modified the SPI connection port of the Process MCU.
Parts:
- C1, C10, C11, C12, C2, C3, C4, C5, C6, C7, C8, C9: footprint Capacitor_SMD:C_0603_1608Metric -> ControlBoard:C_0603_1608Metric
- J1: footprint Connector_Coaxial:SMA_Molex_73251-2200_Horizontal -> ControlBoard:SMA_Molex_73251-2200_Horizontal
- L1: footprint Inductor_SMD:L_0603_1608Metric -> ControlBoard:L_0603_1608Metric
- LCD1: footprint MM32_Library:TFT-LCD1.8inch -> ControlBoard:TFT-LCD1.8inch
- U1: footprint RF_GPS:ublox_NEO -> ControlBoard:ublox_NEO
- U2: footprint Package_SO:TSSOP-16_4.4x5mm_P0.65mm -> ControlBoard:TSSOP-16_4.4x5mm_P0.65mm
Changed lines of the file:
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@@
   (title_block
     (title "MM32_Board")
-    (date "2022-02-09")
-    (rev "1.2.3")
+    (date "2022-02-28")
+    (rev "1.3.1")
   )
   (junction (at 198.755 97.79) (diameter 0) (color 0 0 0 0)
@@
       (effects (font (size 1.27 1.27)) (justify left))
     )
-    (property "Footprint" "Capacitor_SMD:C_0603_1608Metric" (id 2) (at 222.5802 109.22 0)
+    (property "Footprint" "ControlBoard:C_0603_1608Metric" (id 2) (at 222.5802 109.22 0)
       (effects (font (size 1.27 1.27)) hide)
     )
@@
       (effects (font (size 1.27 1.27)) (justify left))
     )
-    (property "Footprint" "Capacitor_SMD:C_0603_1608Metric" (id 2) (at 108.9152 135.255 0)
+    (property "Footprint" "ControlBoard:C_0603_1608Metric" (id 2) (at 108.9152 135.255 0)
       (effects (font (size 1.27 1.27)) hide)
     )
@@
       (effects (font (size 1.27 1.27)) (justify left))
     )
-    (property "Footprint" "Capacitor_SMD:C_0603_1608Metric" (id 2) (at 131.7752 135.255 0)
+    (property "Footprint" "ControlBoard:C_0603_1608Metric" (id 2) (at 131.7752 135.255 0)
       (effects (font (size 1.27 1.27)) hide)
     )
@@
       (effects (font (size 1.27 1.27)) (justify right))
     )
-    (property "Footprint" "Connector_Coaxial:SMA_Molex_73251-2200_Horizontal" (id 2) (at 128.905 57.15 0)
+    (property "Footprint" "ControlBoard:SMA_Molex_73251-2200_Horizontal" (id 2) (at 128.905 57.15 0)
       (effects (font (size 1.27 1.27)) hide)
     )
@@
       (effects (font (size 1.27 1.27)) (justify left))
     )
-    (property "Footprint" "Capacitor_SMD:C_0603_1608Metric" (id 2) (at 96.2152 135.255 0)
+    (property "Footprint" "ControlBoard:C_0603_1608Metric" (id 2) (at 96.2152 135.255 0)
       (effects (font (size 1.27 1.27)) hide)
     )
@@
     (property "Reference" "L1" (id 0) (at 123.19 71.12 90))
     (property "Value" "39nH" (id 1) (at 125.095 75.565 90))
-    (property "Footprint" "Inductor_SMD:L_0603_1608Metric" (id 2) (at 124.46 73.66 0)
+    (property "Footprint" "ControlBoard:L_0603_1608Metric" (id 2) (at 124.46 73.66 0)
       (effects (font (size 1.27 1.27)) hide)
     )
@@
     (property "Reference" "U2" (id 0) (at 183.515 127 0))
     (property "Value" "XPT2046TS" (id 1) (at 197.485 152.4 0))
-    (property "Footprint" "Package_SO:TSSOP-16_4.4x5mm_P0.65mm" (id 2) (at 192.405 153.67 0)
+    (property "Footprint" "ControlBoard:TSSOP-16_4.4x5mm_P0.65mm" (id 2) (at 192.405 153.67 0)
       (effects (font (size 1.27 1.27) italic) hide)
     )
@@
       (effects (font (size 1.27 1.27)) (justify left))
     )
-    (property "Footprint" "Capacitor_SMD:C_0603_1608Metric" (id 2) (at 120.3452 135.255 0)
+    (property "Footprint" "ControlBoard:C_0603_1608Metric" (id 2) (at 120.3452 135.255 0)
       (effects (font (size 1.27 1.27)) hide)
     )
@@
       (effects (font (size 1.27 1.27)) (justify left))
     )
-    (property "Footprint" "Capacitor_SMD:C_0603_1608Metric" (id 2) (at 187.0202 109.22 0)
+    (property "Footprint" "ControlBoard:C_0603_1608Metric" (id 2) (at 187.0202 109.22 0)
       (effects (font (size 1.27 1.27)) hide)
     )
@@
     (property "Reference" "LCD1" (id 0) (at 187.325 53.34 0))
     (property "Value" "1.8inch-TFT-LCD" (id 1) (at 193.675 81.28 0))
-    (property "Footprint" "MM32_Library:TFT-LCD1.8inch" (id 2) (at 187.325 53.34 0)
+    (property "Footprint" "ControlBoard:TFT-LCD1.8inch" (id 2) (at 187.325 53.34 0)
       (effects (font (size 1.27 1.27)) hide)
     )
@@
       (effects (font (size 1.27 1.27)) (justify left))
     )
-    (property "Footprint" "Capacitor_SMD:C_0603_1608Metric" (id 2) (at 84.7852 135.255 0)
+    (property "Footprint" "ControlBoard:C_0603_1608Metric" (id 2) (at 84.7852 135.255 0)
       (effects (font (size 1.27 1.27)) hide)
     )
@@
       (effects (font (size 1.27 1.27)) (justify left))
     )
-    (property "Footprint" "Capacitor_SMD:C_0603_1608Metric" (id 2) (at 164.1602 109.22 0)
+    (property "Footprint" "ControlBoard:C_0603_1608Metric" (id 2) (at 164.1602 109.22 0)
       (effects (font (size 1.27 1.27)) hide)
     )
@@
     (property "Reference" "U1" (id 0) (at 90.17 61.595 0))
     (property "Value" "TAU1201" (id 1) (at 111.125 100.965 0))
-    (property "Footprint" "RF_GPS:ublox_NEO" (id 2) (at 106.045 62.23 0)
+    (property "Footprint" "ControlBoard:ublox_NEO" (id 2) (at 106.045 62.23 0)
       (effects (font (size 1.27 1.27)) hide)
     )
@@
       (effects (font (size 1.27 1.27)) (justify left))
     )
-    (property "Footprint" "Capacitor_SMD:C_0603_1608Metric" (id 2) (at 175.5902 109.22 0)
+    (property "Footprint" "ControlBoard:C_0603_1608Metric" (id 2) (at 175.5902 109.22 0)
       (effects (font (size 1.27 1.27)) hide)
     )
@@
       (effects (font (size 1.27 1.27)) (justify left))
     )
-    (property "Footprint" "Capacitor_SMD:C_0603_1608Metric" (id 2) (at 199.7202 109.22 0)
+    (property "Footprint" "ControlBoard:C_0603_1608Metric" (id 2) (at 199.7202 109.22 0)
       (effects (font (size 1.27 1.27)) hide)
     )
@@
       (effects (font (size 1.27 1.27)) (justify left))
     )
-    (property "Footprint" "Capacitor_SMD:C_0603_1608Metric" (id 2) (at 73.3552 135.255 0)
+    (property "Footprint" "ControlBoard:C_0603_1608Metric" (id 2) (at 73.3552 135.255 0)
       (effects (font (size 1.27 1.27)) hide)
     )
@@
       (effects (font (size 1.27 1.27)) (justify left))
     )
-    (property "Footprint" "Capacitor_SMD:C_0603_1608Metric" (id 2) (at 211.1502 109.22 0)
-      (effects (font (size 1.27 1.27)) hide)
-    )
+    (property "Footprint" "ControlBoard:C_0603_1608Metric" (id 2) (at 211.1502 109.22 0)
+      (effects (font (size 1.27 1.27)) hide)
+    )

Commit message: Modify and complete the circuit schematic to make the interface easier to wire.
Other:
- title: MM32_Board -> MM32 Control Board
Changed lines of the file:
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@@
   (paper "A4")
   (title_block
-    (title "MM32_Board")
-    (date "2022-03-02")
-    (rev "1.3.2")
+    (title "MM32 Control Board")
+    (date "2022-03-03")
+    (rev "1.3.3")
   )
   (junction (at 198.755 97.79) (diameter 0) (color 0 0 0 0)

Commit message: Modify the main control board schematic, replace the IMU device and remove the isolation module.
Parts:
- added J4: BAT_CR1220, ControlBoard:BAT_CR1220, symbol MM32_Periph:BAT_CR1220
- added R24: 1kR, ControlBoard:R_0603_1608Metric, symbol Device:R
Connections:
- net +3.3VP: no longer U1.22 (AVDD_BAK)
- net GND: now also J4.2 (N)
- new net: R24.1, U1.22 (AVDD_BAK)
- new net: J4.1 (P), R24.2
Other:
- moved on the sheet: C1, C2, C3, C4, C5, C6, J1

Commit message: Modify the ControlBoard schematic to add useful features.
Other:
- note added: "Flash"
- moved on the sheet: C1, C10, C11, C12, C2, C3, C4, C5, C6, C7, C8, C9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

Commit message: Modified the main control board schematic by deleting the extra wireframes.
Other:
- note removed: "Flash"
- moved on the sheet: C1, C10, C11, C12, C2, C3, C4, C5, C6, C7, C8, C9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
