File: circuit/control_board/LCD&GPS.kicad_sch (KiCad schematic)
At the start: 19 parts, among them J1 ANT, J4 BAT_CR1220, U1 TAU1201, U2 XPT2046TS

Commit message: Fixed part of the control board circuit and added SD card reading chip.
Parts:
- renumbered J4 to J1, J1 to J2, R24 to R1
Changed lines of the file:
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@@
   (symbol (lib_id "power:GND") (at 84.455 110.49 0) (unit 1)
     (in_bom yes) (on_board yes)
-    (property "Reference" "#PWR02" (id 0) (at 84.455 116.84 0)
+    (property "Reference" "#PWR03" (id 0) (at 84.455 116.84 0)
       (effects (font (size 1.27 1.27)) hide)
     )
@@
   (symbol (lib_id "power:GND") (at 133.35 110.49 0) (unit 1)
     (in_bom yes) (on_board yes)
-    (property "Reference" "#PWR06" (id 0) (at 133.35 116.84 0)
+    (property "Reference" "#PWR07" (id 0) (at 133.35 116.84 0)
       (effects (font (size 1.27 1.27)) hide)
     )
@@
   (symbol (lib_id "power:+3.3VP") (at 81.28 54.61 0) (unit 1)
     (in_bom yes) (on_board yes)
-    (property "Reference" "#PWR01" (id 0) (at 85.09 55.88 0)
+    (property "Reference" "#PWR02" (id 0) (at 85.09 55.88 0)
       (effects (font (size 1.27 1.27)) hide)
     )
@@
   (symbol (lib_id "power:+3.3VP") (at 103.505 130.175 0) (unit 1)
     (in_bom yes) (on_board yes)
-    (property "Reference" "#PWR03" (id 0) (at 107.315 131.445 0)
+    (property "Reference" "#PWR04" (id 0) (at 107.315 131.445 0)
       (effects (font (size 1.27 1.27)) hide)
     )
@@
   (symbol (lib_id "power:+3.3VA") (at 210.82 46.355 0) (unit 1)
     (in_bom yes) (on_board yes)
-    (property "Reference" "#PWR014" (id 0) (at 210.82 50.165 0)
+    (property "Reference" "#PWR015" (id 0) (at 210.82 50.165 0)
       (effects (font (size 1.27 1.27)) hide)
     )
@@
   (symbol (lib_id "power:PWR_FLAG") (at 73.025 92.075 90) (unit 1)
     (in_bom yes) (on_board yes) (fields_autoplaced)
-    (property "Reference" "#FLG0101" (id 0) (at 71.12 92.075 0)
+    (property "Reference" "#FLG01" (id 0) (at 71.12 92.075 0)
       (effects (font (size 1.27 1.27)) hide)
     )
@@
   (symbol (lib_id "power:GND") (at 121.285 110.49 0) (unit 1)
     (in_bom yes) (on_board yes)
-    (property "Reference" "#PWR05" (id 0) (at 121.285 116.84 0)
+    (property "Reference" "#PWR06" (id 0) (at 121.285 116.84 0)
       (effects (font (size 1.27 1.27)) hide)
     )
@@
   (symbol (lib_id "Device:R") (at 73.025 97.79 0) (unit 1)
     (in_bom yes) (on_board yes)
-    (property "Reference" "R24" (id 0) (at 74.803 96.6216 0)
+    (property "Reference" "R1" (id 0) (at 74.803 96.6216 0)
       (effects (font (size 1.27 1.27)) (justify left))
     )
@@
   (symbol (lib_id "Connector_Generic:Conn_01x02") (at 130.81 52.07 90) (unit 1)
     (in_bom yes) (on_board yes)
-    (property "Reference" "J1" (id 0) (at 130.175 48.895 90)
+    (property "Reference" "J2" (id 0) (at 130.175 48.895 90)
       (effects (font (size 1.27 1.27)) (justify right))
     )
@@
   (symbol (lib_id "power:GND") (at 208.28 89.535 0) (unit 1)
     (in_bom yes) (on_board yes)
-    (property "Reference" "#PWR012" (id 0) (at 208.28 95.885 0)
+    (property "Reference" "#PWR013" (id 0) (at 208.28 95.885 0)
       (effects (font (size 1.27 1.27)) hide)
     )
@@
   (symbol (lib_id "power:GND") (at 73.025 110.49 0) (unit 1)
     (in_bom yes) (on_board yes)
-    (property "Reference" "#PWR015" (id 0) (at 73.025 116.84 0)
+    (property "Reference" "#PWR01" (id 0) (at 73.025 116.84 0)
       (effects (font (size 1.27 1.27)) hide)
     )
@@
   (symbol (lib_id "power:GND") (at 194.31 114.935 0) (unit 1)
     (in_bom yes) (on_board yes)
-    (property "Reference" "#PWR011" (id 0) (at 194.31 121.285 0)
+    (property "Reference" "#PWR012" (id 0) (at 194.31 121.285 0)
       (effects (font (size 1.27 1.27)) hide)
     )
@@
   (symbol (lib_id "power:+3.3VA") (at 181.61 46.355 0) (unit 1)
     (in_bom yes) (on_board yes)
-    (property "Reference" "#PWR09" (id 0) (at 181.61 50.165 0)
+    (property "Reference" "#PWR010" (id 0) (at 181.61 50.165 0)
       (effects (font (size 1.27 1.27)) hide)
     )
@@
   (symbol (lib_id "power:GND") (at 103.505 147.955 0) (unit 1)
     (in_bom yes) (on_board yes)
-    (property "Reference" "#PWR04" (id 0) (at 103.505 154.305 0)
+    (property "Reference" "#PWR05" (id 0) (at 103.505 154.305 0)
       (effects (font (size 1.27 1.27)) hide)
     )
@@
   (symbol (lib_id "power:+3.3VA") (at 194.31 97.155 0) (unit 1)
     (in_bom yes) (on_board yes)
-    (property "Reference" "#PWR010" (id 0) (at 194.31 100.965 0)
+    (property "Reference" "#PWR011" (id 0) (at 194.31 100.965 0)
       (effects (font (size 1.27 1.27)) hide)
     )
@@
   (symbol (lib_id "power:GND") (at 172.72 161.925 0) (unit 1)
     (in_bom yes) (on_board yes)
-    (property "Reference" "#PWR07" (id 0) (at 172.72 168.275 0)
+    (property "Reference" "#PWR08" (id 0) (at 172.72 168.275 0)
       (effects (font (size 1.27 1.27)) hide)
     )
@@
   (symbol (lib_id "MM32_Periph:BAT_CR1220") (at 70.485 109.22 0) (unit 1)
     (in_bom yes) (on_board yes)
-    (property "Reference" "J4" (id 0) (at 76.2 106.045 0)
+    (property "Reference" "J1" (id 0) (at 76.2 106.045 0)
       (effects (font (size 1.27 1.27)) (justify left))
     )
@@
   (symbol (lib_id "power:+3.3VP") (at 209.55 122.555 0) (unit 1)
     (in_bom yes) (on_board yes)
-    (property "Reference" "#PWR013" (id 0) (at 213.36 123.825 0)
+    (property "Reference" "#PWR014" (id 0) (at 213.36 123.825 0)
       (effects (font (size 1.27 1.27)) hide)
     )
@@
   (symbol (lib_id "power:GND") (at 179.07 89.535 0) (unit 1)
     (in_bom yes) (on_board yes)
-    (property "Reference" "#PWR08" (id 0) (at 179.07 95.885 0)
-      (effects (font (size 1.27 1.27)) hide)
-    )
+    (property "Reference" "#PWR09" (id 0) (at 179.07 95.885 0)
+      (effects (font (size 1.27 1.27)) hide)
+    )
