File: circuit/control_board/project.kicad_sch (KiCad schematic)
At the start: 0 parts

Commit message: Modified the circuitry of the main control board to add a microcontroller for reading information from the magnetometer and IMU. Modified the SPI connection port of the Process MCU.
Other:
- added sheet Coprocessor (Coprocessor.kicad_sch)
- sheet Compass&Storage ports: added COMPASS_SCL, COMPASS_SDA, EEPROM_SCL, EEPROM_SDA; removed IIC_SCL, IIC_SDA
- sheet Process_MCU ports: added SPI2_MISO, UART8_RX, UART8_TX; removed PD12, PE0, PG10, PG9, SPI1_CLK, SPI1_MISO, SPI1_MOSI, SPI3_MISO

Commit message: Update the main control board schematic and replace the magnetometer with RM3100.
Other:
- sheet Compass&Storage ports: added Compass_CLK, Compass_CS, Compass_DR, Compass_MISO, Compass_MOSI; removed COMPASS_RDY, COMPASS_SCL, COMPASS_SDA
- sheet Coprocessor ports: added PC6, SPI2_CLK, SPI2_MISO, SPI2_MOSI, SPI2_NSS; removed IIC1_SCL, IIC1_SDA, PB2
Changed lines of the file:
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@@
   (title_block
     (title "MM32_Board")
-    (date "2022-02-28")
-    (rev "1.3.1")
+    (date "2022-03-02")
+    (rev "1.3.2")
   )
   (wire (pts (xy 80.645 72.39) (xy 91.44 72.39))
@@
     (stroke (width 0) (type default) (color 0 0 0 0))
   )
-  (wire (pts (xy 201.295 91.44) (xy 213.36 91.44))
-    (stroke (width 0) (type default) (color 0 0 0 0))
-  )
   (wire (pts (xy 80.645 99.695) (xy 125.73 99.695))
     (stroke (width 0) (type default) (color 0 0 0 0))
@@
     (stroke (width 0) (type default) (color 0 0 0 0))
   )
+  (wire (pts (xy 201.295 86.995) (xy 213.36 86.995))
+    (stroke (width 0) (type default) (color 0 0 0 0))
+  )
   (wire (pts (xy 114.3 125.095) (xy 125.73 125.095))
     (stroke (width 0) (type default) (color 0 0 0 0))
@@
     (stroke (width 0) (type default) (color 0 0 0 0))
   )
+  (wire (pts (xy 201.295 94.615) (xy 213.36 94.615))
+    (stroke (width 0) (type default) (color 0 0 0 0))
+  )
   (wire (pts (xy 201.295 133.985) (xy 213.36 133.985))
     (stroke (width 0) (type default) (color 0 0 0 0))
@@
     (stroke (width 0) (type default) (color 0 0 0 0))
   )
-  (wire (pts (xy 201.295 96.52) (xy 213.36 96.52))
+  (wire (pts (xy 201.295 89.535) (xy 213.36 89.535))
+    (stroke (width 0) (type default) (color 0 0 0 0))
+  )
+  (wire (pts (xy 201.295 92.075) (xy 213.36 92.075))
     (stroke (width 0) (type default) (color 0 0 0 0))
   )
@@
     (stroke (width 0) (type default) (color 0 0 0 0))
   )
-  (wire (pts (xy 201.295 93.98) (xy 213.36 93.98))
-    (stroke (width 0) (type default) (color 0 0 0 0))
-  )
   (wire (pts (xy 172.085 67.945) (xy 213.36 67.945))
+    (stroke (width 0) (type default) (color 0 0 0 0))
+  )
+  (wire (pts (xy 201.295 97.79) (xy 213.36 97.79))
     (stroke (width 0) (type default) (color 0 0 0 0))
   )
@@
       (effects (font (size 1.27 1.27)) (justify left top) hide)
     )
-    (pin "COMPASS_RDY" output (at 213.36 96.52 180)
-      (effects (font (size 1.27 1.27)) (justify left))
-    )
-    (pin "COMPASS_SDA" bidirectional (at 213.36 93.98 180)
-      (effects (font (size 1.27 1.27)) (justify left))
-    )
-    (pin "COMPASS_SCL" input (at 213.36 91.44 180)
-      (effects (font (size 1.27 1.27)) (justify left))
-    )
     (pin "EEPROM_SCL" input (at 213.36 67.945 180)
       (effects (font (size 1.27 1.27)) (justify left))
@@
       (effects (font (size 1.27 1.27)) (justify left))
     )
-  )
-  (sheet (at 183.515 86.36) (size 17.78 60.325) (fields_autoplaced)
+    (pin "Compass_MISO" output (at 213.36 94.615 180)
+      (effects (font (size 1.27 1.27)) (justify left))
+    )
+    (pin "Compass_MOSI" input (at 213.36 92.075 180)
+      (effects (font (size 1.27 1.27)) (justify left))
+    )
+    (pin "Compass_CS" input (at 213.36 86.995 180)
+      (effects (font (size 1.27 1.27)) (justify left))
+    )
+    (pin "Compass_CLK" input (at 213.36 89.535 180)
+      (effects (font (size 1.27 1.27)) (justify left))
+    )
+    (pin "Compass_DR" output (at 213.36 97.79 180)
+      (effects (font (size 1.27 1.27)) (justify left))
+    )
+  )
+  (sheet (at 183.515 82.55) (size 17.78 64.135) (fields_autoplaced)
     (stroke (width 0.1524) (type solid) (color 0 0 0 0))
     (fill (color 0 0 0 0.0000))
-    (property "Sheet name" "Coprocessor" (id 0) (at 183.515 85.6484 0)
+    (property "Sheet name" "Coprocessor" (id 0) (at 183.515 81.8384 0)
       (effects (font (size 1.27 1.27)) (justify left bottom))
     )
@@
       (effects (font (size 1.27 1.27)) (justify right))
     )
-    (pin "IIC1_SCL" output (at 201.295 91.44 0)
-      (effects (font (size 1.27 1.27)) (justify right))
-    )
-    (pin "IIC1_SDA" bidirectional (at 201.295 93.98 0)
-      (effects (font (size 1.27 1.27)) (justify right))
-    )
-    (pin "PB2" input (at 201.295 96.52 0)
-      (effects (font (size 1.27 1.27)) (justify right))
-    )
     (pin "PA6" input (at 201.295 136.525 0)
       (effects (font (size 1.27 1.27)) (justify right))
@@
     (pin "UART1_TX" output (at 183.515 106.045 180)
       (effects (font (size 1.27 1.27)) (justify left))
+    )
+    (pin "SPI2_NSS" output (at 201.295 86.995 0)
+      (effects (font (size 1.27 1.27)) (justify right))
+    )
+    (pin "SPI2_MISO" input (at 201.295 94.615 0)
+      (effects (font (size 1.27 1.27)) (justify right))
+    )
+    (pin "SPI2_MOSI" output (at 201.295 92.075 0)
+      (effects (font (size 1.27 1.27)) (justify right))
+    )
+    (pin "SPI2_CLK" output (at 201.295 89.535 0)
+      (effects (font (size 1.27 1.27)) (justify right))
+    )
+    (pin "PC6" input (at 201.295 97.79 0)
+      (effects (font (size 1.27 1.27)) (justify right))
     )
   )
@@
       (reference "#PWR047") (unit 1) (value "GNDA") (footprint "")
     )
-    (path "/364540f7-0c58-4618-8ce3-bea6d054cb4e/45d738b8-f947-423e-a920-41cf36d2f4de"
+    (path "/364540f7-0c58-4618-8ce3-bea6d054cb4e/a6775428-a60b-4f97-b264-253b40d8e192"
       (reference "#PWR048") (unit 1) (value "+3.3VADC") (footprint "")
     )
-    (path "/364540f7-0c58-4618-8ce3-bea6d054cb4e/c3b0e43d-9a6a-4a9f-a714-e08909d82f1b"
-      (reference "#PWR049") (unit 1) (value "+3.3VADC") (footprint "")
-    )
-    (path "/364540f7-0c58-4618-8ce3-bea6d054cb4e/d01e7679-d450-4cdf-b461-a0157d013803"
-      (reference "#PWR050") (unit 1) (value "+3.3VADC") (footprint "")
-    )
-    (path "/364540f7-0c58-4618-8ce3-bea6d054cb4e/ed340206-14a4-455b-8ea9-39768ecd0f28"
-      (reference "#PWR051") (unit 1) (value "GNDA") (footprint "")
+    (path "/364540f7-0c58-4618-8ce3-bea6d054cb4e/41bd3c43-0fc4-48be-bb81-2828e90c227c"
+      (reference "#PWR049") (unit 1) (value "GNDA") (footprint "")
+    )
+    (path "/364540f7-0c58-4618-8ce3-bea6d054cb4e/acb8ee8f-b6db-4402-856e-8cc0d08027b9"
+      (reference "#PWR050") (unit 1) (value "GNDA") (footprint "")
     )
     (path "/364540f7-0c58-4618-8ce3-bea6d054cb4e/4fcaf938-c8f0-4844-b67d-d08f4c665a24"
@@
       (reference "C68") (unit 1) (value "100nF") (footprint "ControlBoard:C_0603_1608Metric")
     )
-    (path "/364540f7-0c58-4618-8ce3-bea6d054cb4e/4eb8beb8-e1a5-4685-9ad8-287b2764f530"
-      (reference "C70") (unit 1) (value "220nF") (footprint "ControlBoard:C_0603_1608Metric")
-    )
     (path "/364540f7-0c58-4618-8ce3-bea6d054cb4e/1f65eb4c-5fc9-47ce-9c25-03b83f3814a4"
       (reference "C71") (unit 1) (value "4.7uF") (footprint "ControlBoard:C_0603_1608Metric")
@@
       (reference "R10") (unit 1) (value "10kR") (footprint "ControlBoard:R_0603_1608Metric")
     )
-    (path "/364540f7-0c58-4618-8ce3-bea6d054cb4e/dffb8a34-d8bd-480f-84de-ac0e68ea6ade"
-      (reference "R11") (unit 1) (value "10kR") (footprint "ControlBoard:R_0603_1608Metric")
+    (path "/364540f7-0c58-4618-8ce3-bea6d054cb4e/67b0ea81-3642-46a2-8355-d60793417e57"
+      (reference "R11") (unit 1) (value "121R") (footprint "ControlBoard:R_0603_1608Metric")
     )
     (path "/364540f7-0c58-4618-8ce3-bea6d054cb4e/2275492a-6359-4cd4-b350-01dd400f86da"
-      (reference "R12") (unit 1) (value "10kR") (footprint "ControlBoard:R_0603_1608Metric")
+      (reference "R12") (unit 1) (value "33kR") (footprint "ControlBoard:R_0603_1608Metric")
     )
     (path "/7c560bda-f929-4e77-960a-fa15837ad328/64061abf-a031-4cf4-b8c4-a6b55a09d428"
@@
       (reference "R15") (unit 1) (value "10kR") (footprint "ControlBoard:R_0603_1608Metric")
     )
+    (path "/364540f7-0c58-4618-8ce3-bea6d054cb4e/dc301244-5e61-4fd0-8b27-8600aa8a128e"
+      (reference "R16") (unit 1) (value "121R") (footprint "ControlBoard:R_0603_1608Metric")
+    )
+    (path "/364540f7-0c58-4618-8ce3-bea6d054cb4e/550032b8-ac1a-4add-998e-66bec0bec8ee"
+      (reference "R17") (unit 1) (value "121R") (footprint "ControlBoard:R_0603_1608Metric")
+    )
+    (path "/364540f7-0c58-4618-8ce3-bea6d054cb4e/9968087a-1796-4fc1-a61c-12224b3cfb36"
+      (reference "R18") (unit 1) (value "121R") (footprint "ControlBoard:R_0603_1608Metric")
+    )
+    (path "/364540f7-0c58-4618-8ce3-bea6d054cb4e/4ef7ac11-d4ed-4ace-be37-e21d7f63f921"
+      (reference "R19") (unit 1) (value "121R") (footprint "ControlBoard:R_0603_1608Metric")
+    )
+    (path "/364540f7-0c58-4618-8ce3-bea6d054cb4e/c5318030-0c39-492d-82c8-f5e8f484d6df"
+      (reference "R20") (unit 1) (value "121R") (footprint "ControlBoard:R_0603_1608Metric")
+    )
+    (path "/364540f7-0c58-4618-8ce3-bea6d054cb4e/72a8a79e-a772-48b4-ab19-23f2cc1e83e2"
+      (reference "R21") (unit 1) (value "PN13101(Z)") (footprint "")
+    )
+    (path "/364540f7-0c58-4618-8ce3-bea6d054cb4e/502d3ff1-5239-4490-b785-a16dc791dfd7"
+      (reference "R22") (unit 1) (value "PN13104(XY)") (footprint "")
+    )
+    (path "/364540f7-0c58-4618-8ce3-bea6d054cb4e/6152da4d-452d-4939-aedd-70eddfb32f6a"
+      (reference "R23") (unit 1) (value "PN13104(XY)") (footprint "")
+    )
     (path "/b932d339-7888-4506-92dc-7b9f4a021ec5/5be3d2d4-2465-422c-8da7-9722bb04468f"
       (reference "SW1") (unit 1) (value "SW_DIP_x02") (footprint "ControlBoard:SW_DIP_SPSTx02_Slide_Copal_CHS-02B_W7.62mm_P1.27mm")
@@
       (reference "U12") (unit 1) (value "CH440R") (footprint "ControlBoard:TSSOP-16_4.4x5mm_P0.65mm")
     )
-    (path "/364540f7-0c58-4618-8ce3-bea6d054cb4e/e9849458-b660-4143-bb2d-8de2b914ecd0"
-      (reference "U13") (unit 1) (value "HMC5883L") (footprint "ControlBoard:QFN-16_3x3_Pitch0.5mm")
+    (path "/364540f7-0c58-4618-8ce3-bea6d054cb4e/9181ff88-2f85-4129-b483-720f264e83b2"
+      (reference "U13") (unit 1) (value "RM3100_13156") (footprint "")
     )
     (path "/364540f7-0c58-4618-8ce3-bea6d054cb4e/0c3ba1b6-7976-4c67-9efa-1457c99ef463"

Commit message: Modify and complete the circuit schematic to make the interface easier to wire.
Other:
- sheet Coprocessor ports: added PC7; removed PA7
- sheet Process_MCU ports: added PE0; removed PF0
- title: MM32_Board -> MM32 Control Board

Commit message: Modify the main control board schematic, replace the IMU device and remove the isolation module.
Other:
- sheet IMU ports: added IMU_INT1, IMU_INT2; removed IMU_DR, IMU_RST

Commit message: Modify the ControlBoard schematic to add useful features.
Other:
- added sheet Flash&USB (Flash&USB.kicad_sch)
- sheet Compass&Storage ports: added none; removed Compass_DR
- sheet Control_MCU ports: added PC0, PE6, PF0, PF1, PF10, PF2, PF3, PF4, PF5, PF6, PF7, PF8, PF9, SPI3_CLK, SPI3_MISO, SPI3_MOSI, SPI3_NSS; removed none
- sheet Coprocessor ports: added IIC_CLK, IIC_SDA; removed PA6
- sheet IMU ports: added IIC_CLK, IIC_SDA; removed none
- sheet Process_MCU ports: added UART2_RX, UART2_TX; removed UART8_RX, UART8_TX

Commit message: The main control board circuit modified the CH372C package, changed the serial port of the GPS and ControlMCU back, and moved the components a bit towards the middle so that they could be screwed on.
Changed lines of the file:
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@@
   (title_block
     (title "MM32 Control Board")
-    (date "2022-04-06")
-    (rev "1.5.2")
+    (date "2022-04-17")
+    (rev "1.5.3")
   )
   (wire (pts (xy 100.33 73.66) (xy 111.125 73.66))
@@
     (stroke (width 0) (type default) (color 0 0 0 0))
   )
-  (wire (pts (xy 220.98 124.46) (xy 233.045 124.46))
+  (wire (pts (xy 220.98 127.635) (xy 233.045 127.635))
     (stroke (width 0) (type default) (color 0 0 0 0))
   )
@@
     (stroke (width 0) (type default) (color 0 0 0 0))
   )
-  (wire (pts (xy 220.98 119.38) (xy 233.045 119.38))
+  (wire (pts (xy 220.98 122.555) (xy 233.045 122.555))
     (stroke (width 0) (type default) (color 0 0 0 0))
   )
@@
     (stroke (width 0) (type default) (color 0 0 0 0))
   )
-  (wire (pts (xy 220.98 115.57) (xy 233.045 115.57))
+  (wire (pts (xy 220.98 118.745) (xy 233.045 118.745))
     (stroke (width 0) (type default) (color 0 0 0 0))
   )
@@
     (stroke (width 0) (type default) (color 0 0 0 0))
   )
-  (wire (pts (xy 220.98 121.92) (xy 233.045 121.92))
+  (wire (pts (xy 220.98 125.095) (xy 233.045 125.095))
     (stroke (width 0) (type default) (color 0 0 0 0))
   )
@@
     (stroke (width 0) (type default) (color 0 0 0 0))
   )
-  (wire (pts (xy 220.98 137.795) (xy 233.045 137.795))
+  (wire (pts (xy 220.98 140.97) (xy 233.045 140.97))
     (stroke (width 0) (type default) (color 0 0 0 0))
   )
@@
     (stroke (width 0) (type default) (color 0 0 0 0))
   )
-  (wire (pts (xy 220.98 113.03) (xy 233.045 113.03))
+  (wire (pts (xy 220.98 116.205) (xy 233.045 116.205))
     (stroke (width 0) (type default) (color 0 0 0 0))
   )
@@
     (stroke (width 0) (type default) (color 0 0 0 0))
   )
-  (wire (pts (xy 220.98 127) (xy 233.045 127))
+  (wire (pts (xy 220.98 130.175) (xy 233.045 130.175))
     (stroke (width 0) (type default) (color 0 0 0 0))
   )
@@
     (stroke (width 0) (type default) (color 0 0 0 0))
   )
-  (wire (pts (xy 220.98 135.255) (xy 233.045 135.255))
+  (wire (pts (xy 220.98 138.43) (xy 233.045 138.43))
     (stroke (width 0) (type default) (color 0 0 0 0))
   )
@@
       (effects (font (size 1.27 1.27)) (justify left))
     )
-    (pin "UART3_TX" output (at 145.415 100.965 180)
+    (pin "UART3_TX" output (at 145.415 112.395 180)
       (effects (font (size 1.27 1.27)) (justify left))
     )
@@
       (effects (font (size 1.27 1.27)) (justify left))
     )
-    (pin "UART4_TX" output (at 145.415 112.395 180)
+    (pin "UART4_TX" output (at 145.415 100.965 180)
       (effects (font (size 1.27 1.27)) (justify left))
     )
@@
       (effects (font (size 1.27 1.27)) (justify left top) hide)
     )
-    (pin "IMU_CS" input (at 233.045 119.38 180)
-      (effects (font (size 1.27 1.27)) (justify left))
-    )
-    (pin "IMU_CLK" input (at 233.045 121.92 180)
-      (effects (font (size 1.27 1.27)) (justify left))
-    )
-    (pin "IMU_MOSI" input (at 233.045 124.46 180)
-      (effects (font (size 1.27 1.27)) (justify left))
-    )
-    (pin "IMU_MISO" output (at 233.045 127 180)
-      (effects (font (size 1.27 1.27)) (justify left))
-    )
-    (pin "IMU_INT1" output (at 233.045 135.255 180)
-      (effects (font (size 1.27 1.27)) (justify left))
-    )
-    (pin "IMU_INT2" output (at 233.045 137.795 180)
-      (effects (font (size 1.27 1.27)) (justify left))
-    )
-    (pin "IIC_SDA" bidirectional (at 233.045 115.57 180)
-      (effects (font (size 1.27 1.27)) (justify left))
-    )
-    (pin "IIC_CLK" input (at 233.045 113.03 180)
+    (pin "IMU_CS" input (at 233.045 122.555 180)
+      (effects (font (size 1.27 1.27)) (justify left))
+    )
+    (pin "IMU_CLK" input (at 233.045 125.095 180)
+      (effects (font (size 1.27 1.27)) (justify left))
+    )
+    (pin "IMU_MOSI" input (at 233.045 127.635 180)
+      (effects (font (size 1.27 1.27)) (justify left))
+    )
+    (pin "IMU_MISO" output (at 233.045 130.175 180)
+      (effects (font (size 1.27 1.27)) (justify left))
+    )
+    (pin "IMU_INT1" output (at 233.045 138.43 180)
+      (effects (font (size 1.27 1.27)) (justify left))
+    )
+    (pin "IMU_INT2" output (at 233.045 140.97 180)
+      (effects (font (size 1.27 1.27)) (justify left))
+    )
+    (pin "IIC_SDA" bidirectional (at 233.045 118.745 180)
+      (effects (font (size 1.27 1.27)) (justify left))
+    )
+    (pin "IIC_CLK" input (at 233.045 116.205 180)
       (effects (font (size 1.27 1.27)) (justify left))
     )
@@
       (effects (font (size 1.27 1.27)) (justify left))
     )
-    (pin "SPI2_NSS" output (at 220.98 119.38 0)
-      (effects (font (size 1.27 1.27)) (justify right))
-    )
-    (pin "SPI2_MISO" input (at 220.98 127 0)
-      (effects (font (size 1.27 1.27)) (justify right))
-    )
-    (pin "SPI2_MOSI" output (at 220.98 124.46 0)
-      (effects (font (size 1.27 1.27)) (justify right))
-    )
-    (pin "SPI2_CLK" output (at 220.98 121.92 0)
-      (effects (font (size 1.27 1.27)) (justify right))
-    )
-    (pin "PC6" input (at 220.98 137.795 0)
-      (effects (font (size 1.27 1.27)) (justify right))
-    )
-    (pin "PC7" input (at 220.98 135.255 0)
-      (effects (font (size 1.27 1.27)) (justify right))
-    )
-    (pin "IIC_SDA" bidirectional (at 220.98 115.57 0)
-      (effects (font (size 1.27 1.27)) (justify right))
-    )
-    (pin "IIC_CLK" output (at 220.98 113.03 0)
+    (pin "SPI2_NSS" output (at 220.98 122.555 0)
+      (effects (font (size 1.27 1.27)) (justify right))
+    )
+    (pin "SPI2_MISO" input (at 220.98 130.175 0)
+      (effects (font (size 1.27 1.27)) (justify right))
+    )
+    (pin "SPI2_MOSI" output (at 220.98 127.635 0)
+      (effects (font (size 1.27 1.27)) (justify right))
+    )
+    (pin "SPI2_CLK" output (at 220.98 125.095 0)
+      (effects (font (size 1.27 1.27)) (justify right))
+    )
+    (pin "PC6" input (at 220.98 140.97 0)
+      (effects (font (size 1.27 1.27)) (justify right))
+    )
+    (pin "PC7" input (at 220.98 138.43 0)
+      (effects (font (size 1.27 1.27)) (justify right))
+    )
+    (pin "IIC_SDA" bidirectional (at 220.98 118.745 0)
+      (effects (font (size 1.27 1.27)) (justify right))
+    )
+    (pin "IIC_CLK" output (at 220.98 116.205 0)
       (effects (font (size 1.27 1.27)) (justify right))
     )
@@
     )
     (path "/99919f16-809b-4d37-b44a-061baa0477d2/161d5af1-f0e2-4af4-a7ec-a33a8da11fd4"
-      (reference "U14") (unit 1) (value "CH372C") (footprint "Package_SO:SSOP-20_4.4x6.5mm_P0.65mm")
+      (reference "U14") (unit 1) (value "CH372C") (footprint "Package_SO:SSOP-20_5.3x7.2mm_P0.65mm")
     )
     (path "/99919f16-809b-4d37-b44a-061baa0477d2/81777fc0-c5a7-4a15-88f6-34092c22851d"
