File: circuit/control_board/project.kicad_sch (KiCad schematic)
At the start: 0 parts

Commit message: Fixed part of the control board circuit and added SD card reading chip.
Other:
- sheet Flash&USB ports: added none; removed USB_A0, USB_CS, USB_D0, USB_D1, USB_D2, USB_D3, USB_D4, USB_D5, USB_D6, USB_D7, USB_INT, USB_RD, USB_WR

Commit message: Update the main control board schematic to complete the SD card reader part.
Other:
- sheet Control_MCU ports: added PG4; removed PC0, PE6, PF0, PF1, PF10, PF2, PF3, PF4, PF5, PF6, PF7, PF8, PF9
- sheet Flash&USB ports: added SELECT; removed none

Commit message: Updated the main control board schematic and switched the geomagnetometer interface sequence.
Other:
- sheet Control_MCU ports: added PD10; removed PG4
Changed lines of the file:
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@@
       (effects (font (size 1.27 1.27)) (justify left))
     )
-    (pin "PG4" output (at 80.01 120.015 180)
+    (pin "PD10" output (at 80.01 120.015 180)
       (effects (font (size 1.27 1.27)) (justify left))
     )
