File: circuit/control_board/Compass&Storage.kicad_sch (KiCad schematic)
At the start: 9 parts, among them U13 HMC5883L, U14 AT24C02

Commit message: Modified the circuitry of the main control board to add a microcontroller for reading information from the magnetometer and IMU. Modified the SPI connection port of the Process MCU.
Parts:
- removed C69, C72: 100nF, Capacitor_SMD:C_0603_1608Metric, symbol Device:C
- added R11, R12: 10kR, ControlBoard:R_0603_1608Metric, symbol Device:R
- C70, C71, C73: footprint Capacitor_SMD:C_0603_1608Metric -> ControlBoard:C_0603_1608Metric
- R10, R9: value 2.2kR -> 10kR; footprint Resistor_SMD:R_0603_1608Metric -> ControlBoard:R_0603_1608Metric
- U13: footprint MM32_Library:QFN-16_3x3_Pitch0.5mm -> ControlBoard:QFN-16_3x3_Pitch0.5mm
- U14: footprint Package_SO:SOP-8_3.9x4.9mm_P1.27mm -> ControlBoard:SOP-8_3.9x4.9mm_P1.27mm
Connections:
- net +3.3VP: no longer U13.13 (VDDIO), U13.2 (VDD), U13.4 (S1)
- net GND: no longer C71.2, U13.11 (GND), U13.9 (GND)
- net IIC_SCL renamed EEPROM_SCL
- net EEPROM_SCL: no longer U13.1 (SCL)
- net IIC_SDA renamed EEPROM_SDA
- net EEPROM_SDA: no longer U13.16 (SDA)
- new net +3.3VADC: R11.1, R12.1, U13.13 (VDDIO), U13.2 (VDD), U13.4 (S1)
- new net COMPASS_SCL: R11.2, U13.1 (SCL)
- new net COMPASS_SDA: R12.2, U13.16 (SDA)
- new net GNDA: C71.2, U13.11 (GND), U13.9 (GND)

Commit message: Update the main control board schematic and replace the magnetometer with RM3100.
Parts:
- removed C70: 220nF, ControlBoard:C_0603_1608Metric, symbol Device:C
- removed U13: HMC5883L, ControlBoard:QFN-16_3x3_Pitch0.5mm, symbol MM32_Periph:HMC5883L
- added R16, R17, R18, R19, R20: 121R, ControlBoard:R_0603_1608Metric, symbol Device:R
- added R21: PN13101(Z), symbol MM32_Periph:PN13101(Z)
- added R22, R23: PN13104(XY), symbol MM32_Periph:PN13104(XY)
- added U13: RM3100_13156, symbol MM32_Periph:RM3100_13156
- R11: value 10kR -> 121R
- R12: value 10kR -> 33kR
Connections:
- net COMPASS_SDA is gone; now on net GNDA: R12.2
- net +3.3VADC: now also C71.1, U13.14 (DVDD), U13.26 (DVDD), U13.4 (AVDD); no longer R11.1, R12.1
- net GNDA: now also U13.19 (DVSS), U13.2 (RES), U13.20 (RES), U13.22 (I2CEN), U13.5 (AVSS)
- net COMPASS_SCL: no longer names the net of R11.2
- net COMPASS_SCL: now also R21.2 (B), U13.7 (ZINP)
- new net: R12.1, U13.25 (REXT)
- new net: R19.1, U13.15 (XDRVP)
- new net: R19.2, R23.2 (B), U13.16 (XINP)
- new net: R18.2, R22.1 (A), U13.12 (YINN)
- new net: R17.2, R22.2 (B), U13.11 (YINP)
- new net: R17.1, U13.10 (YDRVP)
- new net: R20.2, R23.1 (A), U13.17 (XINN)
- new net: R11.1, U13.6 (ZDRVP)
- new net: R16.2, R21.1 (A), U13.8 (ZINN)
- new net: R18.1, U13.13 (YDRVN)
- new net: R20.1, U13.18 (XDRVN)
- new net: R16.1, U13.9 (ZDRVN)
- new net Compass_CLK: U13.27 (SCLK)
- new net Compass_CS: U13.3 (SSN)
- new net Compass_DR: U13.23 (DRDY)
- new net Compass_MISO: U13.28 (MISO)
- new net Compass_MOSI: U13.1 (MOSI)
Other:
- note added: "Compass"
- note removed: "Cmpass"
- moved on the sheet: C71, R12

Commit message: Modify and complete the circuit schematic to make the interface easier to wire.
Parts:
- R16: renamed from R21; footprint (none) -> ControlBoard:PN13101
- R17: renamed from R22; footprint (none) -> ControlBoard:PN13104
- R18: renamed from R23; footprint (none) -> ControlBoard:PN13104
- U11: renamed from U13; footprint (none) -> ControlBoard:QFN-28-1EP_4x4mm_P0.4mm_EP2.4x2.4mm
- renumbered C71 to C65, C73 to C66, R11 to R10, R16 to R11, R17 to R12, R18 to R13, R19 to R14, R20 to R15, R9 to R19, R10 to R20, R12 to R9, U14 to U12
Other:
- title: MM32_Board -> MM32 Control Board

Commit message: Modify the main control board schematic, replace the IMU device and remove the isolation module.
Connections:
- net GNDA is gone; now on net GND: C65.2, R9.2, U11.19 (DVSS), U11.2 (RES), U11.20 (RES), U11.22 (I2CEN), U11.5 (AVSS)
Changed lines of the file:
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@@
   (title_block
     (title "MM32 Control Board")
-    (date "2022-03-03")
-    (rev "1.3.3")
+    (date "2022-03-28")
+    (rev "1.4.1")
   )
   (junction (at 126.365 86.995) (diameter 0) (color 0 0 0 0)
@@
     (pin "1")
   )
-  (symbol (lib_id "power:GNDA") (at 72.39 137.795 0) (unit 1)
-    (in_bom yes) (on_board yes)
-    (property "Reference" "#PWR0160" (id 0) (at 72.39 144.145 0)
-      (effects (font (size 1.27 1.27)) hide)
-    )
-    (property "Value" "GNDA" (id 1) (at 72.39 142.24 0))
-    (property "Footprint" "" (id 2) (at 72.39 137.795 0)
-      (effects (font (size 1.27 1.27)) hide)
-    )
-    (property "Datasheet" "" (id 3) (at 72.39 137.795 0)
+  (symbol (lib_id "power:GND") (at 100.33 137.795 0) (unit 1)
+    (in_bom yes) (on_board yes)
+    (property "Reference" "#PWR0195" (id 0) (at 100.33 144.145 0)
+      (effects (font (size 1.27 1.27)) hide)
+    )
+    (property "Value" "GND" (id 1) (at 100.33 142.24 0))
+    (property "Footprint" "" (id 2) (at 100.33 137.795 0)
+      (effects (font (size 1.27 1.27)) hide)
+    )
+    (property "Datasheet" "" (id 3) (at 100.33 137.795 0)
       (effects (font (size 1.27 1.27)) hide)
     )
@@
     )
     (property "Datasheet" "" (id 3) (at 206.375 132.08 0)
+      (effects (font (size 1.27 1.27)) hide)
+    )
+    (pin "1")
+  )
+  (symbol (lib_id "power:GND") (at 72.39 137.795 0) (unit 1)
+    (in_bom yes) (on_board yes)
+    (property "Reference" "#PWR0196" (id 0) (at 72.39 144.145 0)
+      (effects (font (size 1.27 1.27)) hide)
+    )
+    (property "Value" "GND" (id 1) (at 72.39 142.24 0))
+    (property "Footprint" "" (id 2) (at 72.39 137.795 0)
+      (effects (font (size 1.27 1.27)) hide)
+    )
+    (property "Datasheet" "" (id 3) (at 72.39 137.795 0)
       (effects (font (size 1.27 1.27)) hide)
     )
@@
     (pin "1")
     (pin "2")
-  )
-  (symbol (lib_id "power:GNDA") (at 74.295 102.235 270) (unit 1)
-    (in_bom yes) (on_board yes)
-    (property "Reference" "#PWR0161" (id 0) (at 67.945 102.235 0)
-      (effects (font (size 1.27 1.27)) hide)
-    )
-    (property "Value" "GNDA" (id 1) (at 68.58 102.235 90))
-    (property "Footprint" "" (id 2) (at 74.295 102.235 0)
-      (effects (font (size 1.27 1.27)) hide)
-    )
-    (property "Datasheet" "" (id 3) (at 74.295 102.235 0)
-      (effects (font (size 1.27 1.27)) hide)
-    )
-    (pin "1")
   )
   (symbol (lib_id "MM32_Periph:PN13104(XY)") (at 129.54 111.125 0) (unit 1)
@@
     (pin "2")
   )
+  (symbol (lib_id "power:GND") (at 74.295 102.235 270) (unit 1)
+    (in_bom yes) (on_board yes)
+    (property "Reference" "#PWR0194" (id 0) (at 67.945 102.235 0)
+      (effects (font (size 1.27 1.27)) hide)
+    )
+    (property "Value" "GND" (id 1) (at 69.85 102.235 0))
+    (property "Footprint" "" (id 2) (at 74.295 102.235 0)
+      (effects (font (size 1.27 1.27)) hide)
+    )
+    (property "Datasheet" "" (id 3) (at 74.295 102.235 0)
+      (effects (font (size 1.27 1.27)) hide)
+    )
+    (pin "1")
+  )
   (symbol (lib_id "Device:R") (at 224.155 95.25 0) (unit 1)
     (in_bom yes) (on_board yes)
@@
       (effects (font (size 1.27 1.27)) hide)
     )
-    (pin "1")
-  )
-  (symbol (lib_id "power:GNDA") (at 100.33 137.795 0) (unit 1)
-    (in_bom yes) (on_board yes)
-    (property "Reference" "#PWR0163" (id 0) (at 100.33 144.145 0)
-      (effects (font (size 1.27 1.27)) hide)
-    )
-    (property "Value" "GNDA" (id 1) (at 100.33 142.24 0))
-    (property "Footprint" "" (id 2) (at 100.33 137.795 0)
-      (effects (font (size 1.27 1.27)) hide)
-    )
-    (property "Datasheet" "" (id 3) (at 100.33 137.795 0)
-      (effects (font (size 1.27 1.27)) hide)
-    )

Commit message: Modify the ControlBoard schematic to add useful features.
Connections:
- net +3.3VP renamed +3.3VA
- net Compass_DR: no longer names the net of U11.23 (DRDY)
- no-connect marks 0 -> 1
Changed lines of the file:
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@@
   (title_block
     (title "MM32 Control Board")
-    (date "2022-03-28")
-    (rev "1.4.1")
+    (date "2022-04-06")
+    (rev "1.5.2")
   )
   (junction (at 126.365 86.995) (diameter 0) (color 0 0 0 0)
@@
   (junction (at 76.835 102.235) (diameter 0) (color 0 0 0 0)
   )
+  (no_connect (at 82.55 118.745))
   (wire (pts (xy 123.19 100.965) (xy 126.365 100.965))
     (stroke (width 0) (type default) (color 0 0 0 0))
@@
   )
   (wire (pts (xy 76.835 94.615) (xy 76.835 97.155))
-    (stroke (width 0) (type default) (color 0 0 0 0))
-  )
-  (wire (pts (xy 73.025 118.745) (xy 82.55 118.745))
     (stroke (width 0) (type default) (color 0 0 0 0))
   )
@@
     (effects (font (size 1.27 1.27)) (justify right))
   )
-  (hierarchical_label "Compass_DR" (shape output) (at 73.025 118.745 180)
-    (effects (font (size 1.27 1.27)) (justify right))
-  )
   (hierarchical_label "Compass_CLK" (shape input) (at 73.025 109.855 180)
     (effects (font (size 1.27 1.27)) (justify right))
@@
   (hierarchical_label "Compass_MISO" (shape output) (at 73.025 112.395 180)
     (effects (font (size 1.27 1.27)) (justify right))
-  )
-  (symbol (lib_id "power:+3.3VP") (at 206.375 82.55 0) (unit 1)
-    (in_bom yes) (on_board yes)
-    (property "Reference" "#PWR0167" (id 0) (at 210.185 83.82 0)
-      (effects (font (size 1.27 1.27)) hide)
-    )
-    (property "Value" "+3.3VP" (id 1) (at 206.375 78.105 0))
-    (property "Footprint" "" (id 2) (at 206.375 82.55 0)
-      (effects (font (size 1.27 1.27)) hide)
-    )
-    (property "Datasheet" "" (id 3) (at 206.375 82.55 0)
-      (effects (font (size 1.27 1.27)) hide)
-    )
-    (pin "1")
   )
   (symbol (lib_id "MM32_Periph:AT24C02") (at 185.42 113.03 0) (unit 1)
@@
     (pin "2")
   )
-  (symbol (lib_id "power:+3.3VP") (at 167.005 82.55 0) (unit 1)
-    (in_bom yes) (on_board yes)
-    (property "Reference" "#PWR0164" (id 0) (at 170.815 83.82 0)
-      (effects (font (size 1.27 1.27)) hide)
-    )
-    (property "Value" "+3.3VP" (id 1) (at 167.005 78.105 0))
-    (property "Footprint" "" (id 2) (at 167.005 82.55 0)
-      (effects (font (size 1.27 1.27)) hide)
-    )
-    (property "Datasheet" "" (id 3) (at 167.005 82.55 0)
-      (effects (font (size 1.27 1.27)) hide)
-    )
-    (pin "1")
-  )
   (symbol (lib_id "power:GND") (at 177.8 132.08 0) (unit 1)
     (in_bom yes) (on_board yes)
@@
     (pin "2")
   )
-  (symbol (lib_id "power:+3.3VP") (at 224.155 82.55 0) (unit 1)
-    (in_bom yes) (on_board yes)
-    (property "Reference" "#PWR0170" (id 0) (at 227.965 83.82 0)
-      (effects (font (size 1.27 1.27)) hide)
-    )
-    (property "Value" "+3.3VP" (id 1) (at 224.155 78.105 0))
+  (symbol (lib_id "MM32_Periph:PN13104(XY)") (at 129.54 125.095 0) (unit 1)
+    (in_bom yes) (on_board yes)
+    (property "Reference" "R18" (id 0) (at 132.08 120.65 0)
+      (effects (font (size 1.27 1.27)) (justify left))
+    )
+    (property "Value" "PN13104(XY)" (id 1) (at 138.4808 123.571 0)
+      (effects (font (size 1.27 1.27)) hide)
+    )
+    (property "Footprint" "ControlBoard:PN13104" (id 2) (at 129.54 125.095 0)
+      (effects (font (size 1.27 1.27)) hide)
+    )
+    (property "Datasheet" "" (id 3) (at 129.54 125.095 0)
+      (effects (font (size 1.27 1.27)) hide)
+    )
+    (pin "1")
+    (pin "2")
+  )
+  (symbol (lib_id "power:+3.3VA") (at 224.155 82.55 0) (unit 1)
+    (in_bom yes) (on_board yes)
+    (property "Reference" "#PWR035" (id 0) (at 224.155 86.36 0)
+      (effects (font (size 1.27 1.27)) hide)
+    )
+    (property "Value" "+3.3VA" (id 1) (at 224.155 78.105 0))
     (property "Footprint" "" (id 2) (at 224.155 82.55 0)
       (effects (font (size 1.27 1.27)) hide)
@@
     )
     (pin "1")
-  )
-  (symbol (lib_id "MM32_Periph:PN13104(XY)") (at 129.54 125.095 0) (unit 1)
-    (in_bom yes) (on_board yes)
-    (property "Reference" "R18" (id 0) (at 132.08 120.65 0)
-      (effects (font (size 1.27 1.27)) (justify left))
-    )
-    (property "Value" "PN13104(XY)" (id 1) (at 138.4808 123.571 0)
-      (effects (font (size 1.27 1.27)) hide)
-    )
-    (property "Footprint" "ControlBoard:PN13104" (id 2) (at 129.54 125.095 0)
-      (effects (font (size 1.27 1.27)) hide)
-    )
-    (property "Datasheet" "" (id 3) (at 129.54 125.095 0)
-      (effects (font (size 1.27 1.27)) hide)
-    )
-    (pin "1")
-    (pin "2")
   )
   (symbol (lib_id "Device:R") (at 119.38 86.995 90) (unit 1)
@@
     (pin "2")
   )
+  (symbol (lib_id "power:+3.3VA") (at 167.005 82.55 0) (unit 1)
+    (in_bom yes) (on_board yes)
+    (property "Reference" "#PWR032" (id 0) (at 167.005 86.36 0)
+      (effects (font (size 1.27 1.27)) hide)
+    )
+    (property "Value" "+3.3VA" (id 1) (at 167.005 78.105 0))
+    (property "Footprint" "" (id 2) (at 167.005 82.55 0)
+      (effects (font (size 1.27 1.27)) hide)
+    )
+    (property "Datasheet" "" (id 3) (at 167.005 82.55 0)
+      (effects (font (size 1.27 1.27)) hide)
+    )
+    (pin "1")
+  )
   (symbol (lib_id "MM32_Periph:PN13101(Z)") (at 129.54 95.885 0) (unit 1)
     (in_bom yes) (on_board yes)
@@
     (pin "1")
     (pin "2")
+  )
+  (symbol (lib_id "power:+3.3VA") (at 206.375 82.55 0) (unit 1)
+    (in_bom yes) (on_board yes)
+    (property "Reference" "#PWR033" (id 0) (at 206.375 86.36 0)
+      (effects (font (size 1.27 1.27)) hide)
+    )
+    (property "Value" "+3.3VA" (id 1) (at 206.375 78.105 0))
+    (property "Footprint" "" (id 2) (at 206.375 82.55 0)
+      (effects (font (size 1.27 1.27)) hide)
+    )
+    (property "Datasheet" "" (id 3) (at 206.375 82.55 0)
+      (effects (font (size 1.27 1.27)) hide)
+    )
+    (pin "1")
   )
   (symbol (lib_id "MM32_Periph:RM3100_13156") (at 85.09 125.095 0) (unit 1)
@@
     (pin "2")
   )
-  (symbol (lib_id "power:+3.3VP") (at 215.265 82.55 0) (unit 1)
-    (in_bom yes) (on_board yes)
-    (property "Reference" "#PWR0169" (id 0) (at 219.075 83.82 0)
-      (effects (font (size 1.27 1.27)) hide)
-    )
-    (property "Value" "+3.3VP" (id 1) (at 215.265 78.105 0))
+  (symbol (lib_id "power:+3.3VA") (at 215.265 82.55 0) (unit 1)
+    (in_bom yes) (on_board yes)
+    (property "Reference" "#PWR034" (id 0) (at 215.265 86.36 0)
+      (effects (font (size 1.27 1.27)) hide)
+    )
+    (property "Value" "+3.3VA" (id 1) (at 215.265 78.105 0))
     (property "Footprint" "" (id 2) (at 215.265 82.55 0)
       (effects (font (size 1.27 1.27)) hide)

Commit message: Remove the geomagnetometer from the main control board to enable external connection of the geomagnetometer.
Parts:
- removed R10, R11, R12, R13, R14, R15: 121R, ControlBoard:R_0603_1608Metric, symbol Device:R
- removed R16: PN13101(Z), ControlBoard:PN13101, symbol MM32_Periph:PN13101(Z)
- removed R17, R18: PN13104(XY), ControlBoard:PN13104, symbol MM32_Periph:PN13104(XY)
- removed R9: 33kR, ControlBoard:R_0603_1608Metric, symbol Device:R
- removed U11: RM3100_13156, ControlBoard:QFN-28-1EP_4x4mm_P0.4mm_EP2.4x2.4mm, symbol MM32_Periph:RM3100_13156
- added J5: Conn_01x06, Connector_JST:JST_GH_SM06B-GHS-TB_1x06-1MP_P1.25mm_Horizontal, symbol Connector_Generic:Conn_01x06
Connections:
- net +3.3VADC: now also J5.1 (Pin_1)
- net Compass_CLK: now also J5.3 (Pin_3)
- net Compass_CS: now also J5.2 (Pin_2)
- net Compass_MISO: now also J5.4 (Pin_4)
- net Compass_MOSI: now also J5.5 (Pin_5)
- net GND: now also J5.6 (Pin_6)
- no-connect marks 1 -> 0
Other:
- moved on the sheet: C65

Commit message: Fixed part of the control board circuit and added SD card reading chip.
Parts:
- renumbered J5 to J4, R20 to R10, R19 to R9, U12 to U11
Changed lines of the file:
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@@
   (symbol (lib_id "MM32_Periph:AT24C02") (at 185.42 113.03 0) (unit 1)
     (in_bom yes) (on_board yes)
-    (property "Reference" "U12" (id 0) (at 187.325 99.06 0))
+    (property "Reference" "U11" (id 0) (at 187.325 99.06 0))
     (property "Value" "AT24C02" (id 1) (at 194.31 114.935 0))
     (property "Footprint" "ControlBoard:SOP-8_3.9x4.9mm_P1.27mm" (id 2) (at 193.04 116.84 0)
@@
   (symbol (lib_id "Device:R") (at 215.265 95.25 0) (unit 1)
     (in_bom yes) (on_board yes)
-    (property "Reference" "R19" (id 0) (at 210.82 93.98 0))
+    (property "Reference" "R9" (id 0) (at 210.82 93.98 0))
     (property "Value" "10kR" (id 1) (at 210.82 96.52 0))
     (property "Footprint" "ControlBoard:R_0603_1608Metric" (id 2) (at 213.487 95.25 90)
@@
   (symbol (lib_id "Connector_Generic:Conn_01x06") (at 102.235 104.775 0) (unit 1)
     (in_bom yes) (on_board yes)
-    (property "Reference" "J5" (id 0) (at 101.6 96.52 0)
+    (property "Reference" "J4" (id 0) (at 101.6 96.52 0)
       (effects (font (size 1.27 1.27)) (justify left))
     )
@@
   (symbol (lib_id "power:GND") (at 92.075 127.635 0) (unit 1)
     (in_bom yes) (on_board yes)
-    (property "Reference" "#PWR0195" (id 0) (at 92.075 133.985 0)
+    (property "Reference" "#PWR0161" (id 0) (at 92.075 133.985 0)
       (effects (font (size 1.27 1.27)) hide)
     )
@@
   (symbol (lib_id "power:GND") (at 114.3 127.635 0) (unit 1)
     (in_bom yes) (on_board yes)
-    (property "Reference" "#PWR0196" (id 0) (at 114.3 133.985 0)
+    (property "Reference" "#PWR0163" (id 0) (at 114.3 133.985 0)
       (effects (font (size 1.27 1.27)) hide)
     )
@@
   (symbol (lib_id "power:+3.3VA") (at 224.155 82.55 0) (unit 1)
     (in_bom yes) (on_board yes)
-    (property "Reference" "#PWR035" (id 0) (at 224.155 86.36 0)
+    (property "Reference" "#PWR0170" (id 0) (at 224.155 86.36 0)
       (effects (font (size 1.27 1.27)) hide)
     )
@@
   (symbol (lib_id "power:+3.3VA") (at 167.005 82.55 0) (unit 1)
     (in_bom yes) (on_board yes)
-    (property "Reference" "#PWR032" (id 0) (at 167.005 86.36 0)
+    (property "Reference" "#PWR0164" (id 0) (at 167.005 86.36 0)
       (effects (font (size 1.27 1.27)) hide)
     )
@@
   (symbol (lib_id "power:+3.3VA") (at 206.375 82.55 0) (unit 1)
     (in_bom yes) (on_board yes)
-    (property "Reference" "#PWR033" (id 0) (at 206.375 86.36 0)
+    (property "Reference" "#PWR0167" (id 0) (at 206.375 86.36 0)
       (effects (font (size 1.27 1.27)) hide)
     )
@@
   (symbol (lib_id "Device:R") (at 224.155 95.25 0) (unit 1)
     (in_bom yes) (on_board yes)
-    (property "Reference" "R20" (id 0) (at 219.71 93.98 0))
+    (property "Reference" "R10" (id 0) (at 219.71 93.98 0))
     (property "Value" "10kR" (id 1) (at 219.71 96.52 0))
     (property "Footprint" "ControlBoard:R_0603_1608Metric" (id 2) (at 222.377 95.25 90)
@@
   (symbol (lib_id "power:+3.3VADC") (at 114.3 86.36 0) (unit 1)
     (in_bom yes) (on_board yes)
-    (property "Reference" "#PWR0159" (id 0) (at 118.11 87.63 0)
+    (property "Reference" "#PWR0162" (id 0) (at 118.11 87.63 0)
       (effects (font (size 1.27 1.27)) hide)
     )
@@
   (symbol (lib_id "power:+3.3VADC") (at 92.075 86.36 0) (unit 1)
     (in_bom yes) (on_board yes)
-    (property "Reference" "#PWR0162" (id 0) (at 95.885 87.63 0)
+    (property "Reference" "#PWR0160" (id 0) (at 95.885 87.63 0)
       (effects (font (size 1.27 1.27)) hide)
     )
@@
   (symbol (lib_id "power:+3.3VA") (at 215.265 82.55 0) (unit 1)
     (in_bom yes) (on_board yes)
-    (property "Reference" "#PWR034" (id 0) (at 215.265 86.36 0)
-      (effects (font (size 1.27 1.27)) hide)
-    )
+    (property "Reference" "#PWR0169" (id 0) (at 215.265 86.36 0)
+      (effects (font (size 1.27 1.27)) hide)
+    )
