File: circuit/control_board/Compass&Storage.kicad_sch (KiCad schematic)
At the start: 6 parts, among them J4 Conn_01x06, U11 AT24C02

Commit message: Update the main control board schematic to complete the SD card reader part.
Parts:
- renumbered C65 to C71, C66 to C72
Changed lines of the file:
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@@
   (title_block
     (title "MM32 Control Board")
-    (date "2022-05-18")
-    (rev "1.5.4")
+    (date "2022-07-11")
+    (rev "1.6.1")
   )
   (junction (at 215.265 110.49) (diameter 0) (color 0 0 0 0)
@@
   (symbol (lib_id "Device:C") (at 114.3 106.68 0) (unit 1)
     (in_bom yes) (on_board yes)
-    (property "Reference" "C65" (id 0) (at 117.221 105.5116 0)
+    (property "Reference" "C71" (id 0) (at 117.221 105.5116 0)
       (effects (font (size 1.27 1.27)) (justify left))
     )
@@
   (symbol (lib_id "power:GND") (at 177.8 132.08 0) (unit 1)
     (in_bom yes) (on_board yes)
-    (property "Reference" "#PWR0166" (id 0) (at 177.8 138.43 0)
+    (property "Reference" "#PWR0178" (id 0) (at 177.8 138.43 0)
       (effects (font (size 1.27 1.27)) hide)
     )
@@
   (symbol (lib_id "power:GND") (at 92.075 127.635 0) (unit 1)
     (in_bom yes) (on_board yes)
-    (property "Reference" "#PWR0161" (id 0) (at 92.075 133.985 0)
+    (property "Reference" "#PWR0173" (id 0) (at 92.075 133.985 0)
       (effects (font (size 1.27 1.27)) hide)
     )
@@
   (symbol (lib_id "power:GND") (at 206.375 132.08 0) (unit 1)
     (in_bom yes) (on_board yes)
-    (property "Reference" "#PWR0168" (id 0) (at 206.375 138.43 0)
+    (property "Reference" "#PWR0180" (id 0) (at 206.375 138.43 0)
       (effects (font (size 1.27 1.27)) hide)
     )
@@
   (symbol (lib_id "power:GND") (at 114.3 127.635 0) (unit 1)
     (in_bom yes) (on_board yes)
-    (property "Reference" "#PWR0163" (id 0) (at 114.3 133.985 0)
+    (property "Reference" "#PWR0175" (id 0) (at 114.3 133.985 0)
       (effects (font (size 1.27 1.27)) hide)
     )
@@
   (symbol (lib_id "power:GND") (at 167.005 132.08 0) (unit 1)
     (in_bom yes) (on_board yes)
-    (property "Reference" "#PWR0165" (id 0) (at 167.005 138.43 0)
+    (property "Reference" "#PWR0177" (id 0) (at 167.005 138.43 0)
       (effects (font (size 1.27 1.27)) hide)
     )
@@
   (symbol (lib_id "Device:C") (at 167.005 109.855 0) (unit 1)
     (in_bom yes) (on_board yes)
-    (property "Reference" "C66" (id 0) (at 169.926 108.6866 0)
+    (property "Reference" "C72" (id 0) (at 169.926 108.6866 0)
       (effects (font (size 1.27 1.27)) (justify left))
     )
@@
   (symbol (lib_id "power:+3.3VA") (at 224.155 82.55 0) (unit 1)
     (in_bom yes) (on_board yes)
-    (property "Reference" "#PWR0170" (id 0) (at 224.155 86.36 0)
+    (property "Reference" "#PWR0182" (id 0) (at 224.155 86.36 0)
       (effects (font (size 1.27 1.27)) hide)
     )
@@
   (symbol (lib_id "power:+3.3VA") (at 167.005 82.55 0) (unit 1)
     (in_bom yes) (on_board yes)
-    (property "Reference" "#PWR0164" (id 0) (at 167.005 86.36 0)
+    (property "Reference" "#PWR0176" (id 0) (at 167.005 86.36 0)
       (effects (font (size 1.27 1.27)) hide)
     )
@@
   (symbol (lib_id "power:+3.3VA") (at 206.375 82.55 0) (unit 1)
     (in_bom yes) (on_board yes)
-    (property "Reference" "#PWR0167" (id 0) (at 206.375 86.36 0)
+    (property "Reference" "#PWR0179" (id 0) (at 206.375 86.36 0)
       (effects (font (size 1.27 1.27)) hide)
     )
@@
   (symbol (lib_id "power:+3.3VADC") (at 114.3 86.36 0) (unit 1)
     (in_bom yes) (on_board yes)
-    (property "Reference" "#PWR0162" (id 0) (at 118.11 87.63 0)
+    (property "Reference" "#PWR0174" (id 0) (at 118.11 87.63 0)
       (effects (font (size 1.27 1.27)) hide)
     )
@@
   (symbol (lib_id "power:+3.3VADC") (at 92.075 86.36 0) (unit 1)
     (in_bom yes) (on_board yes)
-    (property "Reference" "#PWR0160" (id 0) (at 95.885 87.63 0)
+    (property "Reference" "#PWR0172" (id 0) (at 95.885 87.63 0)
       (effects (font (size 1.27 1.27)) hide)
     )
@@
   (symbol (lib_id "power:+3.3VA") (at 215.265 82.55 0) (unit 1)
     (in_bom yes) (on_board yes)
-    (property "Reference" "#PWR0169" (id 0) (at 215.265 86.36 0)
-      (effects (font (size 1.27 1.27)) hide)
-    )
+    (property "Reference" "#PWR0181" (id 0) (at 215.265 86.36 0)
+      (effects (font (size 1.27 1.27)) hide)
+    )

Commit message: Updated the main control board schematic and switched the geomagnetometer interface sequence.
Connections:
- net Compass_CLK: now also J4.5 (Pin_5); no longer J4.3 (Pin_3)
- net Compass_MOSI: now also J4.3 (Pin_3); no longer J4.5 (Pin_5)
Changed lines of the file:
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@@
     (effects (font (size 3.81 3.81)) (justify left bottom))
   )
-  (hierarchical_label "Compass_MOSI" (shape input) (at 88.9 109.855 180)
+  (hierarchical_label "Compass_MOSI" (shape input) (at 88.9 104.775 180)
     (effects (font (size 1.27 1.27)) (justify right))
   )
-  (hierarchical_label "Compass_CLK" (shape input) (at 88.9 104.775 180)
+  (hierarchical_label "Compass_CLK" (shape input) (at 88.9 109.855 180)
     (effects (font (size 1.27 1.27)) (justify right))
   )
