File: circuit/control_board/ControlMCU.kicad_sch (KiCad schematic)
At the start: 21 parts, among them U11 MM32F3277G9P, Y2 8MHz

Commit message: Modified the circuitry of the main control board to add a microcontroller for reading information from the magnetometer and IMU. Modified the SPI connection port of the Process MCU.
Parts:
- C52, C53, C54, C55, C56, C57, C58, C59, C60, C61, C62, C63, C64, C65, C66: footprint Capacitor_SMD:C_0603_1608Metric -> ControlBoard:C_0603_1608Metric
- D2: footprint LED_SMD:LED_0603_1608Metric -> ControlBoard:LED_0603_1608Metric
- R4, R5, R6: footprint Resistor_SMD:R_0603_1608Metric -> ControlBoard:R_0603_1608Metric
- U11: footprint Package_QFP:LQFP-144_20x20mm_P0.5mm -> ControlBoard:LQFP-144_20x20mm_P0.5mm
- Y2: footprint Crystal:Crystal_SMD_3225-4Pin_3.2x2.5mm -> ControlBoard:Crystal_SMD_3225-4Pin_3.2x2.5mm
Changed lines of the file:
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@@
   (title_block
     (title "MM32_Board")
-    (date "2022-02-09")
-    (rev "1.2.3")
+    (date "2022-02-28")
+    (rev "1.3.1")
   )
   (junction (at 217.17 134.62) (diameter 0) (color 0 0 0 0)
@@
       (effects (font (size 1.27 1.27)) (justify left))
     )
-    (property "Footprint" "Package_QFP:LQFP-144_20x20mm_P0.5mm" (id 2) (at 176.53 153.67 0)
+    (property "Footprint" "ControlBoard:LQFP-144_20x20mm_P0.5mm" (id 2) (at 176.53 153.67 0)
       (effects (font (size 1.27 1.27)) hide)
     )
@@
       (effects (font (size 1.27 1.27)) (justify left))
     )
-    (property "Footprint" "Crystal:Crystal_SMD_3225-4Pin_3.2x2.5mm" (id 2) (at 222.25 48.26 0)
+    (property "Footprint" "ControlBoard:Crystal_SMD_3225-4Pin_3.2x2.5mm" (id 2) (at 222.25 48.26 0)
       (effects (font (size 1.27 1.27)) hide)
     )
@@
       (effects (font (size 1.27 1.27)) (justify left))
     )
-    (property "Footprint" "Capacitor_SMD:C_0603_1608Metric" (id 2) (at 209.2452 55.88 0)
+    (property "Footprint" "ControlBoard:C_0603_1608Metric" (id 2) (at 209.2452 55.88 0)
       (effects (font (size 1.27 1.27)) hide)
     )
@@
       (effects (font (size 1.27 1.27)) (justify left))
     )
-    (property "Footprint" "Capacitor_SMD:C_0603_1608Metric" (id 2) (at 238.4552 55.88 0)
+    (property "Footprint" "ControlBoard:C_0603_1608Metric" (id 2) (at 238.4552 55.88 0)
       (effects (font (size 1.27 1.27)) hide)
     )
@@
       (effects (font (size 1.27 1.27)) (justify left))
     )
-    (property "Footprint" "Capacitor_SMD:C_0603_1608Metric" (id 2) (at 261.3152 57.15 0)
+    (property "Footprint" "ControlBoard:C_0603_1608Metric" (id 2) (at 261.3152 57.15 0)
       (effects (font (size 1.27 1.27)) hide)
     )
@@
       (effects (font (size 1.27 1.27)) (justify left))
     )
-    (property "Footprint" "Resistor_SMD:R_0603_1608Metric" (id 2) (at 258.572 40.64 90)
+    (property "Footprint" "ControlBoard:R_0603_1608Metric" (id 2) (at 258.572 40.64 90)
       (effects (font (size 1.27 1.27)) hide)
     )
@@
       (effects (font (size 1.27 1.27)) (justify left))
     )
-    (property "Footprint" "Capacitor_SMD:C_0603_1608Metric" (id 2) (at 206.7052 130.81 0)
+    (property "Footprint" "ControlBoard:C_0603_1608Metric" (id 2) (at 206.7052 130.81 0)
       (effects (font (size 1.27 1.27)) hide)
     )
@@
       (effects (font (size 1.27 1.27)) (justify left))
     )
-    (property "Footprint" "Capacitor_SMD:C_0603_1608Metric" (id 2) (at 218.1352 130.81 0)
+    (property "Footprint" "ControlBoard:C_0603_1608Metric" (id 2) (at 218.1352 130.81 0)
       (effects (font (size 1.27 1.27)) hide)
     )
@@
       (effects (font (size 1.27 1.27)) (justify left))
     )
-    (property "Footprint" "Capacitor_SMD:C_0603_1608Metric" (id 2) (at 229.5652 130.81 0)
+    (property "Footprint" "ControlBoard:C_0603_1608Metric" (id 2) (at 229.5652 130.81 0)
       (effects (font (size 1.27 1.27)) hide)
     )
@@
       (effects (font (size 1.27 1.27)) (justify left))
     )
-    (property "Footprint" "Capacitor_SMD:C_0603_1608Metric" (id 2) (at 242.2652 130.81 0)
+    (property "Footprint" "ControlBoard:C_0603_1608Metric" (id 2) (at 242.2652 130.81 0)
       (effects (font (size 1.27 1.27)) hide)
     )
@@
       (effects (font (size 1.27 1.27)) (justify left))
     )
-    (property "Footprint" "Capacitor_SMD:C_0603_1608Metric" (id 2) (at 253.6952 130.81 0)
+    (property "Footprint" "ControlBoard:C_0603_1608Metric" (id 2) (at 253.6952 130.81 0)
       (effects (font (size 1.27 1.27)) hide)
     )
@@
       (effects (font (size 1.27 1.27)) (justify left))
     )
-    (property "Footprint" "Capacitor_SMD:C_0603_1608Metric" (id 2) (at 265.1252 130.81 0)
+    (property "Footprint" "ControlBoard:C_0603_1608Metric" (id 2) (at 265.1252 130.81 0)
       (effects (font (size 1.27 1.27)) hide)
     )
@@
       (effects (font (size 1.27 1.27)) (justify left))
     )
-    (property "Footprint" "Capacitor_SMD:C_0603_1608Metric" (id 2) (at 206.7052 160.02 0)
+    (property "Footprint" "ControlBoard:C_0603_1608Metric" (id 2) (at 206.7052 160.02 0)
       (effects (font (size 1.27 1.27)) hide)
     )
@@
       (effects (font (size 1.27 1.27)) (justify left))
     )
-    (property "Footprint" "Capacitor_SMD:C_0603_1608Metric" (id 2) (at 218.1352 160.02 0)
+    (property "Footprint" "ControlBoard:C_0603_1608Metric" (id 2) (at 218.1352 160.02 0)
       (effects (font (size 1.27 1.27)) hide)
     )
@@
       (effects (font (size 1.27 1.27)) (justify left))
     )
-    (property "Footprint" "Capacitor_SMD:C_0603_1608Metric" (id 2) (at 229.5652 160.02 0)
+    (property "Footprint" "ControlBoard:C_0603_1608Metric" (id 2) (at 229.5652 160.02 0)
       (effects (font (size 1.27 1.27)) hide)
     )
@@
       (effects (font (size 1.27 1.27)) (justify left))
     )
-    (property "Footprint" "Capacitor_SMD:C_0603_1608Metric" (id 2) (at 242.2652 160.02 0)
+    (property "Footprint" "ControlBoard:C_0603_1608Metric" (id 2) (at 242.2652 160.02 0)
       (effects (font (size 1.27 1.27)) hide)
     )
@@
       (effects (font (size 1.27 1.27)) (justify left))
     )
-    (property "Footprint" "Capacitor_SMD:C_0603_1608Metric" (id 2) (at 253.6952 160.02 0)
+    (property "Footprint" "ControlBoard:C_0603_1608Metric" (id 2) (at 253.6952 160.02 0)
       (effects (font (size 1.27 1.27)) hide)
     )
@@
       (effects (font (size 1.27 1.27)) (justify left))
     )
-    (property "Footprint" "Capacitor_SMD:C_0603_1608Metric" (id 2) (at 265.1252 160.02 0)
+    (property "Footprint" "ControlBoard:C_0603_1608Metric" (id 2) (at 265.1252 160.02 0)
       (effects (font (size 1.27 1.27)) hide)
     )
@@
       (effects (font (size 1.27 1.27)) hide)
     )
-    (property "Footprint" "LED_SMD:LED_0603_1608Metric" (id 2) (at 228.6 90.17 0)
+    (property "Footprint" "ControlBoard:LED_0603_1608Metric" (id 2) (at 228.6 90.17 0)
       (effects (font (size 1.27 1.27)) hide)
     )
@@
     (property "Reference" "R5" (id 0) (at 246.38 87.63 90))
     (property "Value" "1kR" (id 1) (at 251.46 91.44 90))
-    (property "Footprint" "Resistor_SMD:R_0603_1608Metric" (id 2) (at 246.38 88.392 90)
+    (property "Footprint" "ControlBoard:R_0603_1608Metric" (id 2) (at 246.38 88.392 90)
       (effects (font (size 1.27 1.27)) hide)
     )
@@
       (effects (font (size 1.27 1.27)) (justify left))
     )
-    (property "Footprint" "Resistor_SMD:R_0603_1608Metric" (id 2) (at 75.692 38.1 90)
-      (effects (font (size 1.27 1.27)) hide)
-    )
+    (property "Footprint" "ControlBoard:R_0603_1608Metric" (id 2) (at 75.692 38.1 90)
+      (effects (font (size 1.27 1.27)) hide)
+    )

Commit message: Modify and complete the circuit schematic to make the interface easier to wire.
Parts:
- renumbered C52 to C48, C53 to C49, C54 to C50, C55 to C51, C56 to C52, C57 to C53, C58 to C54, C59 to C55, C60 to C56, C61 to C57, C62 to C58, C63 to C59, C64 to C60, C65 to C61, C66 to C62, R4 to R5, R5 to R6, R6 to R7, U11 to U9
Other:
- title: MM32_Board -> MM32 Control Board

Commit message: Modify the ControlBoard schematic to add useful features.
Connections:
- net +3.3VP: no longer R6.1
- net LED1: now also U9.36 (PA2); no longer U9.1 (PE2)
- net PF0: now reaches U9.10 (PF0)
- net PF1: now reaches U9.11 (PF1)
- net PF2: now reaches U9.12 (PF2)
- net PF3: now reaches U9.13 (PF3)
- net PF4: now reaches U9.14 (PF4)
- net PF5: now reaches U9.15 (PF5)
- net PF6: now reaches U9.18 (PF6)
- net PF7: now reaches U9.19 (PF7)
- net PF8: now reaches U9.20 (PF8)
- net PF9: now reaches U9.21 (PF9)
- net PF10: now reaches U9.22 (PF10)
- net PC0: now reaches U9.26 (PC0)
- net PE6: now reaches U9.5 (PE6)
- net SPI3_CLK: now reaches U9.81 (PD12)
- net SPI3_MISO: now reaches U9.82 (PD13)
- net SPI3_MOSI: now reaches U9.85 (PD14)
- net SPI3_NSS: now reaches U9.86 (PD15)
- new net +3.3VA: R6.1
- no-connect marks 103 -> 86
