File: circuit/control_board/ControlMCU.kicad_sch (KiCad schematic)
At the start: 21 parts, among them U9 MM32F3277G9P, Y2 8MHz

Commit message: Update the main control board schematic to complete the SD card reader part.
Parts:
- renumbered C48 to C54, C49 to C55, C50 to C56, C51 to C57, C52 to C58, C53 to C59, C54 to C60, C55 to C61, C56 to C62, C57 to C63, C58 to C64, C59 to C65, C60 to C66, C61 to C67, C62 to C68
Connections:
- net PG4: now reaches U9.89 (PG4)
- net PC0: no longer names the net of U9.26 (PC0)
- net PE6: no longer names the net of U9.5 (PE6)
- net PF0: no longer names the net of U9.10 (PF0)
- net PF1: no longer names the net of U9.11 (PF1)
- net PF10: no longer names the net of U9.22 (PF10)
- net PF2: no longer names the net of U9.12 (PF2)
- net PF3: no longer names the net of U9.13 (PF3)
- net PF4: no longer names the net of U9.14 (PF4)
- net PF5: no longer names the net of U9.15 (PF5)
- net PF6: no longer names the net of U9.18 (PF6)
- net PF7: no longer names the net of U9.19 (PF7)
- net PF8: no longer names the net of U9.20 (PF8)
- net PF9: no longer names the net of U9.21 (PF9)
- no-connect marks 86 -> 98

Commit message: Updated the main control board schematic and switched the geomagnetometer interface sequence.
Connections:
- net PD10: now reaches U9.79 (PD10)
- net PG4: no longer names the net of U9.89 (PG4)
Changed lines of the file:
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@@
   (no_connect (at 80.01 151.13))
   (no_connect (at 161.29 80.01))
-  (no_connect (at 161.29 128.27))
+  (no_connect (at 161.29 102.87))
   (no_connect (at 52.07 105.41))
   (no_connect (at 90.17 151.13))
@@
     (stroke (width 0) (type default) (color 0 0 0 0))
   )
-  (wire (pts (xy 161.29 102.87) (xy 175.26 102.87))
+  (wire (pts (xy 161.29 128.27) (xy 175.26 128.27))
     (stroke (width 0) (type default) (color 0 0 0 0))
   )
@@
     (effects (font (size 1.27 1.27)) (justify left))
   )
-  (hierarchical_label "PG4" (shape output) (at 175.26 102.87 0)
-    (effects (font (size 1.27 1.27)) (justify left))
-  )
+  (hierarchical_label "PD10" (shape output) (at 175.26 128.27 0)
+    (effects (font (size 1.27 1.27)) (justify left))
+  )
