File: circuit/control_board/Coprocessor.kicad_sch (KiCad schematic)
At the start: 12 parts, among them J3 Conn_01x04, U6 MM32SPIN27PS, U7 π131M31, Y3 8MHz

Commit message: Update the main control board schematic and replace the magnetometer with RM3100.
Connections:
- net SPI2_NSS: now reaches U6.33 (PB12)
- net SPI2_CLK: now reaches U6.34 (PB13)
- net SPI2_MISO: now reaches U6.35 (PB14)
- net SPI2_MOSI: now reaches U6.36 (PB15)
- net PC6: now reaches U6.37 (PC6)
- net IIC1_SCL: no longer names the net of U6.29 (PB10)
- net IIC1_SDA: no longer names the net of U6.30 (PB11)
- net PB2: no longer names the net of U6.28 (PB2)
- no-connect marks 43 -> 41
Changed lines of the file:
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@@
   (title_block
     (title "MM32_Board")
-    (date "2022-02-28")
-    (rev "1.3.1")
+    (date "2022-03-02")
+    (rev "1.3.2")
   )
   (junction (at 254.635 158.75) (diameter 0) (color 0 0 0 0)
@@
   (junction (at 252.73 55.245) (diameter 0) (color 0 0 0 0)
   )
+  (no_connect (at 103.505 130.81))
   (no_connect (at 122.555 91.44))
   (no_connect (at 122.555 93.98))
+  (no_connect (at 108.585 130.81))
   (no_connect (at 252.095 146.05))
   (no_connect (at 230.505 146.05))
@@
   (no_connect (at 122.555 106.68))
   (no_connect (at 122.555 109.22))
-  (no_connect (at 122.555 111.76))
-  (no_connect (at 122.555 114.3))
-  (no_connect (at 122.555 116.84))
-  (no_connect (at 122.555 119.38))
   (no_connect (at 122.555 86.36))
   (no_connect (at 100.965 130.81))
   (no_connect (at 122.555 83.82))
-  (no_connect (at 122.555 121.92))
   (no_connect (at 98.425 130.81))
   (no_connect (at 95.885 130.81))
@@
   (no_connect (at 98.425 74.93))
   (no_connect (at 100.965 74.93))
+  (no_connect (at 106.045 130.81))
   (wire (pts (xy 227.965 140.97) (xy 230.505 140.97))
     (stroke (width 0) (type default) (color 0 0 0 0))
   )
-  (wire (pts (xy 106.045 130.81) (xy 106.045 149.86))
-    (stroke (width 0) (type default) (color 0 0 0 0))
-  )
   (wire (pts (xy 66.675 111.76) (xy 47.625 111.76))
     (stroke (width 0) (type default) (color 0 0 0 0))
   )
-  (wire (pts (xy 108.585 149.86) (xy 108.585 130.81))
-    (stroke (width 0) (type default) (color 0 0 0 0))
-  )
   (wire (pts (xy 243.205 98.425) (xy 252.095 98.425))
     (stroke (width 0) (type default) (color 0 0 0 0))
@@
     (stroke (width 0) (type default) (color 0 0 0 0))
   )
-  (wire (pts (xy 103.505 130.81) (xy 103.505 149.86))
-    (stroke (width 0) (type default) (color 0 0 0 0))
-  )
   (wire (pts (xy 75.565 55.88) (xy 75.565 74.93))
     (stroke (width 0) (type default) (color 0 0 0 0))
@@
     (stroke (width 0) (type default) (color 0 0 0 0))
   )
+  (wire (pts (xy 122.555 119.38) (xy 141.605 119.38))
+    (stroke (width 0) (type default) (color 0 0 0 0))
+  )
   (wire (pts (xy 166.37 104.14) (xy 166.37 114.935))
     (stroke (width 0) (type default) (color 0 0 0 0))
@@
     (stroke (width 0) (type default) (color 0 0 0 0))
   )
+  (wire (pts (xy 122.555 121.92) (xy 141.605 121.92))
+    (stroke (width 0) (type default) (color 0 0 0 0))
+  )
   (wire (pts (xy 156.21 101.6) (xy 166.37 101.6))
     (stroke (width 0) (type default) (color 0 0 0 0))
   )
+  (wire (pts (xy 122.555 114.3) (xy 141.605 114.3))
+    (stroke (width 0) (type default) (color 0 0 0 0))
+  )
   (wire (pts (xy 90.805 130.81) (xy 90.805 149.86))
     (stroke (width 0) (type default) (color 0 0 0 0))
@@
     (stroke (width 0) (type default) (color 0 0 0 0))
   )
+  (wire (pts (xy 122.555 116.84) (xy 141.605 116.84))
+    (stroke (width 0) (type default) (color 0 0 0 0))
+  )
   (wire (pts (xy 252.095 143.51) (xy 254.635 143.51))
     (stroke (width 0) (type default) (color 0 0 0 0))
@@
   )
   (polyline (pts (xy 267.97 29.845) (xy 190.5 29.845))
+    (stroke (width 0) (type default) (color 0 0 0 0))
+  )
+  (wire (pts (xy 122.555 111.76) (xy 141.605 111.76))
     (stroke (width 0) (type default) (color 0 0 0 0))
   )
@@
     (effects (font (size 1.27 1.27)) (justify right))
   )
-  (hierarchical_label "IIC1_SCL" (shape output) (at 106.045 149.86 270)
-    (effects (font (size 1.27 1.27)) (justify right))
+  (hierarchical_label "SPI2_NSS" (shape output) (at 141.605 121.92 0)
+    (effects (font (size 1.27 1.27)) (justify left))
   )
   (hierarchical_label "UART1_RX" (shape input) (at 222.25 148.59 180)
     (effects (font (size 1.27 1.27)) (justify right))
   )
+  (hierarchical_label "SPI2_MISO" (shape input) (at 141.605 116.84 0)
+    (effects (font (size 1.27 1.27)) (justify left))
+  )
+  (hierarchical_label "SPI2_CLK" (shape output) (at 141.605 119.38 0)
+    (effects (font (size 1.27 1.27)) (justify left))
+  )
   (hierarchical_label "SPI1_MOSI" (shape output) (at 80.645 149.86 270)
     (effects (font (size 1.27 1.27)) (justify right))
@@
     (effects (font (size 1.27 1.27)) (justify right))
   )
-  (hierarchical_label "IIC1_SDA" (shape bidirectional) (at 108.585 149.86 270)
-    (effects (font (size 1.27 1.27)) (justify right))
+  (hierarchical_label "PC6" (shape input) (at 141.605 111.76 0)
+    (effects (font (size 1.27 1.27)) (justify left))
   )
   (hierarchical_label "SPI1_NSS" (shape output) (at 83.185 149.86 270)
     (effects (font (size 1.27 1.27)) (justify right))
   )
-  (hierarchical_label "PB2" (shape input) (at 103.505 149.86 270)
-    (effects (font (size 1.27 1.27)) (justify right))
-  )
   (hierarchical_label "SPI1_MISO" (shape input) (at 78.105 149.86 270)
     (effects (font (size 1.27 1.27)) (justify right))
   )
+  (hierarchical_label "SPI2_MOSI" (shape output) (at 141.605 114.3 0)
+    (effects (font (size 1.27 1.27)) (justify left))
+  )
   (hierarchical_label "PA6" (shape input) (at 88.265 149.86 270)

Commit message: Modify and complete the circuit schematic to make the interface easier to wire.
Parts:
- renumbered C26 to C67, C27 to C68, C28 to C69, C29 to C70, R13 to R21, R14 to R22, R15 to R23, U6 to U13, U7 to U14
Connections:
- net LED1: now also U13.62 (PB9)
- net PC7: now reaches U13.38 (PC7)
- net PA7: no longer names the net of U13.23 (PA7)
- no-connect marks 41 -> 40
Other:
- title: MM32_Board -> MM32 Control Board

Commit message: Modify the main control board schematic, replace the IMU device and remove the isolation module.
Parts:
- removed C67: 100nF, ControlBoard:C_0603_1608Metric, symbol Device:C
- removed U14: π131M31, ControlBoard:SOIC-16_3.9x9.9mm_P1.27mm, symbol MM32_Periph:π131M31
Connections:
- net GNDA is gone; now on net GND: C68.2, C69.2, C70.2, J3.4 (Pin_4), R21.1, U13.12 (VSSA), U13.31 (VSS), U13.63 (VSS), Y3.2, Y3.4
- net UART_RX is gone; now on net UART1_RX: U13.43 (PA10)
- net UART_TX is gone; now on net UART1_TX: U13.42 (PA9)
- no-connect marks 40 -> 38
Other:
- note removed: "Isolation"
- moved on the sheet: C68, C69, C70, D3, R22, R23, Y3

Commit message: Modify the ControlBoard schematic to add useful features.
Parts:
- removed C68, C69: 18pF, ControlBoard:C_0603_1608Metric, symbol Device:C
- removed Y3: 8MHz, ControlBoard:Crystal_SMD_3225-4Pin_3.2x2.5mm, symbol Device:Crystal_GND24
- added R1, R25: 10kR, ControlBoard:R_0603_1608Metric, symbol Device:R
Connections:
- net +3.3VADC: now also R1.1, R25.1
- net LED1: now also U13.51 (PC10); no longer U13.62 (PB9)
- net IIC_SDA: now reaches U13.55 (PB3)
- net IIC_SDA: now also R1.2
- net IIC_CLK: now reaches U13.56 (PB4)
- net IIC_CLK: now also R25.2
- net PA6: no longer names the net of U13.22 (PA6)
- net XTAL_IN: no longer names the net of U13.5 (OSC_IN)
- net XTAL_OUT: no longer names the net of U13.6 (OSC_OUT)
- no-connect marks 38 -> 39
Other:
- note added: "RST"
- note removed: "XTAL & RST"
- moved on the sheet: C70, R23

Commit message: Slightly modify the ControlBoard package
Parts:
- U13: footprint Package_QFP:LQFP-64_10x10mm_P0.5mm -> ControlBoard:LQFP-64_10x10mm_P0.5mm
Changed lines of the file:
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@@
     (property "Reference" "U13" (id 0) (at 118.11 130.81 0))
     (property "Value" "MM32SPIN27PS" (id 1) (at 123.825 133.35 0))
-    (property "Footprint" "Package_QFP:LQFP-64_10x10mm_P0.5mm" (id 2) (at 94.615 137.16 0)
+    (property "Footprint" "ControlBoard:LQFP-64_10x10mm_P0.5mm" (id 2) (at 94.615 137.16 0)
       (effects (font (size 1.27 1.27)) hide)
     )

Commit message: Fixed part of the control board circuit and added SD card reading chip.
Parts:
- renumbered C70 to C67, J3 to J5, R21 to R11, R1 to R12, R25 to R13, R23 to R14, R22 to R15, U13 to U12
Changed lines of the file:
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@@
   (symbol (lib_id "power:GND") (at 78.105 55.88 180) (unit 1)
     (in_bom yes) (on_board yes)
-    (property "Reference" "#PWR0199" (id 0) (at 78.105 49.53 0)
+    (property "Reference" "#PWR0174" (id 0) (at 78.105 49.53 0)
       (effects (font (size 1.27 1.27)) hide)
     )
@@
   (symbol (lib_id "power:+3.3VADC") (at 159.385 132.715 0) (unit 1)
     (in_bom yes) (on_board yes)
-    (property "Reference" "#PWR028" (id 0) (at 163.195 133.985 0)
+    (property "Reference" "#PWR0178" (id 0) (at 163.195 133.985 0)
       (effects (font (size 1.27 1.27)) hide)
     )
@@
   (symbol (lib_id "power:GND") (at 231.14 108.585 0) (unit 1)
     (in_bom yes) (on_board yes)
-    (property "Reference" "#PWR0204" (id 0) (at 231.14 114.935 0)
+    (property "Reference" "#PWR0183" (id 0) (at 231.14 114.935 0)
       (effects (font (size 1.27 1.27)) hide)
     )
@@
   (symbol (lib_id "power:+3.3VADC") (at 254.635 138.43 270) (unit 1)
     (in_bom yes) (on_board yes)
-    (property "Reference" "#PWR0188" (id 0) (at 253.365 142.24 0)
+    (property "Reference" "#PWR0184" (id 0) (at 253.365 142.24 0)
       (effects (font (size 1.27 1.27)) hide)
     )
@@
   (symbol (lib_id "power:+3.3VADC") (at 231.14 80.645 0) (unit 1)
     (in_bom yes) (on_board yes)
-    (property "Reference" "#PWR0189" (id 0) (at 234.95 81.915 0)
+    (property "Reference" "#PWR0182" (id 0) (at 234.95 81.915 0)
       (effects (font (size 1.27 1.27)) hide)
     )
@@
   (symbol (lib_id "Connector_Generic:Conn_01x04") (at 170.18 105.41 0) (unit 1)
     (in_bom yes) (on_board yes)
-    (property "Reference" "J3" (id 0) (at 170.18 93.98 0)
+    (property "Reference" "J5" (id 0) (at 170.18 93.98 0)
       (effects (font (size 1.27 1.27)) (justify left))
     )
@@
   (symbol (lib_id "power:+3.3VADC") (at 166.37 85.725 0) (unit 1)
     (in_bom yes) (on_board yes)
-    (property "Reference" "#PWR0178" (id 0) (at 170.18 86.995 0)
+    (property "Reference" "#PWR0179" (id 0) (at 170.18 86.995 0)
       (effects (font (size 1.27 1.27)) hide)
     )
@@
   (symbol (lib_id "Device:R") (at 85.725 65.405 0) (unit 1)
     (in_bom yes) (on_board yes)
-    (property "Reference" "R21" (id 0) (at 87.503 64.2366 0)
+    (property "Reference" "R11" (id 0) (at 87.503 64.2366 0)
       (effects (font (size 1.27 1.27)) (justify left))
     )
@@
   (symbol (lib_id "power:+3.3VADC") (at 168.91 132.715 0) (unit 1)
     (in_bom yes) (on_board yes)
-    (property "Reference" "#PWR030" (id 0) (at 172.72 133.985 0)
+    (property "Reference" "#PWR0181" (id 0) (at 172.72 133.985 0)
       (effects (font (size 1.27 1.27)) hide)
     )
@@
   (symbol (lib_id "power:GND") (at 47.625 111.76 270) (unit 1)
     (in_bom yes) (on_board yes)
-    (property "Reference" "#PWR0198" (id 0) (at 41.275 111.76 0)
+    (property "Reference" "#PWR0171" (id 0) (at 41.275 111.76 0)
       (effects (font (size 1.27 1.27)) hide)
     )
@@
   (symbol (lib_id "power:GND") (at 166.37 114.935 0) (unit 1)
     (in_bom yes) (on_board yes)
-    (property "Reference" "#PWR0197" (id 0) (at 166.37 121.285 0)
+    (property "Reference" "#PWR0180" (id 0) (at 166.37 121.285 0)
       (effects (font (size 1.27 1.27)) hide)
     )
@@
   (symbol (lib_id "Device:R") (at 241.935 138.43 270) (unit 1)
     (in_bom yes) (on_board yes)
-    (property "Reference" "R22" (id 0) (at 241.935 135.89 90))
+    (property "Reference" "R15" (id 0) (at 241.935 135.89 90))
     (property "Value" "1kR" (id 1) (at 241.935 140.97 90))
     (property "Footprint" "ControlBoard:R_0603_1608Metric" (id 2) (at 241.935 136.652 90)
@@
   (symbol (lib_id "Device:R") (at 168.91 141.605 0) (unit 1)
     (in_bom yes) (on_board yes)
-    (property "Reference" "R25" (id 0) (at 170.688 140.4366 0)
+    (property "Reference" "R13" (id 0) (at 170.688 140.4366 0)
       (effects (font (size 1.27 1.27)) (justify left))
     )
@@
   (symbol (lib_id "Device:R") (at 231.14 89.535 0) (unit 1)
     (in_bom yes) (on_board yes)
-    (property "Reference" "R23" (id 0) (at 232.918 88.3666 0)
+    (property "Reference" "R14" (id 0) (at 232.918 88.3666 0)
       (effects (font (size 1.27 1.27)) (justify left))
     )
@@
   (symbol (lib_id "power:GND") (at 111.125 149.86 0) (unit 1)
     (in_bom yes) (on_board yes)
-    (property "Reference" "#PWR0205" (id 0) (at 111.125 156.21 0)
+    (property "Reference" "#PWR0176" (id 0) (at 111.125 156.21 0)
       (effects (font (size 1.27 1.27)) hide)
     )
@@
   (symbol (lib_id "Device:R") (at 159.385 141.605 0) (unit 1)
     (in_bom yes) (on_board yes)
-    (property "Reference" "R1" (id 0) (at 161.163 140.4366 0)
+    (property "Reference" "R12" (id 0) (at 161.163 140.4366 0)
       (effects (font (size 1.27 1.27)) (justify left))
     )
@@
   (symbol (lib_id "Device:C") (at 231.14 102.235 0) (unit 1)
     (in_bom yes) (on_board yes)
-    (property "Reference" "C70" (id 0) (at 234.061 101.0666 0)
+    (property "Reference" "C67" (id 0) (at 234.061 101.0666 0)
       (effects (font (size 1.27 1.27)) (justify left))
     )
@@
   (symbol (lib_id "power:GND") (at 85.725 55.88 180) (unit 1)
     (in_bom yes) (on_board yes)
-    (property "Reference" "#PWR0200" (id 0) (at 85.725 49.53 0)
+    (property "Reference" "#PWR0175" (id 0) (at 85.725 49.53 0)
       (effects (font (size 1.27 1.27)) hide)
     )
@@
   (symbol (lib_id "MM32_Periph:MM32SPIN27PS") (at 69.215 128.27 0) (unit 1)
     (in_bom yes) (on_board yes)
-    (property "Reference" "U13" (id 0) (at 118.11 130.81 0))
+    (property "Reference" "U12" (id 0) (at 118.11 130.81 0))
     (property "Value" "MM32SPIN27PS" (id 1) (at 123.825 133.35 0))
     (property "Footprint" "ControlBoard:LQFP-64_10x10mm_P0.5mm" (id 2) (at 94.615 137.16 0)
