File: circuit/control_board/Coprocessor.kicad_sch (KiCad schematic)
At the start: 9 parts, among them J5 Conn_01x04, U12 MM32SPIN27PS

Commit message: Update the main control board schematic to complete the SD card reader part.
Parts:
- renumbered C67 to C73
Changed lines of the file:
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@@
   (title_block
     (title "MM32 Control Board")
-    (date "2022-05-18")
-    (rev "1.5.4")
+    (date "2022-07-11")
+    (rev "1.6.1")
   )
   (junction (at 231.14 95.885) (diameter 0) (color 0 0 0 0)
@@
   (symbol (lib_id "power:GND") (at 78.105 55.88 180) (unit 1)
     (in_bom yes) (on_board yes)
-    (property "Reference" "#PWR0174" (id 0) (at 78.105 49.53 0)
+    (property "Reference" "#PWR0186" (id 0) (at 78.105 49.53 0)
       (effects (font (size 1.27 1.27)) hide)
     )
@@
   (symbol (lib_id "power:+3.3VADC") (at 159.385 132.715 0) (unit 1)
     (in_bom yes) (on_board yes)
-    (property "Reference" "#PWR0178" (id 0) (at 163.195 133.985 0)
+    (property "Reference" "#PWR0190" (id 0) (at 163.195 133.985 0)
       (effects (font (size 1.27 1.27)) hide)
     )
@@
   (symbol (lib_id "power:GND") (at 231.14 108.585 0) (unit 1)
     (in_bom yes) (on_board yes)
-    (property "Reference" "#PWR0183" (id 0) (at 231.14 114.935 0)
+    (property "Reference" "#PWR0195" (id 0) (at 231.14 114.935 0)
       (effects (font (size 1.27 1.27)) hide)
     )
@@
   (symbol (lib_id "power:+3.3VADC") (at 254.635 138.43 270) (unit 1)
     (in_bom yes) (on_board yes)
-    (property "Reference" "#PWR0184" (id 0) (at 253.365 142.24 0)
+    (property "Reference" "#PWR0196" (id 0) (at 253.365 142.24 0)
       (effects (font (size 1.27 1.27)) hide)
     )
@@
   (symbol (lib_id "power:+3.3VADC") (at 231.14 80.645 0) (unit 1)
     (in_bom yes) (on_board yes)
-    (property "Reference" "#PWR0182" (id 0) (at 234.95 81.915 0)
+    (property "Reference" "#PWR0194" (id 0) (at 234.95 81.915 0)
       (effects (font (size 1.27 1.27)) hide)
     )
@@
   (symbol (lib_id "power:+3.3VADC") (at 75.565 55.88 0) (unit 1)
     (in_bom yes) (on_board yes)
-    (property "Reference" "#PWR0173" (id 0) (at 79.375 57.15 0)
+    (property "Reference" "#PWR0185" (id 0) (at 79.375 57.15 0)
       (effects (font (size 1.27 1.27)) hide)
     )
@@
   (symbol (lib_id "power:+3.3VADC") (at 166.37 85.725 0) (unit 1)
     (in_bom yes) (on_board yes)
-    (property "Reference" "#PWR0179" (id 0) (at 170.18 86.995 0)
+    (property "Reference" "#PWR0191" (id 0) (at 170.18 86.995 0)
       (effects (font (size 1.27 1.27)) hide)
     )
@@
   (symbol (lib_id "power:+3.3VADC") (at 168.91 132.715 0) (unit 1)
     (in_bom yes) (on_board yes)
-    (property "Reference" "#PWR0181" (id 0) (at 172.72 133.985 0)
+    (property "Reference" "#PWR0193" (id 0) (at 172.72 133.985 0)
       (effects (font (size 1.27 1.27)) hide)
     )
@@
   (symbol (lib_id "power:GND") (at 47.625 111.76 270) (unit 1)
     (in_bom yes) (on_board yes)
-    (property "Reference" "#PWR0171" (id 0) (at 41.275 111.76 0)
+    (property "Reference" "#PWR0183" (id 0) (at 41.275 111.76 0)
       (effects (font (size 1.27 1.27)) hide)
     )
@@
   (symbol (lib_id "power:GND") (at 166.37 114.935 0) (unit 1)
     (in_bom yes) (on_board yes)
-    (property "Reference" "#PWR0180" (id 0) (at 166.37 121.285 0)
+    (property "Reference" "#PWR0192" (id 0) (at 166.37 121.285 0)
       (effects (font (size 1.27 1.27)) hide)
     )
@@
   (symbol (lib_id "power:+3.3VADC") (at 113.665 149.86 180) (unit 1)
     (in_bom yes) (on_board yes)
-    (property "Reference" "#PWR0177" (id 0) (at 109.855 148.59 0)
+    (property "Reference" "#PWR0189" (id 0) (at 109.855 148.59 0)
       (effects (font (size 1.27 1.27)) hide)
     )
@@
   (symbol (lib_id "power:GND") (at 111.125 149.86 0) (unit 1)
     (in_bom yes) (on_board yes)
-    (property "Reference" "#PWR0176" (id 0) (at 111.125 156.21 0)
+    (property "Reference" "#PWR0188" (id 0) (at 111.125 156.21 0)
       (effects (font (size 1.27 1.27)) hide)
     )
@@
   (symbol (lib_id "power:+3.3VADC") (at 47.625 114.3 90) (unit 1)
     (in_bom yes) (on_board yes)
-    (property "Reference" "#PWR0172" (id 0) (at 48.895 110.49 0)
+    (property "Reference" "#PWR0184" (id 0) (at 48.895 110.49 0)
       (effects (font (size 1.27 1.27)) hide)
     )
@@
   (symbol (lib_id "Device:C") (at 231.14 102.235 0) (unit 1)
     (in_bom yes) (on_board yes)
-    (property "Reference" "C67" (id 0) (at 234.061 101.0666 0)
+    (property "Reference" "C73" (id 0) (at 234.061 101.0666 0)
       (effects (font (size 1.27 1.27)) (justify left))
     )
@@
   (symbol (lib_id "power:GND") (at 85.725 55.88 180) (unit 1)
     (in_bom yes) (on_board yes)
-    (property "Reference" "#PWR0175" (id 0) (at 85.725 49.53 0)
-      (effects (font (size 1.27 1.27)) hide)
-    )
+    (property "Reference" "#PWR0187" (id 0) (at 85.725 49.53 0)
+      (effects (font (size 1.27 1.27)) hide)
+    )
