File: circuit/control_board/Debugger.kicad_sch (KiCad schematic)
At the start: 6 parts, among them M1 Debugger, SW1 SW_DIP_x02, U12 CH440R

Commit message: Modified the circuitry of the main control board to add a microcontroller for reading information from the magnetometer and IMU. Modified the SPI connection port of the Process MCU.
Parts:
- C67, C68: footprint Capacitor_SMD:C_0603_1608Metric -> ControlBoard:C_0603_1608Metric
- M1: footprint MM32_Library:Gernic_Debugger -> ControlBoard:Gernic_Debugger
- R7: footprint Resistor_SMD:R_0603_1608Metric -> ControlBoard:R_0603_1608Metric
- SW1: footprint Button_Switch_SMD:SW_DIP_SPSTx02_Slide_Copal_CHS-02B_W7.62mm_P1.27mm -> ControlBoard:SW_DIP_SPSTx02_Slide_Copal_CHS-02B_W7.62mm_P1.27mm
- U12: footprint Package_SO:TSSOP-16_4.4x5mm_P0.65mm -> ControlBoard:TSSOP-16_4.4x5mm_P0.65mm
Changed lines of the file:
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@@
   (title_block
     (title "MM32_Board")
-    (date "2022-02-09")
-    (rev "1.2.3")
+    (date "2022-02-28")
+    (rev "1.3.1")
   )
   (junction (at 229.235 107.95) (diameter 0) (color 0 0 0 0)
@@
     (property "Reference" "M1" (id 0) (at 97.79 100.965 0))
     (property "Value" "Debugger" (id 1) (at 101.6 116.205 0))
-    (property "Footprint" "MM32_Library:Gernic_Debugger" (id 2) (at 97.79 100.965 0)
+    (property "Footprint" "ControlBoard:Gernic_Debugger" (id 2) (at 97.79 100.965 0)
       (effects (font (size 1.27 1.27)) hide)
     )
@@
     (property "Reference" "U12" (id 0) (at 187.325 95.885 0))
     (property "Value" "CH440R" (id 1) (at 197.485 121.285 0))
-    (property "Footprint" "Package_SO:TSSOP-16_4.4x5mm_P0.65mm" (id 2) (at 194.945 123.825 0)
+    (property "Footprint" "ControlBoard:TSSOP-16_4.4x5mm_P0.65mm" (id 2) (at 194.945 123.825 0)
       (effects (font (size 1.27 1.27)) hide)
     )
@@
       (effects (font (size 1.27 1.27)) (justify left))
     )
-    (property "Footprint" "Capacitor_SMD:C_0603_1608Metric" (id 2) (at 134.3152 111.76 0)
+    (property "Footprint" "ControlBoard:C_0603_1608Metric" (id 2) (at 134.3152 111.76 0)
       (effects (font (size 1.27 1.27)) hide)
     )
@@
       (effects (font (size 1.27 1.27)) (justify right) hide)
     )
-    (property "Footprint" "Button_Switch_SMD:SW_DIP_SPSTx02_Slide_Copal_CHS-02B_W7.62mm_P1.27mm" (id 2) (at 231.775 120.015 0)
+    (property "Footprint" "ControlBoard:SW_DIP_SPSTx02_Slide_Copal_CHS-02B_W7.62mm_P1.27mm" (id 2) (at 231.775 120.015 0)
       (effects (font (size 1.27 1.27)) hide)
     )
@@
     (property "Reference" "R7" (id 0) (at 233.045 97.79 0))
     (property "Value" "10kR" (id 1) (at 233.68 100.33 0))
-    (property "Footprint" "Resistor_SMD:R_0603_1608Metric" (id 2) (at 227.457 97.79 90)
+    (property "Footprint" "ControlBoard:R_0603_1608Metric" (id 2) (at 227.457 97.79 90)
       (effects (font (size 1.27 1.27)) hide)
     )
@@
       (effects (font (size 1.27 1.27)) (justify left))
     )
-    (property "Footprint" "Capacitor_SMD:C_0603_1608Metric" (id 2) (at 144.4752 111.76 0)
-      (effects (font (size 1.27 1.27)) hide)
-    )
+    (property "Footprint" "ControlBoard:C_0603_1608Metric" (id 2) (at 144.4752 111.76 0)
+      (effects (font (size 1.27 1.27)) hide)
+    )

Commit message: Modify and complete the circuit schematic to make the interface easier to wire.
Parts:
- renumbered C67 to C63, C68 to C64, R7 to R8, U12 to U10
Other:
- title: MM32_Board -> MM32 Control Board
Changed lines of the file:
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@@
   (paper "A4")
   (title_block
-    (title "MM32_Board")
-    (date "2022-03-02")
-    (rev "1.3.2")
+    (title "MM32 Control Board")
+    (date "2022-03-03")
+    (rev "1.3.3")
   )
   (junction (at 229.235 107.95) (diameter 0) (color 0 0 0 0)
@@
   (symbol (lib_id "power:GND") (at 123.19 131.445 0) (unit 1)
     (in_bom yes) (on_board yes)
-    (property "Reference" "#PWR0165" (id 0) (at 123.19 137.795 0)
+    (property "Reference" "#PWR0149" (id 0) (at 123.19 137.795 0)
       (effects (font (size 1.27 1.27)) hide)
     )
@@
   (symbol (lib_id "power:GND") (at 88.9 131.445 0) (unit 1)
     (in_bom yes) (on_board yes)
-    (property "Reference" "#PWR0163" (id 0) (at 88.9 137.795 0)
+    (property "Reference" "#PWR0147" (id 0) (at 88.9 137.795 0)
       (effects (font (size 1.27 1.27)) hide)
     )
@@
   (symbol (lib_id "power:GND") (at 143.51 131.445 0) (unit 1)
     (in_bom yes) (on_board yes)
-    (property "Reference" "#PWR0169" (id 0) (at 143.51 137.795 0)
+    (property "Reference" "#PWR0153" (id 0) (at 143.51 137.795 0)
       (effects (font (size 1.27 1.27)) hide)
     )
@@
   (symbol (lib_id "MM32_Periph:CH440R") (at 186.055 120.015 0) (unit 1)
     (in_bom yes) (on_board yes)
-    (property "Reference" "U12" (id 0) (at 187.325 95.885 0))
+    (property "Reference" "U10" (id 0) (at 187.325 95.885 0))
     (property "Value" "CH440R" (id 1) (at 197.485 121.285 0))
     (property "Footprint" "ControlBoard:TSSOP-16_4.4x5mm_P0.65mm" (id 2) (at 194.945 123.825 0)
@@
   (symbol (lib_id "Device:C") (at 133.35 107.95 0) (unit 1)
     (in_bom yes) (on_board yes)
-    (property "Reference" "C67" (id 0) (at 136.271 106.7816 0)
+    (property "Reference" "C63" (id 0) (at 136.271 106.7816 0)
       (effects (font (size 1.27 1.27)) (justify left))
     )
@@
   (symbol (lib_id "power:+5V") (at 143.51 88.265 0) (unit 1)
     (in_bom yes) (on_board yes)
-    (property "Reference" "#PWR0168" (id 0) (at 143.51 92.075 0)
+    (property "Reference" "#PWR0152" (id 0) (at 143.51 92.075 0)
       (effects (font (size 1.27 1.27)) hide)
     )
@@
   (symbol (lib_id "power:GND") (at 133.35 131.445 0) (unit 1)
     (in_bom yes) (on_board yes)
-    (property "Reference" "#PWR0167" (id 0) (at 133.35 137.795 0)
+    (property "Reference" "#PWR0151" (id 0) (at 133.35 137.795 0)
       (effects (font (size 1.27 1.27)) hide)
     )
@@
   (symbol (lib_id "power:+5V") (at 208.915 86.995 0) (unit 1)
     (in_bom yes) (on_board yes)
-    (property "Reference" "#PWR0172" (id 0) (at 208.915 90.805 0)
+    (property "Reference" "#PWR0156" (id 0) (at 208.915 90.805 0)
       (effects (font (size 1.27 1.27)) hide)
     )
@@
   (symbol (lib_id "power:GND") (at 177.8 130.81 0) (unit 1)
     (in_bom yes) (on_board yes)
-    (property "Reference" "#PWR0170" (id 0) (at 177.8 137.16 0)
+    (property "Reference" "#PWR0154" (id 0) (at 177.8 137.16 0)
       (effects (font (size 1.27 1.27)) hide)
     )
@@
   (symbol (lib_id "power:+5V") (at 88.9 88.265 0) (unit 1)
     (in_bom yes) (on_board yes)
-    (property "Reference" "#PWR0162" (id 0) (at 88.9 92.075 0)
+    (property "Reference" "#PWR0146" (id 0) (at 88.9 92.075 0)
       (effects (font (size 1.27 1.27)) hide)
     )
@@
   (symbol (lib_id "power:+5V") (at 133.35 88.265 0) (unit 1)
     (in_bom yes) (on_board yes)
-    (property "Reference" "#PWR0166" (id 0) (at 133.35 92.075 0)
+    (property "Reference" "#PWR0150" (id 0) (at 133.35 92.075 0)
       (effects (font (size 1.27 1.27)) hide)
     )
@@
   (symbol (lib_id "Device:R") (at 229.235 97.79 0) (unit 1)
     (in_bom yes) (on_board yes)
-    (property "Reference" "R7" (id 0) (at 233.045 97.79 0))
+    (property "Reference" "R8" (id 0) (at 233.045 97.79 0))
     (property "Value" "10kR" (id 1) (at 233.68 100.33 0))
     (property "Footprint" "ControlBoard:R_0603_1608Metric" (id 2) (at 227.457 97.79 90)
@@
   (symbol (lib_id "power:GND") (at 229.235 130.81 0) (unit 1)
     (in_bom yes) (on_board yes)
-    (property "Reference" "#PWR0174" (id 0) (at 229.235 137.16 0)
+    (property "Reference" "#PWR0158" (id 0) (at 229.235 137.16 0)
       (effects (font (size 1.27 1.27)) hide)
     )
@@
   (symbol (lib_id "power:+5V") (at 123.19 88.265 0) (unit 1)
     (in_bom yes) (on_board yes)
-    (property "Reference" "#PWR0164" (id 0) (at 123.19 92.075 0)
+    (property "Reference" "#PWR0148" (id 0) (at 123.19 92.075 0)
       (effects (font (size 1.27 1.27)) hide)
     )
@@
   (symbol (lib_id "power:GND") (at 205.105 130.81 0) (unit 1)
     (in_bom yes) (on_board yes)
-    (property "Reference" "#PWR0171" (id 0) (at 205.105 137.16 0)
+    (property "Reference" "#PWR0155" (id 0) (at 205.105 137.16 0)
       (effects (font (size 1.27 1.27)) hide)
     )
@@
   (symbol (lib_id "Device:C") (at 143.51 107.95 0) (unit 1)
     (in_bom yes) (on_board yes)
-    (property "Reference" "C68" (id 0) (at 146.431 106.7816 0)
+    (property "Reference" "C64" (id 0) (at 146.431 106.7816 0)
       (effects (font (size 1.27 1.27)) (justify left))
     )
@@
   (symbol (lib_id "power:+5V") (at 229.235 86.995 0) (unit 1)
     (in_bom yes) (on_board yes)
-    (property "Reference" "#PWR0173" (id 0) (at 229.235 90.805 0)
-      (effects (font (size 1.27 1.27)) hide)
-    )
+    (property "Reference" "#PWR0157" (id 0) (at 229.235 90.805 0)
+      (effects (font (size 1.27 1.27)) hide)
+    )

Commit message: Modify the main control board schematic, replace the IMU device and remove the isolation module.
Other:
- moved on the sheet: C63, C64, M1, R8, SW1, U10
