File: circuit/control_board/Debugger.kicad_sch (KiCad schematic)
At the start: 6 parts, among them M1 Debugger, SW1 SW_DIP_x02, U10 CH440R

Commit message: Update the main control board schematic to complete the SD card reader part.
Parts:
- renumbered C63 to C69, C64 to C70
Changed lines of the file:
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@@
   (title_block
     (title "MM32 Control Board")
-    (date "2022-05-18")
-    (rev "1.5.4")
+    (date "2022-07-11")
+    (rev "1.6.1")
   )
   (junction (at 216.535 102.87) (diameter 0) (color 0 0 0 0)
@@
   (symbol (lib_id "power:GND") (at 110.49 126.365 0) (unit 1)
     (in_bom yes) (on_board yes)
-    (property "Reference" "#PWR0150" (id 0) (at 110.49 132.715 0)
+    (property "Reference" "#PWR0162" (id 0) (at 110.49 132.715 0)
       (effects (font (size 1.27 1.27)) hide)
     )
@@
   (symbol (lib_id "power:GND") (at 76.2 126.365 0) (unit 1)
     (in_bom yes) (on_board yes)
-    (property "Reference" "#PWR0148" (id 0) (at 76.2 132.715 0)
+    (property "Reference" "#PWR0160" (id 0) (at 76.2 132.715 0)
       (effects (font (size 1.27 1.27)) hide)
     )
@@
   (symbol (lib_id "power:GND") (at 130.81 126.365 0) (unit 1)
     (in_bom yes) (on_board yes)
-    (property "Reference" "#PWR0154" (id 0) (at 130.81 132.715 0)
+    (property "Reference" "#PWR0166" (id 0) (at 130.81 132.715 0)
       (effects (font (size 1.27 1.27)) hide)
     )
@@
   (symbol (lib_id "Device:C") (at 120.65 102.87 0) (unit 1)
     (in_bom yes) (on_board yes)
-    (property "Reference" "C63" (id 0) (at 123.571 101.7016 0)
+    (property "Reference" "C69" (id 0) (at 123.571 101.7016 0)
       (effects (font (size 1.27 1.27)) (justify left))
     )
@@
   (symbol (lib_id "power:+5V") (at 130.81 83.185 0) (unit 1)
     (in_bom yes) (on_board yes)
-    (property "Reference" "#PWR0153" (id 0) (at 130.81 86.995 0)
+    (property "Reference" "#PWR0165" (id 0) (at 130.81 86.995 0)
       (effects (font (size 1.27 1.27)) hide)
     )
@@
   (symbol (lib_id "power:GND") (at 120.65 126.365 0) (unit 1)
     (in_bom yes) (on_board yes)
-    (property "Reference" "#PWR0152" (id 0) (at 120.65 132.715 0)
+    (property "Reference" "#PWR0164" (id 0) (at 120.65 132.715 0)
       (effects (font (size 1.27 1.27)) hide)
     )
@@
   (symbol (lib_id "power:+5V") (at 196.215 81.915 0) (unit 1)
     (in_bom yes) (on_board yes)
-    (property "Reference" "#PWR0157" (id 0) (at 196.215 85.725 0)
+    (property "Reference" "#PWR0169" (id 0) (at 196.215 85.725 0)
       (effects (font (size 1.27 1.27)) hide)
     )
@@
   (symbol (lib_id "power:GND") (at 165.1 125.73 0) (unit 1)
     (in_bom yes) (on_board yes)
-    (property "Reference" "#PWR0155" (id 0) (at 165.1 132.08 0)
+    (property "Reference" "#PWR0167" (id 0) (at 165.1 132.08 0)
       (effects (font (size 1.27 1.27)) hide)
     )
@@
   (symbol (lib_id "power:+5V") (at 76.2 83.185 0) (unit 1)
     (in_bom yes) (on_board yes)
-    (property "Reference" "#PWR0147" (id 0) (at 76.2 86.995 0)
+    (property "Reference" "#PWR0159" (id 0) (at 76.2 86.995 0)
       (effects (font (size 1.27 1.27)) hide)
     )
@@
   (symbol (lib_id "power:+5V") (at 120.65 83.185 0) (unit 1)
     (in_bom yes) (on_board yes)
-    (property "Reference" "#PWR0151" (id 0) (at 120.65 86.995 0)
+    (property "Reference" "#PWR0163" (id 0) (at 120.65 86.995 0)
       (effects (font (size 1.27 1.27)) hide)
     )
@@
   (symbol (lib_id "power:GND") (at 216.535 125.73 0) (unit 1)
     (in_bom yes) (on_board yes)
-    (property "Reference" "#PWR0159" (id 0) (at 216.535 132.08 0)
+    (property "Reference" "#PWR0171" (id 0) (at 216.535 132.08 0)
       (effects (font (size 1.27 1.27)) hide)
     )
@@
   (symbol (lib_id "power:+5V") (at 110.49 83.185 0) (unit 1)
     (in_bom yes) (on_board yes)
-    (property "Reference" "#PWR0149" (id 0) (at 110.49 86.995 0)
+    (property "Reference" "#PWR0161" (id 0) (at 110.49 86.995 0)
       (effects (font (size 1.27 1.27)) hide)
     )
@@
   (symbol (lib_id "power:GND") (at 192.405 125.73 0) (unit 1)
     (in_bom yes) (on_board yes)
-    (property "Reference" "#PWR0156" (id 0) (at 192.405 132.08 0)
+    (property "Reference" "#PWR0168" (id 0) (at 192.405 132.08 0)
       (effects (font (size 1.27 1.27)) hide)
     )
@@
   (symbol (lib_id "Device:C") (at 130.81 102.87 0) (unit 1)
     (in_bom yes) (on_board yes)
-    (property "Reference" "C64" (id 0) (at 133.731 101.7016 0)
+    (property "Reference" "C70" (id 0) (at 133.731 101.7016 0)
       (effects (font (size 1.27 1.27)) (justify left))
     )
@@
   (symbol (lib_id "power:+5V") (at 216.535 81.915 0) (unit 1)
     (in_bom yes) (on_board yes)
-    (property "Reference" "#PWR0158" (id 0) (at 216.535 85.725 0)
-      (effects (font (size 1.27 1.27)) hide)
-    )
+    (property "Reference" "#PWR0170" (id 0) (at 216.535 85.725 0)
+      (effects (font (size 1.27 1.27)) hide)
+    )
