File: circuit/control_board/Power.kicad_sch (KiCad schematic)
At the start: 10 parts, among them J2 Conn_01x08, U10 HX9193, U9 HX9193

Commit message: Modified the circuitry of the main control board to add a microcontroller for reading information from the magnetometer and IMU. Modified the SPI connection port of the Process MCU.
Parts:
- C45, C46, C47, C48, C49, C50, C51: footprint Capacitor_SMD:C_0603_1608Metric -> ControlBoard:C_0603_1608Metric
- J2: footprint Connector_JST:JST_PH_S8B-PH-K_1x08_P2.00mm_Horizontal -> ControlBoard:JST_PH_S8B-PH-K_1x08_P2.00mm_Horizontal
- U10, U9: footprint Package_TO_SOT_SMD:SOT-23-5 -> ControlBoard:SOT-23-5
Changed lines of the file:
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@@
   (title_block
     (title "MM32_Board")
-    (date "2022-02-09")
-    (rev "1.2.3")
+    (date "2022-02-28")
+    (rev "1.3.1")
   )
   (junction (at 240.03 102.235) (diameter 0) (color 0 0 0 0)
@@
     (property "Reference" "U9" (id 0) (at 140.97 98.425 0))
     (property "Value" "HX9193" (id 1) (at 149.86 111.125 0))
-    (property "Footprint" "Package_TO_SOT_SMD:SOT-23-5" (id 2) (at 146.05 113.665 0)
+    (property "Footprint" "ControlBoard:SOT-23-5" (id 2) (at 146.05 113.665 0)
       (effects (font (size 1.27 1.27)) hide)
     )
@@
       (effects (font (size 1.27 1.27)) (justify left))
     )
-    (property "Footprint" "Capacitor_SMD:C_0603_1608Metric" (id 2) (at 169.8752 120.015 0)
+    (property "Footprint" "ControlBoard:C_0603_1608Metric" (id 2) (at 169.8752 120.015 0)
       (effects (font (size 1.27 1.27)) hide)
     )
@@
       (effects (font (size 1.27 1.27)) (justify left))
     )
-    (property "Footprint" "Capacitor_SMD:C_0603_1608Metric" (id 2) (at 180.0352 111.125 0)
+    (property "Footprint" "ControlBoard:C_0603_1608Metric" (id 2) (at 180.0352 111.125 0)
       (effects (font (size 1.27 1.27)) hide)
     )
@@
       (effects (font (size 1.27 1.27)) hide)
     )
-    (property "Footprint" "Connector_JST:JST_PH_S8B-PH-K_1x08_P2.00mm_Horizontal" (id 2) (at 40.005 105.41 0)
+    (property "Footprint" "ControlBoard:JST_PH_S8B-PH-K_1x08_P2.00mm_Horizontal" (id 2) (at 40.005 105.41 0)
       (effects (font (size 1.27 1.27)) hide)
     )
@@
       (effects (font (size 1.27 1.27)) (justify left))
     )
-    (property "Footprint" "Capacitor_SMD:C_0603_1608Metric" (id 2) (at 240.9952 120.015 0)
+    (property "Footprint" "ControlBoard:C_0603_1608Metric" (id 2) (at 240.9952 120.015 0)
       (effects (font (size 1.27 1.27)) hide)
     )
@@
       (effects (font (size 1.27 1.27)) (justify left))
     )
-    (property "Footprint" "Capacitor_SMD:C_0603_1608Metric" (id 2) (at 87.3252 108.585 0)
+    (property "Footprint" "ControlBoard:C_0603_1608Metric" (id 2) (at 87.3252 108.585 0)
       (effects (font (size 1.27 1.27)) hide)
     )
@@
       (effects (font (size 1.27 1.27)) (justify left))
     )
-    (property "Footprint" "Capacitor_SMD:C_0603_1608Metric" (id 2) (at 75.2602 108.585 0)
+    (property "Footprint" "ControlBoard:C_0603_1608Metric" (id 2) (at 75.2602 108.585 0)
       (effects (font (size 1.27 1.27)) hide)
     )
@@
       (effects (font (size 1.27 1.27)) (justify left))
     )
-    (property "Footprint" "Capacitor_SMD:C_0603_1608Metric" (id 2) (at 251.1552 111.125 0)
+    (property "Footprint" "ControlBoard:C_0603_1608Metric" (id 2) (at 251.1552 111.125 0)
       (effects (font (size 1.27 1.27)) hide)
     )
@@
       (effects (font (size 1.27 1.27)) (justify left))
     )
-    (property "Footprint" "Capacitor_SMD:C_0603_1608Metric" (id 2) (at 97.4852 108.585 0)
+    (property "Footprint" "ControlBoard:C_0603_1608Metric" (id 2) (at 97.4852 108.585 0)
       (effects (font (size 1.27 1.27)) hide)
     )
@@
     (property "Reference" "U10" (id 0) (at 212.09 98.425 0))
     (property "Value" "HX9193" (id 1) (at 220.98 111.125 0))
-    (property "Footprint" "Package_TO_SOT_SMD:SOT-23-5" (id 2) (at 217.17 113.665 0)
-      (effects (font (size 1.27 1.27)) hide)
-    )
+    (property "Footprint" "ControlBoard:SOT-23-5" (id 2) (at 217.17 113.665 0)
+      (effects (font (size 1.27 1.27)) hide)
+    )

Commit message: Modify and complete the circuit schematic to make the interface easier to wire.
Parts:
- C41: renamed from C45; value 10uF -> 680uF; footprint ControlBoard:C_0603_1608Metric -> ControlBoard:Cap_SinkBoard
- renumbered C46 to C42, C47 to C43, C48 to C44, C49 to C45, C50 to C46, C51 to C47, U9 to U7, U10 to U8
Other:
- title: MM32_Board -> MM32 Control Board
Changed lines of the file:
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@@
   (paper "A4")
   (title_block
-    (title "MM32_Board")
-    (date "2022-03-02")
-    (rev "1.3.2")
+    (title "MM32 Control Board")
+    (date "2022-03-03")
+    (rev "1.3.3")
   )
   (junction (at 240.03 102.235) (diameter 0) (color 0 0 0 0)
@@
   (symbol (lib_id "MM32_Periph:HX9193") (at 139.7 109.855 0) (unit 1)
     (in_bom yes) (on_board yes)
-    (property "Reference" "U9" (id 0) (at 140.97 98.425 0))
+    (property "Reference" "U7" (id 0) (at 140.97 98.425 0))
     (property "Value" "HX9193" (id 1) (at 149.86 111.125 0))
     (property "Footprint" "ControlBoard:SOT-23-5" (id 2) (at 146.05 113.665 0)
@@
   (symbol (lib_id "power:+5V") (at 123.19 84.455 0) (unit 1)
     (in_bom yes) (on_board yes)
-    (property "Reference" "#PWR0110" (id 0) (at 123.19 88.265 0)
+    (property "Reference" "#PWR094" (id 0) (at 123.19 88.265 0)
       (effects (font (size 1.27 1.27)) hide)
     )
@@
   (symbol (lib_id "power:GND") (at 123.19 128.905 0) (unit 1)
     (in_bom yes) (on_board yes)
-    (property "Reference" "#PWR0111" (id 0) (at 123.19 135.255 0)
+    (property "Reference" "#PWR095" (id 0) (at 123.19 135.255 0)
       (effects (font (size 1.27 1.27)) hide)
     )
@@
   (symbol (lib_id "power:+5V") (at 129.54 84.455 0) (unit 1)
     (in_bom yes) (on_board yes)
-    (property "Reference" "#PWR0112" (id 0) (at 129.54 88.265 0)
+    (property "Reference" "#PWR096" (id 0) (at 129.54 88.265 0)
       (effects (font (size 1.27 1.27)) hide)
     )
@@
   (symbol (lib_id "power:GND") (at 168.91 128.905 0) (unit 1)
     (in_bom yes) (on_board yes)
-    (property "Reference" "#PWR0114" (id 0) (at 168.91 135.255 0)
+    (property "Reference" "#PWR098" (id 0) (at 168.91 135.255 0)
       (effects (font (size 1.27 1.27)) hide)
     )
@@
   (symbol (lib_id "Device:C") (at 168.91 116.205 0) (unit 1)
     (in_bom yes) (on_board yes)
-    (property "Reference" "C48" (id 0) (at 171.831 115.0366 0)
+    (property "Reference" "C44" (id 0) (at 171.831 115.0366 0)
       (effects (font (size 1.27 1.27)) (justify left))
     )
@@
   (symbol (lib_id "Device:C") (at 179.07 107.315 0) (unit 1)
     (in_bom yes) (on_board yes)
-    (property "Reference" "C49" (id 0) (at 181.991 106.1466 0)
+    (property "Reference" "C45" (id 0) (at 181.991 106.1466 0)
       (effects (font (size 1.27 1.27)) (justify left))
     )
@@
   (symbol (lib_id "power:GND") (at 179.07 128.905 0) (unit 1)
     (in_bom yes) (on_board yes)
-    (property "Reference" "#PWR0116" (id 0) (at 179.07 135.255 0)
+    (property "Reference" "#PWR0100" (id 0) (at 179.07 135.255 0)
       (effects (font (size 1.27 1.27)) hide)
     )
@@
   (symbol (lib_id "power:GND") (at 194.31 128.905 0) (unit 1)
     (in_bom yes) (on_board yes)
-    (property "Reference" "#PWR0118" (id 0) (at 194.31 135.255 0)
+    (property "Reference" "#PWR0102" (id 0) (at 194.31 135.255 0)
       (effects (font (size 1.27 1.27)) hide)
     )
@@
   (symbol (lib_id "power:GND") (at 86.36 128.27 0) (unit 1)
     (in_bom yes) (on_board yes)
-    (property "Reference" "#PWR0107" (id 0) (at 86.36 134.62 0)
+    (property "Reference" "#PWR091" (id 0) (at 86.36 134.62 0)
       (effects (font (size 1.27 1.27)) hide)
     )
@@
   (symbol (lib_id "Device:C") (at 240.03 116.205 0) (unit 1)
     (in_bom yes) (on_board yes)
-    (property "Reference" "C50" (id 0) (at 242.951 115.0366 0)
+    (property "Reference" "C46" (id 0) (at 242.951 115.0366 0)
       (effects (font (size 1.27 1.27)) (justify left))
     )
@@
   (symbol (lib_id "power:+3.3VP") (at 240.03 84.455 0) (unit 1)
     (in_bom yes) (on_board yes)
-    (property "Reference" "#PWR0120" (id 0) (at 243.84 85.725 0)
+    (property "Reference" "#PWR0104" (id 0) (at 243.84 85.725 0)
       (effects (font (size 1.27 1.27)) hide)
     )
@@
   (symbol (lib_id "power:GND") (at 240.03 128.905 0) (unit 1)
     (in_bom yes) (on_board yes)
-    (property "Reference" "#PWR0121" (id 0) (at 240.03 135.255 0)
+    (property "Reference" "#PWR0105" (id 0) (at 240.03 135.255 0)
       (effects (font (size 1.27 1.27)) hide)
     )
@@
   (symbol (lib_id "power:GND") (at 250.19 128.905 0) (unit 1)
     (in_bom yes) (on_board yes)
-    (property "Reference" "#PWR0123" (id 0) (at 250.19 135.255 0)
+    (property "Reference" "#PWR0107" (id 0) (at 250.19 135.255 0)
       (effects (font (size 1.27 1.27)) hide)
     )
@@
   (symbol (lib_id "power:GND") (at 52.705 128.27 0) (unit 1)
     (in_bom yes) (on_board yes)
-    (property "Reference" "#PWR0103" (id 0) (at 52.705 134.62 0)
+    (property "Reference" "#PWR087" (id 0) (at 52.705 134.62 0)
       (effects (font (size 1.27 1.27)) hide)
     )
@@
   (symbol (lib_id "Device:C") (at 86.36 104.775 0) (unit 1)
     (in_bom yes) (on_board yes)
-    (property "Reference" "C46" (id 0) (at 89.281 103.6066 0)
+    (property "Reference" "C42" (id 0) (at 89.281 103.6066 0)
       (effects (font (size 1.27 1.27)) (justify left))
     )
@@
   (symbol (lib_id "power:+5V") (at 74.295 83.185 0) (unit 1)
     (in_bom yes) (on_board yes)
-    (property "Reference" "#PWR0104" (id 0) (at 74.295 86.995 0)
+    (property "Reference" "#PWR088" (id 0) (at 74.295 86.995 0)
       (effects (font (size 1.27 1.27)) hide)
     )
@@
   (symbol (lib_id "Device:C") (at 74.295 104.775 0) (unit 1)
     (in_bom yes) (on_board yes)
-    (property "Reference" "C45" (id 0) (at 77.216 103.6066 0)
-      (effects (font (size 1.27 1.27)) (justify left))
-    )
-    (property "Value" "10uF" (id 1) (at 77.216 105.918 0)
-      (effects (font (size 1.27 1.27)) (justify left))
-    )
-    (property "Footprint" "ControlBoard:C_0603_1608Metric" (id 2) (at 75.2602 108.585 0)
+    (property "Reference" "C41" (id 0) (at 77.216 103.6066 0)
+      (effects (font (size 1.27 1.27)) (justify left))
+    )
+    (property "Value" "680uF" (id 1) (at 77.216 105.918 0)
+      (effects (font (size 1.27 1.27)) (justify left))
+    )
+    (property "Footprint" "ControlBoard:Cap_SinkBoard" (id 2) (at 75.2602 108.585 0)
       (effects (font (size 1.27 1.27)) hide)
     )
@@
   (symbol (lib_id "power:+5V") (at 200.66 84.455 0) (unit 1)
     (in_bom yes) (on_board yes)
-    (property "Reference" "#PWR0119" (id 0) (at 200.66 88.265 0)
+    (property "Reference" "#PWR0103" (id 0) (at 200.66 88.265 0)
       (effects (font (size 1.27 1.27)) hide)
     )
@@
   (symbol (lib_id "power:+5V") (at 86.36 83.185 0) (unit 1)
     (in_bom yes) (on_board yes)
-    (property "Reference" "#PWR0106" (id 0) (at 86.36 86.995 0)
+    (property "Reference" "#PWR090" (id 0) (at 86.36 86.995 0)
       (effects (font (size 1.27 1.27)) hide)
     )
@@
   (symbol (lib_id "power:+5V") (at 96.52 83.185 0) (unit 1)
     (in_bom yes) (on_board yes)
-    (property "Reference" "#PWR0108" (id 0) (at 96.52 86.995 0)
+    (property "Reference" "#PWR092" (id 0) (at 96.52 86.995 0)
       (effects (font (size 1.27 1.27)) hide)
     )
@@
   (symbol (lib_id "power:GND") (at 96.52 128.27 0) (unit 1)
     (in_bom yes) (on_board yes)
-    (property "Reference" "#PWR0109" (id 0) (at 96.52 134.62 0)
+    (property "Reference" "#PWR093" (id 0) (at 96.52 134.62 0)
       (effects (font (size 1.27 1.27)) hide)
     )
@@
   (symbol (lib_id "power:+3.3VA") (at 168.91 84.455 0) (unit 1)
     (in_bom yes) (on_board yes)
-    (property "Reference" "#PWR0113" (id 0) (at 168.91 88.265 0)
+    (property "Reference" "#PWR097" (id 0) (at 168.91 88.265 0)
       (effects (font (size 1.27 1.27)) hide)
     )
@@
   (symbol (lib_id "power:+5V") (at 52.705 83.82 0) (unit 1)
     (in_bom yes) (on_board yes)
-    (property "Reference" "#PWR0102" (id 0) (at 52.705 87.63 0)
+    (property "Reference" "#PWR086" (id 0) (at 52.705 87.63 0)
       (effects (font (size 1.27 1.27)) hide)
     )
@@
   (symbol (lib_id "Device:C") (at 250.19 107.315 0) (unit 1)
     (in_bom yes) (on_board yes)
-    (property "Reference" "C51" (id 0) (at 253.111 106.1466 0)
+    (property "Reference" "C47" (id 0) (at 253.111 106.1466 0)
       (effects (font (size 1.27 1.27)) (justify left))
     )
@@
   (symbol (lib_id "Device:C") (at 96.52 104.775 0) (unit 1)
     (in_bom yes) (on_board yes)
-    (property "Reference" "C47" (id 0) (at 99.441 103.6066 0)
+    (property "Reference" "C43" (id 0) (at 99.441 103.6066 0)
       (effects (font (size 1.27 1.27)) (justify left))
     )
@@
   (symbol (lib_id "MM32_Periph:HX9193") (at 210.82 109.855 0) (unit 1)
     (in_bom yes) (on_board yes)
-    (property "Reference" "U10" (id 0) (at 212.09 98.425 0))
+    (property "Reference" "U8" (id 0) (at 212.09 98.425 0))
     (property "Value" "HX9193" (id 1) (at 220.98 111.125 0))
     (property "Footprint" "ControlBoard:SOT-23-5" (id 2) (at 217.17 113.665 0)
@@
   (symbol (lib_id "power:+3.3VP") (at 250.19 84.455 0) (unit 1)
     (in_bom yes) (on_board yes)
-    (property "Reference" "#PWR0122" (id 0) (at 254 85.725 0)
+    (property "Reference" "#PWR0106" (id 0) (at 254 85.725 0)
       (effects (font (size 1.27 1.27)) hide)
     )
@@
   (symbol (lib_id "power:GND") (at 74.295 128.27 0) (unit 1)
     (in_bom yes) (on_board yes)
-    (property "Reference" "#PWR0105" (id 0) (at 74.295 134.62 0)
+    (property "Reference" "#PWR089" (id 0) (at 74.295 134.62 0)
       (effects (font (size 1.27 1.27)) hide)
     )
@@
   (symbol (lib_id "power:+5V") (at 194.31 84.455 0) (unit 1)
     (in_bom yes) (on_board yes)
-    (property "Reference" "#PWR0117" (id 0) (at 194.31 88.265 0)
+    (property "Reference" "#PWR0101" (id 0) (at 194.31 88.265 0)
       (effects (font (size 1.27 1.27)) hide)
     )
@@
   (symbol (lib_id "power:+3.3VA") (at 179.07 84.455 0) (unit 1)
     (in_bom yes) (on_board yes)
-    (property "Reference" "#PWR0115" (id 0) (at 179.07 88.265 0)
-      (effects (font (size 1.27 1.27)) hide)
-    )
+    (property "Reference" "#PWR099" (id 0) (at 179.07 88.265 0)
+      (effects (font (size 1.27 1.27)) hide)
+    )

Commit message: Modify the main control board schematic, replace the IMU device and remove the isolation module.
Parts:
- added C22: 22uF, ControlBoard:C_0603_1608Metric, symbol Device:C
- added C23: 100nF, ControlBoard:C_0603_1608Metric, symbol Device:C
- added U4: HX9193, ControlBoard:SOT-23-5, symbol MM32_Periph:HX9193
Connections:
- net +5V: now also U4.1 (VIN), U4.3 (EN)
- net GND: now also C22.2, C23.2, U4.2 (GND)
- new net +3.3VADC: C22.1, C23.1, U4.5 (VOUT)
Other:
- moved on the sheet: C41, C42, C43, C44, C45, C46, C47, J2, U7, U8

Commit message: Fixed part of the control board circuit and added SD card reading chip.
Parts:
- renumbered C41 to C39, C42 to C40, C43 to C41, C22 to C42, C23 to C43, C46 to C45, C45 to C46, J2 to J3, U4 to U6
