File: circuit/control_board/Power.kicad_sch (KiCad schematic)
At the start: 13 parts, among them J3 Conn_01x08, U6 HX9193, U7 HX9193, U8 HX9193

Commit message: Update the main control board schematic to complete the SD card reader part.
Parts:
- added C42, C43, C44, C45, C46, C49: 100nF, ControlBoard:C_0603_1608Metric, symbol Device:C
- renumbered C42 to C47, C43 to C48, C44 to C50, C45 to C51, C46 to C52, C47 to C53
Connections:
- net +5V: now also C42.1, C43.1, C44.1, C45.1, C46.1, C49.1
- net GND: now also C42.2, C43.2, C44.2, C45.2, C46.2, C49.2
