File: circuit/control_board/ProcessMCU.kicad_sch (KiCad schematic)
At the start: 21 parts, among them U8 MM32F3277G9P, Y1 8MHz

Commit message: Modified the circuitry of the main control board to add a microcontroller for reading information from the magnetometer and IMU. Modified the SPI connection port of the Process MCU.
Parts:
- C30, C31, C32, C33, C34, C35, C36, C37, C38, C39, C40, C41, C42, C43, C44: footprint Capacitor_SMD:C_0603_1608Metric -> ControlBoard:C_0603_1608Metric
- D1: footprint LED_SMD:LED_0603_1608Metric -> ControlBoard:LED_0603_1608Metric
- R1, R2, R3: footprint Resistor_SMD:R_0603_1608Metric -> ControlBoard:R_0603_1608Metric
- U8: footprint Package_QFP:LQFP-144_20x20mm_P0.5mm -> ControlBoard:LQFP-144_20x20mm_P0.5mm
- Y1: footprint Crystal:Crystal_SMD_3225-4Pin_3.2x2.5mm -> ControlBoard:Crystal_SMD_3225-4Pin_3.2x2.5mm
Connections:
- net UART8_TX: now reaches U8.114 (PD0)
- net UART8_RX: now reaches U8.115 (PD1)
- net SPI2_MISO: now reaches U8.4 (PE5)
- net PD12: no longer names the net of U8.81 (PD12)
- net PE0: no longer names the net of U8.141 (PE0)
- net PG10: no longer names the net of U8.125 (PG10)
- net PG9: no longer names the net of U8.124 (PG9)
- net SPI1_CLK: no longer names the net of U8.133 (PB3)
- net SPI1_MISO: no longer names the net of U8.134 (PB4)
- net SPI1_MOSI: no longer names the net of U8.135 (PB5)
- net SPI3_MISO: no longer names the net of U8.119 (PD5)
- no-connect marks 83 -> 88

Commit message: Modify and complete the circuit schematic to make the interface easier to wire.
Parts:
- renumbered C30 to C26, C31 to C27, C32 to C28, C33 to C29, C34 to C30, C35 to C31, C36 to C32, C37 to C33, C38 to C34, C39 to C35, C40 to C36, C41 to C37, C42 to C38, C43 to C39, C44 to C40, R1 to R2, R2 to R3, R3 to R4, U8 to U6
Connections:
- net PE0: now reaches U6.141 (PE0)
- net PF0: no longer names the net of U6.10 (PF0)
Other:
- title: MM32_Board -> MM32 Control Board

Commit message: Modify the ControlBoard schematic to add useful features.
Connections:
- net +3.3VP is gone; now on net +3.3VA: R3.1
- net LED1: now also U6.40 (PA4); no longer U6.37 (PA3)
- net UART2_TX: now reaches U6.36 (PA2)
- net UART8_RX: no longer names the net of U6.115 (PD1)
- net UART8_TX: no longer names the net of U6.114 (PD0)
- new net UART2_RX: U6.37 (PA3)
Changed lines of the file:
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@@
   (title_block
     (title "MM32 Control Board")
-    (date "2022-03-28")
-    (rev "1.4.1")
+    (date "2022-04-06")
+    (rev "1.5.2")
   )
   (junction (at 217.17 133.985) (diameter 0) (color 0 0 0 0)
@@
   (no_connect (at 161.29 67.31))
   (no_connect (at 135.89 151.13))
+  (no_connect (at 135.89 46.99))
+  (no_connect (at 138.43 46.99))
   (no_connect (at 52.07 85.09))
   (no_connect (at 161.29 138.43))
@@
   (no_connect (at 52.07 72.39))
   (no_connect (at 138.43 151.13))
-  (no_connect (at 69.85 151.13))
   (no_connect (at 161.29 102.87))
   (no_connect (at 120.65 151.13))
@@
   (no_connect (at 133.35 46.99))
   (no_connect (at 161.29 59.69))
-  (no_connect (at 52.07 143.51))
   (no_connect (at 82.55 151.13))
   (no_connect (at 161.29 82.55))
@@
     (stroke (width 0) (type default) (color 0 0 0 0))
   )
-  (wire (pts (xy 138.43 46.99) (xy 138.43 33.02))
+  (wire (pts (xy 52.07 143.51) (xy 38.1 143.51))
     (stroke (width 0) (type default) (color 0 0 0 0))
   )
@@
     (stroke (width 0) (type default) (color 0 0 0 0))
   )
-  (wire (pts (xy 135.89 33.02) (xy 135.89 46.99))
+  (wire (pts (xy 62.23 165.1) (xy 62.23 151.13))
     (stroke (width 0) (type default) (color 0 0 0 0))
   )
@@
     (stroke (width 0) (type default) (color 0 0 0 0))
   )
-  (wire (pts (xy 62.23 151.13) (xy 62.23 171.45))
+  (wire (pts (xy 69.85 151.13) (xy 69.85 171.45))
     (stroke (width 0) (type default) (color 0 0 0 0))
   )
@@
     (effects (font (size 1.27 1.27)) (justify left bottom))
   )
-  (label "LED1" (at 62.23 171.45 90)
+  (label "LED1" (at 69.85 171.45 90)
     (effects (font (size 1.27 1.27)) (justify left bottom))
   )
@@
     (effects (font (size 1.27 1.27)) (justify right))
   )
-  (hierarchical_label "UART8_TX" (shape output) (at 138.43 33.02 90)
-    (effects (font (size 1.27 1.27)) (justify left))
+  (hierarchical_label "UART2_TX" (shape output) (at 38.1 143.51 180)
+    (effects (font (size 1.27 1.27)) (justify right))
   )
   (hierarchical_label "IIC1_SCL" (shape output) (at 173.99 128.27 0)
@@
     (effects (font (size 1.27 1.27)) (justify left))
   )
-  (hierarchical_label "UART8_RX" (shape input) (at 135.89 33.02 90)
-    (effects (font (size 1.27 1.27)) (justify left))
+  (hierarchical_label "UART2_RX" (shape input) (at 62.23 165.1 270)
+    (effects (font (size 1.27 1.27)) (justify right))
   )
   (hierarchical_label "UART3_RX" (shape input) (at 173.99 130.81 0)
@@
     (pin "1")
   )
+  (symbol (lib_id "power:+3.3VA") (at 259.715 90.17 270) (unit 1)
+    (in_bom yes) (on_board yes)
+    (property "Reference" "#PWR0143" (id 0) (at 255.905 90.17 0)
+      (effects (font (size 1.27 1.27)) hide)
+    )
+    (property "Value" "+3.3VA" (id 1) (at 266.065 90.17 90))
+    (property "Footprint" "" (id 2) (at 259.715 90.17 0)
+      (effects (font (size 1.27 1.27)) hide)
+    )
+    (property "Datasheet" "" (id 3) (at 259.715 90.17 0)
+      (effects (font (size 1.27 1.27)) hide)
+    )
+    (pin "1")
+  )
   (symbol (lib_id "power:GND") (at 234.95 135.255 0) (unit 1)
     (in_bom yes) (on_board yes)
@@
       (effects (font (size 1.27 1.27)) hide)
     )
-    (pin "1")
-  )
-  (symbol (lib_id "power:+3.3VP") (at 259.715 90.17 270) (unit 1)
-    (in_bom yes) (on_board yes)
-    (property "Reference" "#PWR083" (id 0) (at 258.445 93.98 0)
-      (effects (font (size 1.27 1.27)) hide)
-    )
-    (property "Value" "+3.3VP" (id 1) (at 266.7 90.17 90))
-    (property "Footprint" "" (id 2) (at 259.715 90.17 0)
-      (effects (font (size 1.27 1.27)) hide)
-    )
-    (property "Datasheet" "" (id 3) (at 259.715 90.17 0)
-      (effects (font (size 1.27 1.27)) hide)
-    )

Commit message: Fixed part of the control board circuit and added SD card reading chip.
Parts:
- renumbered C26 to C24, C27 to C25, C28 to C26, C29 to C27, C30 to C28, C31 to C29, C32 to C30, C33 to C31, C34 to C32, C35 to C33, C36 to C34, C37 to C35, C38 to C36, C39 to C37, C40 to C38, U6 to U5
