File: circuit/control_board/Flash&USB.kicad_sch (KiCad schematic)
At the start: 6 parts, among them P1 USB_C_Plug_USB2.0, U14 CH372C, U15 W25Q64

Commit message: The main control board circuit modified the CH372C package, changed the serial port of the GPS and ControlMCU back, and moved the components a bit towards the middle so that they could be screwed on.
Parts:
- U14: footprint Package_SO:SSOP-20_4.4x6.5mm_P0.65mm -> Package_SO:SSOP-20_5.3x7.2mm_P0.65mm
Changed lines of the file:
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@@
   (title_block
     (title "MM32 Control Board")
-    (date "2022-04-06")
-    (rev "1.5.2")
+    (date "2022-04-17")
+    (rev "1.5.3")
   )
   (junction (at 220.98 104.775) (diameter 0) (color 0 0 0 0)
@@
     (property "Reference" "U14" (id 0) (at 100.33 92.71 0))
     (property "Value" "CH372C" (id 1) (at 109.22 123.19 0))
-    (property "Footprint" "Package_SO:SSOP-20_4.4x6.5mm_P0.65mm" (id 2) (at 104.775 125.73 0)
+    (property "Footprint" "Package_SO:SSOP-20_5.3x7.2mm_P0.65mm" (id 2) (at 104.775 125.73 0)
       (effects (font (size 1.27 1.27)) hide)
     )

Commit message: Slightly modify the ControlBoard package
Parts:
- U14: footprint Package_SO:SSOP-20_5.3x7.2mm_P0.65mm -> ControlBoard:SSOP-20_5.3x7.2mm_P0.65mm
- U15: footprint Package_SO:SOIC-8_5.23x5.23mm_P1.27mm -> ControlBoard:SOIC-8_5.23x5.23mm_P1.27mm
Changed lines of the file:
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@@
     (property "Reference" "U14" (id 0) (at 100.33 92.71 0))
     (property "Value" "CH372C" (id 1) (at 109.22 123.19 0))
-    (property "Footprint" "Package_SO:SSOP-20_5.3x7.2mm_P0.65mm" (id 2) (at 104.775 125.73 0)
+    (property "Footprint" "ControlBoard:SSOP-20_5.3x7.2mm_P0.65mm" (id 2) (at 104.775 125.73 0)
       (effects (font (size 1.27 1.27)) hide)
     )
@@
     (property "Reference" "U15" (id 0) (at 203.2 100.965 0))
     (property "Value" "W25Q64" (id 1) (at 212.09 116.205 0))
-    (property "Footprint" "Package_SO:SOIC-8_5.23x5.23mm_P1.27mm" (id 2) (at 210.82 118.745 0)
+    (property "Footprint" "ControlBoard:SOIC-8_5.23x5.23mm_P1.27mm" (id 2) (at 210.82 118.745 0)
       (effects (font (size 1.27 1.27)) hide)
     )

Commit message: Modified a portion of the main control board circuit schematic.Added TF card and card reader chip.
Parts:
- removed C67, C69: 100nF, ControlBoard:C_0603_1608Metric, symbol Device:C
- removed C68: 10uF, ControlBoard:C_0603_1608Metric, symbol Device:C
- removed U14: CH372C, ControlBoard:SSOP-20_5.3x7.2mm_P0.65mm, symbol MM32_Periph:CH372C
- removed U15: W25Q64, ControlBoard:SOIC-8_5.23x5.23mm_P1.27mm, symbol MM32_Periph:W25Q64
- added U?: CH440R, ControlBoard:TSSOP-16_4.4x5mm_P0.65mm, symbol MM32_Periph:CH440R
- added U?: MKDV1GCL-AB, ControlBoard:LGA-8060_8, symbol MM32_Periph:MKDV1GCL-AB
Connections:
- no-connect marks 1 -> 0

Commit message: Fixed part of the control board circuit and added SD card reading chip.
Parts:
- added U?: GL823K, symbol MM32_Periph:GL823K
- gave numbers to parts that had none: 2
Connections:
- net +3.3VP: now also U14.8 (Vin)
- net GND: now also U14.4 (GND)
- net GL_DP: now reaches P1.A6 (D+), P1.B6 (D+)
- net GL_DP: now also U?.15 (DP)
- net GL_DM: now reaches P1.A7 (D-), P1.B7 (D-)
- net GL_DM: now also U?.16 (DM)
Other:
- moved on the sheet: U13, U14

Commit message: Update the main control board schematic to complete the SD card reader part.
Parts:
- removed U13: CH440R, ControlBoard:TSSOP-16_4.4x5mm_P0.65mm, symbol MM32_Periph:CH440R
- added C74, C75, C76: 100nF, ControlBoard:C_0603_1608Metric, symbol Device:C
- added D4: LED, ControlBoard:LED_0603_1608Metric, symbol Device:LED
- added R16: 100kR, ControlBoard:R_0603_1608Metric, symbol Device:R
- added R17: 4.7kR, ControlBoard:R_0603_1608Metric, symbol Device:R
- added R18, R19: 10kR, ControlBoard:R_0603_1608Metric, symbol Device:R
- added U14: CH440R, ControlBoard:TSSOP-16_4.4x5mm_P0.65mm, symbol MM32_Periph:CH440R
- added U15, U16: CH443K, Package_TO_SOT_SMD:SOT-363_SC-70-6, symbol MM32_Periph:CH443K
- U13: renamed from U?; footprint (none) -> Package_SO:SSOP-16_3.9x4.9mm_P0.635mm
- renumbered U14 to U17
Connections:
- net +3.3VP: now also R18.1, R19.1
- net +5V: now also U13.10 (5V), R17.1, U14.16 (VCC), U15.5 (VCC), U16.5 (VCC)
- net FLASH_CLK: now also U14.10 (S2C)
- net FLASH_CS: now also U14.13 (S2D)
- net FLASH_MISO: now also U14.3 (S2A)
- net FLASH_MOSI: now also U14.6 (S2B)
- net GND: now also U13.1 (VSS), U13.14 (VSS), C74.2, C75.2, C76.2, R16.2, U14.15 (#EN), U14.8 (GND), U15.2 (GND), U16.2 (GND)
- net at U13.11 (GPIO): now also R16.1
- net at U13.12 (LED): now also D4.1 (K)
- net USB_VDD: now reaches U13.13 (VDDA)
- net USB_VDD: now also U13.9 (VDD), C74.1, C75.1, C76.1
- net DATA1: now reaches U13.2 (D1)
- net DATA1: now also U16.3 (CH0)
- net DATA0: now reaches U13.3 (D0)
- net DATA0: now also U14.2 (S1A)
- net CLK: now reaches U13.4 (CLK)
- net CLK: now also U14.11 (S1C)
- net CMD: now reaches U13.5 (CMD)
- net CMD: now also U14.5 (S1B)
- net DATA3: now reaches U13.6 (D3)
- net DATA3: now also U14.14 (S1D)
- net DATA2: now reaches U13.7 (D2)
- net DATA2: now also U15.3 (CH0)
- net SD_D2: now reaches U17.1 (DAT2)
- net SD_D2: now also U15.4 (COM)
- net SD_D3: now reaches U17.2 (DAT3)
- net SD_D3: now also U14.12 (DD)
- net SD_CLK: now reaches U17.3 (CLK)
- net SD_CLK: now also U14.9 (DC)
- net SD_CMD: now reaches U17.5 (CMD)
- net SD_CMD: now also U14.7 (DB)
- net SD_D0: now reaches U17.6 (DAT0)
- net SD_D0: now also U14.4 (DA)
- net SD_D1: now reaches U17.7 (DAT1)
- net SD_D1: now also U16.4 (COM)
- new net: R18.2, U15.1 (CH1)
- new net: D4.2 (A), R17.2
- new net: R19.2, U16.1 (CH1)
- new net SELECT: U14.1 (SEL), U15.6 (SEL), U16.6 (SEL)
- no-connect marks 0 -> 1
Other:
- note added: "Switch"
- moved on the sheet: P1, U13, U17
