File: circuit/geomagnetometer/geomagnetometer.kicad_pcb (KiCad board)
At the start: 2 copper layers, 20 parts, among them J1 Conn_01x06, U1 RM3100_13156

Commit message: Complete the PCB design of the geomagnetometer circuit
Parts:
- moved C2 26.2 mm to (143.9, 114.5), turned to 180 degrees
- moved R4 19.2 mm to (149.2, 111.9)
- moved R9 17.3 mm to (155.9, 114.5), turned to 180 degrees
- moved R10 16.5 mm to (156.0, 105.8), turned to -90 degrees
- moved C6 14.6 mm to (147.3, 114.5)
- moved R3 12.6 mm to (145.8, 111.9), turned to 180 degrees
- moved C1 12.2 mm to (155.9, 103.6)
- moved C7 12.2 mm to (143.1, 104.5), turned to 180 degrees
- moved C3 11.8 mm to (155.9, 101.8)
- moved C5 11.7 mm to (143.1, 106.3), turned to 180 degrees
- moved R5 10.9 mm to (152.4, 111.9), turned to 180 degrees
- moved R7 10.5 mm to (153.2, 106.2), turned to -90 degrees
- moved C4 9.94 mm to (155.9, 99.8)
- moved R8 8.62 mm to (142.4, 112.0), turned to 90 degrees
- moved U1 8.07 mm to (149.3, 108.2)
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Connections:
- net Net-(J1-Pad3) renamed /MISO
- net Net-(J1-Pad5) renamed /CS
- J1 pad 2: Net-(J1-Pad2) -> /CLK
- J1 pad 4: Net-(J1-Pad4) -> /MOSI
- U1 pad 1: Net-(J1-Pad2) -> /MOSI
- U1 pad 27: Net-(J1-Pad4) -> /CLK
- U1 pad 29: (no net) -> GND
Routing:
- net +3.3VADC: track 0.00 -> 50.8 mm, vias 0 -> 6
- net GND: track 0.00 -> 11.2 mm, vias 0 -> 16
- net Net-(R5-Pad2): track 0.00 -> 8.34 mm
- net Net-(R10-Pad2): track 0.00 -> 6.88 mm
- net /CS: track 0.00 -> 6.80 mm
- net Net-(R3-Pad2): track 0.00 -> 6.66 mm
- net Net-(R10-Pad1): track 0.00 -> 6.48 mm
- net /MOSI: track 0.00 -> 5.95 mm
- net Net-(R2-Pad2): track 0.00 -> 5.40 mm
- net /CLK: track 0.00 -> 5.36 mm
- net /MISO: track 0.00 -> 5.05 mm
- net Net-(R4-Pad2): track 0.00 -> 4.73 mm
- net Net-(R5-Pad1): track 0.00 -> 4.17 mm
- net Net-(R7-Pad1): track 0.00 -> 3.92 mm
- net Net-(R3-Pad1): track 0.00 -> 2.91 mm
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- added copper zone on B.Cu, net GND
- added copper zone on F.Cu, net GND
Other:
- board outline added: 17.6 x 19.1 mm
- board text added: "0"
- board text added: "0 mm"
- board text added: "0.01 mm"
- board text added: "0.02"
- board text added: "0.035 mm"
- board text added: "0.2000 mm / 0.1500 mm"
- board text added: "0.3000 mm"
- board text added: "1"
- board text added: "1.51 mm"
- board text added: "1.6000 mm"
- board text added: "17.6500 mm x 19.0500 mm"
- board text added: "2"
- board text added: "3.3"
- board text added: "4.5"
- board text added: "B.Cu"
- board text added: "B.Mask"
- board text added: "B.Paste"
- board text added: "B.Silkscreen"
- board text added: "BOARD CHARACTERISTICS"
- board text added: "Bottom Silk Screen"
- board text added: "Bottom Solder Mask"
- board text added: "Bottom Solder Paste"
- board text added: "Epsilon R（相对介电常数）"
- board text added: "F.Cu"
- board text added: "F.Mask"
- board text added: "F.Paste"
- board text added: "F.Silkscreen"
- board text added: "FR4"
- board text added: "Loss Tangent（损耗角正切）"
- board text added: "None"
- board text added: "Not specified"
- board text added: "Top Silk Screen"
- board text added: "Top Solder Mask"
- board text added: "Top Solder Paste"
- board text added: "copper"
- board text added: "core"
- board text added: "否"
- board text added: "孔最小直径："
- board text added: "层名称"
- board text added: "最小布线/间距："
- board text added: "材料"
- board text added: "板子整体尺寸："
- board text added: "电介质层 1"
- board text added: "电路板厚度："
- board text added: "电镀板边："
- board text added: "类型"
- board text added: "粗细 (mm)"
- board text added: "边缘卡连接器："
- board text added: "邮票孔："
- board text added: "铜层数量："
- board text added: "铜表面处理（镀铜）："
- board text added: "阻抗控制"
- board text added: "颜色"

Commit message: Add silkscreen and name to the geomagnetometer plate.
Other:
- board text added: "2022/07/18"
- board text added: "GDUT Jesus"
- board text added: "Geomagnometer"
- board text added: "Version 1.0.2"
Changed lines of the file:
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@@
     (title "Geomagnetometer")
     (date "2022-07-09")
-    (rev "1.0.1")
+    (rev "1.0.2")
   )
   (layers
@@
   (gr_line (start 168.292859 124.45) (end 168.292859 165.4) (layer "F.Fab") (width 0.1))
   (gr_line (start 21.35 136.945) (end 168.292859 136.945) (layer "F.Fab") (width 0.1))
+  (gr_text "Version 1.0.2" (at 151.8 114.2) (layer "B.SilkS")
+    (effects (font (size 1.1 1.1) (thickness 0.2)) (justify mirror))
+  )
+  (gr_text "Geomagnometer" (at 149.2 112.1) (layer "B.SilkS")
+    (effects (font (size 1.4 1.4) (thickness 0.23)) (justify mirror))
+  )
+  (gr_text "2022/07/18" (at 149.15 101.1) (layer "B.Mask")
+    (effects (font (size 1.5 1.5) (thickness 0.25)) (justify mirror))
+  )
+  (gr_text "GDUT Jesus" (at 149.2 98.75) (layer "B.Mask")
+    (effects (font (size 1.5 1.5) (thickness 0.25)) (justify mirror))
+  )
   (gr_text "阻抗控制 " (at 233.814286 144.665) (layer "F.Fab")
     (effects (font (size 1.5 1.5) (thickness 0.2)) (justify left top))
@@
   (via (at 151.5 103.25) (size 0.6) (drill 0.3) (layers "F.Cu" "B.Cu") (free) (net 2))
   (via (at 156.75 100.75) (size 0.6) (drill 0.3) (layers "F.Cu" "B.Cu") (free) (net 2))
-  (via (at 142.75 101.7) (size 0.6) (drill 0.3) (layers "F.Cu" "B.Cu") (free) (net 2))
+  (via (at 141.5 102.35) (size 0.6) (drill 0.3) (layers "F.Cu" "B.Cu") (free) (net 2))
   (via (at 144.1 107.85) (size 0.6) (drill 0.3) (layers "F.Cu" "B.Cu") (free) (net 2))
   (via (at 156.75 98.85) (size 0.6) (drill 0.3) (layers "F.Cu" "B.Cu") (free) (net 2))
-  (via (at 152.15 102) (size 0.6) (drill 0.3) (layers "F.Cu" "B.Cu") (free) (net 2))
-  (via (at 151.1 100.4) (size 0.6) (drill 0.3) (layers "F.Cu" "B.Cu") (free) (net 2))
+  (via (at 152.25 102.55) (size 0.6) (drill 0.3) (layers "F.Cu" "B.Cu") (free) (net 2))
+  (via (at 150.3 100.1) (size 0.6) (drill 0.3) (layers "F.Cu" "B.Cu") (free) (net 2))
   (via (at 141.2 106.35) (size 0.6) (drill 0.3) (layers "F.Cu" "B.Cu") (free) (net 2))
   (via (at 157.05 108.6) (size 0.6) (drill 0.3) (layers "F.Cu" "B.Cu") (free) (net 2))
