File: circuit/geomagnetometer/geomagnetometer.kicad_sch (KiCad schematic)
At the start: 13 parts

Commit message: Complete the design of the geomagnetometer circuit and update the PCB rules.
Parts:
- added C2, C4: 1uF, ControlBoard:C_0603_1608Metric, symbol Device:C
- added C3: 10uF, ControlBoard:C_0603_1608Metric, symbol Device:C
- added C5, C7: 4.7uF, ControlBoard:C_0603_1608Metric, symbol Device:C
- added C6, C8: 100nF, ControlBoard:C_0603_1608Metric, symbol Device:C
- C1: renamed from C?; value 4.7uF -> 10uF
- gave numbers to parts that had none: 12
Connections:
- net Compass_CLK is gone; now on an unnamed net: U1.27 (SCLK)
- net Compass_CS is gone; now on an unnamed net: U1.3 (SSN)
- net Compass_MISO is gone; now on an unnamed net: U1.28 (MISO)
- net Compass_MOSI is gone; now on an unnamed net: U1.1 (MOSI)
- net +3.3VADC: now also J1.6 (Pin_6), C2.1, C3.1, C4.1, C5.1, C6.1, C7.1, C8.1
- net GND: now also J1.1 (Pin_1), C2.2, C3.2, C4.2, C5.2, C6.2, C7.2, C8.2
Other:
- note added: "Filter"
- moved on the sheet: C1, J1, R1, R10, R2, R3, R4, R5, R6, R7, R8, R9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

Commit message: Complete the PCB design of the geomagnetometer circuit
Connections:
- net CLK: now reaches J1.2 (Pin_2)
- net CLK: now also U1.27 (SCLK); no longer U1.1 (MOSI)
- net MOSI: now reaches J1.4 (Pin_4)
- net MOSI: now also U1.1 (MOSI); no longer U1.27 (SCLK)
- net MISO: now reaches J1.3 (Pin_3), U1.28 (MISO)
- net CS: now reaches J1.5 (Pin_5), U1.3 (SSN)
Other:
- note added: "Connector"
- moved on the sheet: C1, C2, C3, C4, C5, C6, C7, C8, J1, R1, R10, R2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
