File: circuit/power_board/Connector.kicad_sch (KiCad schematic)
At the start: 4 parts, among them J2 GH1.25_1x8, J3 conn_1x3, J4 GH1.25_1X3, J7 CONN_1X7

Commit message: Update the schematic of the power supply board and organize the schematic structure
Parts:
- added J6: XT30, Connector_AMASS:AMASS_XT30UPB-F_1x02_P5.0mm_Vertical, symbol power_Library:XT30
- added J7: XT60, Connector_AMASS:AMASS_XT60-M_1x02_P7.20mm_Vertical, symbol power_Library:XT60
- renumbered J7 to J5
Connections:
- net +3V3 is gone; now on net +5VA: J5.6
- net GND: now also J6.2 (GND), J7.2 (GND)
- new net +15V: J7.1 (BAT)
- new net VCC: J6.1 (VCC)
Other:
- note added: "BAT"
- note added: "ControlBoard"
- note added: "Motor"
- note added: "Remote"
- note added: "Servo"
- moved on the sheet: J2, J3, J4, J5

Commit message: Update the power board PCB file and complete the power board layout wiring.
Parts:
- J2: footprint Connector_JST:JST_GH_SM08B-GHS-TB_1x08-1MP_P1.25mm_Horizontal -> PowerLibrary:JST_GH_SM08B-GHS-TB_1x08-1MP_P1.25mm_Horizontal
- J3: footprint Connector_PinSocket_2.54mm:PinSocket_1x03_P2.54mm_Vertical -> PowerLibrary:PinSocket_1x03_P2.54mm_Vertical
- J4: footprint Connector_JST:JST_GH_SM03B-GHS-TB_1x03-1MP_P1.25mm_Horizontal -> PowerLibrary:JST_GH_SM03B-GHS-TB_1x03-1MP_P1.25mm_Horizontal
- J5: footprint Connector_PinHeader_2.54mm:PinHeader_1x07_P2.54mm_Vertical -> PowerLibrary:PinHeader_1x07_P2.54mm_Vertical
- J6: footprint Connector_AMASS:AMASS_XT30UPB-F_1x02_P5.0mm_Vertical -> PowerLibrary:AMASS_XT30UPB-F_1x02_P5.0mm_Vertical
- J7: footprint Connector_AMASS:AMASS_XT60-M_1x02_P7.20mm_Vertical -> PowerLibrary:AMASS_XT60-M_1x02_P7.20mm_Vertical
Changed lines of the file:
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@@
   (symbol (lib_id "power:PWR_FLAG") (at 241.935 93.345 0) (unit 1)
     (in_bom yes) (on_board yes) (fields_autoplaced)
-    (property "Reference" "#FLG01" (id 0) (at 241.935 91.44 0)
+    (property "Reference" "#FLG03" (id 0) (at 241.935 91.44 0)
       (effects (font (size 1.27 1.27)) hide)
     )
@@
       (effects (font (size 1.27 1.27)) (justify left))
     )
-    (property "Footprint" "Connector_AMASS:AMASS_XT60-M_1x02_P7.20mm_Vertical" (id 2) (at 248.92 102.235 0)
+    (property "Footprint" "PowerLibrary:AMASS_XT60-M_1x02_P7.20mm_Vertical" (id 2) (at 248.92 102.235 0)
       (effects (font (size 1.27 1.27)) hide)
     )
@@
   (symbol (lib_id "power:+6V") (at 117.475 86.36 0) (mirror y) (unit 1)
     (in_bom yes) (on_board yes)
-    (property "Reference" "#PWR031" (id 0) (at 117.475 90.17 0)
+    (property "Reference" "#PWR032" (id 0) (at 117.475 90.17 0)
       (effects (font (size 1.27 1.27)) hide)
     )
@@
   (symbol (lib_id "power:PWR_FLAG") (at 241.935 107.95 180) (unit 1)
     (in_bom yes) (on_board yes) (fields_autoplaced)
-    (property "Reference" "#FLG03" (id 0) (at 241.935 109.855 0)
+    (property "Reference" "#FLG04" (id 0) (at 241.935 109.855 0)
       (effects (font (size 1.27 1.27)) hide)
     )
@@
   (symbol (lib_id "power:PWR_FLAG") (at 119.38 86.36 0) (unit 1)
     (in_bom yes) (on_board yes) (fields_autoplaced)
-    (property "Reference" "#FLG?" (id 0) (at 119.38 84.455 0)
+    (property "Reference" "#FLG02" (id 0) (at 119.38 84.455 0)
       (effects (font (size 1.27 1.27)) hide)
     )
@@
   (symbol (lib_id "power:VCC") (at 240.03 125.095 0) (unit 1)
     (in_bom yes) (on_board yes)
-    (property "Reference" "#PWR038" (id 0) (at 240.03 128.905 0)
+    (property "Reference" "#PWR039" (id 0) (at 240.03 128.905 0)
       (effects (font (size 1.27 1.27)) hide)
     )
@@
       (effects (font (size 1.27 1.27)) (justify left) hide)
     )
-    (property "Footprint" "Connector_JST:JST_GH_SM03B-GHS-TB_1x03-1MP_P1.25mm_Horizontal" (id 2) (at 151.13 129.54 0)
+    (property "Footprint" "PowerLibrary:JST_GH_SM03B-GHS-TB_1x03-1MP_P1.25mm_Horizontal" (id 2) (at 151.13 129.54 0)
       (effects (font (size 1.27 1.27)) hide)
     )
@@
   (symbol (lib_id "power:GND") (at 240.03 139.7 0) (unit 1)
     (in_bom yes) (on_board yes)
-    (property "Reference" "#PWR039" (id 0) (at 240.03 146.05 0)
+    (property "Reference" "#PWR040" (id 0) (at 240.03 146.05 0)
       (effects (font (size 1.27 1.27)) hide)
     )
@@
       (effects (font (size 1.27 1.27)) (justify left) hide)
     )
-    (property "Footprint" "Connector_PinHeader_2.54mm:PinHeader_1x07_P2.54mm_Vertical" (id 2) (at 195.58 130.81 0)
+    (property "Footprint" "PowerLibrary:PinHeader_1x07_P2.54mm_Vertical" (id 2) (at 195.58 130.81 0)
       (effects (font (size 1.27 1.27)) hide)
     )
@@
   (symbol (lib_id "power:GND") (at 202.565 142.24 0) (mirror y) (unit 1)
     (in_bom yes) (on_board yes)
-    (property "Reference" "#PWR035" (id 0) (at 202.565 148.59 0)
+    (property "Reference" "#PWR036" (id 0) (at 202.565 148.59 0)
       (effects (font (size 1.27 1.27)) hide)
     )
@@
   (symbol (lib_id "power:GND") (at 240.03 107.95 0) (unit 1)
     (in_bom yes) (on_board yes)
-    (property "Reference" "#PWR037" (id 0) (at 240.03 114.3 0)
+    (property "Reference" "#PWR038" (id 0) (at 240.03 114.3 0)
       (effects (font (size 1.27 1.27)) hide)
     )
@@
   (symbol (lib_id "power:GND") (at 64.77 142.24 0) (unit 1)
     (in_bom yes) (on_board yes)
-    (property "Reference" "#PWR030" (id 0) (at 64.77 148.59 0)
+    (property "Reference" "#PWR031" (id 0) (at 64.77 148.59 0)
       (effects (font (size 1.27 1.27)) hide)
     )
@@
   (symbol (lib_id "power:+15V") (at 240.03 93.345 0) (unit 1)
     (in_bom yes) (on_board yes)
-    (property "Reference" "#PWR036" (id 0) (at 240.03 97.155 0)
+    (property "Reference" "#PWR037" (id 0) (at 240.03 97.155 0)
       (effects (font (size 1.27 1.27)) hide)
     )
@@
       (effects (font (size 1.27 1.27)) hide)
     )
-    (property "Footprint" "Connector_JST:JST_GH_SM08B-GHS-TB_1x08-1MP_P1.25mm_Horizontal" (id 2) (at 57.15 137.16 0)
+    (property "Footprint" "PowerLibrary:JST_GH_SM08B-GHS-TB_1x08-1MP_P1.25mm_Horizontal" (id 2) (at 57.15 137.16 0)
       (effects (font (size 1.27 1.27)) hide)
     )
@@
   (symbol (lib_id "power:GND") (at 161.29 142.24 0) (mirror y) (unit 1)
     (in_bom yes) (on_board yes)
-    (property "Reference" "#PWR033" (id 0) (at 161.29 148.59 0)
+    (property "Reference" "#PWR034" (id 0) (at 161.29 148.59 0)
       (effects (font (size 1.27 1.27)) hide)
     )
@@
   (symbol (lib_id "power:GND") (at 117.475 142.24 0) (mirror y) (unit 1)
     (in_bom yes) (on_board yes)
-    (property "Reference" "#PWR032" (id 0) (at 117.475 148.59 0)
+    (property "Reference" "#PWR033" (id 0) (at 117.475 148.59 0)
       (effects (font (size 1.27 1.27)) hide)
     )
@@
       (effects (font (size 1.27 1.27)) (justify left) hide)
     )
-    (property "Footprint" "Connector_PinSocket_2.54mm:PinSocket_1x03_P2.54mm_Vertical" (id 2) (at 107.315 124.46 0)
+    (property "Footprint" "PowerLibrary:PinSocket_1x03_P2.54mm_Vertical" (id 2) (at 107.315 124.46 0)
       (effects (font (size 1.27 1.27)) hide)
     )
@@
       (effects (font (size 1.27 1.27)) (justify left))
     )
-    (property "Footprint" "Connector_AMASS:AMASS_XT30UPB-F_1x02_P5.0mm_Vertical" (id 2) (at 246.38 132.715 0)
+    (property "Footprint" "PowerLibrary:AMASS_XT30UPB-F_1x02_P5.0mm_Vertical" (id 2) (at 246.38 132.715 0)
       (effects (font (size 1.27 1.27)) hide)
     )
@@
   (symbol (lib_id "power:PWR_FLAG") (at 66.675 86.36 0) (unit 1)
     (in_bom yes) (on_board yes) (fields_autoplaced)
-    (property "Reference" "#FLG?" (id 0) (at 66.675 84.455 0)
+    (property "Reference" "#FLG01" (id 0) (at 66.675 84.455 0)
       (effects (font (size 1.27 1.27)) hide)
     )
@@
   (symbol (lib_id "power:+5VA") (at 202.565 86.36 0) (unit 1)
     (in_bom yes) (on_board yes)
-    (property "Reference" "#PWR034" (id 0) (at 202.565 90.17 0)
+    (property "Reference" "#PWR035" (id 0) (at 202.565 90.17 0)
       (effects (font (size 1.27 1.27)) hide)
     )
@@
   (symbol (lib_id "power:PWR_FLAG") (at 241.935 125.095 0) (unit 1)
     (in_bom yes) (on_board yes) (fields_autoplaced)
-    (property "Reference" "#FLG02" (id 0) (at 241.935 123.19 0)
+    (property "Reference" "#FLG05" (id 0) (at 241.935 123.19 0)
       (effects (font (size 1.27 1.27)) hide)
     )
@@
   (symbol (lib_id "power:+5VA") (at 64.77 86.36 0) (unit 1)
     (in_bom yes) (on_board yes)
-    (property "Reference" "#PWR029" (id 0) (at 64.77 90.17 0)
-      (effects (font (size 1.27 1.27)) hide)
-    )
+    (property "Reference" "#PWR030" (id 0) (at 64.77 90.17 0)
+      (effects (font (size 1.27 1.27)) hide)
+    )
