File: circuit/power_board/Controller.kicad_sch (KiCad schematic)
At the start: 21 parts, among them J1 conn_2x5, SW1 KEY, U1 MM32SPIN27PS

Commit message: Update the schematic of the power supply board and organize the schematic structure
Parts:
- removed C7: 10uF, Capacitor_SMD:C_0603_1608Metric_Pad1.08x0.95mm_HandSolder, symbol Device:C
- removed SW1: KEY, Button_Switch_SMD:SW_SPST_CK_RS282G05A3, symbol power_Library:KEY
- C6: value 10uF -> 100nF
- renumbered R3 to R1, R1 to R2, R2 to R3
Connections:
- net EN renamed PC6
- net PG1: no longer names the net of U1.40 (PC9)
- net PG2 renamed PC7
- net ~{SD} renamed PC8
- no-connect marks 39 -> 40
Other:
- note added: "Debug"
- note added: "Filter"
- note added: "LEDs"
- note added: "MCU"
- moved on the sheet: C1, C2, D1, D2, D3, J1, R1, R2, R3, R4, R5, R6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

Commit message: Update the power board PCB file and complete the power board layout wiring.
Parts:
- removed J1: conn_2x5, Connector_PinHeader_2.54mm:PinHeader_2x05_P2.54mm_Vertical, symbol power_Library:conn_2x5
- added C2: 100nF, Capacitor_SMD:C_0603_1608Metric_Pad1.08x0.95mm_HandSolder, symbol Device:C
- added J1: Conn_01x04, Connector_PinHeader_2.54mm:PinHeader_1x04_P2.54mm_Vertical, symbol Connector_Generic:Conn_01x04
- added R6: 10kR, Resistor_SMD:R_0603_1608Metric_Pad0.98x0.95mm_HandSolder, symbol Device:R
- renumbered C2 to C3, C3 to C4, C4 to C5, C5 to C6, C6 to C7, R6 to R7, R7 to R8, R8 to R9
Connections:
- net PC6 is gone; now on net LED2: U1.37 (PC6)
- net PC7 is gone; now on net LED1: U1.38 (PC7)
- net +3V3: now also J1.1 (Pin_1)
- net ADC1: now also R6.1; no longer U1.21 (PA5)
- net GND: now also C2.2, J1.4 (Pin_4)
- net LED1: no longer U1.29 (PB10)
- net LED2: no longer U1.23 (PA7)
- net SWCLK: now also J1.2 (Pin_2)
- net SWDIO: now also J1.3 (Pin_3)
- net PA11: now reaches U1.44 (PA11)
- net D0 renamed PA3
- net D1 renamed PD4
- net D2 renamed PD5
- net D3 renamed PA4
- net PC8: no longer names the net of U1.39 (PC8)
- net UART1_RX renamed PA10
- net UART1_TX renamed PA9
- new net Current: C2.1, R6.2, U1.21 (PA5)
Other:
- moved on the sheet: R5
