File: circuit/power_board/Power.kicad_sch (KiCad schematic)
At the start: 70 parts, among them J5 XT30, J6 XT60, J8 conn_1x1, J9 conn_1x1, Q1 S8050, Q2 HSBB4052, Q3 HSBB4052, Q4 ME85P03, SW2 KEY, U2 TPS54540, U3 INA180A2, U4 LTC4365, U5 ETA7014, U6 HX9193-3.3GB, U7 JW5017S

Commit message: Update the schematic of the power supply board and organize the schematic structure
Parts:
- removed J5: XT30, Connector_AMASS:AMASS_XT30UPB-F_1x02_P5.0mm_Vertical, symbol power_Library:XT30
- removed J6: XT60, Connector_AMASS:AMASS_XT60-M_1x02_P7.20mm_Vertical, symbol power_Library:XT60
- removed Q2, Q3: HSBB4052, Library:PRPAK-8_L3.0-W3.0-P0.65-BL-EP, symbol Device:Q_NMOS_SGD
- removed R19: 2700k, Resistor_SMD:R_0603_1608Metric_Pad0.98x0.95mm_HandSolder, symbol Device:R
- removed R20, R24: 100kR, Resistor_SMD:R_0603_1608Metric_Pad0.98x0.95mm_HandSolder, symbol Device:R
- removed R21: 200kR, Resistor_SMD:R_0603_1608Metric_Pad0.98x0.95mm_HandSolder, symbol Device:R
- removed U4: LTC4365, Package_TO_SOT_SMD:TSOT-23-8, symbol power_Library:LTC4365
- C7: renamed from C21; value 10uF_1206 -> 10uF
- D4: value CUS10S30 -> SD103AWS
- D5: renamed from D6; value CUS10S30 -> SD103AWS
- D8: renamed from D5; value Schottky -> SK104C
- F1: value Fuse_Polarized -> Fuse
- Q1: value S8050 -> SS8050
- R14: value 10kR -> 4.7kR
- R16: renamed from R17; value 10mR -> 3mR
- R17: renamed from R18; value 10kR -> 10R
- R9: renamed from R11; value 1kR -> 100R
- renumbered C27 to C10, C30 to C11, C19 to C12, C20 to C13, C13 to C14, C22 to C16, C33 to C17, C34 to C18, C8 to C19, C9 to C20, C10 to C21, C25 to C22, C28 to C23, C29 to C24, C12 to C25, C31 to C26, C23 to C27, C14 to C28, C17 to C29, C18 to C30, C26 to C31, C24 to C8, C11 to C9, D7 to D6, D8 to D7, L2 to L1, L1 to L2, Q4 to Q2, R31 to R10, R12 to R11, R13 to R12, R32 to R13, R33 to R15, R29 to R18, R30 to R19, R34 to R20, R9 to R21, R10 to R22, R15 to R23, R16 to R24, R22 to R25, SW2 to SW1, U7 to U2, U5 to U4, U2 to U5
Connections:
- net +VSW is gone; now on net +6V: C28.2, C29.2, L2.2, R23.2
- net PG1 renamed GATE
- net PG2 renamed DET
- no-connect marks 1 -> 0
Other:
- note added: "3.3V Power"
- note added: "5V Power"
- note added: "5V Protect"
- note added: "Servo Power"
- note added: "Switch"
- moved on the sheet: C10, C11, C12, C13, C14, C15, C16, C17, C18, C19, C20, C21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

Commit message: Update the power board PCB file and complete the power board layout wiring.
Parts:
- F1: footprint Fuse:Fuse_2512_6332Metric -> Fuse:Fuse_1206_3216Metric
- L1: footprint Library:IND-SMD_L4.6-W4.2_SMMS0420 -> PowerLibrary:IND-SMD_L4.6-W4.2_SMMS0420
- renumbered C9 to C10, C10 to C11, C11 to C12, C12 to C13, C13 to C14, C14 to C15, C15 to C16, C16 to C17, C17 to C18, C18 to C19, C19 to C20, C20 to C21, C21 to C22, C22 to C23, C23 to C24, C24 to C25, C25 to C26, C26 to C27, C27 to C28, C28 to C29, C29 to C30, C30 to C31, C31 to C32, C7 to C8, C8 to C9, R9 to R10, R10 to R11, R11 to R12, R12 to R13, R13 to R14, R14 to R15, R15 to R16, R16 to R17, R17 to R18, R18 to R19, R19 to R20, R20 to R21, R21 to R22, R22 to R23, R23 to R24, R24 to R25, R25 to R26
Connections:
- net +15V: no longer D7.2 (A2)
- net +5V: now also C25.1
- net +5VA: no longer C25.1
- net at D6.2 (A2), F1.2, Q2.3 (S)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: now also D7.2 (A2)
Other:
- moved on the sheet: C15, C17, C19, C23, C24, C25, C27, D7, F1, R18, R19, R20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
