File: circuit/power_board/power_board.kicad_pcb (KiCad board)
At the start: 2 copper layers, 50 x 50 mm, 95 parts, among them J1 conn_2x5, J2 GH1.25_1x8, J3 conn_1x3, J4 GH1.25_1X3, J5 XT30, J6 XT60, J7 CONN_1X7, J8 conn_1x1, J9 conn_1x1, Q1 S8050, Q2 HSBB4052, Q3 HSBB4052, Q4 ME85P03, SW1 KEY, SW2 KEY, U1 MM32SPIN27PS, U2 TPS54540, U3 INA180A2, U4 LTC4365, U5 ETA7014, U6 HX9193-3.3GB, U7 JW5017S

Commit message: Update the power board PCB file and complete the power board layout wiring.
Parts:
- removed the C3 at (160.9, 96.5)
- removed the J5 at (126.2, 121.0)
- removed the Q2 at (152.5, 122.7)
- removed Q3: HSBB4052, PowerLibrary:PRPAK-8_L3.0-W3.0-P0.65-BL-EP
- removed the R19 at (155.3, 123.3)
- removed the R20 at (157.2, 123.3)
- removed the R21 at (159.0, 123.3)
- removed the R24 at (161.0, 116.3)
- removed the SW1 at (166.5, 95.8)
- removed the U4 at (157.6, 117.9)
- added C2: 100nF, Capacitor_SMD:C_0603_1608Metric_Pad1.08x0.95mm_HandSolder, F.Cu at (163.0, 80.5)
- added J7: XT60, PowerLibrary:AMASS_XT60-M_1x02_P7.20mm_Vertical, F.Cu at (128.8, 87.2)
- added R6: 10kR, Resistor_SMD:R_0603_1608Metric_Pad0.98x0.95mm_HandSolder, B.Cu at (163.0, 80.5)
- C1, C4, C5: footprint PowerLibrary:C_0603_1608Metric_Pad1.08x0.95mm_HandSolder -> Capacitor_SMD:C_0603_1608Metric_Pad1.08x0.95mm_HandSolder
- C10: renamed from C11; footprint PowerLibrary:C_0603_1608Metric_Pad1.08x0.95mm_HandSolder -> Capacitor_SMD:C_0603_1608Metric_Pad1.08x0.95mm_HandSolder
- C11: renamed from C27; footprint PowerLibrary:C_0603_1608Metric_Pad1.08x0.95mm_HandSolder -> Capacitor_SMD:C_0603_1608Metric_Pad1.08x0.95mm_HandSolder; moved to F.Cu
- C12: renamed from C30; footprint PowerLibrary:C_0603_1608Metric_Pad1.08x0.95mm_HandSolder -> Capacitor_SMD:C_0603_1608Metric_Pad1.08x0.95mm_HandSolder; moved to F.Cu
- C13: renamed from C19; footprint PowerLibrary:C_0603_1608Metric_Pad1.08x0.95mm_HandSolder -> Capacitor_SMD:C_0603_1608Metric_Pad1.08x0.95mm_HandSolder; moved to F.Cu
- C14: renamed from C20; footprint PowerLibrary:C_0603_1608Metric_Pad1.08x0.95mm_HandSolder -> Capacitor_SMD:C_0603_1608Metric_Pad1.08x0.95mm_HandSolder; moved to F.Cu
- C15: renamed from C13; footprint PowerLibrary:C_1206_3216Metric_Pad1.33x1.80mm_HandSolder -> Capacitor_SMD:C_1206_3216Metric_Pad1.33x1.80mm_HandSolder
- C16: renamed from C15; footprint PowerLibrary:C_0603_1608Metric_Pad1.08x0.95mm_HandSolder -> Capacitor_SMD:C_0603_1608Metric_Pad1.08x0.95mm_HandSolder
- C17: renamed from C22; footprint PowerLibrary:C_0603_1608Metric_Pad1.08x0.95mm_HandSolder -> Capacitor_SMD:C_0603_1608Metric_Pad1.08x0.95mm_HandSolder; moved to F.Cu
- C18: renamed from C33; footprint PowerLibrary:C_1206_3216Metric_Pad1.33x1.80mm_HandSolder -> Capacitor_SMD:C_1206_3216Metric_Pad1.33x1.80mm_HandSolder
- C19: renamed from C34; footprint PowerLibrary:C_0603_1608Metric_Pad1.08x0.95mm_HandSolder -> Capacitor_SMD:C_0603_1608Metric_Pad1.08x0.95mm_HandSolder; moved to F.Cu
- C20: renamed from C8; footprint PowerLibrary:C_1206_3216Metric_Pad1.33x1.80mm_HandSolder -> Capacitor_SMD:C_1206_3216Metric_Pad1.33x1.80mm_HandSolder
- C21: renamed from C9; footprint PowerLibrary:C_0603_1608Metric_Pad1.08x0.95mm_HandSolder -> Capacitor_SMD:C_0603_1608Metric_Pad1.08x0.95mm_HandSolder; moved to B.Cu
- C22: renamed from C10; footprint PowerLibrary:C_0603_1608Metric_Pad1.08x0.95mm_HandSolder -> Capacitor_SMD:C_0603_1608Metric_Pad1.08x0.95mm_HandSolder; moved to B.Cu
- C23: renamed from C25; footprint PowerLibrary:C_0603_1608Metric_Pad1.08x0.95mm_HandSolder -> Capacitor_SMD:C_0603_1608Metric_Pad1.08x0.95mm_HandSolder; moved to F.Cu
- C24: renamed from C28; footprint PowerLibrary:C_0603_1608Metric_Pad1.08x0.95mm_HandSolder -> Capacitor_SMD:C_0603_1608Metric_Pad1.08x0.95mm_HandSolder; moved to F.Cu
- C25: renamed from C29; footprint PowerLibrary:CP_Radial_D6.3mm_P2.50mm -> Capacitor_THT:CP_Radial_D6.3mm_P2.50mm
- C26: renamed from C12; footprint PowerLibrary:C_0603_1608Metric_Pad1.08x0.95mm_HandSolder -> Capacitor_SMD:C_0603_1608Metric_Pad1.08x0.95mm_HandSolder
- C27: renamed from C31; footprint PowerLibrary:C_1210_3225Metric_Pad1.33x2.70mm_HandSolder -> Capacitor_SMD:C_1210_3225Metric_Pad1.33x2.70mm_HandSolder
- C28: renamed from C23; footprint PowerLibrary:C_0603_1608Metric_Pad1.08x0.95mm_HandSolder -> Capacitor_SMD:C_0603_1608Metric_Pad1.08x0.95mm_HandSolder; moved to F.Cu
- C29: renamed from C14; footprint PowerLibrary:C_1206_3216Metric_Pad1.33x1.80mm_HandSolder -> Capacitor_SMD:C_1206_3216Metric_Pad1.33x1.80mm_HandSolder; moved to F.Cu
- C3: renamed from C2; footprint PowerLibrary:C_0603_1608Metric_Pad1.08x0.95mm_HandSolder -> Capacitor_SMD:C_0603_1608Metric_Pad1.08x0.95mm_HandSolder; moved to F.Cu
- C30: renamed from C17; footprint PowerLibrary:C_1206_3216Metric_Pad1.33x1.80mm_HandSolder -> Capacitor_SMD:C_1206_3216Metric_Pad1.33x1.80mm_HandSolder
- C31: renamed from C18; footprint PowerLibrary:CP_Radial_D6.3mm_P2.50mm -> Capacitor_THT:CP_Radial_D6.3mm_P2.50mm
- C32: renamed from C26; footprint PowerLibrary:C_0603_1608Metric_Pad1.08x0.95mm_HandSolder -> Capacitor_SMD:C_0603_1608Metric_Pad1.08x0.95mm_HandSolder; moved to F.Cu
- C6: value 10uF -> 100nF; footprint PowerLibrary:C_0603_1608Metric_Pad1.08x0.95mm_HandSolder -> Capacitor_SMD:C_0603_1608Metric_Pad1.08x0.95mm_HandSolder
- C7: value 10uF -> 100nF; footprint PowerLibrary:C_0603_1608Metric_Pad1.08x0.95mm_HandSolder -> Capacitor_SMD:C_0603_1608Metric_Pad1.08x0.95mm_HandSolder; moved to B.Cu
- C8: renamed from C21; value 10uF_1206 -> 10uF; footprint PowerLibrary:C_1206_3216Metric_Pad1.33x1.80mm_HandSolder -> Capacitor_SMD:C_1206_3216Metric_Pad1.33x1.80mm_HandSolder; moved to F.Cu
- C9: renamed from C24; footprint PowerLibrary:C_1206_3216Metric_Pad1.33x1.80mm_HandSolder -> Capacitor_SMD:C_1206_3216Metric_Pad1.33x1.80mm_HandSolder; moved to F.Cu
- D1, D2, D3, D9: footprint PowerLibrary:LED_0603_1608Metric -> LED_SMD:LED_0603_1608Metric
- D4: value CUS10S30 -> SD103AWS; footprint PowerLibrary:D_SOD-323_HandSoldering -> Diode_SMD:D_SOD-323_HandSoldering; moved to F.Cu
- D5: renamed from D6; value CUS10S30 -> SD103AWS; footprint PowerLibrary:D_SOD-323_HandSoldering -> Diode_SMD:D_SOD-323_HandSoldering; moved to F.Cu
- D6: renamed from D7; footprint PowerLibrary:D_SMB -> Diode_SMD:D_SMB; moved to F.Cu
- D7: renamed from D8; footprint PowerLibrary:D_SMB -> Diode_SMD:D_SMB; moved to F.Cu
- D8: renamed from D5; value Schottky -> SK104C; footprint PowerLibrary:D_SMC -> Diode_SMD:D_SMC; moved to B.Cu
- F1: value Fuse_Polarized -> Fuse; footprint PowerLibrary:Fuse_2512_6332Metric -> Fuse:Fuse_1206_3216Metric
- J1: value conn_2x5 -> Conn_01x04; footprint PowerLibrary:PinHeader_2x05_P2.54mm_Vertical -> Connector_PinHeader_2.54mm:PinHeader_1x04_P2.54mm_Vertical
- J6: value XT60 -> XT30; footprint PowerLibrary:AMASS_XT60-M_1x02_P7.20mm_Vertical -> PowerLibrary:AMASS_XT30UPB-F_1x02_P5.0mm_Vertical
- J8, J9: footprint PowerLibrary:PinSocket_1x01_P2.54mm_Vertical -> Connector_PinSocket_2.54mm:PinSocket_1x01_P2.54mm_Vertical
- L1: renamed from L2; moved to F.Cu
- L2: renamed from L1; footprint PowerLibrary:L_10.4x10.4_H4.8 -> Inductor_SMD:L_10.4x10.4_H4.8; moved to F.Cu
- Q1: value S8050 -> SS8050; footprint PowerLibrary:SOT-23 -> Package_TO_SOT_SMD:SOT-23; moved to F.Cu
- Q2: renamed from Q4; footprint PowerLibrary:TO-252-2 -> Package_TO_SOT_SMD:TO-252-2
- R1: renamed from R3; footprint PowerLibrary:R_0603_1608Metric_Pad0.98x0.95mm_HandSolder -> Resistor_SMD:R_0603_1608Metric_Pad0.98x0.95mm_HandSolder
- R10: renamed from R11; value 1kR -> 100R; footprint PowerLibrary:R_0603_1608Metric_Pad0.98x0.95mm_HandSolder -> Resistor_SMD:R_0603_1608Metric_Pad0.98x0.95mm_HandSolder; moved to F.Cu
- R11: renamed from R31; footprint PowerLibrary:R_0603_1608Metric_Pad0.98x0.95mm_HandSolder -> Resistor_SMD:R_0603_1608Metric_Pad0.98x0.95mm_HandSolder; moved to F.Cu
- R12, R13: footprint PowerLibrary:R_0603_1608Metric_Pad0.98x0.95mm_HandSolder -> Resistor_SMD:R_0603_1608Metric_Pad0.98x0.95mm_HandSolder; moved to F.Cu
- R14: renamed from R32; footprint PowerLibrary:R_0603_1608Metric_Pad0.98x0.95mm_HandSolder -> Resistor_SMD:R_0603_1608Metric_Pad0.98x0.95mm_HandSolder; moved to F.Cu
- R15: renamed from R14; value 10kR -> 4.7kR; footprint PowerLibrary:R_0805_2012Metric_Pad1.20x1.40mm_HandSolder -> Resistor_SMD:R_0805_2012Metric_Pad1.20x1.40mm_HandSolder
- R16: renamed from R33; footprint PowerLibrary:R_0603_1608Metric_Pad0.98x0.95mm_HandSolder -> Resistor_SMD:R_0603_1608Metric_Pad0.98x0.95mm_HandSolder; moved to F.Cu
- R17: value 10mR -> 3mR; footprint PowerLibrary:R_2512_6332Metric -> Resistor_SMD:R_2512_6332Metric
- R18: value 10kR -> 10R; footprint PowerLibrary:R_1206_3216Metric -> Resistor_SMD:R_1206_3216Metric
- R19: renamed from R29; footprint PowerLibrary:R_0603_1608Metric_Pad0.98x0.95mm_HandSolder -> Resistor_SMD:R_0603_1608Metric_Pad0.98x0.95mm_HandSolder; moved to F.Cu
- R2: renamed from R1; footprint PowerLibrary:R_0603_1608Metric_Pad0.98x0.95mm_HandSolder -> Resistor_SMD:R_0603_1608Metric_Pad0.98x0.95mm_HandSolder; moved to B.Cu
- R20: renamed from R30; footprint PowerLibrary:R_0603_1608Metric_Pad0.98x0.95mm_HandSolder -> Resistor_SMD:R_0603_1608Metric_Pad0.98x0.95mm_HandSolder; moved to F.Cu
- R21: renamed from R34; footprint PowerLibrary:R_0603_1608Metric_Pad0.98x0.95mm_HandSolder -> Resistor_SMD:R_0603_1608Metric_Pad0.98x0.95mm_HandSolder; moved to F.Cu
- R22: renamed from R9; footprint PowerLibrary:R_0603_1608Metric_Pad0.98x0.95mm_HandSolder -> Resistor_SMD:R_0603_1608Metric_Pad0.98x0.95mm_HandSolder; moved to B.Cu
- R23: renamed from R10; footprint PowerLibrary:R_0603_1608Metric_Pad0.98x0.95mm_HandSolder -> Resistor_SMD:R_0603_1608Metric_Pad0.98x0.95mm_HandSolder; moved to B.Cu
- R24: renamed from R15; footprint PowerLibrary:R_0603_1608Metric_Pad0.98x0.95mm_HandSolder -> Resistor_SMD:R_0603_1608Metric_Pad0.98x0.95mm_HandSolder
- R25: renamed from R16; footprint PowerLibrary:R_0603_1608Metric_Pad0.98x0.95mm_HandSolder -> Resistor_SMD:R_0603_1608Metric_Pad0.98x0.95mm_HandSolder
- R26: renamed from R22; footprint PowerLibrary:R_0603_1608Metric_Pad0.98x0.95mm_HandSolder -> Resistor_SMD:R_0603_1608Metric_Pad0.98x0.95mm_HandSolder
- R3: renamed from R2; footprint PowerLibrary:R_0603_1608Metric_Pad0.98x0.95mm_HandSolder -> Resistor_SMD:R_0603_1608Metric_Pad0.98x0.95mm_HandSolder
- R4, R5: footprint PowerLibrary:R_0603_1608Metric_Pad0.98x0.95mm_HandSolder -> Resistor_SMD:R_0603_1608Metric_Pad0.98x0.95mm_HandSolder
- R7: renamed from R6; footprint PowerLibrary:R_0603_1608Metric_Pad0.98x0.95mm_HandSolder -> Resistor_SMD:R_0603_1608Metric_Pad0.98x0.95mm_HandSolder
- R8: renamed from R7; footprint PowerLibrary:R_0603_1608Metric_Pad0.98x0.95mm_HandSolder -> Resistor_SMD:R_0603_1608Metric_Pad0.98x0.95mm_HandSolder
- R9: renamed from R8; footprint PowerLibrary:R_0603_1608Metric_Pad0.98x0.95mm_HandSolder -> Resistor_SMD:R_0603_1608Metric_Pad0.98x0.95mm_HandSolder
- SW1: renamed from SW2; footprint PowerLibrary:SW_SPST_CK_RS282G05A3 -> Button_Switch_SMD:SW_SPST_CK_RS282G05A3
- U1: footprint PowerLibrary:LQFP-64_10x10mm_P0.5mm -> Package_QFP:LQFP-64_10x10mm_P0.5mm
- U2: renamed from U7; footprint PowerLibrary:SOT-23-6 -> Package_TO_SOT_SMD:SOT-23-6; moved to F.Cu
- U3: footprint PowerLibrary:SOT-23-5 -> Package_TO_SOT_SMD:SOT-23-5
- U4: renamed from U5; footprint PowerLibrary:TSOT-23-6 -> Package_TO_SOT_SMD:TSOT-23-6; moved to F.Cu
- U5: renamed from U2; footprint PowerLibrary:SOIC-8-1EP_3.9x4.9mm_P1.27mm_EP2.29x3mm -> Package_SO:SOIC-8-1EP_3.9x4.9mm_P1.27mm_EP2.29x3mm
- U6: footprint PowerLibrary:SOT-23-5 -> Package_TO_SOT_SMD:SOT-23-5; moved to F.Cu
- moved J6 35.3 mm to (126.8, 121.5), turned to 90 degrees
- moved J8 29.2 mm to (151.6, 80.7), turned to -90 degrees
- moved J9 27.2 mm to (142.9, 80.7), turned to 180 degrees
- moved SW1 25.8 mm to (147.2, 81.9), turned to 0 degrees
- moved C10 25.7 mm to (147.2, 81.9), turned to 180 degrees
- moved C5 22.0 mm to (166.3, 95.4), turned to 180 degrees
- moved C13 20.7 mm to (141.1, 123.5), turned to 180 degrees
- moved D5 20.5 mm to (148.7, 95.8), turned to 180 degrees
- moved D4 18.7 mm to (148.7, 93.4), turned to 0 degrees
- moved C29 17.9 mm to (163.0, 120.1)
- moved R13 17.5 mm to (149.0, 91.2), turned to 180 degrees
- moved C14 17.0 mm to (141.1, 121.6), turned to 180 degrees
- moved C4 16.6 mm to (166.3, 98.5)
- moved C25 16.5 mm to (143.0, 111.0), turned to 0 degrees
- moved R10 16.1 mm to (150.4, 98.8)
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- renumbered J7 to J5
Connections:
- C25 pad 1: +5VA -> +5V
- C29 pad 2: +VSW -> +6V
- C30 pad 2: +VSW -> +6V
- D4 pad 2: /Controller/PG2 -> /Controller/PA9
- D6 pad 2: Net-(D7-Pad2) -> Net-(D6-Pad2)
- D7 pad 2: +15V -> Net-(D6-Pad2)
- F1 pad 2: Net-(D7-Pad2) -> Net-(D6-Pad2)
- J1 pad 2: /Controller/SWDIO -> /Controller/SWCLK
- J1 pad 3: GND -> /Controller/SWDIO
- J1 pad 4: /Controller/SWCLK -> GND
- J5 pad 6: +3V3 -> +5VA
- J6 pad 1: +15V -> VCC
- L2 pad 2: +VSW -> +6V
- Q2 pad 3: Net-(D7-Pad2) -> Net-(D6-Pad2)
- R10 pad 2: /Controller/PG1 -> /Controller/PA10
- R13 pad 1: /Controller/PG2 -> /Controller/PA9
- R15 pad 2: Net-(D7-Pad2) -> Net-(D6-Pad2)
- R24 pad 2: +VSW -> +6V
- U1 pad 17: /Connector/D0 -> /Connector/D3
- U1 pad 18: /Connector/D1 -> /Connector/D2
- U1 pad 19: /Connector/D2 -> /Connector/D1
- U1 pad 20: /Connector/D3 -> /Connector/D0
- U1 pad 21: /Controller/ADC1 -> /Controller/Current
- U1 pad 23: /Controller/LED2 -> unconnected-(U1-Pad23)
- U1 pad 29: /Controller/LED1 -> unconnected-(U1-Pad29)
- U1 pad 37: /Controller/EN -> /Controller/LED2
- U1 pad 38: /Controller/PG2 -> /Controller/LED1
- U1 pad 39: /Controller/~{SD} -> unconnected-(U1-Pad39)
- U1 pad 40: /Controller/PG1 -> unconnected-(U1-Pad40)
- U1 pad 42: /Controller/UART1_TX -> /Controller/PA9
- U1 pad 43: /Controller/UART1_RX -> /Controller/PA10
- U1 pad 44: unconnected-(U1-Pad44) -> /Controller/PA11
- U4 pad 2: /Controller/EN -> /Controller/PA11
Routing:
- net GND: track 52.0 -> 0.00 mm, vias 103 -> 54
- net /Controller/~{SD}: track 49.6 -> 0.00 mm, vias 4 -> 0
- net +3V3: track 109.3 -> 72.5 mm, vias 6 -> 5
- net +5VA: track 15.3 -> 46.8 mm, vias 0 -> 1
- net /Controller/EN: track 30.2 -> 0.00 mm, vias 1 -> 0
- net +VSW: track 26.4 -> 0.00 mm, vias 9 -> 0
- net /Controller/RST: track 30.6 -> 4.24 mm, vias 1 -> 0
- net /Controller/PG2: track 25.6 -> 0.00 mm, vias 1 -> 0
- net /Connector/PWR_RX: track 51.7 -> 27.7 mm
- net /Connector/PWR_TX: track 49.9 -> 27.1 mm
- net /Controller/PG1: track 20.4 -> 0.00 mm, vias 1 -> 0
- net +5V: track 48.3 -> 67.8 mm, vias 1 -> 4
- net /Controller/PA11: track 0.00 -> 15.0 mm
- net Net-(Q2-Pad2) (its old number): track 14.0 -> 0.00 mm, vias 2 -> 0
- net /Controller/UART1_TX: track 13.9 -> 0.00 mm
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- added copper zone on F.Cu, net +6V
- added copper zone on F.Cu, net Net-(C15-Pad2)
- added copper zone on F.Cu, net Net-(D6-Pad2)
- removed copper zone on B.Cu, net +3V3
- removed copper zone on F.Cu, net +3V3
- removed copper zone on B.Cu, net +VSW
- removed copper zone on F.Cu, net +VSW
- removed copper zone on B.Cu, net Net-(C26-Pad1)
- removed copper zone on B.Cu, net Net-(D5-Pad2)
- removed copper zone on F.Cu, net Net-(D5-Pad2)
- removed copper zone on B.Cu, net Net-(D7-Pad2)
- removed copper zone on F.Cu, net Net-(D7-Pad2)
- removed copper zone on F.Cu, net Net-(Q2-Pad1)
- removed copper zone on B.Cu, net VCC
Other:
- board text added: "2022/07/19"
- board text added: "GDUT Jesus Team"
- board text added: "PowerBoard"
- board text added: "Version 1.2.2"
- board text removed: "+"
- board text removed: "-"
- board text removed: "2022/06/018"
- board text removed: "GDUT"
- board text removed: "Jesus"
- board text removed: "R"
- board text removed: "S"
- board text removed: "T"
