File: circuit/power_board/power_board.kicad_sch (KiCad schematic)
At the start: 0 parts

Commit message: Update the schematic of the power supply board and organize the schematic structure
Other:
- sheet Controller ports: added PC6, PC7, PC8; removed EN, PG1, PG2, ~{SD}
- sheet Power ports: added DET, GATE; removed PG1, PG2, ~{SD}

Commit message: Update the power board PCB file and complete the power board layout wiring.
Other:
- sheet Controller ports: added PA10, PA11, PA3, PA4, PA9, PD4, PD5; removed D0, D1, D2, D3, PC6, PC7, PC8
